Commit message: Modified name of head_mount_xtion_frame to head_mount_xtion_link to fix tf tree. The new openni2 driver uses the latter name. Updated simulated drivers to match. Refs #7642
git-svn-id: svn+ssh://server/srv/svn/repos/branches/hydro_migration/pal-ros-pkg/catkin_pkgs/reem_robot@50104 5e370ff8-3418-0410-babe-3378cc20a00d

File: reem_description/urdf/sensors/openni.gazebo.xacro (robot description, xacro)
@@ -13,5 +13,5 @@
 <robot xmlns:xacro="http://ros.org/wiki/xacro">
   <xacro:macro name="openni_camera_gazebo_v0" params="name">
-    <gazebo reference="${name}_frame">
+    <gazebo reference="${name}_link">
       <sensor type="depth" name="${name}_frame_sensor">
         <always_on>true</always_on>

File: reem_description/urdf/sensors/xtion_pro_live.urdf.xacro (robot description, xacro)
@@ -24,7 +24,7 @@
       <insert_block name="origin" />
       <parent link="${parent}"/>
-      <child link="${name}_frame"/>
+      <child link="${name}_link"/>
     </joint>
-    <link name="${name}_frame">
+    <link name="${name}_link">
       <inertial>
         <mass value="0.01" />
@@ -52,5 +52,5 @@
     <joint name="${name}_optical_joint" type="fixed">
       <insert_block name="calibration_origin" />
-      <parent link="${name}_frame"/>
+      <parent link="${name}_link"/>
       <child link="${name}_optical_frame"/>
     </joint>
