Commit message: add a stereo optical frame for both frontal cameras
git-svn-id: svn+ssh://server/srv/svn/repos/trunk/pal-ros-pkg/catkin_pkgs/reem_robot@51150 5e370ff8-3418-0410-babe-3378cc20a00d

File: reem_description/urdf/sensors/stingrayf033c_camera.urdf.xacro (robot description, xacro)
@@ -31,4 +31,20 @@
       </visual>
     </link>
+    <!-- attach optical frame to the camera link -->
+    <joint name="${name}_optical_frame_joint" type="fixed">
+      <origin xyz="0 0 0" rpy="${-M_PI/2} 0.0 ${-M_PI/2}" /> <!-- rotate frame from x-forward to z-forward camera coords -->
+      <parent link="${name}_link"/>
+      <child link="${name}_optical_frame"/>
+    </joint>
+    <!-- optical frame for the stereo camera, with z-forward notation, this is the frame stereo camera images users should refer to -->
+    <link name="${name}_optical_frame" type="camera">
+      <inertial>
+        <mass value="0.01" />
+        <origin xyz="0 0 0" rpy="0 0 0" />
+        <inertia ixx="0"  ixy="0"  ixz="0"
+                 iyy="0"  iyz="0"
+                 izz="0" /> <!-- this inertia is made up for now. -->
+      </inertial>
+    </link>
   </xacro:macro>
 </robot>

Commit message: explanation of the optical frame orientation
git-svn-id: svn+ssh://server/srv/svn/repos/trunk/pal-ros-pkg/catkin_pkgs/reem_robot@51163 5e370ff8-3418-0410-babe-3378cc20a00d

File: reem_description/urdf/sensors/stingrayf033c_camera.urdf.xacro (robot description, xacro)
@@ -33,5 +33,7 @@
     <!-- attach optical frame to the camera link -->
     <joint name="${name}_optical_frame_joint" type="fixed">
-      <origin xyz="0 0 0" rpy="${-M_PI/2} 0.0 ${-M_PI/2}" /> <!-- rotate frame from x-forward to z-forward camera coords -->
+      <!-- rotate frame from x-forward to z-forward camera coords so that
+           the optical frame has z-forward, x-rightwards and y-downwards -->
+      <origin xyz="0 0 0" rpy="${-M_PI/2} 0.0 ${-M_PI/2}" />
       <parent link="${name}_link"/>
       <child link="${name}_optical_frame"/>
