Commit message: reem_description: cherry pick changes to hands in gazebo from github
git-svn-id: svn+ssh://server/srv/svn/repos/branches/hydro_migration/pal-ros-pkg/catkin_pkgs/reem_robot@50158 5e370ff8-3418-0410-babe-3378cc20a00d

File: reem_description/urdf/hand/hand.gazebo.xacro (robot description, xacro)
@@ -27,3 +27,60 @@
       </gazebo>
     </xacro:macro>
+    <xacro:macro name="hand_finger_gazebo" params="finger_name">
+    <gazebo reference="${finger_name}_link">
+      <mu1>0.9</mu1>
+      <mu2>0.9</mu2>
+    </gazebo>
+    <gazebo reference="${finger_name}_1_link">
+      <kp>1000000.0</kp>
+      <kd>100.0</kd>
+      <mu1>1.0</mu1>
+      <mu2>1.0</mu2>
+      <fdir1>0 0 1</fdir1>
+      <maxVel>1.0</maxVel>
+      <minDepth>0.00</minDepth>
+    </gazebo>
+    <gazebo reference="${finger_name}_2_link">
+      <kp>1000000.0</kp>
+      <kd>100.0</kd>
+      <mu1>1.0</mu1>
+      <mu2>1.0</mu2>
+      <fdir1>0 0 1</fdir1>
+      <maxVel>1.0</maxVel>
+      <minDepth>0.00</minDepth>
+    </gazebo>
+    <gazebo reference="${finger_name}_3_link">
+      <kp>1000000.0</kp>
+      <kd>100.0</kd>
+      <mu1>1.0</mu1>
+      <mu2>1.0</mu2>
+      <fdir1>0 0 1</fdir1>
+      <maxVel>1.0</maxVel>
+      <minDepth>0.00</minDepth>
+    </gazebo>
+    <gazebo reference="${finger_name}_joint">
+      <cfmDamping>1</cfmDamping>
+      <provideFeedback>1</provideFeedback>
+    </gazebo>
+    <gazebo reference="${finger_name}_1_joint">
+      <cfmDamping>1</cfmDamping>
+      <provideFeedback>1</provideFeedback>
+    </gazebo>
+    <gazebo reference="${finger_name}_2_joint">
+      <cfmDamping>1</cfmDamping>
+      <provideFeedback>1</provideFeedback>
+    </gazebo>
+    <gazebo reference="${finger_name}_3_joint">
+      <cfmDamping>1</cfmDamping>
+      <provideFeedback>1</provideFeedback>
+    </gazebo>
+    <gazebo>
+      <plugin filename="libgazebo_pal_hand.so" name="gazebo_pal_right_hand_index">
+        <actuatedJoint>${finger_name}_joint</actuatedJoint>
+        <fingerJoint1>${finger_name}_1_joint</fingerJoint1>
+        <fingerJoint2>${finger_name}_2_joint</fingerJoint2>
+        <fingerJoint3>${finger_name}_3_joint</fingerJoint3>
+      </plugin>
+    </gazebo>
+  </xacro:macro>
 </robot>

File: reem_description/urdf/hand/hand.urdf.xacro (robot description, xacro)
@@ -51,11 +51,4 @@
       </collision>
     </link>
-    <gazebo reference="${hand_name}_${hand_side}_${finger_name}_link">
-      <mu1>0.9</mu1>
-      <mu2>0.9</mu2>
-    </gazebo>
-    <gazebo reference="${hand_name}_${hand_side}_${finger_name}_joint">
-       <cfmDamping>1</cfmDamping>
-    </gazebo>
     <!-- Read-only phalanxes-->
     <joint name="${hand_name}_${hand_side}_${finger_name}_1_joint" type="revolute">
@@ -143,25 +136,5 @@
       </collision>
     </link>
-    <gazebo reference="${hand_name}_${hand_side}_${finger_name}_1_link">
-      <mu1>0.9</mu1>
-      <mu2>0.9</mu2>
-    </gazebo>
-    <gazebo reference="${hand_name}_${hand_side}_${finger_name}_2_link">
-      <mu1>0.9</mu1>
-      <mu2>0.9</mu2>
-    </gazebo>
-    <gazebo reference="${hand_name}_${hand_side}_${finger_name}_3_link">
-      <mu1>0.9</mu1>
-      <mu2>0.9</mu2>
-    </gazebo>
-    <gazebo reference="${hand_name}_${hand_side}_${finger_name}_1_joint">
-       <cfmDamping>1</cfmDamping>
-    </gazebo>
-    <gazebo reference="${hand_name}_${hand_side}_${finger_name}_2_joint">
-       <cfmDamping>1</cfmDamping>
-    </gazebo>
-    <gazebo reference="${hand_name}_${hand_side}_${finger_name}_3_joint">
-       <cfmDamping>1</cfmDamping>
-    </gazebo>
+    <xacro:hand_finger_gazebo finger_name="${hand_name}_${hand_side}_${finger_name}"/>
     <xacro:hand_finger_transmission finger_name="${hand_name}_${hand_side}_${finger_name}" actuator_reduction="1"/>
   </xacro:macro>
@@ -194,4 +167,13 @@
       </collision>
     </link>
+    <gazebo reference="${name}_${side}_palm_link">
+     <kp>1000000.0</kp>
+     <kd>100.0</kd>
+     <mu1>1.0</mu1>
+     <mu2>1.0</mu2>
+     <fdir1>0 0 1</fdir1>
+     <maxVel>1.0</maxVel>
+     <minDepth>0.00</minDepth>
+    </gazebo>
     <xacro:hand_gazebo name="${name}_${side}_palm"/>
     <!-- Thumb -->
@@ -229,6 +211,11 @@
     </link>
     <gazebo reference="${name}_${side}_thumb_link">
-      <mu1>0.9</mu1>
-      <mu2>0.9</mu2>
+     <kp>1000000.0</kp>
+     <kd>100.0</kd>
+     <mu1>1.0</mu1>
+     <mu2>1.0</mu2>
+     <fdir1>0 0 1</fdir1>
+     <maxVel>1.0</maxVel>
+     <minDepth>0.00</minDepth>
     </gazebo>
     <gazebo reference="${name}_${side}_thumb_joint">
