Commit message: Merge from 4.0_ROCKIN_CAMP
git-svn-id: svn+ssh://server/srv/svn/repos/trunk/pal-ros-pkg/catkin_pkgs/reem_robot@51334 5e370ff8-3418-0410-babe-3378cc20a00d

File: reem_description/urdf/hand/hand.urdf.xacro (robot description, xacro)
@@ -59,4 +59,5 @@
       <limit lower="${0.0 * deg_to_rad}" upper="${90.0 * deg_to_rad}" effort="2.0" velocity="${hand_max_vel}" />
       <dynamics friction="${hand_friction}" damping="${hand_damping}"/>
+      <mimic joint="${hand_name}_${hand_side}_${finger_name}_joint" multiplier="-1.0" offset="0.0" />
     </joint>
     <link name="${hand_name}_${hand_side}_${finger_name}_1_link">
@@ -87,4 +88,5 @@
       <limit lower="${0.0 * deg_to_rad}" upper="${80.0 * deg_to_rad}" effort="1.0" velocity="${hand_max_vel}" />
       <dynamics friction="${hand_friction}" damping="${hand_damping}"/>
+      <mimic joint="${hand_name}_${hand_side}_${finger_name}_joint" multiplier="-1.0" offset="0.0" />
     </joint>
     <link name="${hand_name}_${hand_side}_${finger_name}_2_link">
@@ -115,4 +117,5 @@
       <limit lower="${0.0 * deg_to_rad}" upper="${80.0 * deg_to_rad}" effort="1.0" velocity="${hand_max_vel}" />
       <dynamics friction="${hand_friction}" damping="${hand_damping}"/>
+      <mimic joint="${hand_name}_${hand_side}_${finger_name}_joint" multiplier="-1.0" offset="0.0" />
     </joint>
     <link name="${hand_name}_${hand_side}_${finger_name}_3_link">
