Commit message: synchronization with github for arm and hand dynamic parameters and wheeled base slipping.
git-svn-id: svn+ssh://server/srv/svn/repos/branches/hydro_migration/pal-ros-pkg/catkin_pkgs/reem_robot@50466 5e370ff8-3418-0410-babe-3378cc20a00d

File: reem_description/urdf/821b41140000_base/base.gazebo.xacro (robot description, xacro)
@@ -1,5 +1,5 @@
 <?xml version="1.0"?>
 <!--
-  Copyright (c) 2011, PAL Robotics, S.L.
+  Copyright (c) 2011-2014, PAL Robotics, S.L.
   All rights reserved.
   This work is licensed under the Creative Commons Attribution-NonCommercial-NoDerivs 3.0 Unported License.

File: reem_description/urdf/821b41140000_base/base.transmission.xacro (robot description, xacro)
@@ -1,5 +1,5 @@
 <?xml version="1.0"?>
 <!--
-  Copyright (c) 2011, PAL Robotics, S.L.
+  Copyright (c) 2011-2014, PAL Robotics, S.L.
   All rights reserved.
   This work is licensed under the Creative Commons Attribution-NonCommercial-NoDerivs 3.0 Unported License.

File: reem_description/urdf/821b41140000_base/base.urdf.xacro (robot description, xacro)
@@ -1,5 +1,5 @@
 <?xml version="1.0"?>
 <!--
-  Copyright (c) 2011-2012, PAL Robotics, S.L.
+  Copyright (c) 2011-2014, PAL Robotics, S.L.
   All rights reserved.
   This work is licensed under the Creative Commons Attribution-NonCommercial-NoDerivs 3.0 Unported License.
@@ -56,12 +56,9 @@
   <!-- contact model for wheel surface -->
    <gazebo reference="wheel_${side}_link">
-     <kp>1000000.0</kp>
-     <kd>100.0</kd>
+     <kp>100000000.0</kp>
+     <kd>10000.0</kd>
      <mu1>1.0</mu1>
      <mu2>1.0</mu2>
-     <fdir1>0 0 1</fdir1>
-     <maxVel>1.0</maxVel>
      <minDepth>0.00</minDepth>
-     <cfmDamping>1</cfmDamping>
    </gazebo>
     <joint name="wheel_${side}_joint" type="continuous">
@@ -126,12 +123,9 @@
    <!-- contact model for caster wheel surface -->
    <gazebo reference="caster_${side}_2_link">
-     <kp>1000000.0</kp>
-     <kd>100.0</kd>
+     <kp>100000000.0</kp>
+     <kd>10000.0</kd>
      <mu1>1.0</mu1>
      <mu2>1.0</mu2>
-     <fdir1>0 0 1</fdir1>
-     <maxVel>1.0</maxVel>
      <minDepth>0.00</minDepth>
-     <cfmDamping>1</cfmDamping>
    </gazebo>
     <joint name="caster_${side}_1_joint" type="continuous">

File: reem_description/urdf/arm/arm.transmission.xacro (robot description, xacro)
@@ -1,5 +1,5 @@
 <?xml version="1.0"?>
 <!--
-  Copyright (c) 2011, PAL Robotics, S.L.
+  Copyright (c) 2011-2014, PAL Robotics, S.L.
   All rights reserved.
   This work is licensed under the Creative Commons Attribution-NonCommercial-NoDerivs 3.0 Unported License.

File: reem_description/urdf/arm/arm.urdf.xacro (robot description, xacro)
@@ -1,5 +1,5 @@
 <?xml version="1.0"?>
 <!--
-  Copyright (c) 2011-2012, PAL Robotics, S.L.
+  Copyright (c) 2011-2014, PAL Robotics, S.L.
   All rights reserved.
   This work is licensed under the Creative Commons Attribution-NonCommercial-NoDerivs 3.0 Unported License.
@@ -24,9 +24,8 @@
     <link name="${name}_${side}_1_link">
       <inertial>
-        <origin xyz="0.0006 -0.0005 ${reflect*0.20739}" rpy="0 0 0"/>
-        <mass value="2.148" />
-        <inertia ixx="0"  ixy="0"  ixz="0" iyy="0" iyz="0" izz="0" />
-<!--         NOTE: Assuming cylinder centered at CoM with r=0.05, h=0.05 with axis parallel to x coordinate -->
-<!--         <inertia ixx="0.0026850"  ixy="0"  ixz="0" iyy="0.0017900" iyz="0" izz="0.0017900" /> -->
+        <origin xyz="0.00701 -0.00011 ${reflect*0.18627}" rpy="0 0 0"/>
+        <mass value="1.53614" />
+<!--        <inertia ixx="0"  ixy="0"  ixz="0" iyy="0" iyz="0" izz="0" /> -->
+        <inertia ixx="0.00327313329"  ixy="-0.00000460054"  ixz="-0.00025121368" iyy="0.00316047802" iyz="0.00000313158" izz="0.00157642528" />
       </inertial>
       <visual>
@@ -58,9 +57,8 @@
    <link name="${name}_${side}_2_link">
       <inertial>
-        <origin xyz="0.0183 -0.09275 ${reflect*0.00478}" rpy="0 0 0"/>
-        <mass value="1.610" />
-        <inertia ixx="0"  ixy="0"  ixz="0" iyy="0" iyz="0" izz="0" />
-        <!-- NOTE: Assuming cylinder centered at CoM with r=0.05, h=0.05 with axis parallel to y coordinate -->
-<!--         <inertia ixx="0.0013417"  ixy="0"  ixz="0" iyy="0.0020125" iyz="0" izz="0.0013417" /> -->
+        <origin xyz="0.01435 -0.06294 ${reflect*0.01039}" rpy="0 0 0"/>
+        <mass value="1.60393" />
+        <!--<inertia ixx="0"  ixy="0"  ixz="0" iyy="0" iyz="0" izz="0" /> -->
+        <inertia ixx="0.0046195621"  ixy="-0.00056769245"  ixz="0.00018376961" iyy="0.00185384237" iyz="-0.00078286958" izz="0.0049356022" />
       </inertial>
       <visual>
@@ -92,9 +90,8 @@
     <link name="${name}_${side}_3_link">
       <inertial>
-        <origin xyz="0.00045 -0.01547 ${reflect * 0.07654}" rpy="0 0 0"/>
-        <mass value="1.656" />
-        <inertia ixx="0"  ixy="0"  ixz="0" iyy="0" iyz="0" izz="0" />
-        <!-- NOTE: Assuming cylinder centered at CoM with r=0.05, h=0.05 with axis parallel to x coordinate -->
-<!--         <inertia ixx="0.0020700"  ixy="0"  ixz="0" iyy="0.0013800" iyz="0" izz="0.0013800" /> -->
+        <origin xyz="0.00606 -0.0113 ${reflect * 0.05748}" rpy="0 0 0"/>
+        <mass value="1.64293" />
+        <!--<inertia ixx="0"  ixy="0"  ixz="0" iyy="0" iyz="0" izz="0" />-->
+        <inertia ixx="0.00372686652"  ixy="-0.00008722874"  ixz="-0.00028800176" iyy="0.00344463026" iyz="0.00042776588" izz="0.00192229026" />
       </inertial>
       <visual>
@@ -129,9 +126,8 @@
     <link name="${name}_${side}_4_link">
       <inertial>
-        <origin xyz="-0.06424 0.01712 ${-reflect * 0.00666}" rpy="0 0 0"/>
-        <mass value="1.013" />
-        <inertia ixx="0"  ixy="0"  ixz="0" iyy="0" iyz="0" izz="0" />
-        <!-- NOTE: Assuming cylinder centered at CoM with r=0.05, h=0.05 with axis parallel to x coordinate -->
-<!--         <inertia ixx="0.0012663"  ixy="0"  ixz="0" iyy="0.00084417" iyz="0" izz="0.00084417" /> -->
+        <origin xyz="-0.04129 0.0118 ${reflect * -0.01387}" rpy="0 0 0"/>
+        <mass value="1.20222" />
+        <!--<inertia ixx="0"  ixy="0"  ixz="0" iyy="0" iyz="0" izz="0" />-->
+        <inertia ixx="0.00156355749"  ixy="-0.000353141"  ixz="0.00053402452" iyy="0.00277186194" iyz="-0.00015541973" izz="0.00307369106" />
       </inertial>
       <visual>

File: reem_description/urdf/arm/wrist.transmission.xacro (robot description, xacro)
@@ -1,5 +1,5 @@
 <?xml version="1.0"?>
 <!--
-  Copyright (c) 2011, PAL Robotics, S.L.
+  Copyright (c) 2011-2014, PAL Robotics, S.L.
   All rights reserved.
   This work is licensed under the Creative Commons Attribution-NonCommercial-NoDerivs 3.0 Unported License.

File: reem_description/urdf/arm/wrist.urdf.xacro (robot description, xacro)
@@ -1,5 +1,5 @@
 <?xml version="1.0"?>
 <!--
-  Copyright (c) 2011-2012, PAL Robotics, S.L.
+  Copyright (c) 2011-2014, PAL Robotics, S.L.
   All rights reserved.
   This work is licensed under the Creative Commons Attribution-NonCommercial-NoDerivs 3.0 Unported License.
@@ -22,9 +22,8 @@
     <link name="${name}_${side}_5_link">
       <inertial>
-        <origin xyz="-0.00045 -0.00009 ${reflect * 0.08726}" rpy="0 0 0"/>
-        <mass value="1.858" />
-        <inertia ixx="0"  ixy="0"  ixz="0" iyy="0" iyz="0" izz="0" />
-        <!-- NOTE: Assuming cylinder centered at CoM with r=0.05, h=0.1 with axis parallel to z coordinate -->
-<!--         <inertia ixx="0.0027096"  ixy="0"  ixz="0" iyy="0.0027096" iyz="0" izz="0.0023225" /> -->
+        <origin xyz="-0.00044 0.00012 ${reflect * 0.07445}" rpy="0 0 0"/>
+        <mass value="1.21524" />
+        <!--<inertia ixx="0"  ixy="0"  ixz="0" iyy="0" iyz="0" izz="0" />-->
+        <inertia ixx="0.00193499547"  ixy="-0.00000027528"  ixz="-0.00001268153" iyy="0.00177767506" iyz="-0.00000466638" izz="0.00057101196" />
       </inertial>
       <visual>
@@ -56,9 +55,8 @@
     <link name="${name}_${side}_6_link">
       <inertial>
-        <origin xyz="-0.0002 -0.01155 ${reflect * 0.00002}" rpy="0 0 0"/>
-        <mass value="0.255" />
-        <inertia ixx="0"  ixy="0"  ixz="0" iyy="0" iyz="0" izz="0" />
-        <!-- NOTE: Assuming cylinder centered at CoM with r=0.02, h=0.08 with axis parallel to z coordinate -->
-<!--         <inertia ixx="0.0001615"  ixy="0"  ixz="0" iyy="0.0001615" iyz="0" izz="0.000051" /> -->
+        <origin xyz="-0.00005 -0.00252 ${reflect * 0.00007}" rpy="0 0 0"/>
+        <mass value="0.41597" />
+        <!--<inertia ixx="0"  ixy="0"  ixz="0" iyy="0" iyz="0" izz="0" />-->
+        <inertia ixx="0.00020339659"  ixy="-0.00000071703"  ixz="-0.00000006654" iyy="0.00015240261" iyz="0.00000014315" izz="0.0001671881" />
       </inertial>
       <visual>
@@ -91,9 +89,8 @@
       <inertial>
         <!--TODO: Verify these inertial parameters-->
-        <origin xyz="0 0 ${reflect * 0.109404509 / 2}" rpy="0 0 0"/>
-        <mass value="0.152461831" />
-        <inertia ixx="0"  ixy="0"  ixz="0" iyy="0" iyz="0" izz="0" />
-        <!-- NOTE: Assuming point mass -->
-<!--         <inertia ixx="0"  ixy="0"  ixz="0" iyy="0" iyz="0" izz="0" /> -->
+        <origin xyz="-0.00004 0 ${reflect * -0.02887}" rpy="0 0 0"/>
+        <mass value="0.06697" />
+        <!--<inertia ixx="0"  ixy="0"  ixz="0" iyy="0" iyz="0" izz="0" />-->
+        <inertia ixx="0.0000123718"  ixy="0.00000000002"  ixz="0.00000002403" iyy="0.00001242132" iyz="0.00000000001" izz="0.0000059514" />
       </inertial>
       <visual>

File: reem_description/urdf/hand/hand.gazebo.xacro (robot description, xacro)
@@ -1,5 +1,5 @@
 <?xml version="1.0"?>
 <!--
-  Copyright (c) 2011, PAL Robotics, S.L.
+  Copyright (c) 2011-2014, PAL Robotics, S.L.
   All rights reserved.
   This work is licensed under the Creative Commons Attribution-NonCommercial-NoDerivs 3.0 Unported License.

File: reem_description/urdf/hand/hand.transmission.xacro (robot description, xacro)
@@ -1,5 +1,5 @@
 <?xml version="1.0"?>
 <!--
-  Copyright (c) 2011, PAL Robotics, S.L.
+  Copyright (c) 2011-2014, PAL Robotics, S.L.
   All rights reserved.
   This work is licensed under the Creative Commons Attribution-NonCommercial-NoDerivs 3.0 Unported License.

File: reem_description/urdf/hand/hand.urdf.xacro (robot description, xacro)
@@ -1,5 +1,5 @@
 <?xml version="1.0"?>
 <!--
-  Copyright (c) 2011, PAL Robotics, S.L.
+  Copyright (c) 2011-2014, PAL Robotics, S.L.
   All rights reserved.
   This work is licensed under the Creative Commons Attribution-NonCommercial-NoDerivs 3.0 Unported License.
@@ -33,7 +33,7 @@
     <link name="${hand_name}_${hand_side}_${finger_name}_link">
       <inertial>
-        <origin xyz="0 0 0" rpy="0 0 0" /> <!--TODO: Fill up-->
-        <mass value="0.05" />
-        <inertia ixx="0"  ixy="0"  ixz="0" iyy="0" iyz="0" izz="0" /> <!--TODO: Fill up-->
+        <origin xyz="0.00175 -0.01837 -0.00198" rpy="0 0 0" />
+        <mass value="0.055" />
+        <inertia ixx="0.00001450121"  ixy="-0.00000065488"  ixz="-0.00000039654" iyy="0.0000072995" iyz="0.00000012168" izz="0.00001262409" />
       </inertial>
       <visual>
@@ -62,7 +62,7 @@
     <link name="${hand_name}_${hand_side}_${finger_name}_1_link">
       <inertial>
-        <origin xyz="0 0 0" rpy="0 0 0" /> <!--TODO: Fill up-->
-        <mass value="0.05" />
-        <inertia ixx="0"  ixy="0"  ixz="0" iyy="0" iyz="0" izz="0" /> <!--TODO: Fill up-->
+        <origin xyz="0.00175 -0.01837 -0.00198" rpy="0 0 0" />
+        <mass value="0.055" />
+        <inertia ixx="0.00001450121"  ixy="-0.00000065488"  ixz="-0.00000039654" iyy="0.0000072995" iyz="0.00000012168" izz="0.00001262409" />
       </inertial>
       <visual>
@@ -90,7 +90,7 @@
     <link name="${hand_name}_${hand_side}_${finger_name}_2_link">
       <inertial>
-        <origin xyz="0 0 0" rpy="0 0 0" /> <!--TODO: Fill up-->
-        <mass value="0.05" />
-        <inertia ixx="0"  ixy="0"  ixz="0" iyy="0" iyz="0" izz="0" /> <!--TODO: Fill up-->
+        <origin xyz="0.00181 -0.01275 -0.00064" rpy="0 0 0" />
+        <mass value="0.02972" />
+        <inertia ixx="0.00000428193"  ixy="-0.00000049978"  ixz="-0.00000002985" iyy="0.00000254434" iyz="0.00000007762" izz="0.00000345152" />
       </inertial>
       <visual>
@@ -118,7 +118,7 @@
     <link name="${hand_name}_${hand_side}_${finger_name}_3_link">
       <inertial>
-        <origin xyz="0 0 0" rpy="0 0 0" /> <!--TODO: Fill up-->
-        <mass value="0.05" />
-        <inertia ixx="0"  ixy="0"  ixz="0" iyy="0" iyz="0" izz="0" /> <!--TODO: Fill up-->
+        <origin xyz="0 -0.00704 0.00019" rpy="0 0 0" />
+        <mass value="0.01522" />
+        <inertia ixx="0.00000128478"  ixy="-0.00000008056"  ixz="-0.00000001698" iyy="0.00000080139" iyz="-0.00000002884" izz="0.00000090928" />
       </inertial>
       <visual>
@@ -148,8 +148,7 @@
     <link name="${name}_${side}_palm_link">
       <inertial>
-        <!--<origin xyz="0.07547 ${-reflect * 0.00468} 0.00291" rpy="0 0 0" />-->
-        <origin xyz="0 ${-reflect * 0.07547} 0 " rpy="0 0 0" /> <!--TODO: This does not make sense!, there must be a bug in how Gazebo bungles the CoM of a chain of fixed joints-->
-        <mass value="0.41066" /> <!--NOTE: Assigning 0.05kg to each of the ten phalanxes-->
-        <inertia ixx="0"  ixy="0"  ixz="0" iyy="0" iyz="0" izz="0" />
+        <origin xyz="0.05904 ${-reflect * 0.00925} -0.00075 " rpy="0 0 0" /> <!--TODO: This does not make sense!, there must be a bug in how Gazebo bungles the CoM of a chain of fixed joints-->
+        <mass value="0.68275" />
+        <inertia ixx="0.00045643484"  ixy="0.00001885321"  ixz="-0.0000103596" iyy="0.00076077407" iyz="-0.00000266311" izz="0.00052521525" />
       </inertial>
       <visual>
@@ -192,7 +191,7 @@
     <link name="${name}_${side}_thumb_link">
       <inertial>
-        <origin xyz="0 0 0" rpy="0 0 0" /> <!--TODO: Fill up-->
-        <mass value="0.05" />
-        <inertia ixx="0"  ixy="0"  ixz="0" iyy="0" iyz="0" izz="0" /> <!--TODO: Fill up-->
+        <origin xyz="0.00049 0.00451 ${-reflect*0.04179}" rpy="0 0 0" />
+        <mass value="0.07088" />
+        <inertia ixx="0.0000699364"  ixy="0.00000345915"  ixz="0.00000425008" iyy="0.00002675459" iyz="0.00002381865" izz="0.00004787167" />
       </inertial>
       <visual>
