Commit message: refs #8173 : adds offset_x param
git-svn-id: svn+ssh://server/srv/svn/repos/trunk/pal-ros-pkg/catkin_pkgs/ant_robot@52599 5e370ff8-3418-0410-babe-3378cc20a00d

File: ant_description/urdf/wheels/caster.urdf.xacro (robot description, xacro)
@@ -10,5 +10,5 @@
   <xacro:include filename="$(find ant_description)/urdf/wheels/caster.transmission.xacro"/>
   <xacro:include filename="$(find ant_description)/urdf/wheels/caster.gazebo.xacro"/>
-  <xacro:macro name="caster_ant" params="side reflect radius width separation trailing parent">
+  <xacro:macro name="caster_ant" params="side reflect radius width separation trailing offset_x parent">
     <link name="caster_${side}_1_link">
       <inertial>
@@ -56,5 +56,5 @@
       <parent link="${parent}_link"/>
       <child link="caster_${side}_1_link"/>
-      <origin xyz="-0.3805 ${-separation / 2 * reflect} ${radius}" rpy="0 0 0"/>
+      <origin xyz="${offset_x} ${-separation / 2 * reflect} ${radius}" rpy="0 0 0"/>
       <axis xyz="0 0 1"/>
     </joint>
