Commit message: uses caster 1&2 v2.0 and base v2.0 STL

File: ant_description/urdf/wheels/caster_v2.urdf.xacro (robot description, xacro)
@@ -22,5 +22,5 @@
         <origin xyz="0 0 0" rpy="0 0 0"/>
         <geometry>
-          <mesh filename="package://ant_description/meshes/wheels/caster.stl"/>
+          <mesh filename="package://ant_description/meshes/wheels/caster_1_v2.stl"/>
         </geometry>
         <material name="Grey"/>
@@ -29,5 +29,5 @@
         <origin xyz="0 0 0" rpy="0 0 0"/>
         <geometry>
-          <mesh filename="package://ant_description/meshes/wheels/caster.stl"/>
+          <mesh filename="package://ant_description/meshes/wheels/caster_1_v2.stl"/>
         </geometry>
       </collision>
@@ -44,5 +44,5 @@
         <origin xyz="0 0 0" rpy="0 0 0"/>
         <geometry>
-          <cylinder radius="${radius}" length="${width}"/>
+          <mesh filename="package://ant_description/meshes/wheels/caster_2_v2.stl"/>
         </geometry>
         <material name="DarkGrey"/>
