Commit message: removes ant from bumper
git-svn-id: svn+ssh://server/srv/svn/repos/trunk/pal-ros-pkg/catkin_pkgs/ant_robot@52884 5e370ff8-3418-0410-babe-3378cc20a00d

File: ant_description/urdf/sensors/bumper.gazebo.xacro (robot description, xacro)
@@ -8,5 +8,5 @@
 -->
 <robot xmlns:xacro="http://ros.org/wiki/xacro">
-  <xacro:macro name="bumper_ant_gazebo" params="name ros_topic update_rate">
+  <xacro:macro name="bumper_gazebo" params="name ros_topic update_rate">
     <gazebo reference="${name}_link">
       <selfCollide>false</selfCollide>
@@ -15,5 +15,5 @@
         <update_rate>${update_rate}</update_rate>
         <visualize>false</visualize>
-        <plugin filename="libgazebo_ros_bumper.so" name="gazebo_ant_ros_bumper">
+        <plugin filename="libgazebo_ros_bumper.so" name="gazebo_ros_bumper">
           <alwaysOn>true</alwaysOn>
           <updateRate>${update_rate}</updateRate>

File: ant_description/urdf/sensors/bumper.urdf.xacro (robot description, xacro)
@@ -9,5 +9,5 @@
 <robot xmlns:xacro="http://ros.org/wiki/xacro">
   <xacro:include filename="$(find ant_description)/urdf/sensors/bumper.gazebo.xacro" />
-  <xacro:macro name="bumper_ant" params="name parent ros_topic update_rate *origin">
+  <xacro:macro name="bumper" params="name parent ros_topic update_rate *origin">
      <joint name="${name}_joint" type="fixed">
         <axis xyz="0 1 0" />
@@ -37,5 +37,5 @@
        </link>
     <!-- gazebo extensions -->
-    <xacro:bumper_ant_gazebo name="${name}" ros_topic="${ros_topic}" update_rate="${update_rate}" />
+    <xacro:bumper_gazebo name="${name}" ros_topic="${ros_topic}" update_rate="${update_rate}" />
   </xacro:macro>
 </robot>
