Commit message: removes ant from range gazebo
git-svn-id: svn+ssh://server/srv/svn/repos/trunk/pal-ros-pkg/catkin_pkgs/ant_robot@52885 5e370ff8-3418-0410-babe-3378cc20a00d

File: ant_description/urdf/sensors/range.gazebo.xacro (robot description, xacro)
@@ -8,5 +8,5 @@
 -->
 <robot xmlns:xacro="http://ros.org/wiki/xacro">
-  <xacro:macro name="range_ant_gazebo" params="name ros_topic update_rate maxRange minRange fov radiation" >
+  <xacro:macro name="range_gazebo" params="name ros_topic update_rate maxRange minRange fov radiation" >
     <gazebo reference="${name}_link">
       <sensor type="ray" name="${name}">

File: ant_description/urdf/sensors/range.urdf.xacro (robot description, xacro)
@@ -24,5 +24,5 @@
     </joint>
     <!-- gazebo extensions -->
-    <xacro:range_ant_gazebo name="${name}" ros_topic="${ros_topic}" update_rate="${update_rate}" maxRange="${maxRange}" minRange="${minRange}" fov="${fov}" radiation="${radiation}"/>
+    <xacro:range_gazebo name="${name}" ros_topic="${ros_topic}" update_rate="${update_rate}" maxRange="${maxRange}" minRange="${minRange}" fov="${fov}" radiation="${radiation}"/>
   </xacro:macro>
 </robot>
