Commit message: reduces frequency from 1kHz to 100Hz and removes visual
git-svn-id: svn+ssh://server/srv/svn/repos/trunk/pal-ros-pkg/catkin_pkgs/ant_robot@52928 5e370ff8-3418-0410-babe-3378cc20a00d

File: ant_description/urdf/sensors/imu.urdf.xacro (robot description, xacro)
@@ -15,10 +15,10 @@
         <inertia ixx="0.000001" ixy="0" ixz="0" iyy="0.000001" iyz="0" izz="0.000001"/>
       </inertial>
-      <visual>
+      <!--visual>
         <origin rpy="0 0 0" xyz="0 0 0"/>
         <geometry>
           <box size="0.01 0.01 0.01"/>
         </geometry>
-      </visual>
+      </visual-->
     </link>
     <joint name="${name}_joint" type="fixed">
@@ -30,5 +30,5 @@
       <sensor name="${name}_sensor" type="imu">
         <always_on>1</always_on>
-        <update_rate>1000.0</update_rate>
+        <update_rate>100.0</update_rate>
         <imu>
           <noise>
