Commit message: reduces height
git-svn-id: svn+ssh://server/srv/svn/repos/trunk/pal-ros-pkg/catkin_pkgs/ant_robot@52929 5e370ff8-3418-0410-babe-3378cc20a00d

File: ant_description/urdf/sensors/bumper.urdf.xacro (robot description, xacro)
@@ -24,5 +24,5 @@
            <origin xyz="0 0 0" rpy="0 0 0" />
            <geometry>
-              <box size="0.01 0.25 0.05"/>
+              <box size="0.01 0.25 0.04"/>
            </geometry>
            <material name="DarkGrey"/>
@@ -31,5 +31,5 @@
            <origin xyz="0 0 0" rpy="0 0 0" />
            <geometry>
-              <box size="0.01 0.25 0.05"/>
+              <box size="0.01 0.25 0.04"/>
            </geometry>
            <material name="DarkGrey" />
