Commit message: refs #8415 : adds IR receiver visual
git-svn-id: svn+ssh://server/srv/svn/repos/trunk/pal-ros-pkg/catkin_pkgs/ant_robot@55177 5e370ff8-3418-0410-babe-3378cc20a00d

File: ant_description/urdf/sensors/ir_receiver.urdf.xacro (robot description, xacro)
@@ -16,4 +16,11 @@
         <inertia ixx="0.0001" ixy="0" ixz="0" iyy="0.000001" iyz="0" izz="0.0001" />
       </inertial>
+      <visual>
+        <origin xyz="0 0 0" rpy="0 0 0" />
+        <geometry>
+          <cylinder radius="0.01" length="0.01" />
+        </geometry>
+        <material name="DarkGrey" />
+      </visual>
     </link>
     <joint name="${name}_joint" type="fixed">
