Commit message: fixes softkinetic DS311 URDF
NOTE now it uses the same topic names as the real driver


git-svn-id: svn+ssh://server/srv/svn/repos/trunk/pal-ros-pkg/catkin_pkgs/ant_robot@57763 5e370ff8-3418-0410-babe-3378cc20a00d

File: ant_description/urdf/sensors/softkinetic_ds311_rgbd_camera.gazebo.xacro (robot description, xacro)
@@ -12,9 +12,9 @@
 -->
 <robot xmlns:xacro="http://ros.org/wiki/xacro">
-  <xacro:macro name="openni_camera_gazebo_v0" params="name">
+  <xacro:macro name="softkinetic_ds311_rgbd_camera_gazebo" params="name">
     <gazebo reference="${name}_link">
       <sensor type="depth" name="${name}_frame_sensor">
         <always_on>true</always_on>
-        <update_rate>30.0</update_rate>
+        <update_rate>10.0</update_rate>
         <camera>
           <horizontal_fov>${58.0 * deg_to_rad}</horizontal_fov>
@@ -31,42 +31,11 @@
         <plugin name="${name}_frame_controller" filename="libgazebo_ros_openni_kinect.so">
           <alwaysOn>true</alwaysOn>
-          <updateRate>30.0</updateRate>
-          <cameraName>${name}</cameraName>
-          <imageTopicName>ir/image_raw</imageTopicName>
-          <cameraInfoTopicName>/ir/camera_info</cameraInfoTopicName>
-          <depthImageTopicName>depth/image_raw</depthImageTopicName>
-          <depthImageCameraInfoTopicName>depth/camera_info</depthImageCameraInfoTopicName>
-          <pointCloudTopicName>depth/points</pointCloudTopicName>
-          <frameName>${name}_optical_frame</frameName>
-          <pointCloudCutoff>0.5</pointCloudCutoff>
-          <distortionK1>0.00000001</distortionK1>
-          <distortionK2>0.00000001</distortionK2>
-          <distortionK3>0.00000001</distortionK3>
-          <distortionT1>0.00000001</distortionT1>
-          <distortionT2>0.00000001</distortionT2>
-        </plugin>
-      </sensor>
-      <sensor type="depth" name="${name}_frame_sensor">
-        <always_on>true</always_on>
-        <update_rate>30.0</update_rate>
-        <camera>
-          <horizontal_fov>${58.0 * deg_to_rad}</horizontal_fov>
-          <image>
-            <format>R8G8B8</format>
-            <width>640</width>
-            <height>480</height>
-          </image>
-          <clip>
-            <near>0.8</near>
-            <far>3.5</far>
-          </clip>
-        </camera>
-        <plugin name="${name}_frame_controller" filename="libgazebo_ros_openni_kinect.so">
-          <alwaysOn>true</alwaysOn>
-          <updateRate>30.0</updateRate>
-          <cameraName>${name}</cameraName>
-          <imageTopicName>rgb/image_raw</imageTopicName>
-          <pointCloudTopicName>rgb/points</pointCloudTopicName>
-          <cameraInfoTopicName>rgb/camera_info</cameraInfoTopicName>
+          <updateRate>10.0</updateRate>
+          <cameraName>softkinetic_camera</cameraName>
+          <imageTopicName>rgb_data/image_raw</imageTopicName>
+          <cameraInfoTopicName>rgb_data/camera_info</cameraInfoTopicName>
+          <depthImageTopicName>depth_registered/image_raw</depthImageTopicName>
+          <depthImageCameraInfoTopicName>depth_registered/camera_info</depthImageCameraInfoTopicName>
+          <pointCloudTopicName>depth_registered/points</pointCloudTopicName>
           <frameName>${name}_optical_frame</frameName>
           <pointCloudCutoff>0.5</pointCloudCutoff>

File: ant_description/urdf/sensors/softkinetic_ds311_rgbd_camera.urdf.xacro (robot description, xacro)
@@ -8,5 +8,5 @@
 -->
 <robot xmlns:xacro="http://ros.org/wiki/xacro">
-  <xacro:include filename="$(find ant_description)/urdf/sensors/openni.gazebo.xacro" />
+  <xacro:include filename="$(find ant_description)/urdf/sensors/softkinetic_ds311_rgbd_camera.gazebo.xacro" />
   <!-- Macro -->
   <xacro:macro name="softkinetic_ds311_rgbd_camera" params="name parent *origin *calibration_origin">
@@ -18,14 +18,14 @@
     <link name="${name}_link">
       <inertial>
-        <mass value="0.01" />
+        <mass value="0.01"/>
         <origin xyz="0 0 0" rpy="0 0 0"/>
         <inertia ixx="0.0"  ixy="0.0"  ixz="0.0"
                  iyy="0.0"  iyz="0.0"
-                 izz="0.0" />
+                 izz="0.0"/>
       </inertial>
       <visual>
         <origin xyz="0 0 0" rpy="0 0 0"/>
         <geometry>
-          <mesh filename="package://ant_description/meshes/sensors/softkinetic/softkinetic.dae" />
+          <mesh filename="package://ant_description/meshes/sensors/softkinetic/softkinetic.dae"/>
         </geometry>
         <material name="Grey">
@@ -41,5 +41,5 @@
     </link>
     <joint name="${name}_optical_joint" type="fixed">
-      <insert_block name="calibration_origin" />
+      <insert_block name="calibration_origin"/>
       <parent link="${name}_link"/>
       <child link="${name}_optical_frame"/>
@@ -47,13 +47,13 @@
     <link name="${name}_optical_frame">
       <inertial>
-        <mass value="0.01" />
+        <mass value="0.01"/>
         <origin xyz="0 0 0" rpy="0 0 0"/>
         <inertia ixx="0.0"  ixy="0.0"  ixz="0.0"
                  iyy="0.0"  iyz="0.0"
-                 izz="0.0" />
+                 izz="0.0"/>
       </inertial>
     </link>
     <!-- extensions -->
-    <xacro:openni_camera_gazebo_v0 name="${name}" />
+    <xacro:softkinetic_ds311_rgbd_camera_gazebo name="${name}"/>
   </xacro:macro>
 </robot>
