Commit message: stl was converted to m (no scaling needed anymore)
git-svn-id: svn+ssh://server/srv/svn/repos/trunk/pal-ros-pkg/catkin_pkgs/ant_robot@52938 5e370ff8-3418-0410-babe-3378cc20a00d

File: ant_description/urdf/sensors/hokuyo_urg_04lx_ug01_laser.urdf.xacro (robot description, xacro)
@@ -19,5 +19,5 @@
         <origin xyz="0 0 0" rpy="0 0 0" />
         <geometry>
-          <mesh filename="package://ant_description/meshes/sensors/urg-04lx-ug01.stl" scale="0.001 0.001 0.001"/>
+          <mesh filename="package://ant_description/meshes/sensors/urg-04lx-ug01.stl"/>
         </geometry>
         <material name="DarkGrey" />

Commit message: renames hokuyo STL

File: ant_description/urdf/sensors/hokuyo_urg_04lx_ug01_laser.urdf.xacro (robot description, xacro)
@@ -21,5 +21,5 @@
         <origin xyz="0 0 0" rpy="0 0 0" />
         <geometry>
-          <mesh filename="package://ant_description/meshes/sensors/urg-04lx-ug01.stl"/>
+          <mesh filename="package://ant_description/meshes/sensors/hokuyo_urg_04lx_ug01.stl"/>
         </geometry>
         <material name="DarkGrey" />
