Commit message: replaces fixed by revolute joint for softkinetic

File: ant_description/urdf/sensors/softkinetic_ds311_rgbd_camera.urdf.xacro (robot description, xacro)
@@ -11,6 +11,8 @@
   <!-- Macro -->
   <xacro:macro name="softkinetic_ds311_rgbd_camera" params="name parent *origin *optical_origin">
-    <joint name="${name}_frame_joint" type="fixed">
-      <insert_block name="origin" />
+    <joint name="${name}_frame_joint" type="revolute">
+      <insert_block name="origin"/>
+      <axis xyz="0 0 1"/>
+      <limit lower="0" upper="0.001" effort="100" velocity="0.01"/>
       <parent link="${parent}_link"/>
       <child link="${name}_link"/>

Commit message: updates joint name

File: ant_description/urdf/sensors/softkinetic_ds311_rgbd_camera.urdf.xacro (robot description, xacro)
@@ -11,5 +11,5 @@
   <!-- Macro -->
   <xacro:macro name="softkinetic_ds311_rgbd_camera" params="name parent *origin *optical_origin">
-    <joint name="${name}_frame_joint" type="revolute">
+    <joint name="${name}_joint" type="revolute">
       <insert_block name="origin"/>
       <axis xyz="0 0 1"/>
