Commit message: renames gazebo macro

File: ant_description/urdf/sensors/xtion_pro_live.gazebo.xacro (robot description, xacro)
@@ -12,6 +12,7 @@
 -->
 <robot xmlns:xacro="http://ros.org/wiki/xacro">
-  <xacro:macro name="openni_camera_gazebo_v0" params="name">
+  <xacro:macro name="xtion_pro_live_rgbd_camera_gazebo" params="name">
     <gazebo reference="${name}_link">
+      <!-- IR + depth -->
       <sensor type="depth" name="${name}_frame_sensor">
         <always_on>true</always_on>
@@ -47,4 +48,5 @@
         </plugin>
       </sensor>
+      <!-- RGB -->
       <sensor type="depth" name="${name}_frame_sensor">
         <always_on>true</always_on>

File: ant_description/urdf/sensors/xtion_pro_live.urdf.xacro (robot description, xacro)
@@ -69,5 +69,5 @@
     </link>
     <!-- extensions -->
-    <xacro:openni_camera_gazebo_v0 name="${name}" />
+    <xacro:xtion_pro_live_rgbd_camera_gazebo name="${name}" />
   </xacro:macro>
 </robot>
