Commit message: adds rgbd (with xtion) urdf
git-svn-id: svn+ssh://server/srv/svn/repos/trunk/pal-ros-pkg/catkin_pkgs/ant_robot@57368 5e370ff8-3418-0410-babe-3378cc20a00d

File: ant_description/urdf/sensors/xtion_pro_live.urdf.xacro (robot description, xacro)
@@ -23,5 +23,5 @@
     <joint name="${name}_frame_joint" type="fixed">
       <insert_block name="origin" />
-      <parent link="${parent}"/>
+      <parent link="${parent}_link"/>
       <child link="${name}_link"/>
     </joint>

Commit message: replace fixed by revolute joint
Fixed joints are not fully supported by Gazebo. The joint specifying the pose of the xtion camera wrt base_link has been replaced by a 0 limits revolute joint. Fixes #10160

File: ant_description/urdf/sensors/xtion_pro_live.urdf.xacro (robot description, xacro)
@@ -21,6 +21,8 @@
   <!-- Macro -->
   <xacro:macro name="xtion_pro_live" params="name parent *origin *optical_origin">
-    <joint name="${name}_frame_joint" type="fixed">
+   <joint name="${name}_frame_joint" type="revolute">
       <insert_block name="origin" />
+      <axis xyz="0 0 1" />
+      <limit lower="0" upper="0.001" effort="100" velocity="0.01"/>
       <parent link="${parent}_link"/>
       <child link="${name}_link"/>

Commit message: fix

File: ant_description/urdf/sensors/xtion_pro_live.urdf.xacro (robot description, xacro)
@@ -21,7 +21,8 @@
   <!-- Macro -->
   <xacro:macro name="xtion_pro_live" params="name parent *origin *optical_origin">
-   <joint name="${name}_frame_joint" type="revolute">
-      <insert_block name="origin" />
-      <axis xyz="0 0 1" />
+    <!-- frames in the center of the camera -->
+    <joint name="${name}_joint" type="revolute">
+      <insert_block name="origin"/>
+      <axis xyz="0 0 1"/>
       <limit lower="0" upper="0.001" effort="100" velocity="0.01"/>
       <parent link="${parent}_link"/>

Commit message: adds inertia tensor
without this the simulation was crashing

File: ant_description/urdf/sensors/xtion_pro_live.urdf.xacro (robot description, xacro)
@@ -33,7 +33,8 @@
         <mass value="0.01" />
         <origin xyz="0 0 0" rpy="0 0 0"/>
-        <inertia ixx="0.0"  ixy="0.0"  ixz="0.0"
-                 iyy="0.0"  iyz="0.0"
-                 izz="0.0" />
+        <!-- inertia tensor computed analytically for a solid cuboid -->
+        <inertia ixx="0.000030"  ixy="0.0"  ixz="0.0"
+                 iyy="0.000030"  iyz="0.0"
+                 izz="0.000002" />
       </inertial>
       <visual>

Commit message: adds depth and rgb frames

File: ant_description/urdf/sensors/xtion_pro_live.urdf.xacro (robot description, xacro)
@@ -68,4 +68,30 @@
       </inertial>
     </link>
+    <!-- frames of the depth sensor -->
+    <joint name="${name}_depth_joint" type="fixed">
+      <origin xyz="0.0 0.049 0.0" rpy="0 0 0" />
+      <parent link="${name}_link" />
+      <child link="${name}_depth_frame"/>
+    </joint>
+    <link name="${name}_depth_frame"/>
+    <joint name="${name}_depth_optical_joint" type="fixed">
+      <origin xyz="0 0 0" rpy="${-90.0 * deg_to_rad} 0.0 ${-90.0 * deg_to_rad}" />
+      <parent link="${name}_depth_frame" />
+      <child link="${name}_depth_optical_frame"/>
+    </joint>
+    <link name="${name}_depth_optical_frame"/>
+    <!-- frames of the rgb sensor -->
+    <joint name="${name}_rgb_joint" type="fixed">
+      <origin xyz="0.0 0.022 0.0" rpy="0 0 0" />
+      <parent link="${name}_link" />
+      <child link="${name}_rgb_frame"/>
+    </joint>
+    <link name="${name}_rgb_frame"/>
+    <joint name="${name}_rgb_optical_joint" type="fixed">
+      <origin xyz="0 0 0" rpy="${-90.0 * deg_to_rad} 0.0 ${-90.0 * deg_to_rad}" />
+      <parent link="${name}_rgb_frame" />
+      <child link="${name}_rgb_optical_frame"/>
+    </joint>
+    <link name="${name}_rgb_optical_frame"/>
     <!-- extensions -->
     <xacro:xtion_pro_live_rgbd_camera_gazebo name="${name}" />
