Commit message: refs #8415 : disables gazebo emitter part
NOTE the plugin is NOT available yet


git-svn-id: svn+ssh://server/srv/svn/repos/trunk/pal-ros-pkg/catkin_pkgs/ant_robot@55186 5e370ff8-3418-0410-babe-3378cc20a00d

File: ant_description/urdf/dock/dock.urdf.xacro (robot description, xacro)
@@ -48,4 +48,16 @@
       <parent link="${name}_footprint"/>
     </joint>
+    <!-- IR emitter -->
+    <xacro:ir_emitter name="${name}_ir_emitter_01" parent="${name}" code="0" range_min="0.0" range_max="0.75" fov="0.5">
+      <origin xyz="0.17131 0.0 0.280" rpy="0.0 0.0 0.0" />
+    </xacro:ir_emitter>
+    <!-- IR emitter -->
+    <xacro:ir_emitter name="${name}_ir_emitter_02" parent="${name}" code="0" range_min="0.0" range_max="0.75" fov="0.5">
+      <origin xyz="0.16919 0.14919 0.280" rpy="0.0 0.0 0.349" />
+    </xacro:ir_emitter>
+    <!-- IR emitter -->
+    <xacro:ir_emitter name="${name}_ir_emitter_03" parent="${name}" code="0" range_min="0.0" range_max="0.75" fov="0.5">
+      <origin xyz="0.16919 -0.14919 0.280" rpy="0.0 0.0 -0.349" />
+    </xacro:ir_emitter>
   </xacro:macro>
 </robot>

File: ant_description/urdf/sensors/ir_emitter.urdf.xacro (robot description, xacro)
@@ -31,5 +31,5 @@
     </joint>
     <!-- gazebo extensions -->
-    <xacro:ir_emitter_gazebo name="${name}" code="${code}" range_min="${range_min}" range_max="${range_max}" fov="${fov}"/>
+    <!--xacro:ir_emitter_gazebo name="${name}" code="${code}" range_min="${range_min}" range_max="${range_max}" fov="${fov}"/-->
   </xacro:macro>
 </robot>
