Commit message: refs #8173 : removes sick laser and uses hokuyo one (also removes torso laser)
git-svn-id: svn+ssh://server/srv/svn/repos/trunk/pal-ros-pkg/catkin_pkgs/ant_robot@51926 5e370ff8-3418-0410-babe-3378cc20a00d

File: ant_description/urdf/base/base.urdf.xacro (robot description, xacro)
@@ -11,15 +11,14 @@
   <xacro:include filename="$(find ant_description)/urdf/base/base.gazebo.xacro" />
   <xacro:include filename="$(find ant_description)/urdf/base/base.transmission.xacro" />
-  <xacro:include filename="$(find ant_description)/urdf/sensors/sick_laser_ant.urdf.xacro" />
   <xacro:include filename="$(find ant_description)/urdf/sensors/range.urdf.xacro" />
-  <xacro:include filename="$(find ant_description)/urdf/sensors/hokuyo_laser_ant.urdf.xacro" />
+  <xacro:include filename="$(find ant_description)/urdf/sensors/hokuyo_urg_04lx_ug01_laser.urdf.xacro" />
   <xacro:include filename="$(find ant_description)/urdf/sensors/imu.urdf.xacro"/>
   <xacro:include filename="$(find ant_description)/urdf/sensors/bumper.urdf.xacro" />
   <!--wheel characteristics-->
-  <property name="dist_between_wheels" value="0.540" />
-  <property name="wheel_radius" value="0.093" />
-  <property name="wheel_width" value="0.044" />
-  <property name="wheel_torque" value="50.0" />
-  <property name="wheel_velocity" value="1.5" /> <!-- m/s -->
+  <property name="wheel_separation" value="0.540" />
+  <property name="wheel_radius"     value="0.093" />
+  <property name="wheel_width"      value="0.044" />
+  <property name="wheel_torque"     value="50.0" />
+  <property name="wheel_velocity"   value="1.0" /> <!-- m/s -->
  <!--caster characteristics-->
   <property name="dist_between_casters" value="0.300" />
@@ -65,5 +64,5 @@
       <parent link="base_link" />
       <child link="wheel_${side}_link" />
-      <origin xyz="0 ${-dist_between_wheels / 2 * reflect} ${wheel_radius}" rpy="${-90.0 * deg_to_rad} 0 0" />
+      <origin xyz="0 ${-wheel_separation / 2 * reflect} ${wheel_radius}" rpy="${-90.0 * deg_to_rad} 0 0" />
       <axis xyz="0 0 1" />
       <limit effort="${wheel_torque}" velocity="${wheel_velocity / wheel_radius}"/>
@@ -142,12 +141,8 @@
     </joint>
   </xacro:macro>
-  <!-- simplified box collision geometry for sick laser -->
+  <!-- simplified box collision geometry for the laser -->
   <property name="base_laser_x" value="0.0468" />
   <property name="base_laser_y" value="0.0" />
   <property name="base_laser_z" value="0.081" />
-  <!-- simplified box collision geometry for hokuyo laser -->
-  <property name="torso_laser_x" value="0.0073" />
-  <property name="torso_laser_y" value="0.0" />
-  <property name="torso_laser_z" value="0.77" />
   <!-- base_link x-axis offset -->
   <property name="base_link_offset_x" value="-0.0327"/>
@@ -229,61 +224,57 @@
       <parent link="${name}_link"/>
     </joint>
-   <!-- base laser -->
-    <xacro:sick_ant_laser name="${name}_laser" parent="${name}" ros_topic="scan_filtered" update_rate="25" min_angle="${-79 * deg_to_rad}" max_angle="${79 * deg_to_rad}" >
-      <origin xyz="${base_laser_x} ${base_laser_y} ${base_laser_z}" rpy="${180.0 * deg_to_rad} 0 0" />
-    </xacro:sick_ant_laser>
-   <!-- torso laser -->
-    <xacro:hokuyo_ant_laser name="${name}_torso_laser" parent="${name}" ros_topic="hokuyo/LAS_01" update_rate="10" min_angle="${-63 * deg_to_rad}" max_angle="${63 * deg_to_rad}" >
-      <origin xyz="${torso_laser_x} ${torso_laser_y} ${torso_laser_z}" rpy="-0.03 ${52 * deg_to_rad} -0.05" />
-    </xacro:hokuyo_ant_laser>
-    <!-- base sonar -->
+    <!-- laser -->
+    <xacro:hokuyo_urg_04lx_ug01_laser name="${name}_laser" parent="${name}" ros_topic="scan" update_rate="10" min_angle="${-120 * deg_to_rad}" max_angle="${120 * deg_to_rad}" >
+      <origin xyz="${base_laser_x} ${base_laser_y} ${base_laser_z}" rpy="0 0 0" />
+    </xacro:hokuyo_urg_04lx_ug01_laser>
+    <!-- sonar -->
     <xacro:range_ant name="${name}_sonar_02" parent="${name}" ros_topic="sonar_base" update_rate="5" maxRange="0.75" minRange="0.01" fov="0.5" radiation="ultrasound">
       <origin xyz="${0.17131 + base_link_offset_x} 0.0 0.280" rpy="0.0 0.0 0.0" />
     </xacro:range_ant>
-    <!-- base sonar -->
+    <!-- sonar -->
     <xacro:range_ant name="${name}_sonar_03" parent="${name}" ros_topic="sonar_base" update_rate="5" maxRange="0.75" minRange="0.01" fov="0.5" radiation="ultrasound">
       <origin xyz="${0.16919 + base_link_offset_x} 0.14919 0.280" rpy="0.0 0.0 0.349" />
     </xacro:range_ant>
-   <!-- base sonar -->
+    <!-- sonar -->
     <xacro:range_ant name="${name}_sonar_01" parent="${name}" ros_topic="sonar_base" update_rate="5" maxRange="0.75" minRange="0.01" fov="0.5" radiation="ultrasound">
       <origin xyz="${0.16919 + base_link_offset_x} -0.14919 0.280" rpy="0.0 0.0 -0.349" />
     </xacro:range_ant>
-   <!-- base sonar -->
+    <!-- sonar -->
     <xacro:range_ant name="${name}_sonar_04" parent="${name}" ros_topic="sonar_base" update_rate="5" maxRange="0.75" minRange="0.01" fov="0.5" radiation="ultrasound">
       <origin xyz="${0.13676 + base_link_offset_x} 0.27111 0.280" rpy="0.0 0.0 0.8377" />
     </xacro:range_ant>
-   <!-- base sonar -->
+    <!-- sonar -->
     <xacro:range_ant name="${name}_sonar_12" parent="${name}" ros_topic="sonar_base" update_rate="5" maxRange="0.75" minRange="0.01" fov="0.5" radiation="ultrasound">
       <origin xyz="${0.13676 + base_link_offset_x} -0.27111 0.280" rpy="0.0 0.0 -0.8377" />
     </xacro:range_ant>
-   <!-- base sonar -->
+    <!-- sonar -->
     <xacro:range_ant name="${name}_sonar_05" parent="${name}" ros_topic="sonar_base" update_rate="5" maxRange="0.5" minRange="0.01" fov="0.5" radiation="ultrasound">
       <origin xyz="${-0.14 + base_link_offset_x} 0.33455 0.27" rpy="0.0 0.0 1.5708" />
     </xacro:range_ant>
-   <!-- base sonar -->
+    <!-- sonar -->
     <xacro:range_ant name="${name}_sonar_11" parent="${name}" ros_topic="sonar_base" update_rate="5" maxRange="0.5" minRange="0.01" fov="0.5" radiation="ultrasound">
       <origin xyz="${-0.14 + base_link_offset_x} -0.33455 0.27" rpy="0.0 0.0 -1.5708" />
     </xacro:range_ant>
-   <!-- base sonar -->
+    <!-- sonar -->
     <xacro:range_ant name="${name}_sonar_06" parent="${name}" ros_topic="sonar_base" update_rate="5" maxRange="0.5" minRange="0.005" fov="0.5" radiation="ultrasound">
       <origin xyz="${-0.35563 + base_link_offset_x} 0.28266 0.25" rpy="0.0 0.0 1.9547" />
     </xacro:range_ant>
-   <!-- base sonar -->
+    <!-- sonar -->
     <xacro:range_ant name="${name}_sonar_10" parent="${name}" ros_topic="sonar_base" update_rate="5" maxRange="0.5" minRange="0.005" fov="0.5" radiation="ultrasound">
       <origin xyz="${-0.35563 + base_link_offset_x} -0.28266 0.25" rpy="0.0 0.0 -1.9547" />
     </xacro:range_ant>
-   <!-- base sonar -->
+    <!-- sonar -->
     <xacro:range_ant name="${name}_sonar_07" parent="${name}" ros_topic="sonar_base" update_rate="5" maxRange="0.7" minRange="0.01" fov="0.5" radiation="ultrasound">
       <origin xyz="${-0.48412 + base_link_offset_x} 0.15127 0.29" rpy="0.0 0.0 2.6354" />
     </xacro:range_ant>
-   <!-- base sonar -->
+    <!-- sonar -->
     <xacro:range_ant name="${name}_sonar_09" parent="${name}" ros_topic="sonar_base" update_rate="5" maxRange="0.7" minRange="0.01" fov="0.5" radiation="ultrasound">
       <origin xyz="${-0.48412 + base_link_offset_x} -0.15127 0.29" rpy="0.0 0.0 -2.6354" />
     </xacro:range_ant>
-   <!-- base sonar -->
+    <!-- sonar -->
     <xacro:range_ant name="${name}_sonar_08" parent="${name}" ros_topic="sonar_base" update_rate="5" maxRange="0.7" minRange="0.01" fov="0.5" radiation="ultrasound">
       <origin xyz="${-0.51188 + base_link_offset_x} 0.0 0.26" rpy="0.0 0.0 -3.1415" />
     </xacro:range_ant>
-   <!-- base ir -->
+    <!-- ir -->
     <xacro:range_ant name="${name}_ir_01" parent="${name}" ros_topic="ir_base" update_rate="10" maxRange="1.45" minRange="0.01" fov="0.1" radiation="infrared">
       <origin xyz="${0.1804 + base_link_offset_x} -0.12463 0.22" rpy="0.0 -0.8726 0.0" />

File: ant_description/urdf/sensors/hokuyo_urg_04lx_ug01_laser.gazebo.xacro (robot description, xacro)
@@ -6,11 +6,12 @@
   To view a copy of this license, visit http://creativecommons.org/licenses/by-nc-nd/3.0/ or send a letter to
   Creative Commons, 444 Castro Street, Suite 900, Mountain View, California, 94041, USA.
+  Laser configuraiton according with the Hokuyo URG-04LX-UG01 product specification:
+  http://www.hokuyo-aut.jp/02sensor/07scanner/download/products/urg-04lx-ug01/data/URG-04LX_UG01_spec_en.pdf
 -->
 <robot xmlns:xacro="http://ros.org/wiki/xacro">
-  <xacro:include filename="$(find ant_description)/urdf/deg_to_rad.xacro" />
-  <xacro:macro name="sick_ant_laser_gazebo" params="name ros_topic update_rate min_angle max_angle">
+  <xacro:macro name="hokuyo_urg_04lx_ug01_laser_gazebo" params="name ros_topic update_rate min_angle max_angle">
     <gazebo reference="${name}_link">
       <sensor type="ray" name="${name}">
-        <pose>0 0 0 ${180 * deg_to_rad} 0 0</pose>
+        <pose>0 0 0 0 0 0</pose>
         <update_rate>${update_rate}</update_rate>
         <visualize>true</visualize>
@@ -18,6 +19,7 @@
           <scan>
             <horizontal>
-              <samples>513</samples>
-              <resolution>1</resolution>
+              <!-- 683 steps in 240deg fov -->
+              <samples>${683*(max_angle - min_angle)/(240.0 * deg_to_rad)}</samples>
+              <resolution>1</resolution> <!-- not the sensor resolution; just 1 -->
               <min_angle>${min_angle}</min_angle>
               <max_angle>${max_angle}</max_angle>
@@ -25,11 +27,11 @@
           </scan>
           <range>
-            <min>0.08</min>
-            <max>20.0</max>
-            <resolution>0.01</resolution>
+            <min>0.02</min>
+            <max>4.0</max>
+            <resolution>0.001</resolution>
           </range>
         </ray>
-        <plugin filename="libgazebo_ros_laser.so" name="gazebo_ros_sick_laser">
-          <gaussianNoise>0.005</gaussianNoise>
+        <plugin filename="libgazebo_ros_laser.so" name="gazebo_ros_hokuyo_laser">
+          <gaussianNoise>0.03</gaussianNoise>
           <alwaysOn>true</alwaysOn>
           <updateRate>${update_rate}</updateRate>

File: ant_description/urdf/sensors/hokuyo_urg_04lx_ug01_laser.urdf.xacro (robot description, xacro)
@@ -8,34 +8,30 @@
 -->
 <robot xmlns:xacro="http://ros.org/wiki/xacro">
-  <xacro:include filename="$(find ant_description)/urdf/sensors/sick_laser_ant.gazebo.xacro" />
-  <xacro:macro name="sick_ant_laser" params="name parent *origin ros_topic update_rate min_angle max_angle">
+  <xacro:include filename="$(find ant_description)/urdf/sensors/hokuyo_urg_04lx_ug01_laser.gazebo.xacro" />
+  <xacro:macro name="hokuyo_urg_04lx_ug01_laser" params="name parent *origin ros_topic update_rate min_angle max_angle">
      <link name="${name}_link" type="laser">
       <inertial>
-        <mass value="1" />
         <origin xyz="0 0 0" rpy="0 0 0" />
-        <inertia ixx="0.0001" ixy="0" ixz="0" iyy="0.000001" iyz="0" izz="0.0001" />
+        <mass value="0.001" />
+        <inertia iyy="4.2412e-05" ixy="4.9927e-08" iyz="-9.8165e-09" ixx="3.7174e-05" ixz="1.1015e-05" izz="4.167e-05" />
       </inertial>
       <visual>
         <origin xyz="0 0 0" rpy="0 0 0" />
         <geometry>
-          <box size="0.05 0.05 0.05" />
+          <mesh filename="package://ant_description/meshes/sensors/urg-04lx-ug01.stl" scale="0.001 0.001 0.001"/>
         </geometry>
         <material name="DarkGrey" />
       </visual>
-      <collision>
-        <origin xyz="0 0 0" rpy="0 0 0" />
-        <geometry>
-          <box size=".05 .05 .05" />
-        </geometry>
-      </collision>
     </link>
     <joint name="${name}_joint" type="fixed">
       <axis xyz="0 1 0" />
       <insert_block name="origin" />
-      <parent link="base_link"/>
-      <child link="${name}_link"/>
+      <parent link="${parent}_link"/>
+      <child  link="${name}_link"/>
+      <dynamics friction="1.0" damping="1"/>
+      <limit lower="0" upper="0" effort="60" velocity="20" />
     </joint>
     <!-- gazebo extensions -->
-    <xacro:sick_ant_laser_gazebo name="${name}" ros_topic="${ros_topic}" update_rate="${update_rate}" min_angle="${min_angle}" max_angle="${max_angle}" />
+    <xacro:hokuyo_urg_04lx_ug01_laser_gazebo name="${name}" ros_topic="${ros_topic}" update_rate="${update_rate}" min_angle="${min_angle}" max_angle="${max_angle}" />
   </xacro:macro>
 </robot>

Commit message: refs #8137 : removes cargo and updates some wheel params
git-svn-id: svn+ssh://server/srv/svn/repos/trunk/pal-ros-pkg/catkin_pkgs/ant_robot@51939 5e370ff8-3418-0410-babe-3378cc20a00d

File: ant_description/urdf/base/base.urdf.xacro (robot description, xacro)
@@ -15,9 +15,9 @@
   <xacro:include filename="$(find ant_description)/urdf/sensors/bumper.urdf.xacro" />
   <!--wheel characteristics-->
-  <property name="wheel_separation" value="0.540" />
-  <property name="wheel_radius"     value="0.093" />
-  <property name="wheel_width"      value="0.044" />
-  <property name="wheel_torque"     value="50.0" />
-  <property name="wheel_velocity"   value="1.0" /> <!-- m/s -->
+  <property name="wheel_separation" value="0.42"/>
+  <property name="wheel_radius"     value="0.1016"/>
+  <property name="wheel_width"      value="0.044"/>
+  <property name="wheel_torque"     value="50.0"/>
+  <property name="wheel_velocity"   value="1.0"/>
  <!--caster characteristics-->
   <property name="dist_between_casters" value="0.300" />
@@ -315,48 +315,12 @@
     <!-- imu -->
     <xacro:ant_imu name="base_inclinometer" parent="${name}_link" update_rate="100.0">
-      <origin xyz="-0.02977 -0.1497 0.164" rpy="0 ${M_PI} 0"/>
+      <origin xyz="-0.02977 -0.1497 0.164" rpy="0 ${180 * deg_to_rad} 0"/>
     </xacro:ant_imu>
     <!-- wheels -->
-    <xacro:ant_wheel side="right" reflect="1.0" />
-    <xacro:ant_wheel side="left" reflect="-1.0" />
+    <xacro:ant_wheel side="right" reflect=" 1.0"/>
+    <xacro:ant_wheel side="left"  reflect="-1.0"/>
     <!-- casters -->
-    <xacro:ant_caster side="right" reflect=" 1.0" />
-    <xacro:ant_caster side="left"  reflect="-1.0" />
-    <!-- extensions -->
-    <xacro:ant_base_controllers />
-  </xacro:macro>
-  <xacro:macro name="ant_cargo" params="name">
-    <!--************************-->
-    <!--        CARGO           -->
-    <!--************************-->
-    <link name="${name}_cargo_link">
-      <inertial>
-        <mass value="1.0" />
-        <origin xyz="0 0 0" />
-        <inertia ixx="0.01" ixy="0.0" ixz="0.0"
-                 iyy="0.01" iyz="0.0" izz="0.01" />
-        <!--<mass value="1.0" />
-        <origin xyz="0 0 -0.5" />
-        <inertia ixx="0.0" ixy="0.0" ixz="0.0" iyy="0.0" iyz="0.0" izz="0.0" />-->
-      </inertial>
-      <visual>
-        <origin xyz="0 0 -0.5" rpy="0 0 0" />
-        <geometry>
-          <box size="0.001 0.001 0.001" />
-        </geometry>
-        <material name="Green" />
-      </visual>
-      <collision>
-        <origin xyz="0.05 0 0.02" rpy="0 0 0" />
-        <geometry>
-          <box size="0.30 0.30 0.25" /> <!-- Generous hand luggage size allowed in an airplane is 0.55x0.45x0.25. This slightly smaller. -->
-        </geometry>
-      </collision>
-    </link>
-    <joint name="${name}_cargo_link" type="fixed">
-      <origin xyz="${-0.41 + base_link_offset_x} 0 ${0.605 + 0.029}" rpy="0 0.18 0" />
-      <child link="${name}_cargo_link" />
-      <parent link="${name}_link"/>
-    </joint>
+    <xacro:ant_caster side="right" reflect=" 1.0"/>
+    <xacro:ant_caster side="left"  reflect="-1.0"/>
   </xacro:macro>
 </robot>

Commit message: refs #8173 : sets sonars update rate to 10Hz (instead of 5Hz)
git-svn-id: svn+ssh://server/srv/svn/repos/trunk/pal-ros-pkg/catkin_pkgs/ant_robot@52026 5e370ff8-3418-0410-babe-3378cc20a00d

File: ant_description/urdf/base/base.urdf.xacro (robot description, xacro)
@@ -155,8 +155,4 @@
         <mass value="63.58850" />
         <inertia ixx="3.42"  ixy="0"  ixz="0" iyy="4.33" iyz="0" izz="5.08" /> <!-- assuming d=0.6, w=0.5, h=0.4 -->
-<!--         <origin xyz="-0.15006 -0.00031 0.24965" rpy="0 0 0" /> -->
-<!--         <mass value="64.063" /> -->
-        <!-- NOTE: Assuming box with d=0.6, w=0.5, h=0.4 -->
-<!--         <inertia ixx="3.42"  ixy="0"  ixz="0" iyy="4.33" iyz="0" izz="5.08" /> -->
       </inertial>
       <visual>
@@ -228,49 +224,49 @@
     </xacro:hokuyo_urg_04lx_ug01_laser>
     <!-- sonar -->
-    <xacro:range_ant name="${name}_sonar_02" parent="${name}" ros_topic="sonar_base" update_rate="5" maxRange="0.75" minRange="0.01" fov="0.5" radiation="ultrasound">
+    <xacro:range_ant name="${name}_sonar_02" parent="${name}" ros_topic="sonar_base" update_rate="10" maxRange="0.75" minRange="0.01" fov="0.5" radiation="ultrasound">
       <origin xyz="${0.17131 + base_link_offset_x} 0.0 0.280" rpy="0.0 0.0 0.0" />
     </xacro:range_ant>
     <!-- sonar -->
-    <xacro:range_ant name="${name}_sonar_03" parent="${name}" ros_topic="sonar_base" update_rate="5" maxRange="0.75" minRange="0.01" fov="0.5" radiation="ultrasound">
+    <xacro:range_ant name="${name}_sonar_03" parent="${name}" ros_topic="sonar_base" update_rate="10" maxRange="0.75" minRange="0.01" fov="0.5" radiation="ultrasound">
       <origin xyz="${0.16919 + base_link_offset_x} 0.14919 0.280" rpy="0.0 0.0 0.349" />
     </xacro:range_ant>
     <!-- sonar -->
-    <xacro:range_ant name="${name}_sonar_01" parent="${name}" ros_topic="sonar_base" update_rate="5" maxRange="0.75" minRange="0.01" fov="0.5" radiation="ultrasound">
+    <xacro:range_ant name="${name}_sonar_01" parent="${name}" ros_topic="sonar_base" update_rate="10" maxRange="0.75" minRange="0.01" fov="0.5" radiation="ultrasound">
       <origin xyz="${0.16919 + base_link_offset_x} -0.14919 0.280" rpy="0.0 0.0 -0.349" />
     </xacro:range_ant>
     <!-- sonar -->
-    <xacro:range_ant name="${name}_sonar_04" parent="${name}" ros_topic="sonar_base" update_rate="5" maxRange="0.75" minRange="0.01" fov="0.5" radiation="ultrasound">
+    <xacro:range_ant name="${name}_sonar_04" parent="${name}" ros_topic="sonar_base" update_rate="10" maxRange="0.75" minRange="0.01" fov="0.5" radiation="ultrasound">
       <origin xyz="${0.13676 + base_link_offset_x} 0.27111 0.280" rpy="0.0 0.0 0.8377" />
     </xacro:range_ant>
     <!-- sonar -->
-    <xacro:range_ant name="${name}_sonar_12" parent="${name}" ros_topic="sonar_base" update_rate="5" maxRange="0.75" minRange="0.01" fov="0.5" radiation="ultrasound">
+    <xacro:range_ant name="${name}_sonar_12" parent="${name}" ros_topic="sonar_base" update_rate="10" maxRange="0.75" minRange="0.01" fov="0.5" radiation="ultrasound">
       <origin xyz="${0.13676 + base_link_offset_x} -0.27111 0.280" rpy="0.0 0.0 -0.8377" />
     </xacro:range_ant>
     <!-- sonar -->
-    <xacro:range_ant name="${name}_sonar_05" parent="${name}" ros_topic="sonar_base" update_rate="5" maxRange="0.5" minRange="0.01" fov="0.5" radiation="ultrasound">
+    <xacro:range_ant name="${name}_sonar_05" parent="${name}" ros_topic="sonar_base" update_rate="10" maxRange="0.5" minRange="0.01" fov="0.5" radiation="ultrasound">
       <origin xyz="${-0.14 + base_link_offset_x} 0.33455 0.27" rpy="0.0 0.0 1.5708" />
     </xacro:range_ant>
     <!-- sonar -->
-    <xacro:range_ant name="${name}_sonar_11" parent="${name}" ros_topic="sonar_base" update_rate="5" maxRange="0.5" minRange="0.01" fov="0.5" radiation="ultrasound">
+    <xacro:range_ant name="${name}_sonar_11" parent="${name}" ros_topic="sonar_base" update_rate="10" maxRange="0.5" minRange="0.01" fov="0.5" radiation="ultrasound">
       <origin xyz="${-0.14 + base_link_offset_x} -0.33455 0.27" rpy="0.0 0.0 -1.5708" />
     </xacro:range_ant>
     <!-- sonar -->
-    <xacro:range_ant name="${name}_sonar_06" parent="${name}" ros_topic="sonar_base" update_rate="5" maxRange="0.5" minRange="0.005" fov="0.5" radiation="ultrasound">
+    <xacro:range_ant name="${name}_sonar_06" parent="${name}" ros_topic="sonar_base" update_rate="10" maxRange="0.5" minRange="0.005" fov="0.5" radiation="ultrasound">
       <origin xyz="${-0.35563 + base_link_offset_x} 0.28266 0.25" rpy="0.0 0.0 1.9547" />
     </xacro:range_ant>
     <!-- sonar -->
-    <xacro:range_ant name="${name}_sonar_10" parent="${name}" ros_topic="sonar_base" update_rate="5" maxRange="0.5" minRange="0.005" fov="0.5" radiation="ultrasound">
+    <xacro:range_ant name="${name}_sonar_10" parent="${name}" ros_topic="sonar_base" update_rate="10" maxRange="0.5" minRange="0.005" fov="0.5" radiation="ultrasound">
       <origin xyz="${-0.35563 + base_link_offset_x} -0.28266 0.25" rpy="0.0 0.0 -1.9547" />
     </xacro:range_ant>
     <!-- sonar -->
-    <xacro:range_ant name="${name}_sonar_07" parent="${name}" ros_topic="sonar_base" update_rate="5" maxRange="0.7" minRange="0.01" fov="0.5" radiation="ultrasound">
+    <xacro:range_ant name="${name}_sonar_07" parent="${name}" ros_topic="sonar_base" update_rate="10" maxRange="0.7" minRange="0.01" fov="0.5" radiation="ultrasound">
       <origin xyz="${-0.48412 + base_link_offset_x} 0.15127 0.29" rpy="0.0 0.0 2.6354" />
     </xacro:range_ant>
     <!-- sonar -->
-    <xacro:range_ant name="${name}_sonar_09" parent="${name}" ros_topic="sonar_base" update_rate="5" maxRange="0.7" minRange="0.01" fov="0.5" radiation="ultrasound">
+    <xacro:range_ant name="${name}_sonar_09" parent="${name}" ros_topic="sonar_base" update_rate="10" maxRange="0.7" minRange="0.01" fov="0.5" radiation="ultrasound">
       <origin xyz="${-0.48412 + base_link_offset_x} -0.15127 0.29" rpy="0.0 0.0 -2.6354" />
     </xacro:range_ant>
     <!-- sonar -->
-    <xacro:range_ant name="${name}_sonar_08" parent="${name}" ros_topic="sonar_base" update_rate="5" maxRange="0.7" minRange="0.01" fov="0.5" radiation="ultrasound">
+    <xacro:range_ant name="${name}_sonar_08" parent="${name}" ros_topic="sonar_base" update_rate="10" maxRange="0.7" minRange="0.01" fov="0.5" radiation="ultrasound">
       <origin xyz="${-0.51188 + base_link_offset_x} 0.0 0.26" rpy="0.0 0.0 -3.1415" />
     </xacro:range_ant>
