Commit message: refs #8173 : sets caster wheel radius to 16.4mm
git-svn-id: svn+ssh://server/srv/svn/repos/trunk/pal-ros-pkg/catkin_pkgs/ant_robot@52074 5e370ff8-3418-0410-babe-3378cc20a00d

File: ant_description/urdf/base/base.urdf.xacro (robot description, xacro)
@@ -23,5 +23,5 @@
   <property name="dist_between_casters" value="0.300"/>
   <property name="caster_radius"        value="0.025"/>
-  <property name="caster_width"         value="0.037"/>
+  <property name="caster_width"         value="0.0164"/>
   <property name="caster_trailing_dist" value="0.038"/>
   <xacro:macro name="ant_wheel" params="side reflect" parent="base_link">
@@ -145,5 +145,5 @@
   <property name="base_laser_z" value="0.081" />
   <!-- base_link x-axis offset -->
-  <property name="base_link_offset_x" value="-0.0327"/>
+  <property name="base_link_offset_x" value="0.0"/>
   <xacro:macro name="ant_base" params="name">
     <!--************************-->
@@ -152,5 +152,5 @@
     <link name="${name}_link">
       <inertial>
-        <origin xyz="-0.14527 -0.00003 0.24721" rpy="0 0 0" /> <!-- assuming d=0.6, w=0.5, h=0.4 -->
+        <origin xyz="0.0 0.0 0.24721" rpy="0 0 0" /> <!-- assuming d=0.6, w=0.5, h=0.4 -->
         <mass value="63.58850" />
         <inertia ixx="3.42"  ixy="0"  ixz="0" iyy="4.33" iyz="0" izz="5.08" /> <!-- assuming d=0.6, w=0.5, h=0.4 -->

Commit message: removes IRs (pointing up)
git-svn-id: svn+ssh://server/srv/svn/repos/trunk/pal-ros-pkg/catkin_pkgs/ant_robot@52510 5e370ff8-3418-0410-babe-3378cc20a00d

File: ant_description/urdf/base/base.urdf.xacro (robot description, xacro)
@@ -271,14 +271,4 @@
       <origin xyz="${-0.51188 + base_link_offset_x} 0.0 0.26" rpy="0.0 0.0 -3.1415" />
     </xacro:range_ant>
-    <!-- ir -->
-    <xacro:range_ant name="${name}_ir_01" parent="${name}" ros_topic="ir_base" update_rate="10" maxRange="1.45" minRange="0.01" fov="0.1" radiation="infrared">
-      <origin xyz="${0.1804 + base_link_offset_x} -0.12463 0.22" rpy="0.0 -0.8726 0.0" />
-    </xacro:range_ant>
-    <xacro:range_ant name="${name}_ir_02" parent="${name}" ros_topic="ir_base" update_rate="10" maxRange="1.45" minRange="0.01" fov="0.1" radiation="infrared">
-      <origin xyz="${0.18574 + base_link_offset_x} 0.0 0.22" rpy="0.0 -0.8726 0.0" />
-    </xacro:range_ant>
-    <xacro:range_ant name="${name}_ir_03" parent="${name}" ros_topic="ir_base" update_rate="10" maxRange="1.45" minRange="0.01" fov="0.1" radiation="infrared">
-      <origin xyz="${0.1804 + base_link_offset_x} 0.12463 0.22" rpy="0.0 -0.8726 0.0" />
-    </xacro:range_ant>
     <!-- bumper front right -->
     <xacro:bumper_ant name="${name}_bumper_01" parent="${name}" ros_topic="bumper_base" update_rate="25" >

Commit message: refs #8173 : removes sonars outside the front
git-svn-id: svn+ssh://server/srv/svn/repos/trunk/pal-ros-pkg/catkin_pkgs/ant_robot@52511 5e370ff8-3418-0410-babe-3378cc20a00d

File: ant_description/urdf/base/base.urdf.xacro (robot description, xacro)
@@ -235,40 +235,4 @@
       <origin xyz="${0.16919 + base_link_offset_x} -0.14919 0.280" rpy="0.0 0.0 -0.349" />
     </xacro:range_ant>
-    <!-- sonar -->
-    <xacro:range_ant name="${name}_sonar_04" parent="${name}" ros_topic="sonar_base" update_rate="10" maxRange="0.75" minRange="0.01" fov="0.5" radiation="ultrasound">
-      <origin xyz="${0.13676 + base_link_offset_x} 0.27111 0.280" rpy="0.0 0.0 0.8377" />
-    </xacro:range_ant>
-    <!-- sonar -->
-    <xacro:range_ant name="${name}_sonar_12" parent="${name}" ros_topic="sonar_base" update_rate="10" maxRange="0.75" minRange="0.01" fov="0.5" radiation="ultrasound">
-      <origin xyz="${0.13676 + base_link_offset_x} -0.27111 0.280" rpy="0.0 0.0 -0.8377" />
-    </xacro:range_ant>
-    <!-- sonar -->
-    <xacro:range_ant name="${name}_sonar_05" parent="${name}" ros_topic="sonar_base" update_rate="10" maxRange="0.5" minRange="0.01" fov="0.5" radiation="ultrasound">
-      <origin xyz="${-0.14 + base_link_offset_x} 0.33455 0.27" rpy="0.0 0.0 1.5708" />
-    </xacro:range_ant>
-    <!-- sonar -->
-    <xacro:range_ant name="${name}_sonar_11" parent="${name}" ros_topic="sonar_base" update_rate="10" maxRange="0.5" minRange="0.01" fov="0.5" radiation="ultrasound">
-      <origin xyz="${-0.14 + base_link_offset_x} -0.33455 0.27" rpy="0.0 0.0 -1.5708" />
-    </xacro:range_ant>
-    <!-- sonar -->
-    <xacro:range_ant name="${name}_sonar_06" parent="${name}" ros_topic="sonar_base" update_rate="10" maxRange="0.5" minRange="0.005" fov="0.5" radiation="ultrasound">
-      <origin xyz="${-0.35563 + base_link_offset_x} 0.28266 0.25" rpy="0.0 0.0 1.9547" />
-    </xacro:range_ant>
-    <!-- sonar -->
-    <xacro:range_ant name="${name}_sonar_10" parent="${name}" ros_topic="sonar_base" update_rate="10" maxRange="0.5" minRange="0.005" fov="0.5" radiation="ultrasound">
-      <origin xyz="${-0.35563 + base_link_offset_x} -0.28266 0.25" rpy="0.0 0.0 -1.9547" />
-    </xacro:range_ant>
-    <!-- sonar -->
-    <xacro:range_ant name="${name}_sonar_07" parent="${name}" ros_topic="sonar_base" update_rate="10" maxRange="0.7" minRange="0.01" fov="0.5" radiation="ultrasound">
-      <origin xyz="${-0.48412 + base_link_offset_x} 0.15127 0.29" rpy="0.0 0.0 2.6354" />
-    </xacro:range_ant>
-    <!-- sonar -->
-    <xacro:range_ant name="${name}_sonar_09" parent="${name}" ros_topic="sonar_base" update_rate="10" maxRange="0.7" minRange="0.01" fov="0.5" radiation="ultrasound">
-      <origin xyz="${-0.48412 + base_link_offset_x} -0.15127 0.29" rpy="0.0 0.0 -2.6354" />
-    </xacro:range_ant>
-    <!-- sonar -->
-    <xacro:range_ant name="${name}_sonar_08" parent="${name}" ros_topic="sonar_base" update_rate="10" maxRange="0.7" minRange="0.01" fov="0.5" radiation="ultrasound">
-      <origin xyz="${-0.51188 + base_link_offset_x} 0.0 0.26" rpy="0.0 0.0 -3.1415" />
-    </xacro:range_ant>
     <!-- bumper front right -->
     <xacro:bumper_ant name="${name}_bumper_01" parent="${name}" ros_topic="bumper_base" update_rate="25" >

Commit message: refs #8173 : removes bumpers outside the front
git-svn-id: svn+ssh://server/srv/svn/repos/trunk/pal-ros-pkg/catkin_pkgs/ant_robot@52512 5e370ff8-3418-0410-babe-3378cc20a00d

File: ant_description/urdf/base/base.urdf.xacro (robot description, xacro)
@@ -243,24 +243,4 @@
       <origin xyz="${0.225 + base_link_offset_x} 0.15 0.20" rpy="0 0 ${15.0 * deg_to_rad}" />
     </xacro:bumper_ant>
-    <!-- bumper left 1 -->
-    <xacro:bumper_ant name="${name}_bumper_03" parent="${name}" ros_topic="bumper_base" update_rate="25" >
-      <origin xyz="${-0.04 + base_link_offset_x} 0.33 0.1" rpy="0 0 ${90.0 * deg_to_rad}" />
-    </xacro:bumper_ant>
-    <!-- bumper left 2 -->
-    <xacro:bumper_ant name="${name}_bumper_04" parent="${name}" ros_topic="bumper_base" update_rate="25" >
-      <origin xyz="${-0.3 + base_link_offset_x} 0.31 0.1" rpy="0 0 ${100.0 * deg_to_rad}" />
-    </xacro:bumper_ant>
-    <!-- bumper back -->
-    <xacro:bumper_ant name="${name}_bumper_05" parent="${name}" ros_topic="bumper_base" update_rate="25" >
-      <origin xyz="${-0.545 + base_link_offset_x} 0.0 0.1" rpy="0 0 ${180.0 * deg_to_rad}" />
-    </xacro:bumper_ant>
-    <!-- bumper right 2 -->
-    <xacro:bumper_ant name="${name}_bumper_06" parent="${name}" ros_topic="bumper_base" update_rate="25" >
-      <origin xyz="${-0.3 + base_link_offset_x} -0.31 0.1" rpy="0 0 ${-100.0 * deg_to_rad}" />
-    </xacro:bumper_ant>
-    <!-- bumper right 1 -->
-    <xacro:bumper_ant name="${name}_bumper_07" parent="${name}" ros_topic="bumper_base" update_rate="25" >
-      <origin xyz="${-0.04 + base_link_offset_x} -0.33 0.1" rpy="0 0 ${-90.0 * deg_to_rad}" />
-    </xacro:bumper_ant>
     <!-- imu -->
     <xacro:ant_imu name="base_inclinometer" parent="${name}_link" update_rate="100.0">

Commit message: refs #8173 : cleans
git-svn-id: svn+ssh://server/srv/svn/repos/trunk/pal-ros-pkg/catkin_pkgs/ant_robot@52513 5e370ff8-3418-0410-babe-3378cc20a00d

File: ant_description/urdf/base/base.urdf.xacro (robot description, xacro)
@@ -81,7 +81,4 @@
                   iyy="0.015218160428" iyz="-0.000004273467"
                   izz="0.011763977943" />
-        <!--<origin xyz="0 0 0" rpy="0 0 0"/>
-        <mass value="0.1" />
-        <inertia  ixx="0" ixy="0" ixz="0" iyy="0" iyz="0" izz="0" />-->
       </inertial>
       <visual>
@@ -193,5 +190,5 @@
       <parent link="${name}_footprint"/>
     </joint>
-   <link name="${name}_center">
+    <link name="${name}_center">
       <inertial>
         <mass value="1.0" />
@@ -214,5 +211,5 @@
       </collision>
     </link>
-   <joint name="${name}_center_joint" type="fixed">
+    <joint name="${name}_center_joint" type="fixed">
       <origin xyz="${-0.195 + base_link_offset_x} 0 0" rpy="0 0 0" />
       <child link="${name}_center" />

Commit message: refs #8173 : adds xacro macros for the wheels
git-svn-id: svn+ssh://server/srv/svn/repos/trunk/pal-ros-pkg/catkin_pkgs/ant_robot@52520 5e370ff8-3418-0410-babe-3378cc20a00d

File: ant_description/urdf/base/base.urdf.xacro (robot description, xacro)
@@ -10,4 +10,5 @@
   <xacro:include filename="$(find ant_description)/urdf/deg_to_rad.xacro" />
   <xacro:include filename="$(find ant_description)/urdf/base/base.transmission.xacro" />
+  <xacro:include filename="$(find ant_description)/urdf/wheels/wheel.urdf.xacro" />
   <xacro:include filename="$(find ant_description)/urdf/sensors/range.urdf.xacro" />
   <xacro:include filename="$(find ant_description)/urdf/sensors/hokuyo_urg_04lx_ug01_laser.urdf.xacro" />
@@ -25,49 +26,4 @@
   <property name="caster_width"         value="0.0164"/>
   <property name="caster_trailing_dist" value="0.038"/>
-  <xacro:macro name="ant_wheel" params="side reflect" parent="base_link">
-    <!--************************-->
-    <!--        WHEELS          -->
-    <!--************************-->
-    <link name="wheel_${side}_link">
-      <inertial>
-        <origin xyz="0 0 0" rpy="0 0 0" />
-        <mass value="1.0" />
-        <inertia ixx="1"  ixy="0"  ixz="0" iyy="1" iyz="0" izz="1" />
-        <!--<origin xyz="0 0 0" rpy="0 0 0" />
-        <mass value="3.5" />
-        <inertia ixx="0.00156"  ixy="0"  ixz="0" iyy="0.00156" iyz="0" izz="0.0273" />-->
-      </inertial>
-      <visual>
-        <origin xyz="0 0 0" rpy="0 0 0" />
-        <geometry>
-          <cylinder radius="${wheel_radius}" length="${wheel_width}" />
-        </geometry>
-        <material name="DarkGrey" />
-      </visual>
-      <collision>
-        <origin xyz="0 0 0" rpy="0 0 0" />
-        <geometry>
-          <cylinder radius="${wheel_radius}" length="${wheel_width}" />
-        </geometry>
-      </collision>
-    </link>
-    <!-- contact model for wheel surface -->
-    <gazebo reference="wheel_${side}_link">
-      <kp>100000000.0</kp>
-      <kd>10000.0</kd>
-      <mu1>1.0</mu1>
-      <mu2>1.0</mu2>
-      <minDepth>0.00</minDepth>
-    </gazebo>
-    <joint name="wheel_${side}_joint" type="continuous">
-      <parent link="base_link" />
-      <child link="wheel_${side}_link" />
-      <origin xyz="0 ${-wheel_separation / 2 * reflect} ${wheel_radius}" rpy="${-90.0 * deg_to_rad} 0 0" />
-      <axis xyz="0 0 1" />
-      <limit effort="${wheel_torque}" velocity="${wheel_velocity / wheel_radius}"/>
-    </joint>
-    <!-- extensions -->
-    <xacro:ant_wheel_transmission side="${side}" />
-  </xacro:macro>
   <xacro:macro name="ant_caster" params="side reflect">
     <!--************************-->
@@ -143,4 +99,7 @@
   <!-- base_link x-axis offset -->
   <property name="base_link_offset_x" value="0.0"/>
+  <property name="base_radius" value="${(wheel_separation - wheel_width)/2 - 0.01}"/>
+  <property name="base_length" value="0.04"/>
+  <property name="base_link_offset_z" value="${base_length + 0.01}"/>
   <xacro:macro name="ant_base" params="name">
     <!--************************-->
@@ -154,14 +113,16 @@
       </inertial>
       <visual>
-        <origin xyz="${base_link_offset_x} 0 0" rpy="0 0 0" />
-        <geometry>
-          <mesh filename="package://ant_description/meshes/base/base.dae" />
+        <origin xyz="${base_link_offset_x} 0 ${base_link_offset_z}" rpy="0 0 0" />
+        <geometry>
+          <cylinder radius="${base_radius}" length="${base_length}"/>
+          <!--mesh filename="package://ant_description/meshes/base/base.dae" /-->
         </geometry>
         <material name="LightGrey" />
       </visual>
       <collision>
-        <origin xyz="${base_link_offset_x} 0 0" rpy="0 0 0" />
-        <geometry>
-          <mesh filename="package://ant_description/meshes/base/base_collision.stl" />
+        <origin xyz="${base_link_offset_x} 0 ${base_link_offset_z}" rpy="0 0 0" />
+        <geometry>
+          <cylinder radius="${base_radius}" length="${base_length}"/>
+          <!--mesh filename="package://ant_description/meshes/base/base_collision.stl" /-->
         </geometry>
         <material name="LightGrey" />
@@ -245,6 +206,8 @@
     </xacro:ant_imu>
     <!-- wheels -->
-    <xacro:ant_wheel side="right" reflect=" 1.0"/>
-    <xacro:ant_wheel side="left"  reflect="-1.0"/>
+    <xacro:wheel_ant side="right" reflect=" 1.0" radius="${wheel_radius}" width="${wheel_width}" torque="${wheel_torque}" velocity="${wheel_velocity}" separation="${wheel_separation}" parent="${name}"/>
+    <xacro:ant_wheel_transmission side="right"/>
+    <xacro:wheel_ant side="left"  reflect="-1.0" radius="${wheel_radius}" width="${wheel_width}" torque="${wheel_torque}" velocity="${wheel_velocity}" separation="${wheel_separation}" parent="${name}"/>
+    <xacro:ant_wheel_transmission side="left"/>
     <!-- casters -->
     <xacro:ant_caster side="right" reflect=" 1.0"/>

Commit message: refs #8173 : uses caster wheel xacro files
git-svn-id: svn+ssh://server/srv/svn/repos/trunk/pal-ros-pkg/catkin_pkgs/ant_robot@52593 5e370ff8-3418-0410-babe-3378cc20a00d

File: ant_description/urdf/base/base.urdf.xacro (robot description, xacro)
@@ -11,9 +11,10 @@
   <xacro:include filename="$(find ant_description)/urdf/base/base.transmission.xacro" />
   <xacro:include filename="$(find ant_description)/urdf/wheels/wheel.urdf.xacro" />
+  <xacro:include filename="$(find ant_description)/urdf/wheels/caster.urdf.xacro" />
   <xacro:include filename="$(find ant_description)/urdf/sensors/range.urdf.xacro" />
   <xacro:include filename="$(find ant_description)/urdf/sensors/hokuyo_urg_04lx_ug01_laser.urdf.xacro" />
   <xacro:include filename="$(find ant_description)/urdf/sensors/imu.urdf.xacro"/>
   <xacro:include filename="$(find ant_description)/urdf/sensors/bumper.urdf.xacro" />
-  <!--wheel characteristics-->
+  <!-- Wheel characteristics -->
   <property name="wheel_separation" value="0.42"/>
   <property name="wheel_radius"     value="0.09931"/>
@@ -21,80 +22,9 @@
   <property name="wheel_torque"     value="50.0"/>
   <property name="wheel_velocity"   value="1.0"/>
-  <!--caster characteristics-->
-  <property name="dist_between_casters" value="0.300"/>
-  <property name="caster_radius"        value="0.025"/>
-  <property name="caster_width"         value="0.0164"/>
-  <property name="caster_trailing_dist" value="0.038"/>
-  <xacro:macro name="ant_caster" params="side reflect">
-    <!--************************-->
-    <!--        CASTERS         -->
-    <!--************************-->
-    <link name="caster_${side}_1_link">
-      <inertial>
-        <origin xyz="0 0 0" rpy="0 0 0"/>
-        <mass value="0.1" />
-        <inertia  ixx="0.012411765597" ixy="-0.000711733678" ixz="0.00050272983"
-                  iyy="0.015218160428" iyz="-0.000004273467"
-                  izz="0.011763977943" />
-      </inertial>
-      <visual>
-        <origin xyz="${0.5 * caster_radius - caster_trailing_dist} 0 ${0.5 * caster_radius}" rpy="0 0 0" />
-        <geometry>
-          <box size="${caster_radius} ${1.2 * caster_width} ${caster_radius}"/>
-        </geometry>
-        <material name="DarkGrey" />
-      </visual>
-      <collision>
-        <origin xyz="${0.5 * caster_radius - caster_trailing_dist} 0 ${0.5 * caster_radius}" rpy="0 0 0" />
-        <geometry>
-          <box size="${caster_radius} ${1.2 * caster_width} ${caster_radius}"/>
-        </geometry>
-      </collision>
-    </link>
-    <link name="caster_${side}_2_link">
-      <inertial>
-        <origin xyz="0 0 0" rpy="0 0 0"/>
-        <mass value="0.4" />
-        <inertia  ixx="0.00044" ixy="0" ixz="0" iyy="0.00044" iyz="0" izz="0.00078" />
-        </inertial>
-      <visual>
-        <origin xyz="0 0 0" rpy="0 0 0" />
-        <geometry>
-          <cylinder radius="${caster_radius}" length="${caster_width}"/>
-        </geometry>
-        <material name="DarkGrey" />
-      </visual>
-      <collision>
-        <origin xyz="0 0 0" rpy="0 0 0" />
-        <geometry>
-          <cylinder radius="${caster_radius}" length="${caster_width}"/>
-        </geometry>
-      </collision>
-    </link>
-    <!-- contact model for caster wheel surface -->
-    <gazebo reference="caster_${side}_2_link">
-      <kp>100000000.0</kp>
-      <kd>10000.0</kd>
-      <mu1>1.0</mu1>
-      <mu2>1.0</mu2>
-      <minDepth>0.00</minDepth>
-    </gazebo>
-    <joint name="caster_${side}_1_joint" type="continuous">
-      <parent link="base_link" />
-      <child link="caster_${side}_1_link" />
-      <origin xyz="-0.3805 ${-dist_between_casters / 2 * reflect} ${caster_radius}" rpy="0 0 0" />
-      <axis xyz="0 0 1" />
-    </joint>
-    <joint name="caster_${side}_2_joint" type="continuous">
-      <parent link="caster_${side}_1_link" />
-      <child link="caster_${side}_2_link" />
-      <origin xyz="${-caster_trailing_dist} 0 0" rpy="${-90.0 * deg_to_rad} 0 0" />
-      <axis xyz="0 0 1" />
-    </joint>
-  </xacro:macro>
-  <!-- simplified box collision geometry for the laser -->
-  <property name="base_laser_x" value="0.0468" />
-  <property name="base_laser_y" value="0.0" />
-  <property name="base_laser_z" value="0.081" />
+  <!-- Caster wheel characteristics -->
+  <property name="caster_separation" value="0.300"/>
+  <property name="caster_radius"     value="0.025"/>
+  <property name="caster_width"      value="0.0164"/>
+  <property name="caster_trailing"   value="0.138"/>
   <!-- base_link x-axis offset -->
   <property name="base_link_offset_x" value="0.0"/>
@@ -102,4 +32,8 @@
   <property name="base_length" value="0.04"/>
   <property name="base_link_offset_z" value="${base_length + 0.01}"/>
+  <!-- simplified box collision geometry for the laser -->
+  <property name="base_laser_x" value="0.15"/>
+  <property name="base_laser_y" value="0.0"/>
+  <property name="base_laser_z" value="0.081"/>
   <xacro:macro name="ant_base" params="name">
     <!--************************-->
@@ -177,40 +111,40 @@
       <parent link="${name}_link"/>
     </joint>
-    <!-- laser -->
+    <!-- Laser -->
     <xacro:hokuyo_urg_04lx_ug01_laser name="${name}_laser" parent="${name}" ros_topic="scan" update_rate="10" min_angle="${-120 * deg_to_rad}" max_angle="${120 * deg_to_rad}" >
       <origin xyz="${base_laser_x} ${base_laser_y} ${base_laser_z}" rpy="0 0 0" />
     </xacro:hokuyo_urg_04lx_ug01_laser>
-    <!-- sonar -->
+    <!-- Sonar -->
     <xacro:range_ant name="${name}_sonar_02" parent="${name}" ros_topic="sonar_base" update_rate="10" maxRange="0.75" minRange="0.01" fov="0.5" radiation="ultrasound">
       <origin xyz="${0.17131 + base_link_offset_x} 0.0 0.280" rpy="0.0 0.0 0.0" />
     </xacro:range_ant>
-    <!-- sonar -->
+    <!-- Sonar -->
     <xacro:range_ant name="${name}_sonar_03" parent="${name}" ros_topic="sonar_base" update_rate="10" maxRange="0.75" minRange="0.01" fov="0.5" radiation="ultrasound">
       <origin xyz="${0.16919 + base_link_offset_x} 0.14919 0.280" rpy="0.0 0.0 0.349" />
     </xacro:range_ant>
-    <!-- sonar -->
+    <!-- Sonar -->
     <xacro:range_ant name="${name}_sonar_01" parent="${name}" ros_topic="sonar_base" update_rate="10" maxRange="0.75" minRange="0.01" fov="0.5" radiation="ultrasound">
       <origin xyz="${0.16919 + base_link_offset_x} -0.14919 0.280" rpy="0.0 0.0 -0.349" />
     </xacro:range_ant>
-    <!-- bumper front right -->
+    <!-- Bumper front right -->
     <xacro:bumper_ant name="${name}_bumper_01" parent="${name}" ros_topic="bumper_base" update_rate="25" >
       <origin xyz="${0.225 + base_link_offset_x} -0.15 0.20" rpy="0 0 ${-15.0 * deg_to_rad}" />
     </xacro:bumper_ant>
-    <!-- bumper front left -->
+    <!-- Bumper front left -->
     <xacro:bumper_ant name="${name}_bumper_02" parent="${name}" ros_topic="bumper_base" update_rate="25" >
       <origin xyz="${0.225 + base_link_offset_x} 0.15 0.20" rpy="0 0 ${15.0 * deg_to_rad}" />
     </xacro:bumper_ant>
-    <!-- imu -->
+    <!-- IMU -->
     <xacro:ant_imu name="base_inclinometer" parent="${name}_link" update_rate="100.0">
       <origin xyz="-0.02977 -0.1497 0.164" rpy="0 ${180 * deg_to_rad} 0"/>
     </xacro:ant_imu>
-    <!-- wheels -->
+    <!-- Wheels -->
     <xacro:wheel_ant side="right" reflect=" 1.0" radius="${wheel_radius}" width="${wheel_width}" torque="${wheel_torque}" velocity="${wheel_velocity}" separation="${wheel_separation}" parent="${name}"/>
     <xacro:ant_wheel_transmission side="right"/>
     <xacro:wheel_ant side="left"  reflect="-1.0" radius="${wheel_radius}" width="${wheel_width}" torque="${wheel_torque}" velocity="${wheel_velocity}" separation="${wheel_separation}" parent="${name}"/>
     <xacro:ant_wheel_transmission side="left"/>
-    <!-- casters -->
-    <xacro:ant_caster side="right" reflect=" 1.0"/>
-    <xacro:ant_caster side="left"  reflect="-1.0"/>
+    <!-- Casters wheels -->
+    <xacro:caster_ant side="right" reflect=" 1.0" radius="${caster_radius}" width="${caster_width}" separation="${caster_separation}" trailing="${caster_trailing}" parent="${name}"/>
+    <xacro:caster_ant side="left"  reflect="-1.0" radius="${caster_radius}" width="${caster_width}" separation="${caster_separation}" trailing="${caster_trailing}" parent="${name}"/>
   </xacro:macro>
 </robot>
