Commit message: refs #8173 : removes center link, and base footprint visual
git-svn-id: svn+ssh://server/srv/svn/repos/trunk/pal-ros-pkg/catkin_pkgs/ant_robot@52594 5e370ff8-3418-0410-babe-3378cc20a00d

File: ant_description/urdf/base/base.urdf.xacro (robot description, xacro)
@@ -66,11 +66,4 @@
     using the navigation stack -->
     <link name="${name}_footprint">
-      <visual>
-        <origin xyz="0 0 0.2" rpy="0 0 0" />
-        <geometry>
-          <box size="0.01 0.01 0.01" />
-        </geometry>
-        <material name="White" />
-      </visual>
       <collision>
         <origin xyz="0 0 0.2" rpy="0 0 0" />
@@ -84,30 +77,4 @@
       <child link="${name}_link" />
       <parent link="${name}_footprint"/>
-    </joint>
-    <link name="${name}_center">
-      <inertial>
-        <mass value="1.0" />
-        <origin xyz="-0.0 0 0" />
-        <inertia ixx="0.01" ixy="0.0" ixz="0.0"
-                 iyy="0.01" iyz="0.0" izz="0.01" />
-      </inertial>
-      <visual>
-        <origin xyz="-0.0 0 0" rpy="0 0 0" />
-        <geometry>
-          <box size="0.01 0.01 0.01" />
-        </geometry>
-        <material name="White" />
-      </visual>
-      <collision>
-        <origin xyz="-0.0 0 0.2" rpy="0 0 0" />
-        <geometry>
-          <box size="0.001 0.001 0.001" />
-        </geometry>
-      </collision>
-    </link>
-    <joint name="${name}_center_joint" type="fixed">
-      <origin xyz="${-0.195 + base_link_offset_x} 0 0" rpy="0 0 0" />
-      <child link="${name}_center" />
-      <parent link="${name}_link"/>
     </joint>
     <!-- Laser -->

Commit message: refs #8173 : puts transmission in the wheel/caster xacro files
git-svn-id: svn+ssh://server/srv/svn/repos/trunk/pal-ros-pkg/catkin_pkgs/ant_robot@52595 5e370ff8-3418-0410-babe-3378cc20a00d

File: ant_description/urdf/base/base.urdf.xacro (robot description, xacro)
@@ -9,5 +9,4 @@
 <robot xmlns:xacro="http://ros.org/wiki/xacro">
   <xacro:include filename="$(find ant_description)/urdf/deg_to_rad.xacro" />
-  <xacro:include filename="$(find ant_description)/urdf/base/base.transmission.xacro" />
   <xacro:include filename="$(find ant_description)/urdf/wheels/wheel.urdf.xacro" />
   <xacro:include filename="$(find ant_description)/urdf/wheels/caster.urdf.xacro" />
@@ -108,7 +107,5 @@
     <!-- Wheels -->
     <xacro:wheel_ant side="right" reflect=" 1.0" radius="${wheel_radius}" width="${wheel_width}" torque="${wheel_torque}" velocity="${wheel_velocity}" separation="${wheel_separation}" parent="${name}"/>
-    <xacro:ant_wheel_transmission side="right"/>
     <xacro:wheel_ant side="left"  reflect="-1.0" radius="${wheel_radius}" width="${wheel_width}" torque="${wheel_torque}" velocity="${wheel_velocity}" separation="${wheel_separation}" parent="${name}"/>
-    <xacro:ant_wheel_transmission side="left"/>
     <!-- Casters wheels -->
     <xacro:caster_ant side="right" reflect=" 1.0" radius="${caster_radius}" width="${caster_width}" separation="${caster_separation}" trailing="${caster_trailing}" parent="${name}"/>

File: ant_description/urdf/wheels/caster.urdf.xacro (robot description, xacro)
@@ -8,4 +8,5 @@
 -->
 <robot xmlns:xacro="http://ros.org/wiki/xacro">
+  <xacro:include filename="$(find ant_description)/urdf/wheels/caster.transmission.xacro"/>
   <xacro:include filename="$(find ant_description)/urdf/wheels/caster.gazebo.xacro"/>
   <xacro:macro name="caster_ant" params="side reflect radius width separation trailing parent">
@@ -64,5 +65,7 @@
       <axis xyz="0 0 1"/>
     </joint>
-    <!-- gazebo extensions -->
+    <!-- Transmission -->
+    <!--xacro:ant_caster_transmission name="" side="${side}" number="" reduction=""-->
+    <!-- Gazebo extensions -->
     <xacro:caster_ant_gazebo side="${side}"/>
   </xacro:macro>

File: ant_description/urdf/wheels/wheel.transmission.xacro (robot description, xacro)
@@ -8,5 +8,5 @@
 -->
 <robot xmlns:xacro="http://ros.org/wiki/xacro">
-  <!-- wheels transmission -->
+  <!-- Wheel transmission -->
   <xacro:macro name="ant_wheel_transmission" params="side">
     <transmission name="wheel_${side}_trans">
@@ -20,15 +20,3 @@
     </transmission>
   </xacro:macro>
-  <!-- caster transmissions -->
-  <xacro:macro name="ant_caster_simple_transmission" params="name side number reduction" >
-    <transmission name="${name}_${side}_${number}_trans">
-      <type>transmission_interface/SimpleTransmission</type>
-      <actuator name="${name}_${side}_${number}_motor" >
-        <mechanicalReduction>${reduction}</mechanicalReduction>
-      </actuator>
-      <joint name="${name}_${side}_${number}_joint" >
-        <hardwareInterface>hardware_interface/JointStateInterface</hardwareInterface>
-      </joint>
-    </transmission>
-  </xacro:macro>
 </robot>

File: ant_description/urdf/wheels/wheel.urdf.xacro (robot description, xacro)
@@ -8,4 +8,5 @@
 -->
 <robot xmlns:xacro="http://ros.org/wiki/xacro">
+  <xacro:include filename="$(find ant_description)/urdf/wheels/wheel.transmission.xacro"/>
   <xacro:include filename="$(find ant_description)/urdf/wheels/wheel.gazebo.xacro"/>
   <xacro:macro name="wheel_ant" params="side reflect radius width torque velocity separation parent">
@@ -37,5 +38,7 @@
       <limit effort="${torque}" velocity="${velocity / radius}"/>
     </joint>
-    <!-- gazebo extensions -->
+    <!-- Transmission -->
+    <xacro:ant_wheel_transmission side="${side}"/>
+    <!-- Gazebo extensions -->
     <xacro:wheel_ant_gazebo side="${side}"/>
   </xacro:macro>

Commit message: refs #8173 : puts caster wheels in good position (but not real)
git-svn-id: svn+ssh://server/srv/svn/repos/trunk/pal-ros-pkg/catkin_pkgs/ant_robot@52600 5e370ff8-3418-0410-babe-3378cc20a00d

File: ant_description/urdf/base/base.urdf.xacro (robot description, xacro)
@@ -22,26 +22,25 @@
   <property name="wheel_velocity"   value="1.0"/>
   <!-- Caster wheel characteristics -->
-  <property name="caster_separation" value="0.300"/>
+  <property name="caster_separation" value="0.200"/>
   <property name="caster_radius"     value="0.025"/>
   <property name="caster_width"      value="0.0164"/>
   <property name="caster_trailing"   value="0.038"/>
+  <property name="caster_offset_x"   value="0.140"/>
   <!-- base_link x-axis offset -->
   <property name="base_link_offset_x" value="0.0"/>
   <property name="base_radius" value="${(wheel_separation - wheel_width)/2 - 0.01}"/>
   <property name="base_length" value="0.04"/>
-  <property name="base_link_offset_z" value="${base_length + 0.01}"/>
+  <property name="base_link_offset_z" value="${base_length + 0.031}"/>
   <!-- simplified box collision geometry for the laser -->
   <property name="base_laser_x" value="0.15"/>
   <property name="base_laser_y" value="0.0"/>
-  <property name="base_laser_z" value="0.081"/>
+  <property name="base_laser_z" value="0.093"/>
   <xacro:macro name="ant_base" params="name">
-    <!--************************-->
-    <!--        BASE            -->
-    <!--************************-->
+    <!-- Base -->
     <link name="${name}_link">
       <inertial>
-        <origin xyz="0.0 0.0 0.24721" rpy="0 0 0" /> <!-- assuming d=0.6, w=0.5, h=0.4 -->
+        <origin xyz="0.0 0.0 0.26721" rpy="0 0 0" />
         <mass value="63.58850" />
-        <inertia ixx="3.42"  ixy="0"  ixz="0" iyy="4.33" iyz="0" izz="5.08" /> <!-- assuming d=0.6, w=0.5, h=0.4 -->
+        <inertia ixx="3.42" ixy="0" ixz="0" iyy="4.33" iyz="0" izz="5.08" />
       </inertial>
       <visual>
@@ -78,5 +77,5 @@
     </joint>
     <!-- Laser -->
-    <xacro:hokuyo_urg_04lx_ug01_laser name="${name}_laser" parent="${name}" ros_topic="scan" update_rate="10" min_angle="${-120 * deg_to_rad}" max_angle="${120 * deg_to_rad}" >
+    <xacro:hokuyo_urg_04lx_ug01_laser name="${name}_laser" parent="${name}" ros_topic="scan" update_rate="10" min_angle="${-100 * deg_to_rad}" max_angle="${100 * deg_to_rad}" >
       <origin xyz="${base_laser_x} ${base_laser_y} ${base_laser_z}" rpy="0 0 0" />
     </xacro:hokuyo_urg_04lx_ug01_laser>
@@ -109,6 +108,6 @@
     <xacro:wheel_ant side="left"  reflect="-1.0" radius="${wheel_radius}" width="${wheel_width}" torque="${wheel_torque}" velocity="${wheel_velocity}" separation="${wheel_separation}" parent="${name}"/>
     <!-- Casters wheels -->
-    <xacro:caster_ant side="right" reflect=" 1.0" radius="${caster_radius}" width="${caster_width}" separation="${caster_separation}" trailing="${caster_trailing}" parent="${name}"/>
-    <xacro:caster_ant side="left"  reflect="-1.0" radius="${caster_radius}" width="${caster_width}" separation="${caster_separation}" trailing="${caster_trailing}" parent="${name}"/>
+    <xacro:caster_ant side="right" reflect=" 1.0" radius="${caster_radius}" width="${caster_width}" separation="${caster_separation}" trailing="${caster_trailing}" offset_x="${caster_offset_x}" parent="${name}"/>
+    <xacro:caster_ant side="left"  reflect="-1.0" radius="${caster_radius}" width="${caster_width}" separation="${caster_separation}" trailing="${caster_trailing}" offset_x="${caster_offset_x}" parent="${name}"/>
   </xacro:macro>
 </robot>

Commit message: removes ant_ prefix from wheels and base
git-svn-id: svn+ssh://server/srv/svn/repos/trunk/pal-ros-pkg/catkin_pkgs/ant_robot@52879 5e370ff8-3418-0410-babe-3378cc20a00d

File: ant_description/urdf/base/base.urdf.xacro (robot description, xacro)
@@ -36,5 +36,5 @@
   <property name="base_laser_y" value="0.0"/>
   <property name="base_laser_z" value="0.093"/>
-  <xacro:macro name="ant_base" params="name">
+  <xacro:macro name="base" params="name">
     <!-- Base -->
     <link name="${name}_link">
@@ -104,11 +104,11 @@
     </xacro:ant_imu>
     <!-- Wheels -->
-    <xacro:wheel_ant side="right" reflect=" 1.0" radius="${wheel_radius}" width="${wheel_width}" torque="${wheel_torque}" velocity="${wheel_velocity}" separation="${wheel_separation}" parent="${name}"/>
-    <xacro:wheel_ant side="left"  reflect="-1.0" radius="${wheel_radius}" width="${wheel_width}" torque="${wheel_torque}" velocity="${wheel_velocity}" separation="${wheel_separation}" parent="${name}"/>
+    <xacro:wheel side="right" reflect=" 1.0" radius="${wheel_radius}" width="${wheel_width}" torque="${wheel_torque}" velocity="${wheel_velocity}" separation="${wheel_separation}" parent="${name}"/>
+    <xacro:wheel side="left"  reflect="-1.0" radius="${wheel_radius}" width="${wheel_width}" torque="${wheel_torque}" velocity="${wheel_velocity}" separation="${wheel_separation}" parent="${name}"/>
     <!-- Casters wheels -->
-    <xacro:caster_ant side="front_right" reflect=" 1.0" radius="${caster_radius}" width="${caster_width}" separation="${caster_separation}" trailing="${caster_trailing}" offset_x="${caster_offset_x}" parent="${name}"/>
-    <xacro:caster_ant side="front_left"  reflect="-1.0" radius="${caster_radius}" width="${caster_width}" separation="${caster_separation}" trailing="${caster_trailing}" offset_x="${caster_offset_x}" parent="${name}"/>
-    <xacro:caster_ant side="back_right" reflect=" 1.0" radius="${caster_radius}" width="${caster_width}" separation="${caster_separation}" trailing="${caster_trailing}" offset_x="${-caster_offset_x}" parent="${name}"/>
-    <xacro:caster_ant side="back_left"  reflect="-1.0" radius="${caster_radius}" width="${caster_width}" separation="${caster_separation}" trailing="${caster_trailing}" offset_x="${-caster_offset_x}" parent="${name}"/>
+    <xacro:caster side="front_right" reflect=" 1.0" radius="${caster_radius}" width="${caster_width}" separation="${caster_separation}" trailing="${caster_trailing}" offset_x="${caster_offset_x}" parent="${name}"/>
+    <xacro:caster side="front_left"  reflect="-1.0" radius="${caster_radius}" width="${caster_width}" separation="${caster_separation}" trailing="${caster_trailing}" offset_x="${caster_offset_x}" parent="${name}"/>
+    <xacro:caster side="back_right" reflect=" 1.0" radius="${caster_radius}" width="${caster_width}" separation="${caster_separation}" trailing="${caster_trailing}" offset_x="${-caster_offset_x}" parent="${name}"/>
+    <xacro:caster side="back_left"  reflect="-1.0" radius="${caster_radius}" width="${caster_width}" separation="${caster_separation}" trailing="${caster_trailing}" offset_x="${-caster_offset_x}" parent="${name}"/>
   </xacro:macro>
 </robot>

File: ant_description/urdf/wheels/caster.gazebo.xacro (robot description, xacro)
@@ -8,5 +8,5 @@
 -->
 <robot xmlns:xacro="http://ros.org/wiki/xacro">
-  <xacro:macro name="caster_ant_gazebo" params="side">
+  <xacro:macro name="caster_gazebo" params="side">
     <!-- Contact model for the caster wheel surface -->
     <gazebo reference="caster_${side}_link">

File: ant_description/urdf/wheels/caster.transmission.xacro (robot description, xacro)
@@ -9,5 +9,5 @@
 <robot xmlns:xacro="http://ros.org/wiki/xacro">
   <!-- Caster transmissions -->
-  <xacro:macro name="ant_caster_transmission" params="name side number reduction" >
+  <xacro:macro name="caster_transmission" params="name side number reduction" >
     <transmission name="${name}_${side}_${number}_trans">
       <type>transmission_interface/SimpleTransmission</type>

File: ant_description/urdf/wheels/caster.urdf.xacro (robot description, xacro)
@@ -10,5 +10,5 @@
   <xacro:include filename="$(find ant_description)/urdf/wheels/caster.transmission.xacro"/>
   <xacro:include filename="$(find ant_description)/urdf/wheels/caster.gazebo.xacro"/>
-  <xacro:macro name="caster_ant" params="side reflect radius width separation trailing offset_x parent">
+  <xacro:macro name="caster" params="side reflect radius width separation trailing offset_x parent">
     <link name="caster_${side}_1_link">
       <inertial>
@@ -66,7 +66,7 @@
     </joint>
     <!-- Transmission -->
-    <!--xacro:ant_caster_transmission name="" side="${side}" number="" reduction=""-->
+    <!--xacro:caster_transmission name="" side="${side}" number="" reduction=""-->
     <!-- Gazebo extensions -->
-    <xacro:caster_ant_gazebo side="${side}"/>
+    <xacro:caster_gazebo side="${side}"/>
   </xacro:macro>
 </robot>

File: ant_description/urdf/wheels/wheel.gazebo.xacro (robot description, xacro)
@@ -8,5 +8,5 @@
 -->
 <robot xmlns:xacro="http://ros.org/wiki/xacro">
-  <xacro:macro name="wheel_ant_gazebo" params="side">
+  <xacro:macro name="wheel_gazebo" params="side">
     <!-- Contact model for the wheel surface -->
     <gazebo reference="wheel_${side}_link">

File: ant_description/urdf/wheels/wheel.transmission.xacro (robot description, xacro)
@@ -9,5 +9,5 @@
 <robot xmlns:xacro="http://ros.org/wiki/xacro">
   <!-- Wheel transmission -->
-  <xacro:macro name="ant_wheel_transmission" params="side">
+  <xacro:macro name="wheel_transmission" params="side">
     <transmission name="wheel_${side}_trans">
       <type>transmission_interface/SimpleTransmission</type>

File: ant_description/urdf/wheels/wheel.urdf.xacro (robot description, xacro)
@@ -10,5 +10,5 @@
   <xacro:include filename="$(find ant_description)/urdf/wheels/wheel.transmission.xacro"/>
   <xacro:include filename="$(find ant_description)/urdf/wheels/wheel.gazebo.xacro"/>
-  <xacro:macro name="wheel_ant" params="side reflect radius width torque velocity separation parent">
+  <xacro:macro name="wheel" params="side reflect radius width torque velocity separation parent">
     <link name="wheel_${side}_link">
       <inertial>
@@ -39,7 +39,7 @@
     </joint>
     <!-- Transmission -->
-    <xacro:ant_wheel_transmission side="${side}"/>
+    <xacro:wheel_transmission side="${side}"/>
     <!-- Gazebo extensions -->
-    <xacro:wheel_ant_gazebo side="${side}"/>
+    <xacro:wheel_gazebo side="${side}"/>
   </xacro:macro>
 </robot>
