Commit message: removes ant and uses sensor prefix
git-svn-id: svn+ssh://server/srv/svn/repos/trunk/pal-ros-pkg/catkin_pkgs/ant_robot@52886 5e370ff8-3418-0410-babe-3378cc20a00d

File: ant_description/urdf/base/base.urdf.xacro (robot description, xacro)
@@ -8,11 +8,12 @@
 -->
 <robot xmlns:xacro="http://ros.org/wiki/xacro">
-  <xacro:include filename="$(find ant_description)/urdf/deg_to_rad.xacro" />
-  <xacro:include filename="$(find ant_description)/urdf/wheels/wheel.urdf.xacro" />
-  <xacro:include filename="$(find ant_description)/urdf/wheels/caster.urdf.xacro" />
-  <xacro:include filename="$(find ant_description)/urdf/sensors/range.urdf.xacro" />
-  <xacro:include filename="$(find ant_description)/urdf/sensors/hokuyo_urg_04lx_ug01_laser.urdf.xacro" />
+  <xacro:include filename="$(find ant_description)/urdf/deg_to_rad.xacro"/>
+  <xacro:include filename="$(find ant_description)/urdf/wheels/wheel.urdf.xacro"/>
+  <xacro:include filename="$(find ant_description)/urdf/wheels/caster.urdf.xacro"/>
+  <xacro:include filename="$(find ant_description)/urdf/sensors/range.urdf.xacro"/>
+  <xacro:include filename="$(find ant_description)/urdf/sensors/hokuyo_urg_04lx_ug01_laser.urdf.xacro"/>
   <xacro:include filename="$(find ant_description)/urdf/sensors/imu.urdf.xacro"/>
-  <xacro:include filename="$(find ant_description)/urdf/sensors/bumper.urdf.xacro" />
+  <xacro:include filename="$(find ant_description)/urdf/sensors/bumper.urdf.xacro"/>
+  <xacro:include filename="$(find ant_description)/urdf/sensors/ir_receiver.urdf.xacro"/>
   <!-- Wheel characteristics -->
   <property name="wheel_separation" value="0.42"/>
@@ -27,9 +28,8 @@
   <property name="caster_trailing"   value="0.038"/>
   <property name="caster_offset_x"   value="0.140"/>
-  <!-- base_link x-axis offset -->
-  <property name="base_link_offset_x" value="0.0"/>
   <property name="base_radius" value="${(wheel_separation - wheel_width)/2 - 0.01}"/>
   <property name="base_length" value="0.04"/>
-  <property name="base_link_offset_z" value="${base_length + 0.031}"/>
+  <property name="base_offset_x" value="0.0"/>
+  <property name="base_offset_z" value="${base_length + 0.031}"/>
   <!-- simplified box collision geometry for the laser -->
   <property name="base_laser_x" value="0.15"/>
@@ -45,5 +45,5 @@
       </inertial>
       <visual>
-        <origin xyz="${base_link_offset_x} 0 ${base_link_offset_z}" rpy="0 0 0" />
+        <origin xyz="${base_offset_x} 0 ${base_offset_z}" rpy="0 0 0" />
         <geometry>
           <cylinder radius="${base_radius}" length="${base_length}"/>
@@ -53,5 +53,5 @@
       </visual>
       <collision>
-        <origin xyz="${base_link_offset_x} 0 ${base_link_offset_z}" rpy="0 0 0" />
+        <origin xyz="${base_offset_x} 0 ${base_offset_z}" rpy="0 0 0" />
         <geometry>
           <cylinder radius="${base_radius}" length="${base_length}"/>
@@ -80,27 +80,39 @@
     </xacro:hokuyo_urg_04lx_ug01_laser>
     <!-- Sonar -->
-    <xacro:range_ant name="${name}_sonar_02" parent="${name}" ros_topic="sonar_base" update_rate="10" maxRange="0.75" minRange="0.01" fov="0.5" radiation="ultrasound">
-      <origin xyz="${0.17131 + base_link_offset_x} 0.0 0.280" rpy="0.0 0.0 0.0" />
-    </xacro:range_ant>
+    <xacro:range_sensor name="${name}_sonar_02" parent="${name}" ros_topic="sonar_base" update_rate="10" maxRange="0.75" minRange="0.01" fov="0.5" radiation="ultrasound">
+      <origin xyz="${0.17131 + base_offset_x} 0.0 0.280" rpy="0.0 0.0 0.0" />
+    </xacro:range_sensor>
     <!-- Sonar -->
-    <xacro:range_ant name="${name}_sonar_03" parent="${name}" ros_topic="sonar_base" update_rate="10" maxRange="0.75" minRange="0.01" fov="0.5" radiation="ultrasound">
-      <origin xyz="${0.16919 + base_link_offset_x} 0.14919 0.280" rpy="0.0 0.0 0.349" />
-    </xacro:range_ant>
+    <xacro:range_sensor name="${name}_sonar_03" parent="${name}" ros_topic="sonar_base" update_rate="10" maxRange="0.75" minRange="0.01" fov="0.5" radiation="ultrasound">
+      <origin xyz="${0.16919 + base_offset_x} 0.14919 0.280" rpy="0.0 0.0 0.349" />
+    </xacro:range_sensor>
     <!-- Sonar -->
-    <xacro:range_ant name="${name}_sonar_01" parent="${name}" ros_topic="sonar_base" update_rate="10" maxRange="0.75" minRange="0.01" fov="0.5" radiation="ultrasound">
-      <origin xyz="${0.16919 + base_link_offset_x} -0.14919 0.280" rpy="0.0 0.0 -0.349" />
-    </xacro:range_ant>
+    <xacro:range_sensor name="${name}_sonar_01" parent="${name}" ros_topic="sonar_base" update_rate="10" maxRange="0.75" minRange="0.01" fov="0.5" radiation="ultrasound">
+      <origin xyz="${0.16919 + base_offset_x} -0.14919 0.280" rpy="0.0 0.0 -0.349" />
+    </xacro:range_sensor>
     <!-- Bumper front right -->
-    <xacro:bumper_ant name="${name}_bumper_01" parent="${name}" ros_topic="bumper_base" update_rate="25" >
-      <origin xyz="${0.225 + base_link_offset_x} -0.15 0.20" rpy="0 0 ${-15.0 * deg_to_rad}" />
-    </xacro:bumper_ant>
+    <xacro:bumper name="${name}_bumper_01" parent="${name}" ros_topic="bumper_base" update_rate="25" >
+      <origin xyz="${0.225 + base_offset_x} -0.15 0.20" rpy="0 0 ${-15.0 * deg_to_rad}" />
+    </xacro:bumper>
     <!-- Bumper front left -->
-    <xacro:bumper_ant name="${name}_bumper_02" parent="${name}" ros_topic="bumper_base" update_rate="25" >
-      <origin xyz="${0.225 + base_link_offset_x} 0.15 0.20" rpy="0 0 ${15.0 * deg_to_rad}" />
-    </xacro:bumper_ant>
+    <xacro:bumper name="${name}_bumper_02" parent="${name}" ros_topic="bumper_base" update_rate="25" >
+      <origin xyz="${0.225 + base_offset_x} 0.15 0.20" rpy="0 0 ${15.0 * deg_to_rad}" />
+    </xacro:bumper>
     <!-- IMU -->
-    <xacro:ant_imu name="base_inclinometer" parent="${name}_link" update_rate="100.0">
+    <xacro:imu_sensor name="base_inclinometer" parent="${name}_link" update_rate="100.0">
       <origin xyz="-0.02977 -0.1497 0.164" rpy="0 ${180 * deg_to_rad} 0"/>
-    </xacro:ant_imu>
+    </xacro:imu_sensor>
+    <!-- IR receiver -->
+    <!--xacro:ir_receiver name="${name}_ir_receiver_01" parent="${name}" ros_topic="ir_receiver_base" update_rate="10" range_min="0.0" range_max="0.75" fov="0.5" code="1">
+      <origin xyz="${0.17131 + base_offset_x} 0.0 0.280" rpy="0.0 0.0 0.0" />
+    </xacro:ir_receiver-->
+    <!-- IR receiver -->
+    <!--xacro:ir_receiver name="${name}_ir_receiver_02" parent="${name}" ros_topic="ir_receiver_base" update_rate="10" range_min="0.0" range_max="0.75" fov="0.5" code="2">
+      <origin xyz="${0.16919 + base_offset_x} 0.14919 0.280" rpy="0.0 0.0 0.349" />
+    </xacro:ir_receiver-->
+    <!-- IR receiver -->
+    <!--xacro:ir_receiver name="${name}_ir_receiver_03" parent="${name}" ros_topic="ir_receiver_base" update_rate="10" range_min="0.0" range_max="0.75" fov="0.5" code="3">
+      <origin xyz="${0.16919 + base_offset_x} -0.14919 0.280" rpy="0.0 0.0 -0.349" />
+    </xacro:ir_receiver-->
     <!-- Wheels -->
     <xacro:wheel side="right" reflect=" 1.0" radius="${wheel_radius}" width="${wheel_width}" torque="${wheel_torque}" velocity="${wheel_velocity}" separation="${wheel_separation}" parent="${name}"/>

File: ant_description/urdf/sensors/imu.urdf.xacro (robot description, xacro)
@@ -8,5 +8,5 @@
 -->
 <robot xmlns:xacro="http://ros.org/wiki/xacro">
-  <xacro:macro name="ant_imu" params="name parent *origin update_rate">
+  <xacro:macro name="imu_sensor" params="name parent *origin update_rate">
     <link name="${name}_link">
       <inertial>
@@ -28,7 +28,4 @@
     </joint>
     <gazebo reference="${name}_link">
-      <!-- this is expected to be reparented to pelvis with appropriate offset
-          when imu_link is reduced by fixed joint reduction -->
-      <!-- todo: this is working with gazebo 1.4, need to write a unit test -->
       <sensor name="${name}_sensor" type="imu">
         <always_on>1</always_on>

File: ant_description/urdf/sensors/range.urdf.xacro (robot description, xacro)
@@ -9,5 +9,5 @@
 <robot xmlns:xacro="http://ros.org/wiki/xacro">
   <xacro:include filename="$(find ant_description)/urdf/sensors/range.gazebo.xacro" />
-  <xacro:macro name="range_ant" params="name parent *origin ros_topic update_rate maxRange minRange fov radiation">
+  <xacro:macro name="range_sensor" params="name parent *origin ros_topic update_rate maxRange minRange fov radiation">
     <link name="${name}_link">
       <inertial>

Commit message: removes base_offset_x (was 0.0) and adapts sensors' positions
git-svn-id: svn+ssh://server/srv/svn/repos/trunk/pal-ros-pkg/catkin_pkgs/ant_robot@52930 5e370ff8-3418-0410-babe-3378cc20a00d

File: ant_description/urdf/base/base.urdf.xacro (robot description, xacro)
@@ -30,5 +30,4 @@
   <property name="base_radius" value="${(wheel_separation - wheel_width)/2 - 0.01}"/>
   <property name="base_length" value="0.04"/>
-  <property name="base_offset_x" value="0.0"/>
   <property name="base_offset_z" value="${base_length + 0.031}"/>
   <!-- simplified box collision geometry for the laser -->
@@ -45,5 +44,5 @@
       </inertial>
       <visual>
-        <origin xyz="${base_offset_x} 0 ${base_offset_z}" rpy="0 0 0" />
+        <origin xyz="0 0 ${base_offset_z}" rpy="0 0 0" />
         <geometry>
           <cylinder radius="${base_radius}" length="${base_length}"/>
@@ -53,5 +52,5 @@
       </visual>
       <collision>
-        <origin xyz="${base_offset_x} 0 ${base_offset_z}" rpy="0 0 0" />
+        <origin xyz="0 0 ${base_offset_z}" rpy="0 0 0" />
         <geometry>
           <cylinder radius="${base_radius}" length="${base_length}"/>
@@ -81,37 +80,37 @@
     <!-- Sonar -->
     <xacro:range_sensor name="${name}_sonar_02" parent="${name}" ros_topic="sonar_base" update_rate="10" maxRange="0.75" minRange="0.01" fov="0.5" radiation="ultrasound">
-      <origin xyz="${0.17131 + base_offset_x} 0.0 0.280" rpy="0.0 0.0 0.0" />
+      <origin xyz="0.18 0.0 0.1" rpy="0.0 0.0 0.0" />
     </xacro:range_sensor>
     <!-- Sonar -->
     <xacro:range_sensor name="${name}_sonar_03" parent="${name}" ros_topic="sonar_base" update_rate="10" maxRange="0.75" minRange="0.01" fov="0.5" radiation="ultrasound">
-      <origin xyz="${0.16919 + base_offset_x} 0.14919 0.280" rpy="0.0 0.0 0.349" />
+      <origin xyz="0.15 0.1 0.1" rpy="0.0 0.0 ${40.0 * deg_to_rad}" />
     </xacro:range_sensor>
     <!-- Sonar -->
     <xacro:range_sensor name="${name}_sonar_01" parent="${name}" ros_topic="sonar_base" update_rate="10" maxRange="0.75" minRange="0.01" fov="0.5" radiation="ultrasound">
-      <origin xyz="${0.16919 + base_offset_x} -0.14919 0.280" rpy="0.0 0.0 -0.349" />
+      <origin xyz="0.15 -0.1 0.1" rpy="0.0 0.0 ${-40.0 * deg_to_rad}" />
     </xacro:range_sensor>
-    <!-- Bumper front right -->
+    <!-- Bumper right -->
     <xacro:bumper name="${name}_bumper_01" parent="${name}" ros_topic="bumper_base" update_rate="25" >
-      <origin xyz="${0.225 + base_offset_x} -0.15 0.20" rpy="0 0 ${-15.0 * deg_to_rad}" />
+      <origin xyz="0.16 -0.12 0.07" rpy="0 0 ${-20.0 * deg_to_rad}" />
     </xacro:bumper>
-    <!-- Bumper front left -->
+    <!-- Bumper left -->
     <xacro:bumper name="${name}_bumper_02" parent="${name}" ros_topic="bumper_base" update_rate="25" >
-      <origin xyz="${0.225 + base_offset_x} 0.15 0.20" rpy="0 0 ${15.0 * deg_to_rad}" />
+      <origin xyz="0.16 0.12 0.07" rpy="0 0 ${20.0 * deg_to_rad}" />
     </xacro:bumper>
     <!-- IMU -->
     <xacro:imu_sensor name="base_inclinometer" parent="${name}_link" update_rate="100.0">
-      <origin xyz="-0.02977 -0.1497 0.164" rpy="0 ${180 * deg_to_rad} 0"/>
+      <origin xyz="0 0 0.1" rpy="0 0 0"/>
     </xacro:imu_sensor>
     <!-- IR receiver -->
     <!--xacro:ir_receiver name="${name}_ir_receiver_01" parent="${name}" ros_topic="ir_receiver_base" update_rate="10" range_min="0.0" range_max="0.75" fov="0.5" code="1">
-      <origin xyz="${0.17131 + base_offset_x} 0.0 0.280" rpy="0.0 0.0 0.0" />
+      <origin xyz="0.17131 0.0 0.280" rpy="0.0 0.0 0.0" />
     </xacro:ir_receiver-->
     <!-- IR receiver -->
     <!--xacro:ir_receiver name="${name}_ir_receiver_02" parent="${name}" ros_topic="ir_receiver_base" update_rate="10" range_min="0.0" range_max="0.75" fov="0.5" code="2">
-      <origin xyz="${0.16919 + base_offset_x} 0.14919 0.280" rpy="0.0 0.0 0.349" />
+      <origin xyz="0.16919 0.14919 0.280" rpy="0.0 0.0 0.349" />
     </xacro:ir_receiver-->
     <!-- IR receiver -->
     <!--xacro:ir_receiver name="${name}_ir_receiver_03" parent="${name}" ros_topic="ir_receiver_base" update_rate="10" range_min="0.0" range_max="0.75" fov="0.5" code="3">
-      <origin xyz="${0.16919 + base_offset_x} -0.14919 0.280" rpy="0.0 0.0 -0.349" />
+      <origin xyz="0.16919 -0.14919 0.280" rpy="0.0 0.0 -0.349" />
     </xacro:ir_receiver-->
     <!-- Wheels -->

Commit message: puts the sonars higher and looking up, so they don't see the ground (affecting speed limit)
git-svn-id: svn+ssh://server/srv/svn/repos/trunk/pal-ros-pkg/catkin_pkgs/ant_robot@52942 5e370ff8-3418-0410-babe-3378cc20a00d

File: ant_description/urdf/base/base.urdf.xacro (robot description, xacro)
@@ -80,13 +80,13 @@
     <!-- Sonar -->
     <xacro:range_sensor name="${name}_sonar_02" parent="${name}" ros_topic="sonar_base" update_rate="10" maxRange="0.75" minRange="0.01" fov="0.5" radiation="ultrasound">
-      <origin xyz="0.18 0.0 0.1" rpy="0.0 0.0 0.0" />
+      <origin xyz="0.18 0.0 0.12" rpy="0.0 ${-10.0 * deg_to_rad} 0.0" />
     </xacro:range_sensor>
     <!-- Sonar -->
     <xacro:range_sensor name="${name}_sonar_03" parent="${name}" ros_topic="sonar_base" update_rate="10" maxRange="0.75" minRange="0.01" fov="0.5" radiation="ultrasound">
-      <origin xyz="0.15 0.1 0.1" rpy="0.0 0.0 ${40.0 * deg_to_rad}" />
+      <origin xyz="0.15 0.1 0.12" rpy="0.0 ${-10.0 * deg_to_rad} ${40.0 * deg_to_rad}" />
     </xacro:range_sensor>
     <!-- Sonar -->
     <xacro:range_sensor name="${name}_sonar_01" parent="${name}" ros_topic="sonar_base" update_rate="10" maxRange="0.75" minRange="0.01" fov="0.5" radiation="ultrasound">
-      <origin xyz="0.15 -0.1 0.1" rpy="0.0 0.0 ${-40.0 * deg_to_rad}" />
+      <origin xyz="0.15 -0.1 0.12" rpy="0.0 ${-10.0 * deg_to_rad} ${-40.0 * deg_to_rad}" />
     </xacro:range_sensor>
     <!-- Bumper right -->

Commit message: adds ir_receiver (WIP)
NOTE the ir_receiver.gazebo.xacro uses a ray sensor as a workaround!


git-svn-id: svn+ssh://server/srv/svn/repos/trunk/pal-ros-pkg/catkin_pkgs/ant_robot@55120 5e370ff8-3418-0410-babe-3378cc20a00d

File: ant_description/urdf/base/base.urdf.xacro (robot description, xacro)
@@ -104,15 +104,15 @@
     </xacro:imu_sensor>
     <!-- IR receiver -->
-    <!--xacro:ir_receiver name="${name}_ir_receiver_01" parent="${name}" ros_topic="ir_receiver_base" update_rate="10" range_min="0.0" range_max="0.75" fov="0.5" code="1">
+    <xacro:ir_receiver name="${name}_ir_receiver_01" parent="${name}" ros_topic="ir_receiver_base" update_rate="10" range_min="0.0" range_max="0.75" fov="0.5" code="1">
       <origin xyz="0.17131 0.0 0.280" rpy="0.0 0.0 0.0" />
-    </xacro:ir_receiver-->
+    </xacro:ir_receiver>
     <!-- IR receiver -->
-    <!--xacro:ir_receiver name="${name}_ir_receiver_02" parent="${name}" ros_topic="ir_receiver_base" update_rate="10" range_min="0.0" range_max="0.75" fov="0.5" code="2">
+    <xacro:ir_receiver name="${name}_ir_receiver_02" parent="${name}" ros_topic="ir_receiver_base" update_rate="10" range_min="0.0" range_max="0.75" fov="0.5" code="2">
       <origin xyz="0.16919 0.14919 0.280" rpy="0.0 0.0 0.349" />
-    </xacro:ir_receiver-->
+    </xacro:ir_receiver>
     <!-- IR receiver -->
-    <!--xacro:ir_receiver name="${name}_ir_receiver_03" parent="${name}" ros_topic="ir_receiver_base" update_rate="10" range_min="0.0" range_max="0.75" fov="0.5" code="3">
+    <xacro:ir_receiver name="${name}_ir_receiver_03" parent="${name}" ros_topic="ir_receiver_base" update_rate="10" range_min="0.0" range_max="0.75" fov="0.5" code="3">
       <origin xyz="0.16919 -0.14919 0.280" rpy="0.0 0.0 -0.349" />
-    </xacro:ir_receiver-->
+    </xacro:ir_receiver>
     <!-- Wheels -->
     <xacro:wheel side="right" reflect=" 1.0" radius="${wheel_radius}" width="${wheel_width}" torque="${wheel_torque}" velocity="${wheel_velocity}" separation="${wheel_separation}" parent="${name}"/>

File: ant_description/urdf/sensors/ir_receiver.gazebo.xacro (robot description, xacro)
@@ -8,10 +8,31 @@
 -->
 <robot xmlns:xacro="http://ros.org/wiki/xacro">
-  <xacro:macro name="ir_receiver_gazebo" params="name ros_topic update_rate range_min range_max fov code">
+  <xacro:macro name="ir_receiver_gazebo" params="name ros_topic update_rate range_min range_max fov code" >
     <gazebo reference="${name}_link">
-      <sensor type="rfid" name="${name}">
+      <sensor type="ray" name="${name}">
         <pose>0 0 0 0 0 0</pose>
         <update_rate>${update_rate}</update_rate>
         <visualize>false</visualize>
+        <ray>
+          <scan>
+            <horizontal>
+              <samples>5</samples>
+              <resolution>1</resolution>
+              <min_angle>-${fov/2}</min_angle>
+              <max_angle>${fov/2}</max_angle>
+            </horizontal>
+            <vertical>
+              <samples>5</samples>
+              <resolution>1</resolution>
+              <min_angle>-${fov/2}</min_angle>
+              <max_angle>${fov/2}</max_angle>
+            </vertical>
+          </scan>
+          <range>
+            <min>${range_min}</min>
+            <max>${range_max}</max>
+            <resolution>0.01</resolution>
+          </range>
+        </ray>
         <plugin filename="libgazebo_ros_ir_receiver.so" name="gazebo_ros_ir_receiver">
           <alwaysOn>true</alwaysOn>

Commit message: refs #8415 : removes not needed code SDF param
NTOE also removes horizontal part of scan/ray used
as ir_receiver sensor, and set the samples dependant on
the FOV


git-svn-id: svn+ssh://server/srv/svn/repos/trunk/pal-ros-pkg/catkin_pkgs/ant_robot@55176 5e370ff8-3418-0410-babe-3378cc20a00d

File: ant_description/urdf/base/base.urdf.xacro (robot description, xacro)
@@ -104,13 +104,13 @@
     </xacro:imu_sensor>
     <!-- IR receiver -->
-    <xacro:ir_receiver name="${name}_ir_receiver_01" parent="${name}" ros_topic="ir_receiver_base" update_rate="10" range_min="0.0" range_max="0.75" fov="0.5" code="1">
+    <xacro:ir_receiver name="${name}_ir_receiver_01" parent="${name}" ros_topic="ir_receiver_base" update_rate="10" range_min="0.0" range_max="0.75" fov="0.5">
       <origin xyz="0.17131 0.0 0.280" rpy="0.0 0.0 0.0" />
     </xacro:ir_receiver>
     <!-- IR receiver -->
-    <xacro:ir_receiver name="${name}_ir_receiver_02" parent="${name}" ros_topic="ir_receiver_base" update_rate="10" range_min="0.0" range_max="0.75" fov="0.5" code="2">
+    <xacro:ir_receiver name="${name}_ir_receiver_02" parent="${name}" ros_topic="ir_receiver_base" update_rate="10" range_min="0.0" range_max="0.75" fov="0.5">
       <origin xyz="0.16919 0.14919 0.280" rpy="0.0 0.0 0.349" />
     </xacro:ir_receiver>
     <!-- IR receiver -->
-    <xacro:ir_receiver name="${name}_ir_receiver_03" parent="${name}" ros_topic="ir_receiver_base" update_rate="10" range_min="0.0" range_max="0.75" fov="0.5" code="3">
+    <xacro:ir_receiver name="${name}_ir_receiver_03" parent="${name}" ros_topic="ir_receiver_base" update_rate="10" range_min="0.0" range_max="0.75" fov="0.5">
       <origin xyz="0.16919 -0.14919 0.280" rpy="0.0 0.0 -0.349" />
     </xacro:ir_receiver>

File: ant_description/urdf/sensors/ir_receiver.gazebo.xacro (robot description, xacro)
@@ -8,24 +8,18 @@
 -->
 <robot xmlns:xacro="http://ros.org/wiki/xacro">
-  <xacro:macro name="ir_receiver_gazebo" params="name ros_topic update_rate range_min range_max fov code" >
+  <xacro:macro name="ir_receiver_gazebo" params="name ros_topic update_rate range_min range_max fov" >
     <gazebo reference="${name}_link">
       <sensor type="ray" name="${name}">
         <pose>0 0 0 0 0 0</pose>
         <update_rate>${update_rate}</update_rate>
-        <visualize>false</visualize>
+        <visualize>true</visualize>
         <ray>
           <scan>
             <horizontal>
-              <samples>5</samples>
+              <samples>${100 * fov/(360 * deg_to_rad)}</samples>
               <resolution>1</resolution>
               <min_angle>-${fov/2}</min_angle>
               <max_angle>${fov/2}</max_angle>
             </horizontal>
-            <vertical>
-              <samples>5</samples>
-              <resolution>1</resolution>
-              <min_angle>-${fov/2}</min_angle>
-              <max_angle>${fov/2}</max_angle>
-            </vertical>
           </scan>
           <range>
@@ -43,5 +37,4 @@
           <maxRange>${range_max}</maxRange>
           <fov>${fov}</fov>
-          <code>${code}</code>
         </plugin>
       </sensor>

File: ant_description/urdf/sensors/ir_receiver.urdf.xacro (robot description, xacro)
@@ -9,5 +9,5 @@
 <robot xmlns:xacro="http://ros.org/wiki/xacro">
   <xacro:include filename="$(find ant_description)/urdf/sensors/ir_receiver.gazebo.xacro" />
-  <xacro:macro name="ir_receiver" params="name parent *origin ros_topic update_rate range_min range_max fov code">
+  <xacro:macro name="ir_receiver" params="name parent *origin ros_topic update_rate range_min range_max fov">
     <link name="${name}_link">
       <inertial>
@@ -24,5 +24,5 @@
     </joint>
     <!-- gazebo extensions -->
-    <xacro:ir_receiver_gazebo name="${name}" ros_topic="${ros_topic}" update_rate="${update_rate}" range_min="${range_min}" range_max="${range_max}" fov="${fov}" code="${code}"/>
+    <xacro:ir_receiver_gazebo name="${name}" ros_topic="${ros_topic}" update_rate="${update_rate}" range_min="${range_min}" range_max="${range_max}" fov="${fov}"/>
   </xacro:macro>
 </robot>
