Commit message: refs #8415 : fixes base_footprint position and casters
git-svn-id: svn+ssh://server/srv/svn/repos/trunk/pal-ros-pkg/catkin_pkgs/ant_robot@55431 5e370ff8-3418-0410-babe-3378cc20a00d

File: ant_description/urdf/base/base.urdf.xacro (robot description, xacro)
@@ -17,33 +17,32 @@
   <xacro:include filename="$(find ant_description)/urdf/sensors/ir_receiver.urdf.xacro"/>
   <!-- Wheel characteristics -->
-  <!-- Note that we temporary use Rebujito's -->
-  <property name="wheel_separation" value="0.444"/>
   <property name="wheel_radius"     value="0.08"/>
   <property name="wheel_width"      value="0.044"/>
+  <property name="wheel_separation" value="0.444"/>
   <property name="wheel_torque"     value="50.0"/>
   <property name="wheel_velocity"   value="1.0"/>
   <!-- Caster wheel characteristics -->
-  <property name="caster_separation" value="0.200"/>
-  <property name="caster_radius"     value="0.025"/>
-  <property name="caster_width"      value="0.0164"/>
-  <property name="caster_trailing"   value="0.038"/>
-  <property name="caster_offset_x"   value="0.140"/>
+  <property name="caster_radius"       value="0.025"/>
+  <property name="caster_width"        value="0.0164"/>
+  <property name="caster_separation_x" value="0.140"/>
+  <property name="caster_separation_y" value="0.200"/>
+  <property name="caster_offset_z"     value="-0.02"/> <!-- ${-base_length / 2} -->
+  <!-- Base characteristics -->
   <property name="base_radius" value="${(wheel_separation - wheel_width)/2 - 0.01}"/>
   <property name="base_length" value="0.04"/>
-  <property name="base_offset_z" value="${base_length + 0.031}"/>
-  <!-- simplified box collision geometry for the laser -->
+  <!-- Laser characteristics -->
   <property name="base_laser_x" value="0.15"/>
   <property name="base_laser_y" value="0.0"/>
-  <property name="base_laser_z" value="0.153"/>
+  <property name="base_laser_z" value="0.083"/>
   <xacro:macro name="base" params="name">
     <!-- Base -->
     <link name="${name}_link">
       <inertial>
-        <origin xyz="0.0 0.0 0.26721" rpy="0 0 0" />
-        <mass value="63.58850" />
-        <inertia ixx="3.42" ixy="0" ixz="0" iyy="4.33" iyz="0" izz="5.08" />
+        <origin xyz="0.0 0.0 0.0" rpy="0 0 0" />
+        <mass value="10.0" />
+        <inertia ixx="1.0" ixy="0" ixz="0" iyy="1.0" iyz="0" izz="1.0" />
       </inertial>
       <visual>
-        <origin xyz="0 0 ${base_offset_z}" rpy="0 0 0" />
+        <origin xyz="0 0 0" rpy="0 0 0" />
         <geometry>
           <cylinder radius="${base_radius}" length="${base_length}"/>
@@ -53,5 +52,5 @@
       </visual>
       <collision>
-        <origin xyz="0 0 ${base_offset_z}" rpy="0 0 0" />
+        <origin xyz="0 0 0" rpy="0 0 0" />
         <geometry>
           <cylinder radius="${base_radius}" length="${base_length}"/>
@@ -62,14 +61,7 @@
     </link>
     <!-- Base footprint -->
-    <link name="${name}_footprint">
-      <collision>
-        <origin xyz="0 0 0.2" rpy="0 0 0" />
-        <geometry>
-          <box size="0.001 0.001 0.001" />
-        </geometry>
-      </collision>
-    </link>
+    <link name="${name}_footprint"/>
     <joint name="${name}_footprint_joint" type="fixed">
-      <origin xyz="0 0 0" rpy="0 0 0" />
+      <origin xyz="0 0 ${wheel_radius}" rpy="0 0 0" />
       <child link="${name}_link" />
       <parent link="${name}_footprint"/>
@@ -81,25 +73,25 @@
     <!-- Sonar -->
     <xacro:range_sensor name="${name}_sonar_02" parent="${name}" ros_topic="sonar_base" update_rate="10" maxRange="0.75" minRange="0.01" fov="0.5" radiation="ultrasound">
-      <origin xyz="0.18 0.0 0.12" rpy="0.0 ${-10.0 * deg_to_rad} 0.0" />
+      <origin xyz="0.18 0.0 0.04" rpy="0.0 ${-10.0 * deg_to_rad} 0.0" />
     </xacro:range_sensor>
     <!-- Sonar -->
     <xacro:range_sensor name="${name}_sonar_03" parent="${name}" ros_topic="sonar_base" update_rate="10" maxRange="0.75" minRange="0.01" fov="0.5" radiation="ultrasound">
-      <origin xyz="0.15 0.1 0.12" rpy="0.0 ${-10.0 * deg_to_rad} ${40.0 * deg_to_rad}" />
+      <origin xyz="0.15 0.1 0.04" rpy="0.0 ${-10.0 * deg_to_rad} ${40.0 * deg_to_rad}" />
     </xacro:range_sensor>
     <!-- Sonar -->
     <xacro:range_sensor name="${name}_sonar_01" parent="${name}" ros_topic="sonar_base" update_rate="10" maxRange="0.75" minRange="0.01" fov="0.5" radiation="ultrasound">
-      <origin xyz="0.15 -0.1 0.12" rpy="0.0 ${-10.0 * deg_to_rad} ${-40.0 * deg_to_rad}" />
+      <origin xyz="0.15 -0.1 0.04" rpy="0.0 ${-10.0 * deg_to_rad} ${-40.0 * deg_to_rad}" />
     </xacro:range_sensor>
     <!-- Bumper right -->
     <xacro:bumper name="${name}_bumper_01" parent="${name}" ros_topic="bumper_base" update_rate="25" >
-      <origin xyz="0.16 -0.12 0.07" rpy="0 0 ${-20.0 * deg_to_rad}" />
+      <origin xyz="0.16 -0.12 0.00" rpy="0 0 ${-20.0 * deg_to_rad}" />
     </xacro:bumper>
     <!-- Bumper left -->
     <xacro:bumper name="${name}_bumper_02" parent="${name}" ros_topic="bumper_base" update_rate="25" >
-      <origin xyz="0.16 0.12 0.07" rpy="0 0 ${20.0 * deg_to_rad}" />
+      <origin xyz="0.16 0.12 0.00" rpy="0 0 ${20.0 * deg_to_rad}" />
     </xacro:bumper>
     <!-- IMU -->
     <xacro:imu_sensor name="base_inclinometer" parent="${name}_link" update_rate="100.0">
-      <origin xyz="0 0 0.1" rpy="0 0 0"/>
+      <origin xyz="0 0 0.2" rpy="0 0 0"/>
     </xacro:imu_sensor>
     <!-- IR receiver -->
@@ -119,8 +111,8 @@
     <xacro:wheel side="left"  reflect="-1.0" radius="${wheel_radius}" width="${wheel_width}" torque="${wheel_torque}" velocity="${wheel_velocity}" separation="${wheel_separation}" parent="${name}"/>
     <!-- Casters wheels -->
-    <xacro:caster side="front_right" reflect=" 1.0" radius="${caster_radius}" width="${caster_width}" separation="${caster_separation}" trailing="${caster_trailing}" offset_x="${caster_offset_x}" parent="${name}"/>
-    <xacro:caster side="front_left"  reflect="-1.0" radius="${caster_radius}" width="${caster_width}" separation="${caster_separation}" trailing="${caster_trailing}" offset_x="${caster_offset_x}" parent="${name}"/>
-    <xacro:caster side="back_right" reflect=" 1.0" radius="${caster_radius}" width="${caster_width}" separation="${caster_separation}" trailing="${caster_trailing}" offset_x="${-caster_offset_x}" parent="${name}"/>
-    <xacro:caster side="back_left"  reflect="-1.0" radius="${caster_radius}" width="${caster_width}" separation="${caster_separation}" trailing="${caster_trailing}" offset_x="${-caster_offset_x}" parent="${name}"/>
+    <xacro:caster side="front_right" radius="${caster_radius}" width="${caster_width}" separation_x="${ caster_separation_x}" separation_y="${ caster_separation_y}" offset_z="${caster_offset_z}" parent="${name}"/>
+    <xacro:caster side="front_left"  radius="${caster_radius}" width="${caster_width}" separation_x="${ caster_separation_x}" separation_y="${-caster_separation_y}" offset_z="${caster_offset_z}" parent="${name}"/>
+    <xacro:caster side="back_right"  radius="${caster_radius}" width="${caster_width}" separation_x="${-caster_separation_x}" separation_y="${ caster_separation_y}" offset_z="${caster_offset_z}" parent="${name}"/>
+    <xacro:caster side="back_left"   radius="${caster_radius}" width="${caster_width}" separation_x="${-caster_separation_x}" separation_y="${-caster_separation_y}" offset_z="${caster_offset_z}" parent="${name}"/>
   </xacro:macro>
 </robot>

File: ant_description/urdf/wheels/caster.urdf.xacro (robot description, xacro)
@@ -10,5 +10,5 @@
   <xacro:include filename="$(find ant_description)/urdf/wheels/caster.transmission.xacro"/>
   <xacro:include filename="$(find ant_description)/urdf/wheels/caster.gazebo.xacro"/>
-  <xacro:macro name="caster" params="side reflect radius width separation trailing offset_x parent">
+  <xacro:macro name="caster" params="side radius width separation_x separation_y offset_z parent">
     <link name="caster_${side}_1_link">
       <inertial>
@@ -20,5 +20,5 @@
       </inertial>
       <visual>
-        <origin xyz="${0.5 * radius - trailing} 0 ${0.5 * radius}" rpy="0 0 0"/>
+        <origin xyz="0 0 0" rpy="0 0 0"/>
         <geometry>
           <box size="${radius} ${1.2 * width} ${radius}"/>
@@ -27,5 +27,5 @@
       </visual>
       <collision>
-        <origin xyz="${0.5 * radius - trailing} 0 ${0.5 * radius}" rpy="0 0 0"/>
+        <origin xyz="0 0 0" rpy="0 0 0"/>
         <geometry>
           <box size="${radius} ${1.2 * width} ${radius}"/>
@@ -56,5 +56,5 @@
       <parent link="${parent}_link"/>
       <child link="caster_${side}_1_link"/>
-      <origin xyz="${offset_x} ${-separation / 2 * reflect} ${radius}" rpy="0 0 0"/>
+      <origin xyz="${separation_x} ${-separation_y / 2} ${offset_z - radius / 2}" rpy="0 0 0"/>
       <axis xyz="0 0 1"/>
     </joint>
@@ -62,5 +62,5 @@
       <parent link="caster_${side}_1_link"/>
       <child link="caster_${side}_2_link"/>
-      <origin xyz="${-trailing} 0 0" rpy="${-90.0 * deg_to_rad} 0 0"/>
+      <origin xyz="${-radius / 2} 0 ${-radius + 0.0025}" rpy="${-90.0 * deg_to_rad} 0 0"/>
       <axis xyz="0 0 1"/>
     </joint>

File: ant_description/urdf/wheels/wheel.urdf.xacro (robot description, xacro)
@@ -34,5 +34,5 @@
       <parent link="${parent}_link"/>
       <child link="wheel_${side}_link"/>
-      <origin xyz="0 ${-separation / 2 * reflect} ${radius}" rpy="${-90.0 * deg_to_rad} 0 0"/>
+      <origin xyz="0 ${-separation / 2 * reflect} 0" rpy="${-90.0 * deg_to_rad} 0 0"/>
       <axis xyz="0 0 1"/>
       <limit effort="${torque}" velocity="${velocity / radius}"/>

Commit message: refs #8415 : fixes inclinometer and ir receivers position (z-axis)
git-svn-id: svn+ssh://server/srv/svn/repos/trunk/pal-ros-pkg/catkin_pkgs/ant_robot@55436 5e370ff8-3418-0410-babe-3378cc20a00d

File: ant_description/urdf/base/base.urdf.xacro (robot description, xacro)
@@ -93,17 +93,17 @@
     <!-- IMU -->
     <xacro:imu_sensor name="base_inclinometer" parent="${name}_link" update_rate="100.0">
-      <origin xyz="0 0 0.2" rpy="0 0 0"/>
+      <origin xyz="0 0 ${base_length / 2}" rpy="0 0 0"/>
     </xacro:imu_sensor>
     <!-- IR receiver -->
     <xacro:ir_receiver name="${name}_ir_receiver_01" parent="${name}" ros_topic="ir_receiver_base" update_rate="10" range_min="0.0" range_max="0.75" fov="0.5">
-      <origin xyz="0.17131 0.0 0.280" rpy="0.0 0.0 0.0" />
+      <origin xyz="0.17131 0.0 0.180" rpy="0.0 0.0 0.0" />
     </xacro:ir_receiver>
     <!-- IR receiver -->
     <xacro:ir_receiver name="${name}_ir_receiver_02" parent="${name}" ros_topic="ir_receiver_base" update_rate="10" range_min="0.0" range_max="0.75" fov="0.5">
-      <origin xyz="0.16919 0.14919 0.280" rpy="0.0 0.0 0.349" />
+      <origin xyz="0.16919 0.14919 0.180" rpy="0.0 0.0 0.349" />
     </xacro:ir_receiver>
     <!-- IR receiver -->
     <xacro:ir_receiver name="${name}_ir_receiver_03" parent="${name}" ros_topic="ir_receiver_base" update_rate="10" range_min="0.0" range_max="0.75" fov="0.5">
-      <origin xyz="0.16919 -0.14919 0.280" rpy="0.0 0.0 -0.349" />
+      <origin xyz="0.16919 -0.14919 0.180" rpy="0.0 0.0 -0.349" />
     </xacro:ir_receiver>
     <!-- Wheels -->

Commit message: adds base stl (note the final one)
git-svn-id: svn+ssh://server/srv/svn/repos/trunk/pal-ros-pkg/catkin_pkgs/ant_robot@55596 5e370ff8-3418-0410-babe-3378cc20a00d

File: ant_description/urdf/base/base.urdf.xacro (robot description, xacro)
@@ -46,5 +46,6 @@
         <origin xyz="0 0 0" rpy="0 0 0" />
         <geometry>
-          <cylinder radius="${base_radius}" length="${base_length}"/>
+          <!--cylinder radius="${base_radius}" length="${base_length}"/-->
+          <mesh filename="package://ant_description/meshes/base/base.stl" />
           <!--mesh filename="package://ant_description/meshes/base/base.dae" /-->
         </geometry>

Commit message: fixes base STL and updates links positions
NOTE mass and CoM, and inertias not set yet


git-svn-id: svn+ssh://server/srv/svn/repos/trunk/pal-ros-pkg/catkin_pkgs/ant_robot@55653 5e370ff8-3418-0410-babe-3378cc20a00d

File: ant_description/urdf/base/base.urdf.xacro (robot description, xacro)
@@ -17,22 +17,22 @@
   <xacro:include filename="$(find ant_description)/urdf/sensors/ir_receiver.urdf.xacro"/>
   <!-- Wheel characteristics -->
-  <property name="wheel_radius"     value="0.08"/>
+  <property name="wheel_radius"     value="0.100"/>
   <property name="wheel_width"      value="0.044"/>
-  <property name="wheel_separation" value="0.444"/>
-  <property name="wheel_torque"     value="50.0"/>
+  <property name="wheel_separation" value="0.43408"/>
+  <property name="wheel_torque"     value="50.0"/><!--@todo try this: 6Nm-->
   <property name="wheel_velocity"   value="1.0"/>
   <!-- Caster wheel characteristics -->
   <property name="caster_radius"       value="0.025"/>
-  <property name="caster_width"        value="0.0164"/>
-  <property name="caster_separation_x" value="0.140"/>
-  <property name="caster_separation_y" value="0.200"/>
-  <property name="caster_offset_z"     value="-0.02"/> <!-- ${-base_length / 2} -->
+  <property name="caster_width"        value="0.020"/>
+  <property name="caster_separation_x" value="0.36734"/>
+  <property name="caster_separation_y" value="0.20362"/>
+  <property name="caster_offset_z"     value="-0.04252"/>
   <!-- Base characteristics -->
   <property name="base_radius" value="${(wheel_separation - wheel_width)/2 - 0.01}"/>
   <property name="base_length" value="0.04"/>
   <!-- Laser characteristics -->
-  <property name="base_laser_x" value="0.15"/>
+  <property name="base_laser_x" value="0.185"/>
   <property name="base_laser_y" value="0.0"/>
-  <property name="base_laser_z" value="0.083"/>
+  <property name="base_laser_z" value="0.05275"/>
   <xacro:macro name="base" params="name">
     <!-- Base -->
@@ -69,43 +69,44 @@
     </joint>
     <!-- Laser -->
-    <xacro:hokuyo_urg_04lx_ug01_laser name="${name}_laser" parent="${name}" ros_topic="scan" update_rate="10" min_angle="${-100 * deg_to_rad}" max_angle="${100 * deg_to_rad}" >
+    <xacro:hokuyo_urg_04lx_ug01_laser name="${name}_laser" parent="${name}" ros_topic="scan" update_rate="10" min_angle="${-90 * deg_to_rad}" max_angle="${90 * deg_to_rad}" >
       <origin xyz="${base_laser_x} ${base_laser_y} ${base_laser_z}" rpy="0 0 0" />
     </xacro:hokuyo_urg_04lx_ug01_laser>
     <!-- Sonar -->
-    <xacro:range_sensor name="${name}_sonar_02" parent="${name}" ros_topic="sonar_base" update_rate="10" maxRange="0.75" minRange="0.01" fov="0.5" radiation="ultrasound">
+    <!--xacro:range_sensor name="${name}_sonar_02" parent="${name}" ros_topic="sonar_base" update_rate="10" maxRange="0.75" minRange="0.01" fov="0.5" radiation="ultrasound">
       <origin xyz="0.18 0.0 0.04" rpy="0.0 ${-10.0 * deg_to_rad} 0.0" />
-    </xacro:range_sensor>
+    </xacro:range_sensor-->
     <!-- Sonar -->
-    <xacro:range_sensor name="${name}_sonar_03" parent="${name}" ros_topic="sonar_base" update_rate="10" maxRange="0.75" minRange="0.01" fov="0.5" radiation="ultrasound">
+    <!--xacro:range_sensor name="${name}_sonar_03" parent="${name}" ros_topic="sonar_base" update_rate="10" maxRange="0.75" minRange="0.01" fov="0.5" radiation="ultrasound">
       <origin xyz="0.15 0.1 0.04" rpy="0.0 ${-10.0 * deg_to_rad} ${40.0 * deg_to_rad}" />
-    </xacro:range_sensor>
+    </xacro:range_sensor-->
     <!-- Sonar -->
-    <xacro:range_sensor name="${name}_sonar_01" parent="${name}" ros_topic="sonar_base" update_rate="10" maxRange="0.75" minRange="0.01" fov="0.5" radiation="ultrasound">
+    <!--xacro:range_sensor name="${name}_sonar_01" parent="${name}" ros_topic="sonar_base" update_rate="10" maxRange="0.75" minRange="0.01" fov="0.5" radiation="ultrasound">
       <origin xyz="0.15 -0.1 0.04" rpy="0.0 ${-10.0 * deg_to_rad} ${-40.0 * deg_to_rad}" />
-    </xacro:range_sensor>
+    </xacro:range_sensor-->
     <!-- Bumper right -->
-    <xacro:bumper name="${name}_bumper_01" parent="${name}" ros_topic="bumper_base" update_rate="25" >
+    <!--xacro:bumper name="${name}_bumper_01" parent="${name}" ros_topic="bumper_base" update_rate="25" >
       <origin xyz="0.16 -0.12 0.00" rpy="0 0 ${-20.0 * deg_to_rad}" />
-    </xacro:bumper>
+    </xacro:bumper-->
     <!-- Bumper left -->
-    <xacro:bumper name="${name}_bumper_02" parent="${name}" ros_topic="bumper_base" update_rate="25" >
+    <!--xacro:bumper name="${name}_bumper_02" parent="${name}" ros_topic="bumper_base" update_rate="25" >
       <origin xyz="0.16 0.12 0.00" rpy="0 0 ${20.0 * deg_to_rad}" />
-    </xacro:bumper>
+    </xacro:bumper-->
     <!-- IMU -->
+    <!-- @todo ant_hardware_gazebo needs an IMU!  -->
     <xacro:imu_sensor name="base_inclinometer" parent="${name}_link" update_rate="100.0">
       <origin xyz="0 0 ${base_length / 2}" rpy="0 0 0"/>
     </xacro:imu_sensor>
     <!-- IR receiver -->
-    <xacro:ir_receiver name="${name}_ir_receiver_01" parent="${name}" ros_topic="ir_receiver_base" update_rate="10" range_min="0.0" range_max="0.75" fov="0.5">
+    <!--xacro:ir_receiver name="${name}_ir_receiver_01" parent="${name}" ros_topic="ir_receiver_base" update_rate="10" range_min="0.0" range_max="0.75" fov="0.5">
       <origin xyz="0.17131 0.0 0.180" rpy="0.0 0.0 0.0" />
-    </xacro:ir_receiver>
+    </xacro:ir_receiver-->
     <!-- IR receiver -->
-    <xacro:ir_receiver name="${name}_ir_receiver_02" parent="${name}" ros_topic="ir_receiver_base" update_rate="10" range_min="0.0" range_max="0.75" fov="0.5">
+    <!--xacro:ir_receiver name="${name}_ir_receiver_02" parent="${name}" ros_topic="ir_receiver_base" update_rate="10" range_min="0.0" range_max="0.75" fov="0.5">
       <origin xyz="0.16919 0.14919 0.180" rpy="0.0 0.0 0.349" />
-    </xacro:ir_receiver>
+    </xacro:ir_receiver-->
     <!-- IR receiver -->
-    <xacro:ir_receiver name="${name}_ir_receiver_03" parent="${name}" ros_topic="ir_receiver_base" update_rate="10" range_min="0.0" range_max="0.75" fov="0.5">
+    <!--xacro:ir_receiver name="${name}_ir_receiver_03" parent="${name}" ros_topic="ir_receiver_base" update_rate="10" range_min="0.0" range_max="0.75" fov="0.5">
       <origin xyz="0.16919 -0.14919 0.180" rpy="0.0 0.0 -0.349" />
-    </xacro:ir_receiver>
+    </xacro:ir_receiver-->
     <!-- Wheels -->
     <xacro:wheel side="right" reflect=" 1.0" radius="${wheel_radius}" width="${wheel_width}" torque="${wheel_torque}" velocity="${wheel_velocity}" separation="${wheel_separation}" parent="${name}"/>

File: ant_description/urdf/wheels/caster.urdf.xacro (robot description, xacro)
@@ -64,5 +64,5 @@
       <parent link="${parent}_link"/>
       <child link="caster_${side}_1_link"/>
-      <origin xyz="${separation_x} ${-separation_y / 2} ${offset_z - radius / 2}" rpy="0 0 0"/>
+      <origin xyz="${separation_x / 2} ${-separation_y / 2} ${offset_z}" rpy="0 0 0"/>
       <axis xyz="0 0 1"/>
     </joint>
@@ -70,5 +70,5 @@
       <parent link="caster_${side}_1_link"/>
       <child link="caster_${side}_2_link"/>
-      <origin xyz="${-radius / 2} 0 ${-radius + 0.0025}" rpy="${-90.0 * deg_to_rad} 0 0"/>
+      <origin xyz="0.017 0.0003 -0.032" rpy="${-90.0 * deg_to_rad} 0 0"/>
       <axis xyz="0 0 1"/>
     </joint>

Commit message: updates caster and wheel position, angle and STL
git-svn-id: svn+ssh://server/srv/svn/repos/trunk/pal-ros-pkg/catkin_pkgs/ant_robot@55687 5e370ff8-3418-0410-babe-3378cc20a00d

File: ant_description/urdf/base/base.urdf.xacro (robot description, xacro)
@@ -56,4 +56,5 @@
         <geometry>
           <cylinder radius="${base_radius}" length="${base_length}"/>
+          <!-- @todo base_collision.stl still the same as base.stl -->
           <!--mesh filename="package://ant_description/meshes/base/base_collision.stl" /-->
         </geometry>

File: ant_description/urdf/wheels/caster.urdf.xacro (robot description, xacro)
@@ -22,5 +22,6 @@
         <origin xyz="0 0 0" rpy="0 0 0"/>
         <geometry>
-          <box size="${radius} ${1.2 * width} ${radius}"/>
+          <!--box size="${radius} ${1.2 * width} ${radius}"/-->
+          <mesh filename="package://ant_description/meshes/wheels/caster.stl"/>
         </geometry>
         <material name="DarkGrey"/>
@@ -29,5 +30,6 @@
         <origin xyz="0 0 0" rpy="0 0 0"/>
         <geometry>
-          <box size="${radius} ${1.2 * width} ${radius}"/>
+          <!--box size="${radius} ${1.2 * width} ${radius}"/-->
+          <mesh filename="package://ant_description/meshes/wheels/caster.stl"/>
         </geometry>
       </collision>
@@ -70,5 +72,5 @@
       <parent link="caster_${side}_1_link"/>
       <child link="caster_${side}_2_link"/>
-      <origin xyz="0.017 0.0003 -0.032" rpy="${-90.0 * deg_to_rad} 0 0"/>
+      <origin xyz="-0.017 0.0003 -0.032" rpy="${90.0 * deg_to_rad} 0 0"/>
       <axis xyz="0 0 1"/>
     </joint>

File: ant_description/urdf/wheels/wheel.urdf.xacro (robot description, xacro)
@@ -42,5 +42,5 @@
       <parent link="${parent}_link"/>
       <child link="wheel_${side}_link"/>
-      <origin xyz="0 ${-separation / 2 * reflect} 0" rpy="${-90.0 * deg_to_rad} 0 0"/>
+      <origin xyz="0 ${-separation / 2 * reflect} 0" rpy="${90.0 * deg_to_rad} 0 0"/>
       <axis xyz="0 0 1"/>
       <limit effort="${torque}" velocity="${velocity / radius}"/>
