Commit message: refs #8219 : sets CoM and mass
git-svn-id: svn+ssh://server/srv/svn/repos/trunk/pal-ros-pkg/catkin_pkgs/ant_robot@55689 5e370ff8-3418-0410-babe-3378cc20a00d

File: ant_description/urdf/base/base.urdf.xacro (robot description, xacro)
@@ -39,6 +39,6 @@
     <link name="${name}_link">
       <inertial>
-        <origin xyz="0.0 0.0 0.0" rpy="0 0 0" />
-        <mass value="10.0" />
+        <origin xyz="0.0123 0.0071 0.064" rpy="0 0 0" />
+        <mass value="7.95534" />
         <inertia ixx="1.0" ixy="0" ixz="0" iyy="1.0" iyz="0" izz="1.0" />
       </inertial>

File: ant_description/urdf/sensors/hokuyo_urg_04lx_ug01_laser.urdf.xacro (robot description, xacro)
@@ -12,6 +12,6 @@
      <link name="${name}_link" type="laser">
       <inertial>
-        <origin xyz="0 0 0" rpy="0 0 0" />
-        <mass value="0.001" />
+        <origin xyz="0 0 -0.04225" rpy="0 0 0" />
+        <mass value="0.160" />
         <inertia iyy="4.2412e-05" ixy="4.9927e-08" iyz="-9.8165e-09" ixx="3.7174e-05" ixz="1.1015e-05" izz="4.167e-05" />
       </inertial>

File: ant_description/urdf/wheels/caster.urdf.xacro (robot description, xacro)
@@ -13,6 +13,6 @@
     <link name="caster_${side}_1_link">
       <inertial>
-        <origin xyz="0 0 0" rpy="0 0 0"/>
-        <mass value="0.1"/>
+        <origin xyz="-0.00653 -0.00008 -0.01177" rpy="0 0 0"/>
+        <mass value="0.09556"/>
         <inertia  ixx="0.012411765597" ixy="-0.000711733678" ixz="0.00050272983"
                   iyy="0.015218160428" iyz="-0.000004273467"
@@ -38,5 +38,5 @@
       <inertial>
         <origin xyz="0 0 0" rpy="0 0 0"/>
-        <mass value="0.4"/>
+        <mass value="0.02425"/>
         <inertia  ixx="0.00044" ixy="0" ixz="0" iyy="0.00044" iyz="0" izz="0.00078"/>
         </inertial>

File: ant_description/urdf/wheels/wheel.urdf.xacro (robot description, xacro)
@@ -13,6 +13,6 @@
     <link name="wheel_${side}_link">
       <inertial>
-        <origin xyz="0 0 0" rpy="0 0 0"/>
-        <mass value="1.0"/>
+        <origin xyz="0 0 -0.0016" rpy="0 0 0"/>
+        <mass value="3.33926"/>
         <inertia ixx="1" ixy="0" ixz="0" iyy="1" iyz="0" izz="1"/>
       </inertial>

Commit message: refs #8219 : sets inertias
git-svn-id: svn+ssh://server/srv/svn/repos/trunk/pal-ros-pkg/catkin_pkgs/ant_robot@55692 5e370ff8-3418-0410-babe-3378cc20a00d

File: ant_description/urdf/base/base.urdf.xacro (robot description, xacro)
@@ -41,5 +41,7 @@
         <origin xyz="0.0123 0.0071 0.064" rpy="0 0 0" />
         <mass value="7.95534" />
-        <inertia ixx="1.0" ixy="0" ixz="0" iyy="1.0" iyz="0" izz="1.0" />
+        <inertia ixx="0.19540233297" ixy="-0.00188862789" ixz="-0.00370655921"
+                 iyy="0.23325457568" iyz="0.00387528692"
+                 izz="0.3312456162" />
       </inertial>
       <visual>

File: ant_description/urdf/sensors/hokuyo_urg_04lx_ug01_laser.urdf.xacro (robot description, xacro)
@@ -14,5 +14,7 @@
         <origin xyz="0 0 -0.04225" rpy="0 0 0" />
         <mass value="0.160" />
-        <inertia iyy="4.2412e-05" ixy="4.9927e-08" iyz="-9.8165e-09" ixx="3.7174e-05" ixz="1.1015e-05" izz="4.167e-05" />
+        <inertia ixx="0.00008631543" ixy="-0.00000088815" ixz="-0.00000094079"
+                 iyy="0.00008461544" iyz="0.00000139389"
+                 izz="0.00005947238" />
       </inertial>
       <visual>

File: ant_description/urdf/wheels/caster.urdf.xacro (robot description, xacro)
@@ -15,7 +15,7 @@
         <origin xyz="-0.00653 -0.00008 -0.01177" rpy="0 0 0"/>
         <mass value="0.09556"/>
-        <inertia  ixx="0.012411765597" ixy="-0.000711733678" ixz="0.00050272983"
-                  iyy="0.015218160428" iyz="-0.000004273467"
-                  izz="0.011763977943"/>
+        <inertia  ixx="0.00002195406" ixy="0.00000000009" ixz="0.00000370909"
+                  iyy="0.00001717745" iyz="-0.00000000032"
+                  izz="0.00002240463"/>
       </inertial>
       <visual>
@@ -39,5 +39,7 @@
         <origin xyz="0 0 0" rpy="0 0 0"/>
         <mass value="0.02425"/>
-        <inertia  ixx="0.00044" ixy="0" ixz="0" iyy="0.00044" iyz="0" izz="0.00078"/>
+        <inertia  ixx="0.00000464376" ixy="0" ixz="0"
+                  iyy="0.00000464377" iyz="0"
+                  izz="0.00000802779"/>
         </inertial>
       <visual>
@@ -72,5 +74,5 @@
       <parent link="caster_${side}_1_link"/>
       <child link="caster_${side}_2_link"/>
-      <origin xyz="-0.017 0.0003 -0.032" rpy="${90.0 * deg_to_rad} 0 0"/>
+      <origin xyz="-0.017 0.0003 -0.032" rpy="${-90.0 * deg_to_rad} 0 0"/>
       <axis xyz="0 0 1"/>
     </joint>

File: ant_description/urdf/wheels/wheel.urdf.xacro (robot description, xacro)
@@ -15,5 +15,7 @@
         <origin xyz="0 0 -0.0016" rpy="0 0 0"/>
         <mass value="3.33926"/>
-        <inertia ixx="1" ixy="0" ixz="0" iyy="1" iyz="0" izz="1"/>
+        <inertia ixx="0.00668369447" ixy="0.00000007414" ixz="0.00000024433"
+                 iyy="0.00668332554" iyz="-0.00000005662"
+                 izz="0.01088090651"/>
       </inertial>
       <visual>
@@ -42,5 +44,5 @@
       <parent link="${parent}_link"/>
       <child link="wheel_${side}_link"/>
-      <origin xyz="0 ${-separation / 2 * reflect} 0" rpy="${90.0 * deg_to_rad} 0 0"/>
+      <origin xyz="0 ${-separation / 2 * reflect} 0" rpy="${-90.0 * deg_to_rad} 0 0"/>
       <axis xyz="0 0 1"/>
       <limit effort="${torque}" velocity="${velocity / radius}"/>

Commit message: puts more similar colors
git-svn-id: svn+ssh://server/srv/svn/repos/trunk/pal-ros-pkg/catkin_pkgs/ant_robot@56490 5e370ff8-3418-0410-babe-3378cc20a00d

File: ant_description/urdf/base/base.urdf.xacro (robot description, xacro)
@@ -52,5 +52,5 @@
           <!--mesh filename="package://ant_description/meshes/base/base.dae" /-->
         </geometry>
-        <material name="LightGrey" />
+        <material name="DarkGrey" />
       </visual>
       <collision>
@@ -61,5 +61,5 @@
           <!--mesh filename="package://ant_description/meshes/base/base_collision.stl" /-->
         </geometry>
-        <material name="LightGrey" />
+        <material name="DarkGrey" />
       </collision>
     </link>

File: ant_description/urdf/wheels/caster.urdf.xacro (robot description, xacro)
@@ -25,5 +25,5 @@
           <mesh filename="package://ant_description/meshes/wheels/caster.stl"/>
         </geometry>
-        <material name="DarkGrey"/>
+        <material name="Grey"/>
       </visual>
       <collision>

File: ant_description/urdf/wheels/wheel.urdf.xacro (robot description, xacro)
@@ -24,5 +24,5 @@
           <cylinder radius="${radius}" length="${width}"/>
         </geometry>
-        <material name="DarkGrey"/>
+        <material name="LightGrey"/>
       </visual>
       <collision>
