Commit message: adds RGBD sensor with laser
NOTE with robot:=rgbd_only we have only the RGBD
(and we can use the depthimage_to_laserscan to simulate a laser)


git-svn-id: svn+ssh://server/srv/svn/repos/trunk/pal-ros-pkg/catkin_pkgs/ant_robot@57443 5e370ff8-3418-0410-babe-3378cc20a00d

File: ant_description/urdf/base/base_rgbd_only.urdf.xacro (robot description, xacro)
@@ -12,5 +12,4 @@
   <xacro:include filename="$(find ant_description)/urdf/wheels/caster.urdf.xacro"/>
   <xacro:include filename="$(find ant_description)/urdf/sensors/range.urdf.xacro"/>
-  <xacro:include filename="$(find ant_description)/urdf/sensors/hokuyo_urg_04lx_ug01_laser.urdf.xacro"/>
   <xacro:include filename="$(find ant_description)/urdf/sensors/xtion_pro_live.urdf.xacro"/>
   <xacro:include filename="$(find ant_description)/urdf/sensors/imu.urdf.xacro"/>
@@ -32,12 +31,8 @@
   <property name="base_radius" value="${(wheel_separation - wheel_width)/2 - 0.01}"/>
   <property name="base_length" value="0.04"/>
-  <!-- Laser characteristics -->
-  <property name="base_laser_x" value="0.185"/>
-  <property name="base_laser_y" value="0.0"/>
-  <property name="base_laser_z" value="0.05275"/>
   <!-- RGBD characteristics -->
   <property name="base_rgbd_x" value="0.185"/>
   <property name="base_rgbd_y" value="0.0"/>
-  <property name="base_rgbd_z" value="0.23"/>
+  <property name="base_rgbd_z" value="0.05275"/>
   <xacro:macro name="base" params="name">
     <!-- Base -->
@@ -76,8 +71,4 @@
       <parent link="${name}_footprint"/>
     </joint>
-    <!-- Laser -->
-    <xacro:hokuyo_urg_04lx_ug01_laser name="${name}_laser" parent="${name}" ros_topic="scan" update_rate="10" min_angle="${-90 * deg_to_rad}" max_angle="${90 * deg_to_rad}" >
-      <origin xyz="${base_laser_x} ${base_laser_y} ${base_laser_z}" rpy="0 0 0" />
-    </xacro:hokuyo_urg_04lx_ug01_laser>
     <!-- RGBD -->
     <xacro:xtion_pro_live name="${name}_xtion" parent="${name}">

Commit message: adds softkinetic with hfov (rotated)
git-svn-id: svn+ssh://server/srv/svn/repos/trunk/pal-ros-pkg/catkin_pkgs/ant_robot@58003 5e370ff8-3418-0410-babe-3378cc20a00d

File: ant_description/urdf/base/base_rgbd_only.urdf.xacro (robot description, xacro)
@@ -76,5 +76,5 @@
       <origin xyz="${base_rgbd_x} ${base_rgbd_y} ${base_rgbd_z}" rpy="0 0 0"/>
       <!-- Pose of optical frame wrt to sensor -->
-      <origin xyz="0 0 0" rpy="${-90 * deg_to_rad} 0 ${-90 * deg_to_rad}"/>
+      <optical_origin xyz="0 0 0" rpy="${-90 * deg_to_rad} 0 ${-90 * deg_to_rad}"/>
     </xacro:xtion_pro_live>
     <!-- Sonar -->

File: ant_description/urdf/base/base_softkinetic_ds311.urdf.xacro (robot description, xacro)
@@ -85,5 +85,5 @@
       <origin xyz="${base_rgbd_x} ${base_rgbd_y} ${base_rgbd_z}" rpy="0 0 0"/>
       <!-- Pose of optical frame wrt to sensor -->
-      <origin xyz="0 0 0" rpy="${-90 * deg_to_rad} 0 ${-90 * deg_to_rad}"/>
+      <optical_origin xyz="0 0 0" rpy="${-90 * deg_to_rad} 0 ${-90 * deg_to_rad}"/>
     </xacro:softkinetic_ds311_rgbd_camera>
     <!-- Sonar -->

File: ant_description/urdf/base/base_softkinetic_ds311_hfov.urdf.xacro (robot description, xacro)
@@ -13,5 +13,5 @@
   <xacro:include filename="$(find ant_description)/urdf/sensors/range.urdf.xacro"/>
   <xacro:include filename="$(find ant_description)/urdf/sensors/hokuyo_urg_04lx_ug01_laser.urdf.xacro"/>
-  <xacro:include filename="$(find ant_description)/urdf/sensors/xtion_pro_live.urdf.xacro"/>
+  <xacro:include filename="$(find ant_description)/urdf/sensors/softkinetic_ds311_rgbd_camera.urdf.xacro"/>
   <xacro:include filename="$(find ant_description)/urdf/sensors/imu.urdf.xacro"/>
   <xacro:include filename="$(find ant_description)/urdf/sensors/bumper.urdf.xacro"/>
@@ -37,7 +37,7 @@
   <property name="base_laser_z" value="0.05275"/>
   <!-- RGBD characteristics -->
-  <property name="base_rgbd_x" value="0.185"/>
+  <property name="base_rgbd_x" value="0.0"/>
   <property name="base_rgbd_y" value="0.0"/>
-  <property name="base_rgbd_z" value="0.23"/>
+  <property name="base_rgbd_z" value="1.00"/>
   <xacro:macro name="base" params="name">
     <!-- Base -->
@@ -81,10 +81,11 @@
     </xacro:hokuyo_urg_04lx_ug01_laser>
     <!-- RGBD -->
-    <xacro:xtion_pro_live name="${name}_xtion" parent="${name}">
+    <xacro:softkinetic_ds311_rgbd_camera name="${name}_rgbd_camera" parent="${name}">
       <!-- Pose of sensor frame wrt to base -->
-      <origin xyz="${base_rgbd_x} ${base_rgbd_y} ${base_rgbd_z}" rpy="0 0 0"/>
+      <origin xyz="${base_rgbd_x} ${base_rgbd_y} ${base_rgbd_z}" rpy="0 ${30 * deg_to_rad} 0"/>
+      <!--origin xyz="${base_rgbd_x} ${base_rgbd_y} ${base_rgbd_z}" rpy="${90 * deg_to_rad} ${30 * deg_to_rad} 0"/-->
       <!-- Pose of optical frame wrt to sensor -->
       <optical_origin xyz="0 0 0" rpy="${-90 * deg_to_rad} 0 ${-90 * deg_to_rad}"/>
-    </xacro:xtion_pro_live>
+    </xacro:softkinetic_ds311_rgbd_camera>
     <!-- Sonar -->
     <!--xacro:range_sensor name="${name}_sonar_02" parent="${name}" ros_topic="sonar_base" update_rate="10" maxRange="0.75" minRange="0.01" fov="0.5" radiation="ultrasound">

File: ant_description/urdf/sensors/softkinetic_ds311_rgbd_camera.gazebo.xacro (robot description, xacro)
@@ -19,13 +19,13 @@
         <update_rate>10.0</update_rate>
         <camera>
-          <horizontal_fov>${58.0 * deg_to_rad}</horizontal_fov>
+          <horizontal_fov>${57.3 * deg_to_rad}</horizontal_fov>
           <image>
             <format>R8G8B8</format>
-            <width>640</width>
-            <height>480</height>
+            <width>160</width>
+            <height>120</height>
           </image>
           <clip>
             <near>0.1</near>
-            <far>100.0</far>
+            <far>4.0</far>
           </clip>
         </camera>
@@ -40,5 +40,6 @@
           <pointCloudTopicName>depth_registered/points</pointCloudTopicName>
           <frameName>${name}_optical_frame</frameName>
-          <pointCloudCutoff>0.8</pointCloudCutoff>
+          <pointCloudCutoff>0.0</pointCloudCutoff>
+          <rangeMax>4.0</rangeMax>
           <distortionK1>0.00000001</distortionK1>
           <distortionK2>0.00000001</distortionK2>
@@ -53,5 +54,5 @@
         <update_rate>10.0</update_rate>
         <camera>
-          <horizontal_fov>${58.0 * deg_to_rad}</horizontal_fov>
+          <horizontal_fov>${50.0 * deg_to_rad}</horizontal_fov>
           <image>
             <format>R8G8B8</format>
@@ -61,5 +62,5 @@
           <clip>
             <near>0.1</near>
-            <far>100.0</far>
+            <far>4.0</far>
           </clip>
         </camera>
@@ -72,5 +73,6 @@
           <pointCloudTopicName>rgbd_data/points</pointCloudTopicName>
           <frameName>${name}_optical_frame</frameName>
-          <pointCloudCutoff>0.8</pointCloudCutoff>
+          <pointCloudCutoff>0.0</pointCloudCutoff>
+          <rangeMax>4.0</rangeMax>
           <distortionK1>0.00000001</distortionK1>
           <distortionK2>0.00000001</distortionK2>

File: ant_description/urdf/sensors/softkinetic_ds311_rgbd_camera.urdf.xacro (robot description, xacro)
@@ -10,5 +10,5 @@
   <xacro:include filename="$(find ant_description)/urdf/sensors/softkinetic_ds311_rgbd_camera.gazebo.xacro" />
   <!-- Macro -->
-  <xacro:macro name="softkinetic_ds311_rgbd_camera" params="name parent *origin *calibration_origin">
+  <xacro:macro name="softkinetic_ds311_rgbd_camera" params="name parent *origin *optical_origin">
     <joint name="${name}_frame_joint" type="fixed">
       <insert_block name="origin" />
@@ -41,5 +41,5 @@
     </link>
     <joint name="${name}_optical_joint" type="fixed">
-      <insert_block name="calibration_origin"/>
+      <insert_block name="optical_origin"/>
       <parent link="${name}_link"/>
       <child link="${name}_optical_frame"/>

File: ant_description/urdf/sensors/xtion_pro_live.urdf.xacro (robot description, xacro)
@@ -20,5 +20,5 @@
   <xacro:include filename="$(find ant_description)/urdf/sensors/xtion_pro_live.gazebo.xacro" />
   <!-- Macro -->
-  <xacro:macro name="xtion_pro_live" params="name parent *origin *calibration_origin">
+  <xacro:macro name="xtion_pro_live" params="name parent *origin *optical_origin">
     <joint name="${name}_frame_joint" type="fixed">
       <insert_block name="origin" />
@@ -51,5 +51,5 @@
     </link>
     <joint name="${name}_optical_joint" type="fixed">
-      <insert_block name="calibration_origin" />
+      <insert_block name="optical_origin" />
       <parent link="${name}_link"/>
       <child link="${name}_optical_frame"/>
