Commit message: fixes base_rebujito
git-svn-id: svn+ssh://server/srv/svn/repos/trunk/pal-ros-pkg/catkin_pkgs/ant_robot@57748 5e370ff8-3418-0410-babe-3378cc20a00d

File: ant_description/urdf/base/base_rebujito.urdf.xacro (robot description, xacro)
@@ -24,12 +24,11 @@
   <property name="wheel_velocity"   value="1.0"/>
   <!-- Caster wheel characteristics -->
-  <property name="caster_separation" value="0.200"/>
   <property name="caster_radius"     value="0.025"/>
   <property name="caster_width"      value="0.0164"/>
-  <property name="caster_trailing"   value="0.038"/>
-  <property name="caster_offset_x"   value="0.140"/>
+  <property name="caster_separation" value="0.35764"/>
+  <property name="caster_offset_z"   value="-0.028"/>
   <property name="base_radius" value="${(wheel_separation - wheel_width)/2 - 0.01}"/>
-  <property name="base_length" value="0.04"/>
-  <property name="base_offset_z" value="${base_length + 0.031}"/>
+  <!-- @todo once the mesh has the laser whole, we can reduce this base_offset_z -->
+  <property name="base_offset_z" value="0.2"/>
   <!-- simplified box collision geometry for the laser -->
   <property name="base_laser_x" value="0.15"/>
@@ -104,24 +103,10 @@
       <origin xyz="0 0 0.1" rpy="0 0 0"/>
     </xacro:imu_sensor>
-    <!-- IR receiver -->
-    <xacro:ir_receiver name="${name}_ir_receiver_01" parent="${name}" ros_topic="ir_receiver_base" update_rate="10" range_min="0.0" range_max="0.75" fov="0.5">
-      <origin xyz="0.17131 0.0 0.280" rpy="0.0 0.0 0.0" />
-    </xacro:ir_receiver>
-    <!-- IR receiver -->
-    <xacro:ir_receiver name="${name}_ir_receiver_02" parent="${name}" ros_topic="ir_receiver_base" update_rate="10" range_min="0.0" range_max="0.75" fov="0.5">
-      <origin xyz="0.16919 0.14919 0.280" rpy="0.0 0.0 0.349" />
-    </xacro:ir_receiver>
-    <!-- IR receiver -->
-    <xacro:ir_receiver name="${name}_ir_receiver_03" parent="${name}" ros_topic="ir_receiver_base" update_rate="10" range_min="0.0" range_max="0.75" fov="0.5">
-      <origin xyz="0.16919 -0.14919 0.280" rpy="0.0 0.0 -0.349" />
-    </xacro:ir_receiver>
     <!-- Wheels -->
     <xacro:wheel side="right" reflect=" 1.0" radius="${wheel_radius}" width="${wheel_width}" torque="${wheel_torque}" velocity="${wheel_velocity}" separation="${wheel_separation}" parent="${name}"/>
     <xacro:wheel side="left"  reflect="-1.0" radius="${wheel_radius}" width="${wheel_width}" torque="${wheel_torque}" velocity="${wheel_velocity}" separation="${wheel_separation}" parent="${name}"/>
     <!-- Casters wheels -->
-    <xacro:caster side="front_right" radius="${caster_radius}" width="${caster_width}" separation="${caster_separation}" trailing="${caster_trailing}" offset_x="${caster_offset_x}" parent="${name}"/>
-    <xacro:caster side="front_left"  radius="${caster_radius}" width="${caster_width}" separation="${caster_separation}" trailing="${caster_trailing}" offset_x="${caster_offset_x}" parent="${name}"/>
-    <xacro:caster side="back_right" radius="${caster_radius}" width="${caster_width}" separation="${caster_separation}" trailing="${caster_trailing}" offset_x="${-caster_offset_x}" parent="${name}"/>
-    <xacro:caster side="back_left"  radius="${caster_radius}" width="${caster_width}" separation="${caster_separation}" trailing="${caster_trailing}" offset_x="${-caster_offset_x}" parent="${name}"/>
+    <xacro:caster side="front" radius="${caster_radius}" width="${caster_width}" separation_x="${ caster_separation}" separation_y="0" offset_z="${caster_offset_z}" parent="${name}"/>
+    <xacro:caster side="back"  radius="${caster_radius}" width="${caster_width}" separation_x="${-caster_separation}" separation_y="0" offset_z="${caster_offset_z}" parent="${name}"/>
   </xacro:macro>
 </robot>

Commit message: fixes non-supported used of properties to defined another property (suspicious)
git-svn-id: svn+ssh://server/srv/svn/repos/trunk/pal-ros-pkg/catkin_pkgs/ant_robot@58046 5e370ff8-3418-0410-babe-3378cc20a00d

File: ant_description/urdf/base/base_rebujito.urdf.xacro (robot description, xacro)
@@ -30,5 +30,6 @@
   <property name="caster_offset_z"   value="-0.028"/>
   <!-- Antennas characteristics -->
-  <property name="antenna_separation_y" value="${wheel_separation + wheel_width}"/>
+  <!-- @todo ${wheel_separation + wheel_width} fails -->
+  <property name="antenna_separation_y" value="0.48"/>
   <property name="antenna_height_0"     value="0.2"/>
   <property name="antenna_height_inc"   value="0.35"/>

File: ant_description/urdf/base/base_softkinetic_ds311_hfov.urdf.xacro (robot description, xacro)
@@ -31,5 +31,6 @@
   <property name="caster_offset_z"     value="-0.04252"/>
   <!-- Antennas characteristics -->
-  <property name="antenna_separation_y" value="${wheel_separation + wheel_width}"/>
+  <!-- @todo ${wheel_separation + wheel_width} fails -->
+  <property name="antenna_separation_y" value="0.48"/>
   <property name="antenna_height_0"     value="0.2"/>
   <property name="antenna_height_inc"   value="0.35"/>
@@ -88,5 +89,6 @@
     <xacro:softkinetic_ds311_rgbd_camera name="${name}_rgbd_camera" parent="${name}">
       <!-- Pose of sensor frame wrt to base -->
-      <origin xyz="${base_rgbd_x} ${base_rgbd_y} ${base_rgbd_z}" rpy="${90 * deg_to_rad} ${0 * deg_to_rad} 0"/>
+      <!-- @todo r=90, p=30 doesn't work (see http://answers.gazebosim.org/question/7005/gazebo_ros_openni_kinect-plugin-with-roll-pitch/) -->
+      <origin xyz="${base_rgbd_x} ${base_rgbd_y} ${base_rgbd_z}" rpy="${0 * deg_to_rad} ${30 * deg_to_rad} 0"/>
       <!-- Pose of optical frame wrt to sensor -->
       <origin xyz="0 0 0" rpy="${-90 * deg_to_rad} 0 ${-90 * deg_to_rad}"/>
