Commit message: uses the base v2.0 STL for the collision
A cylinder close the laser window!

File: ant_description/urdf/base/base_v2.urdf.xacro (robot description, xacro)
@@ -29,6 +29,6 @@
   <property name="caster_offset_z"     value="-0.0335"/>
   <!-- Base characteristics -->
-  <property name="base_radius" value="${(wheel_separation - wheel_width)/2 - 0.01}"/>
-  <property name="base_length" value="0.04"/>
+  <property name="base_radius" value="${(wheel_separation + wheel_width)/2}"/>
+  <property name="base_length" value="0.235"/>
   <!-- Laser characteristics -->
   <property name="base_laser_x" value="0.185"/>
@@ -55,5 +55,6 @@
         <origin xyz="0 0 0" rpy="0 0 0" />
         <geometry>
-          <cylinder radius="${base_radius}" length="${base_length}"/>
+          <mesh filename="package://ant_description/meshes/base/base_v2.stl" />
+          <!--cylinder radius="${base_radius}" length="${base_length}"/-->
         </geometry>
         <material name="DarkGrey" />

Commit message: removes cylinder for the base collision
and also related params; we keep this commit to have the approximate
values of them

File: ant_description/urdf/base/base_v2.urdf.xacro (robot description, xacro)
@@ -28,7 +28,4 @@
   <property name="caster_separation_y" value="0.20168"/>
   <property name="caster_offset_z"     value="-0.0335"/>
-  <!-- Base characteristics -->
-  <property name="base_radius" value="${(wheel_separation + wheel_width)/2}"/>
-  <property name="base_length" value="0.235"/>
   <!-- Laser characteristics -->
   <property name="base_laser_x" value="0.185"/>
@@ -56,5 +53,4 @@
         <geometry>
           <mesh filename="package://ant_description/meshes/base/base_v2.stl" />
-          <!--cylinder radius="${base_radius}" length="${base_length}"/-->
         </geometry>
         <material name="DarkGrey" />
@@ -95,5 +91,5 @@
     <!-- @todo ant_hardware_gazebo needs an IMU!  -->
     <xacro:imu_sensor name="base_inclinometer" parent="${name}_link" update_rate="100.0">
-      <origin xyz="0 0 ${base_length / 2}" rpy="0 0 0"/>
+      <origin xyz="0 0 0" rpy="0 0 0"/>
     </xacro:imu_sensor>
     <!-- IR receiver -->

Commit message: adds SICK TiM511 laser to URDF

File: ant_description/urdf/base/base_v2.urdf.xacro (robot description, xacro)
@@ -12,5 +12,5 @@
   <xacro:include filename="$(find ant_description)/urdf/wheels/caster_v2.urdf.xacro"/>
   <xacro:include filename="$(find ant_description)/urdf/sensors/range.urdf.xacro"/>
-  <xacro:include filename="$(find ant_description)/urdf/sensors/hokuyo_urg_04lx_ug01_laser.urdf.xacro"/>
+  <xacro:include filename="$(find ant_description)/urdf/sensors/sick_tim511_laser.urdf.xacro"/>
   <xacro:include filename="$(find ant_description)/urdf/sensors/imu.urdf.xacro"/>
   <xacro:include filename="$(find ant_description)/urdf/sensors/bumper.urdf.xacro"/>
@@ -29,5 +29,5 @@
   <property name="caster_offset_z"     value="-0.0335"/>
   <!-- Laser characteristics -->
-  <property name="base_laser_x" value="0.185"/>
+  <property name="base_laser_x" value="0.185"/> <!-- measured value it's approx. 0.1593 -->
   <property name="base_laser_y" value="0.0"/>
   <property name="base_laser_z" value="0.0498"/>
@@ -65,7 +65,7 @@
     </joint>
     <!-- Laser -->
-    <xacro:hokuyo_urg_04lx_ug01_laser name="${name}_laser" parent="${name}" ros_topic="scan" update_rate="10" min_angle="${-110 * deg_to_rad}" max_angle="${110 * deg_to_rad}" >
+    <xacro:sick_tim511_laser name="${name}_laser" parent="${name}" ros_topic="scan" update_rate="15" min_angle="${-110 * deg_to_rad}" max_angle="${110 * deg_to_rad}" >
       <origin xyz="${base_laser_x} ${base_laser_y} ${base_laser_z}" rpy="0 0 0" />
-    </xacro:hokuyo_urg_04lx_ug01_laser>
+    </xacro:sick_tim511_laser>
     <!-- Sonar -->
     <!--xacro:range_sensor name="${name}_sonar_02" parent="${name}" ros_topic="sonar_base" update_rate="10" maxRange="0.75" minRange="0.01" fov="0.5" radiation="ultrasound">

File: ant_description/urdf/sensors/sick_tim511_laser.gazebo.xacro (robot description, xacro)
@@ -6,9 +6,9 @@
   To view a copy of this license, visit http://creativecommons.org/licenses/by-nc-nd/3.0/ or send a letter to
   Creative Commons, 444 Castro Street, Suite 900, Mountain View, California, 94041, USA.
-  Laser configuration according with the Hokuyo URG-04LX-UG01 product specification:
-  http://www.hokuyo-aut.jp/02sensor/07scanner/download/products/urg-04lx-ug01/data/URG-04LX_UG01_spec_en.pdf
+  Laser configuration according with the SICK TiM 511 product specification:
+  http://www.sick.com/group/DE/home/pr/events/robot_day/Documents/TIM551-2050001_en.pdf
 -->
 <robot xmlns:xacro="http://ros.org/wiki/xacro">
-  <xacro:macro name="hokuyo_urg_04lx_ug01_laser_gazebo" params="name ros_topic update_rate min_angle max_angle">
+  <xacro:macro name="sick_tim511_laser_gazebo" params="name ros_topic update_rate min_angle max_angle">
     <gazebo reference="${name}_link">
       <sensor type="ray" name="${name}">
@@ -19,6 +19,6 @@
           <scan>
             <horizontal>
-              <!-- 683 steps in 240deg fov -->
-              <samples>${683*(max_angle - min_angle)/(240.0 * deg_to_rad)}</samples>
+              <!-- 270 steps in 270deg fov -->
+              <samples>${270*(max_angle - min_angle)/(270.0 * deg_to_rad)}</samples>
               <resolution>1</resolution> <!-- not the sensor resolution; just 1 -->
               <min_angle>${min_angle}</min_angle>
@@ -27,11 +27,11 @@
           </scan>
           <range>
-            <min>0.02</min>
-            <max>5.6</max>
+            <min>0.05</min>
+            <max>10.0</max>
             <resolution>0.001</resolution>
           </range>
         </ray>
-        <plugin filename="libgazebo_ros_laser.so" name="gazebo_ros_hokuyo_laser">
-          <gaussianNoise>0.03</gaussianNoise>
+        <plugin filename="libgazebo_ros_laser.so" name="gazebo_ros_sick_laser">
+          <gaussianNoise>0.06</gaussianNoise>
           <alwaysOn>true</alwaysOn>
           <updateRate>${update_rate}</updateRate>

Commit message: adds base collision mesh and reduces laser FOV
with the theoretic 2*110deg FOV the laser measurements touches
the collision mesh, so it's been reduced to 2*108deg

File: ant_description/urdf/base/base_v2.urdf.xacro (robot description, xacro)
@@ -52,5 +52,5 @@
         <origin xyz="0 0 0" rpy="0 0 0" />
         <geometry>
-          <mesh filename="package://ant_description/meshes/base/base_v2.stl" />
+          <mesh filename="package://ant_description/meshes/base/base_v2_collision.stl" />
         </geometry>
         <material name="DarkGrey" />
@@ -65,5 +65,6 @@
     </joint>
     <!-- Laser -->
-    <xacro:sick_tim511_laser name="${name}_laser" parent="${name}" ros_topic="scan" update_rate="15" min_angle="${-110 * deg_to_rad}" max_angle="${110 * deg_to_rad}" >
+    <!-- Theoretic FOV = 220º -->
+    <xacro:sick_tim511_laser name="${name}_laser" parent="${name}" ros_topic="scan" update_rate="15" min_angle="${-108 * deg_to_rad}" max_angle="${108 * deg_to_rad}" >
       <origin xyz="${base_laser_x} ${base_laser_y} ${base_laser_z}" rpy="0 0 0" />
     </xacro:sick_tim511_laser>

Commit message: renames TiM511 to TiM551 (the right name)

File: ant_description/urdf/base/base_v2.urdf.xacro (robot description, xacro)
@@ -12,5 +12,5 @@
   <xacro:include filename="$(find ant_description)/urdf/wheels/caster_v2.urdf.xacro"/>
   <xacro:include filename="$(find ant_description)/urdf/sensors/range.urdf.xacro"/>
-  <xacro:include filename="$(find ant_description)/urdf/sensors/sick_tim511_laser.urdf.xacro"/>
+  <xacro:include filename="$(find ant_description)/urdf/sensors/sick_tim551_laser.urdf.xacro"/>
   <xacro:include filename="$(find ant_description)/urdf/sensors/imu.urdf.xacro"/>
   <xacro:include filename="$(find ant_description)/urdf/sensors/bumper.urdf.xacro"/>
@@ -66,7 +66,7 @@
     <!-- Laser -->
     <!-- Theoretic FOV = 220º -->
-    <xacro:sick_tim511_laser name="${name}_laser" parent="${name}" ros_topic="scan" update_rate="15" min_angle="${-110 * deg_to_rad}" max_angle="${110 * deg_to_rad}" >
+    <xacro:sick_tim551_laser name="${name}_laser" parent="${name}" ros_topic="scan" update_rate="15" min_angle="${-110 * deg_to_rad}" max_angle="${110 * deg_to_rad}" >
       <origin xyz="${base_laser_x} ${base_laser_y} ${base_laser_z}" rpy="0 0 0" />
-    </xacro:sick_tim511_laser>
+    </xacro:sick_tim551_laser>
     <!-- Sonar -->
     <!--xacro:range_sensor name="${name}_sonar_02" parent="${name}" ros_topic="sonar_base" update_rate="10" maxRange="0.75" minRange="0.01" fov="0.5" radiation="ultrasound">

File: ant_description/urdf/sensors/sick_tim551_laser.gazebo.xacro (robot description, xacro)
@@ -6,9 +6,9 @@
   To view a copy of this license, visit http://creativecommons.org/licenses/by-nc-nd/3.0/ or send a letter to
   Creative Commons, 444 Castro Street, Suite 900, Mountain View, California, 94041, USA.
-  Laser configuration according with the SICK TiM 511 product specification:
+  Laser configuration according with the SICK TiM 551 product specification:
   http://www.sick.com/group/DE/home/pr/events/robot_day/Documents/TIM551-2050001_en.pdf
 -->
 <robot xmlns:xacro="http://ros.org/wiki/xacro">
-  <xacro:macro name="sick_tim511_laser_gazebo" params="name ros_topic update_rate min_angle max_angle">
+  <xacro:macro name="sick_tim551_laser_gazebo" params="name ros_topic update_rate min_angle max_angle">
     <gazebo reference="${name}_link">
       <sensor type="ray" name="${name}">

File: ant_description/urdf/sensors/sick_tim551_laser.urdf.xacro (robot description, xacro)
@@ -8,6 +8,6 @@
 -->
 <robot xmlns:xacro="http://ros.org/wiki/xacro">
-  <xacro:include filename="$(find ant_description)/urdf/sensors/sick_tim511_laser.gazebo.xacro" />
-  <xacro:macro name="sick_tim511_laser" params="name parent *origin ros_topic update_rate min_angle max_angle">
+  <xacro:include filename="$(find ant_description)/urdf/sensors/sick_tim551_laser.gazebo.xacro" />
+  <xacro:macro name="sick_tim551_laser" params="name parent *origin ros_topic update_rate min_angle max_angle">
      <link name="${name}_link" type="laser">
       <inertial>
@@ -21,5 +21,5 @@
         <origin xyz="0 0 0" rpy="0 0 0" />
         <geometry>
-          <mesh filename="package://ant_description/meshes/sensors/sick_tim511.stl"/>
+          <mesh filename="package://ant_description/meshes/sensors/sick_tim551.stl"/>
         </geometry>
         <material name="DarkGrey" />
@@ -35,5 +35,5 @@
     </joint>
     <!-- gazebo extensions -->
-    <xacro:sick_tim511_laser_gazebo name="${name}" ros_topic="${ros_topic}" update_rate="${update_rate}" min_angle="${min_angle}" max_angle="${max_angle}" />
+    <xacro:sick_tim551_laser_gazebo name="${name}" ros_topic="${ros_topic}" update_rate="${update_rate}" min_angle="${min_angle}" max_angle="${max_angle}" />
   </xacro:macro>
 </robot>
