Commit message: fixes origin (must be origin twice, not optical_origin)
git-svn-id: svn+ssh://server/srv/svn/repos/trunk/pal-ros-pkg/catkin_pkgs/ant_robot@58060 5e370ff8-3418-0410-babe-3378cc20a00d

File: ant_description/urdf/base/base_softkinetic_ds311.urdf.xacro (robot description, xacro)
@@ -85,5 +85,5 @@
       <origin xyz="${base_rgbd_x} ${base_rgbd_y} ${base_rgbd_z}" rpy="0 0 0"/>
       <!-- Pose of optical frame wrt to sensor -->
-      <optical_origin xyz="0 0 0" rpy="${-90 * deg_to_rad} 0 ${-90 * deg_to_rad}"/>
+      <origin xyz="0 0 0" rpy="${-90 * deg_to_rad} 0 ${-90 * deg_to_rad}"/>
     </xacro:softkinetic_ds311_rgbd_camera>
     <!-- Sonar -->

File: ant_description/urdf/base/base_xtion_pro_live.urdf.xacro (robot description, xacro)
@@ -85,5 +85,5 @@
       <origin xyz="${base_rgbd_x} ${base_rgbd_y} ${base_rgbd_z}" rpy="0 0 0"/>
       <!-- Pose of optical frame wrt to sensor -->
-      <optical_origin xyz="0 0 0" rpy="${-90 * deg_to_rad} 0 ${-90 * deg_to_rad}"/>
+      <origin xyz="0 0 0" rpy="${-90 * deg_to_rad} 0 ${-90 * deg_to_rad}"/>
     </xacro:xtion_pro_live>
     <!-- Sonar -->

File: ant_description/urdf/base/base_xtion_pro_live_only.urdf.xacro (robot description, xacro)
@@ -76,5 +76,5 @@
       <origin xyz="${base_rgbd_x} ${base_rgbd_y} ${base_rgbd_z}" rpy="0 0 0"/>
       <!-- Pose of optical frame wrt to sensor -->
-      <optical_origin xyz="0 0 0" rpy="${-90 * deg_to_rad} 0 ${-90 * deg_to_rad}"/>
+      <origin xyz="0 0 0" rpy="${-90 * deg_to_rad} 0 ${-90 * deg_to_rad}"/>
     </xacro:xtion_pro_live>
     <!-- Sonar -->

Commit message: refs #9791 : single urdf for softkinetic_ds311 with several poses
git-svn-id: svn+ssh://server/srv/svn/repos/trunk/pal-ros-pkg/catkin_pkgs/ant_robot@58081 5e370ff8-3418-0410-babe-3378cc20a00d

File: ant_description/urdf/base/base_softkinetic_ds311.urdf.xacro (robot description, xacro)
@@ -37,7 +37,37 @@
   <property name="base_laser_z" value="0.05275"/>
   <!-- RGBD characteristics -->
+  <!-- Setups: see :https://docs.google.com/a/pal-robotics.com/presentation/d/1AfR5_-aYmT7fTs_w-cQlUHA08lY2gSzhnPvTg2bpwMU/edit#slide=id.g36ad429de_037 -->
+  <!-- Setup #1: Similar to page #4 -->
+  <!--
   <property name="base_rgbd_x" value="0.185"/>
   <property name="base_rgbd_y" value="0.0"/>
   <property name="base_rgbd_z" value="0.23"/>
+  <property name="base_rgbd_r" value="0.0"/>
+  <property name="base_rgbd_p" value="0.0"/>
+  <property name="base_rgbd_y" value="0.0"/>
+  -->
+  <!-- Setup #2: Similar to page #8 -->
+  <property name="base_rgbd_x" value="0.045"/>
+  <property name="base_rgbd_y" value="0.0"/>
+  <property name="base_rgbd_z" value="0.87"/>
+  <property name="base_rgbd_r" value="0.0"/>
+  <property name="base_rgbd_p" value="0.0"/>
+  <property name="base_rgbd_y" value="0.0"/>
+  <!-- Setup #3: Similar to page #8 -->
+  <property name="base_rgbd_x" value="0.045"/>
+  <property name="base_rgbd_y" value="0.0"/>
+  <property name="base_rgbd_z" value="0.87"/>
+  <property name="base_rgbd_r" value="0.0"/>
+  <property name="base_rgbd_p" value="30.0"/>
+  <property name="base_rgbd_y" value="0.0"/>
+  <!-- Setup #4: Similar to page #12 -->
+  <!--
+  <property name="base_rgbd_x" value="0.045"/>
+  <property name="base_rgbd_y" value="0.0"/>
+  <property name="base_rgbd_z" value="0.87"/>
+  <property name="base_rgbd_r" value="0.0"/>
+  <property name="base_rgbd_p" value="0.0"/>
+  <property name="base_rgbd_y" value="0.0"/>
+  -->
   <xacro:macro name="base" params="name">
     <!-- Base -->
@@ -83,5 +113,5 @@
     <xacro:softkinetic_ds311_rgbd_camera name="${name}_rgbd_camera" parent="${name}">
       <!-- Pose of sensor frame wrt to base -->
-      <origin xyz="${base_rgbd_x} ${base_rgbd_y} ${base_rgbd_z}" rpy="0 0 0"/>
+      <origin xyz="${base_rgbd_x} ${base_rgbd_y} ${base_rgbd_z}" rpy="${base_rgbd_r * deg_to_rad} ${base_rgbd_p * deg_to_rad} ${base_rgbd_y * deg_to_rad}"/>
       <!-- Pose of optical frame wrt to sensor -->
       <origin xyz="0 0 0" rpy="${-90 * deg_to_rad} 0 ${-90 * deg_to_rad}"/>

Commit message: refs #10350 : fixes base_rgbd_y collision (y, yaw)
also sets the yaw to 7.1º (current value on the real robot)

File: ant_description/urdf/base/base_softkinetic_ds311.urdf.xacro (robot description, xacro)
@@ -43,7 +43,7 @@
   <property name="base_rgbd_y" value="0.0"/>
   <property name="base_rgbd_z" value="0.23"/>
-  <property name="base_rgbd_r" value="0.0"/>
-  <property name="base_rgbd_p" value="0.0"/>
-  <property name="base_rgbd_y" value="0.0"/>
+  <property name="base_rgbd_R" value="0.0"/>
+  <property name="base_rgbd_P" value="0.0"/>
+  <property name="base_rgbd_Y" value="0.0"/>
   -->
   <!-- Setup #2: Similar to page #8 -->
@@ -52,7 +52,7 @@
   <property name="base_rgbd_y" value="0.0"/>
   <property name="base_rgbd_z" value="0.87"/>
-  <property name="base_rgbd_r" value="0.0"/>
-  <property name="base_rgbd_p" value="0.0"/>
-  <property name="base_rgbd_y" value="0.0"/>
+  <property name="base_rgbd_R" value="0.0"/>
+  <property name="base_rgbd_P" value="0.0"/>
+  <property name="base_rgbd_Y" value="0.0"/>
   -->
   <!-- Setup #3: Similar to page #8 -->
@@ -61,7 +61,7 @@
   <property name="base_rgbd_y" value="0.0"/>
   <property name="base_rgbd_z" value="0.87"/>
-  <property name="base_rgbd_r" value="0.0"/>
-  <property name="base_rgbd_p" value="30.0"/>
-  <property name="base_rgbd_y" value="0.0"/>
+  <property name="base_rgbd_R" value="0.0"/>
+  <property name="base_rgbd_P" value="30.0"/>
+  <property name="base_rgbd_Y" value="0.0"/>
   -->
   <!-- Setup #4: Similar to page #12 -->
@@ -69,7 +69,7 @@
   <property name="base_rgbd_y" value="0.0"/>
   <property name="base_rgbd_z" value="1.05"/>
-  <property name="base_rgbd_r" value="90.0"/>
-  <property name="base_rgbd_p" value="0.0"/>
-  <property name="base_rgbd_y" value="0.0"/>
+  <property name="base_rgbd_R" value="90.0"/>
+  <property name="base_rgbd_P" value="0.0"/>
+  <property name="base_rgbd_Y" value="0.0"/>
   <xacro:macro name="base" params="name">
     <!-- Base -->
@@ -111,5 +111,5 @@
     <xacro:softkinetic_ds311_rgbd_camera name="${name}_rgbd_camera" parent="${name}">
       <!-- Pose of sensor frame wrt to base -->
-      <origin xyz="${base_rgbd_x} ${base_rgbd_y} ${base_rgbd_z}" rpy="${base_rgbd_r * deg_to_rad} ${base_rgbd_p * deg_to_rad} ${base_rgbd_y * deg_to_rad}"/>
+      <origin xyz="${base_rgbd_x} ${base_rgbd_y} ${base_rgbd_z}" rpy="${base_rgbd_R * deg_to_rad} ${base_rgbd_P * deg_to_rad} ${base_rgbd_Y * deg_to_rad}"/>
       <!-- Pose of optical frame wrt to sensor -->
       <origin xyz="0 0 0" rpy="${-90 * deg_to_rad} 0 ${-90 * deg_to_rad}"/>

File: ant_description/urdf/base/base_v2_vertical_xtion_pro_live.urdf.xacro (robot description, xacro)
@@ -37,7 +37,7 @@
   <property name="base_rgbd_y" value="0.05"/>
   <property name="base_rgbd_z" value="1.1"/>
-  <property name="base_rgbd_r" value="90.0"/>
-  <property name="base_rgbd_p" value="30.0"/>
-  <property name="base_rgbd_y" value="0.0"/>
+  <property name="base_rgbd_R" value="90.0"/>
+  <property name="base_rgbd_P" value="30.0"/>
+  <property name="base_rgbd_Y" value="7.1"/>
   <xacro:macro name="base" params="name">
     <!-- Base -->
@@ -80,5 +80,5 @@
     <xacro:xtion_pro_live name="${name}_rgbd_camera" parent="${name}">
       <!-- Pose of sensor frame wrt to base -->
-      <origin xyz="${base_rgbd_x} ${base_rgbd_y} ${base_rgbd_z}" rpy="${base_rgbd_r * deg_to_rad} ${base_rgbd_p * deg_to_rad} ${base_rgbd_y * deg_to_rad}"/>
+      <origin xyz="${base_rgbd_x} ${base_rgbd_y} ${base_rgbd_z}" rpy="${base_rgbd_R * deg_to_rad} ${base_rgbd_P * deg_to_rad} ${base_rgbd_Y * deg_to_rad}"/>
       <!-- Pose of optical frame wrt to sensor -->
       <origin xyz="0 0 0" rpy="${-90 * deg_to_rad} 0 ${-90 * deg_to_rad}"/>

File: ant_description/urdf/base/base_v2_xtion_pro_live.urdf.xacro (robot description, xacro)
@@ -37,7 +37,7 @@
   <property name="base_rgbd_y" value="0.0"/>
   <property name="base_rgbd_z" value="0.6"/>
-  <property name="base_rgbd_r" value="0.0"/>
-  <property name="base_rgbd_p" value="0.0"/>
-  <property name="base_rgbd_y" value="0.0"/>
+  <property name="base_rgbd_R" value="0.0"/>
+  <property name="base_rgbd_P" value="0.0"/>
+  <property name="base_rgbd_Y" value="0.0"/>
   <xacro:macro name="base" params="name">
     <!-- Base -->
@@ -80,5 +80,5 @@
     <xacro:xtion_pro_live name="${name}_rgbd_camera" parent="${name}">
       <!-- Pose of sensor frame wrt to base -->
-      <origin xyz="${base_rgbd_x} ${base_rgbd_y} ${base_rgbd_z}" rpy="${base_rgbd_r * deg_to_rad} ${base_rgbd_p * deg_to_rad} ${base_rgbd_y * deg_to_rad}"/>
+      <origin xyz="${base_rgbd_x} ${base_rgbd_y} ${base_rgbd_z}" rpy="${base_rgbd_R * deg_to_rad} ${base_rgbd_P * deg_to_rad} ${base_rgbd_Y * deg_to_rad}"/>
       <!-- Pose of optical frame wrt to sensor -->
       <origin xyz="0 0 0" rpy="${-90 * deg_to_rad} 0 ${-90 * deg_to_rad}"/>
