Commit message: updates antenna urdf files (more modular)
They will be also used for the ant with softkinetic


git-svn-id: svn+ssh://server/srv/svn/repos/trunk/pal-ros-pkg/catkin_pkgs/ant_robot@57996 5e370ff8-3418-0410-babe-3378cc20a00d

File: ant_description/robots/ant_rebujito.urdf.xacro (robot description, xacro)
@@ -15,12 +15,16 @@
   <!-- Base -->
   <xacro:include filename="$(find ant_description)/urdf/base/base_rebujito.urdf.xacro" />
-  <xacro:include filename="$(find ant_description)/urdf/antennas/antennas.urdf.xacro" />
+  <xacro:include filename="$(find ant_description)/urdf/antennas/antenna_array.urdf.xacro" />
   <!-- Generic simulator_gazebo plugins -->
   <xacro:include filename="$(find ant_description)/gazebo/gazebo.urdf.xacro" />
   <!-- Materials for visualization -->
   <xacro:include filename="$(find ant_description)/urdf/materials.urdf.xacro" />
+  <!-- Properties -->
+  <xacro:property name="separation_y" value="0.48"/>
+  <xacro:property name="height_0"   value="0.2"/>
+  <xacro:property name="height_inc" value="0.35"/>
   <!-- Now we can start using the macros included above to define the actual robot -->
   <xacro:base name="base"/>
-  <xacro:antenna name="antenna" parent="base_link" side="left"  reflect=" 1.0" />
-  <xacro:antenna name="antenna" parent="base_link" side="right" reflect="-1.0" />
+  <xacro:antenna_array name="antenna" parent="base_link" side="left"  reflect=" 1.0" separation_y="${separation_y}" height_0="${height_0}" height_inc="${height_inc}" />
+  <xacro:antenna_array name="antenna" parent="base_link" side="right" reflect="-1.0" separation_y="${separation_y}" height_0="${height_0}" height_inc="${height_inc}" />
 </robot>

Commit message: adds antennas and move them inside base
git-svn-id: svn+ssh://server/srv/svn/repos/trunk/pal-ros-pkg/catkin_pkgs/ant_robot@58045 5e370ff8-3418-0410-babe-3378cc20a00d

File: ant_description/robots/ant_rebujito.urdf.xacro (robot description, xacro)
@@ -15,16 +15,9 @@
   <!-- Base -->
   <xacro:include filename="$(find ant_description)/urdf/base/base_rebujito.urdf.xacro" />
-  <xacro:include filename="$(find ant_description)/urdf/antennas/antenna_array.urdf.xacro" />
   <!-- Generic simulator_gazebo plugins -->
   <xacro:include filename="$(find ant_description)/gazebo/gazebo.urdf.xacro" />
   <!-- Materials for visualization -->
   <xacro:include filename="$(find ant_description)/urdf/materials.urdf.xacro" />
-  <!-- Properties -->
-  <xacro:property name="separation_y" value="0.48"/>
-  <xacro:property name="height_0"   value="0.2"/>
-  <xacro:property name="height_inc" value="0.35"/>
   <!-- Now we can start using the macros included above to define the actual robot -->
   <xacro:base name="base"/>
-  <xacro:antenna_array name="antenna" parent="base_link" side="left"  reflect=" 1.0" separation_y="${separation_y}" height_0="${height_0}" height_inc="${height_inc}" />
-  <xacro:antenna_array name="antenna" parent="base_link" side="right" reflect="-1.0" separation_y="${separation_y}" height_0="${height_0}" height_inc="${height_inc}" />
 </robot>

File: ant_description/urdf/base/base_rebujito.urdf.xacro (robot description, xacro)
@@ -16,4 +16,5 @@
   <xacro:include filename="$(find ant_description)/urdf/sensors/bumper.urdf.xacro"/>
   <xacro:include filename="$(find ant_description)/urdf/sensors/ir_receiver.urdf.xacro"/>
+  <xacro:include filename="$(find ant_description)/urdf/antennas/antenna_array.urdf.xacro"/>
   <!-- Wheel characteristics -->
   <!-- Note that we temporary use Rebujito's -->
@@ -28,4 +29,8 @@
   <property name="caster_separation" value="0.35764"/>
   <property name="caster_offset_z"   value="-0.028"/>
+  <!-- Antennas characteristics -->
+  <property name="antenna_separation_y" value="${wheel_separation + wheel_width}"/>
+  <property name="antenna_height_0"     value="0.2"/>
+  <property name="antenna_height_inc"   value="0.35"/>
   <property name="base_radius" value="${(wheel_separation - wheel_width)/2 - 0.01}"/>
   <!-- @todo once the mesh has the laser whole, we can reduce this base_offset_z -->
@@ -109,4 +114,7 @@
     <xacro:caster side="front" radius="${caster_radius}" width="${caster_width}" separation_x="${ caster_separation}" separation_y="0" offset_z="${caster_offset_z}" parent="${name}"/>
     <xacro:caster side="back"  radius="${caster_radius}" width="${caster_width}" separation_x="${-caster_separation}" separation_y="0" offset_z="${caster_offset_z}" parent="${name}"/>
+    <!-- Antennas -->
+    <xacro:antenna_array name="antenna" parent="base_link" side="left"  reflect=" 1.0" separation_y="${antenna_separation_y}" height_0="${antenna_height_0}" height_inc="${antenna_height_inc}" />
+    <xacro:antenna_array name="antenna" parent="base_link" side="right" reflect="-1.0" separation_y="${antenna_separation_y}" height_0="${antenna_height_0}" height_inc="${antenna_height_inc}" />
   </xacro:macro>
 </robot>

File: ant_description/urdf/base/base_softkinetic_ds311_hfov.urdf.xacro (robot description, xacro)
@@ -17,4 +17,5 @@
   <xacro:include filename="$(find ant_description)/urdf/sensors/bumper.urdf.xacro"/>
   <xacro:include filename="$(find ant_description)/urdf/sensors/ir_receiver.urdf.xacro"/>
+  <xacro:include filename="$(find ant_description)/urdf/antennas/antenna_array.urdf.xacro"/>
   <!-- Wheel characteristics -->
   <property name="wheel_radius"     value="0.100"/>
@@ -29,4 +30,8 @@
   <property name="caster_separation_y" value="0.20362"/>
   <property name="caster_offset_z"     value="-0.04252"/>
+  <!-- Antennas characteristics -->
+  <property name="antenna_separation_y" value="${wheel_separation + wheel_width}"/>
+  <property name="antenna_height_0"     value="0.2"/>
+  <property name="antenna_height_inc"   value="0.35"/>
   <!-- Base characteristics -->
   <property name="base_radius" value="${(wheel_separation - wheel_width)/2 - 0.01}"/>
@@ -83,8 +88,7 @@
     <xacro:softkinetic_ds311_rgbd_camera name="${name}_rgbd_camera" parent="${name}">
       <!-- Pose of sensor frame wrt to base -->
-      <origin xyz="${base_rgbd_x} ${base_rgbd_y} ${base_rgbd_z}" rpy="0 ${30 * deg_to_rad} 0"/>
-      <!--origin xyz="${base_rgbd_x} ${base_rgbd_y} ${base_rgbd_z}" rpy="${90 * deg_to_rad} ${30 * deg_to_rad} 0"/-->
+      <origin xyz="${base_rgbd_x} ${base_rgbd_y} ${base_rgbd_z}" rpy="${90 * deg_to_rad} ${0 * deg_to_rad} 0"/>
       <!-- Pose of optical frame wrt to sensor -->
-      <optical_origin xyz="0 0 0" rpy="${-90 * deg_to_rad} 0 ${-90 * deg_to_rad}"/>
+      <origin xyz="0 0 0" rpy="${-90 * deg_to_rad} 0 ${-90 * deg_to_rad}"/>
     </xacro:softkinetic_ds311_rgbd_camera>
     <!-- Sonar -->
@@ -133,4 +137,7 @@
     <xacro:caster side="back_right"  radius="${caster_radius}" width="${caster_width}" separation_x="${-caster_separation_x}" separation_y="${ caster_separation_y}" offset_z="${caster_offset_z}" parent="${name}"/>
     <xacro:caster side="back_left"   radius="${caster_radius}" width="${caster_width}" separation_x="${-caster_separation_x}" separation_y="${-caster_separation_y}" offset_z="${caster_offset_z}" parent="${name}"/>
+    <!-- Antennas -->
+    <xacro:antenna_array name="antenna" parent="base_link" side="left"  reflect=" 1.0" separation_y="${antenna_separation_y}" height_0="${antenna_height_0}" height_inc="${antenna_height_inc}" />
+    <xacro:antenna_array name="antenna" parent="base_link" side="right" reflect="-1.0" separation_y="${antenna_separation_y}" height_0="${antenna_height_0}" height_inc="${antenna_height_inc}" />
   </xacro:macro>
 </robot>
