Commit message: use base_v2 rather than base urdf

File: ant_description/robots/ant_vertical_xtion_pro_live_v2.urdf.xacro (robot description, xacro)
@@ -11,5 +11,5 @@
   <!-- The following included files set up definitions of parts of the robot body -->
   <!-- Base -->
-  <xacro:include filename="$(find ant_description)/urdf/base/base_vertical_xtion_pro_live.urdf.xacro" />
+  <xacro:include filename="$(find ant_description)/urdf/base/base_v2_vertical_xtion_pro_live.urdf.xacro" />
   <!-- Generic simulator_gazebo plugins -->
   <xacro:include filename="$(find ant_description)/gazebo/gazebo.urdf.xacro" />

File: ant_description/urdf/base/base_v2_vertical_xtion_pro_live.urdf.xacro (robot description, xacro)
@@ -9,8 +9,8 @@
 <robot xmlns:xacro="http://ros.org/wiki/xacro">
   <xacro:include filename="$(find ant_description)/urdf/deg_to_rad.xacro"/>
-  <xacro:include filename="$(find ant_description)/urdf/wheels/wheel.urdf.xacro"/>
-  <xacro:include filename="$(find ant_description)/urdf/wheels/caster.urdf.xacro"/>
+  <xacro:include filename="$(find ant_description)/urdf/wheels/wheel_v2.urdf.xacro"/>
+  <xacro:include filename="$(find ant_description)/urdf/wheels/caster_v2.urdf.xacro"/>
   <xacro:include filename="$(find ant_description)/urdf/sensors/range.urdf.xacro"/>
-  <xacro:include filename="$(find ant_description)/urdf/sensors/hokuyo_urg_04lx_ug01_laser.urdf.xacro"/>
+  <xacro:include filename="$(find ant_description)/urdf/sensors/sick_tim551_laser.urdf.xacro"/>
   <xacro:include filename="$(find ant_description)/urdf/sensors/xtion_pro_live.urdf.xacro"/>
   <xacro:include filename="$(find ant_description)/urdf/sensors/imu.urdf.xacro"/>
@@ -18,22 +18,19 @@
   <xacro:include filename="$(find ant_description)/urdf/sensors/ir_receiver.urdf.xacro"/>
   <!-- Wheel characteristics -->
-  <property name="wheel_radius"     value="0.100"/>
-  <property name="wheel_width"      value="0.044"/>
-  <property name="wheel_separation" value="0.43408"/>
+  <property name="wheel_radius"     value="0.0985"/>
+  <property name="wheel_width"      value="0.040"/>
+  <property name="wheel_separation" value="0.4226"/>
   <property name="wheel_torque"     value="6.0"/>
   <property name="wheel_velocity"   value="1.0"/>
   <!-- Caster wheel characteristics -->
   <property name="caster_radius"       value="0.025"/>
-  <property name="caster_width"        value="0.020"/>
-  <property name="caster_separation_x" value="0.36734"/>
-  <property name="caster_separation_y" value="0.20362"/>
-  <property name="caster_offset_z"     value="-0.04252"/>
-  <!-- Base characteristics -->
-  <property name="base_radius" value="${(wheel_separation - wheel_width)/2 - 0.01}"/>
-  <property name="base_length" value="0.04"/>
+  <property name="caster_width"        value="0.015"/>
+  <property name="caster_separation_x" value="0.36384"/>
+  <property name="caster_separation_y" value="0.20168"/>
+  <property name="caster_offset_z"     value="-0.0335"/>
   <!-- Laser characteristics -->
-  <property name="base_laser_x" value="0.185"/>
+  <property name="base_laser_x" value="0.185"/> <!-- measured value it's approx. 0.1593 -->
   <property name="base_laser_y" value="0.0"/>
-  <property name="base_laser_z" value="0.05275"/>
+  <property name="base_laser_z" value="0.0498"/>
   <!-- RGBD characteristics -->
   <property name="base_rgbd_x" value="0.05"/>
@@ -47,14 +44,14 @@
     <link name="${name}_link">
       <inertial>
-        <origin xyz="0.0123 0.0071 0.064" rpy="0 0 0" />
-        <mass value="7.95534" />
-        <inertia ixx="0.19540233297" ixy="-0.00188862789" ixz="-0.00370655921"
-                 iyy="0.23325457568" iyz="0.00387528692"
-                 izz="0.3312456162" />
+        <origin xyz="0.00144 0.00003 0.06711" rpy="0 0 0" />
+        <mass value="24.73813" />
+        <inertia ixx="0.50215676906" ixy="0.00014630224" ixz="-0.00851406322"
+                 iyy="0.41873574615" iyz="0.00001868612"
+                 izz="0.64067017495" />
       </inertial>
       <visual>
         <origin xyz="0 0 0" rpy="0 0 0" />
         <geometry>
-          <mesh filename="package://ant_description/meshes/base/base.stl" />
+          <mesh filename="package://ant_description/meshes/base/base_v2.stl" />
         </geometry>
         <material name="DarkGrey" />
@@ -63,5 +60,5 @@
         <origin xyz="0 0 0" rpy="0 0 0" />
         <geometry>
-          <cylinder radius="${base_radius}" length="${base_length}"/>
+          <mesh filename="package://ant_description/meshes/base/base_v2_collision.stl" />
         </geometry>
         <material name="DarkGrey" />
@@ -76,7 +73,8 @@
     </joint>
     <!-- Laser -->
-    <xacro:hokuyo_urg_04lx_ug01_laser name="${name}_laser" parent="${name}" ros_topic="scan" update_rate="10" min_angle="${-90 * deg_to_rad}" max_angle="${90 * deg_to_rad}" >
+    <!-- Theoretic FOV = 220º -->
+    <xacro:sick_tim551_laser name="${name}_laser" parent="${name}" ros_topic="scan" update_rate="15" min_angle="${-110 * deg_to_rad}" max_angle="${110 * deg_to_rad}" >
       <origin xyz="${base_laser_x} ${base_laser_y} ${base_laser_z}" rpy="0 0 0" />
-    </xacro:hokuyo_urg_04lx_ug01_laser>
+    </xacro:sick_tim551_laser>
     <!-- RGBD -->
     <xacro:xtion_pro_live name="${name}_rgbd_camera" parent="${name}">
@@ -109,5 +107,5 @@
     <!-- @todo ant_hardware_gazebo needs an IMU!  -->
     <xacro:imu_sensor name="base_inclinometer" parent="${name}_link" update_rate="100.0">
-      <origin xyz="0 0 ${base_length / 2}" rpy="0 0 0"/>
+      <origin xyz="0 0 0" rpy="0 0 0"/>
     </xacro:imu_sensor>
     <!-- IR receiver -->
