Commit message: Divide antenna_array into 4 and 6 antenna variants, add antenna to ant

File: ant_description/urdf/antennas/antenna_array.urdf.xacro (robot description, xacro)
@@ -10,9 +10,12 @@
   <!--File includes-->
   <xacro:include filename="$(find ant_description)/urdf/antennas/antenna.urdf.xacro" />
-  <xacro:macro name="antenna_array" params="name parent side reflect separation_y height_0 height_inc">
+  <xacro:macro name="antenna_array_4" params="name parent side reflect separation_y height_0 height_inc">
       <xacro:antenna name="${name}" parent="${parent}" side="${side}" reflect="${reflect}" num="1" separation_y="${separation_y}" height="${height_0}" />
       <xacro:antenna name="${name}" parent="${parent}" side="${side}" reflect="${reflect}" num="2" separation_y="${separation_y}" height="${height_0 +     height_inc}"  />
       <xacro:antenna name="${name}" parent="${parent}" side="${side}" reflect="${reflect}" num="3" separation_y="${separation_y}" height="${height_0 + 2 * height_inc}" />
       <xacro:antenna name="${name}" parent="${parent}" side="${side}" reflect="${reflect}" num="4" separation_y="${separation_y}" height="${height_0 + 3 * height_inc}" />
+  </xacro:macro>
+  <xacro:macro name="antenna_array_6" params="name parent side reflect separation_y height_0 height_inc">
+      <xacro:antenna_array_4 name="${name}" parent="${parent}" side="${side}" reflect="${reflect}" separation_y="${separation_y}" height_0="${height_0}" height_inc="${height_inc}" />
       <xacro:antenna name="${name}" parent="${parent}" side="${side}" reflect="${reflect}" num="5" separation_y="${separation_y}" height="${height_0 + 4 * height_inc}"/>
       <xacro:antenna name="${name}" parent="${parent}" side="${side}" reflect="${reflect}" num="6" separation_y="${separation_y}" height="${height_0 + 5 * height_inc}" />

File: ant_description/urdf/base/base_rebujito.urdf.xacro (robot description, xacro)
@@ -113,6 +113,6 @@
     <xacro:caster side="back"  radius="${caster_radius}" width="${caster_width}" separation_x="${-caster_separation}" separation_y="0" offset_z="${caster_offset_z}" parent="${name}"/>
     <!-- Antennas -->
-    <xacro:antenna_array name="antenna" parent="base_link" side="left"  reflect=" 1.0" separation_y="${antenna_separation_y}" height_0="${antenna_height_0}" height_inc="${antenna_height_inc}" />
-    <xacro:antenna_array name="antenna" parent="base_link" side="right" reflect="-1.0" separation_y="${antenna_separation_y}" height_0="${antenna_height_0}" height_inc="${antenna_height_inc}" />
+    <xacro:antenna_array_6 name="antenna" parent="base_link" side="left"  reflect=" 1.0" separation_y="${antenna_separation_y}" height_0="${antenna_height_0}" height_inc="${antenna_height_inc}" />
+    <xacro:antenna_array_6 name="antenna" parent="base_link" side="right" reflect="-1.0" separation_y="${antenna_separation_y}" height_0="${antenna_height_0}" height_inc="${antenna_height_inc}" />
   </xacro:macro>
 </robot>

File: ant_description/urdf/base/base_v2_vertical_xtion_pro_live.urdf.xacro (robot description, xacro)
@@ -40,4 +40,9 @@
   <property name="base_rgbd_P" value="30.0"/>
   <property name="base_rgbd_Y" value="8.0"/>
+  <!-- Antennas characteristics -->
+  <!-- @todo ${wheel_separation + wheel_width} fails -->
+  <property name="antenna_separation_y" value="0.2"/>
+  <property name="antenna_height_0"     value="0.5"/>
+  <property name="antenna_height_inc"   value="0.45"/>
   <xacro:macro name="base" params="name">
     <!-- Base -->
@@ -129,4 +134,7 @@
     <xacro:caster side="back_right"  radius="${caster_radius}" width="${caster_width}" separation_x="${-caster_separation_x}" separation_y="${ caster_separation_y}" offset_z="${caster_offset_z}" parent="${name}"/>
     <xacro:caster side="back_left"   radius="${caster_radius}" width="${caster_width}" separation_x="${-caster_separation_x}" separation_y="${-caster_separation_y}" offset_z="${caster_offset_z}" parent="${name}"/>
+    <!-- Antennas -->
+    <xacro:antenna_array_4 name="antenna" parent="base_link" side="left"  reflect=" 1.0" separation_y="${antenna_separation_y}" height_0="${antenna_height_0}" height_inc="${antenna_height_inc}" />
+    <xacro:antenna_array_4 name="antenna" parent="base_link" side="right" reflect="-1.0" separation_y="${antenna_separation_y}" height_0="${antenna_height_0}" height_inc="${antenna_height_inc}" />
   </xacro:macro>
 </robot>
