Commit message: Use base_footprint_link

File: pmb2_description/urdf/objects/battery_atp.urdf.xacro (robot description, xacro)
@@ -22,5 +22,5 @@
           <mesh filename="package://pmb2_description/meshes/objects/battery_atp.stl"/>
         </geometry>
-        <material name="LightGrey"/>
+        <material name="DarkGrey"/>
       </visual>
       <collision>

File: pmb2_description/urdf/objects/battery_atp_2.urdf.xacro (robot description, xacro)
@@ -22,5 +22,5 @@
           <mesh filename="package://pmb2_description/meshes/objects/battery_atp_2.stl"/>
         </geometry>
-        <material name="LightGrey"/>
+        <material name="DarkGrey"/>
       </visual>
       <collision>

File: pmb2_description/urdf/objects/battery_tlh.urdf.xacro (robot description, xacro)
@@ -22,5 +22,5 @@
           <mesh filename="package://pmb2_description/meshes/objects/battery_tlh.stl"/>
         </geometry>
-        <material name="LightGrey"/>
+        <material name="DarkGrey"/>
       </visual>
       <collision>

File: pmb2_description/urdf/objects/battery_tlh_2.urdf.xacro (robot description, xacro)
@@ -22,5 +22,5 @@
           <mesh filename="package://pmb2_description/meshes/objects/battery_tlh_2.stl"/>
         </geometry>
-        <material name="LightGrey"/>
+        <material name="DarkGrey"/>
       </visual>
       <collision>

File: pmb2_description/urdf/objects/charger.urdf.xacro (robot description, xacro)
@@ -22,5 +22,5 @@
           <mesh filename="package://pmb2_description/meshes/objects/charger.stl"/>
         </geometry>
-        <material name="LightGrey"/>
+        <material name="DarkGrey"/>
       </visual>
       <collision>
