Commit message: New meshes

File: pmb2_description/urdf/objects/cover.urdf.xacro (robot description, xacro)
@@ -28,5 +28,5 @@
       <parent link="${parent}"/>
       <child link="${name}_link"/>
-      <origin xyz="0 0 0.15" rpy="0 0 0"/>
+      <origin xyz="0 0 0.13" rpy="0 0 0"/>
     </joint>
     <gazebo reference="${name}_link">
