Commit message: Add collision to antenna

File: pmb2_description/urdf/objects/antenna.urdf.xacro (robot description, xacro)
@@ -24,4 +24,11 @@
         <material name="Black"/>
       </visual>
+      <collision>
+        <origin xyz="0 0 0.085" rpy="0 0 0"/>
+        <geometry>
+          <cylinder radius="0.005" length="0.17"/>
+        </geometry>
+        <material name="Black"/>
+      </collision>
     </link>
     <gazebo reference="${name}_link">
