Commit message: Make rgbd camera fixed

File: pmb2_description/urdf/sensors/xtion_pro_live_revolute.urdf.xacro (robot description, xacro)
@@ -22,6 +22,8 @@
   <xacro:macro name="xtion_pro_live" params="name parent *origin *optical_origin">
     <!-- frames in the center of the camera -->
-    <joint name="${name}_joint" type="fixed">
+    <joint name="${name}_joint" type="revolute">
       <insert_block name="origin"/>
+      <axis xyz="0 0 1"/>
+      <limit lower="0" upper="0.001" effort="100" velocity="0.01"/>
       <parent link="${parent}_link"/>
       <child link="${name}_link"/>
