Commit message: Add inertial block to xtion pro live

File: pmb2_description/urdf/sensors/xtion_pro_live.urdf.xacro (robot description, xacro)
@@ -48,5 +48,13 @@
       <child link="${name}_optical_frame"/>
     </joint>
-    <link name="${name}_optical_frame"/>
+    <link name="${name}_optical_frame">
+      <inertial>
+        <origin xyz="0 0 0" rpy="0 0 0"/>
+        <mass value="0.001"/>
+        <inertia ixx="0.00001" ixy="0" ixz="0"
+                 iyy="0.00001" iyz="0"
+                 izz="0.00001"/>
+      </inertial>
+    </link>
     <!-- frames of the depth sensor -->
     <joint name="${name}_depth_joint" type="fixed">
@@ -55,5 +63,13 @@
       <child link="${name}_depth_frame"/>
     </joint>
-    <link name="${name}_depth_frame"/>
+    <link name="${name}_depth_frame">
+      <inertial>
+        <origin xyz="0 0 0" rpy="0 0 0"/>
+        <mass value="0.001"/>
+        <inertia ixx="0.00001" ixy="0" ixz="0"
+                 iyy="0.00001" iyz="0"
+                 izz="0.00001"/>
+      </inertial>
+    </link>
     <joint name="${name}_depth_optical_joint" type="fixed">
       <origin xyz="0 0 0" rpy="${-90.0 * deg_to_rad} 0.0 ${-90.0 * deg_to_rad}" />
@@ -61,5 +77,13 @@
       <child link="${name}_depth_optical_frame"/>
     </joint>
-    <link name="${name}_depth_optical_frame"/>
+    <link name="${name}_depth_optical_frame">
+      <inertial>
+        <origin xyz="0 0 0" rpy="0 0 0"/>
+        <mass value="0.001"/>
+        <inertia ixx="0.00001" ixy="0" ixz="0"
+                 iyy="0.00001" iyz="0"
+                 izz="0.00001"/>
+      </inertial>
+    </link>
     <!-- frames of the rgb sensor -->
     <joint name="${name}_rgb_joint" type="fixed">
@@ -68,5 +92,13 @@
       <child link="${name}_rgb_frame"/>
     </joint>
-    <link name="${name}_rgb_frame"/>
+    <link name="${name}_rgb_frame">
+      <inertial>
+        <origin xyz="0 0 0" rpy="0 0 0"/>
+        <mass value="0.001"/>
+        <inertia ixx="0.00001" ixy="0" ixz="0"
+                 iyy="0.00001" iyz="0"
+                 izz="0.00001"/>
+      </inertial>
+    </link>
     <joint name="${name}_rgb_optical_joint" type="fixed">
       <origin xyz="0 0 0" rpy="${-90.0 * deg_to_rad} 0.0 ${-90.0 * deg_to_rad}" />
@@ -74,5 +106,13 @@
       <child link="${name}_rgb_optical_frame"/>
     </joint>
-    <link name="${name}_rgb_optical_frame"/>
+    <link name="${name}_rgb_optical_frame">
+      <inertial>
+        <origin xyz="0 0 0" rpy="0 0 0"/>
+        <mass value="0.001"/>
+        <inertia ixx="0.00001" ixy="0" ixz="0"
+                 iyy="0.00001" iyz="0"
+                 izz="0.00001"/>
+      </inertial>
+    </link>
     <!-- extensions -->
     <xacro:xtion_pro_live_rgbd_camera_gazebo name="${name}" />

File: pmb2_description/urdf/sensors/xtion_pro_live_revolute.urdf.xacro (robot description, xacro)
@@ -50,5 +50,13 @@
       <child link="${name}_optical_frame"/>
     </joint>
-    <link name="${name}_optical_frame"/>
+    <link name="${name}_optical_frame">
+      <inertial>
+        <origin xyz="0 0 0" rpy="0 0 0"/>
+        <mass value="0.001"/>
+        <inertia ixx="0.00001" ixy="0" ixz="0"
+                 iyy="0.00001" iyz="0"
+                 izz="0.00001"/>
+      </inertial>
+    </link>
     <!-- frames of the depth sensor -->
     <joint name="${name}_depth_joint" type="fixed">
@@ -57,5 +65,13 @@
       <child link="${name}_depth_frame"/>
     </joint>
-    <link name="${name}_depth_frame"/>
+    <link name="${name}_depth_frame">
+      <inertial>
+        <origin xyz="0 0 0" rpy="0 0 0"/>
+        <mass value="0.001"/>
+        <inertia ixx="0.00001" ixy="0" ixz="0"
+                 iyy="0.00001" iyz="0"
+                 izz="0.00001"/>
+      </inertial>
+    </link>
     <joint name="${name}_depth_optical_joint" type="fixed">
       <origin xyz="0 0 0" rpy="${-90.0 * deg_to_rad} 0.0 ${-90.0 * deg_to_rad}" />
@@ -63,5 +79,13 @@
       <child link="${name}_depth_optical_frame"/>
     </joint>
-    <link name="${name}_depth_optical_frame"/>
+    <link name="${name}_depth_optical_frame">
+      <inertial>
+        <origin xyz="0 0 0" rpy="0 0 0"/>
+        <mass value="0.001"/>
+        <inertia ixx="0.00001" ixy="0" ixz="0"
+                 iyy="0.00001" iyz="0"
+                 izz="0.00001"/>
+      </inertial>
+    </link>
     <!-- frames of the rgb sensor -->
     <joint name="${name}_rgb_joint" type="fixed">
@@ -70,5 +94,13 @@
       <child link="${name}_rgb_frame"/>
     </joint>
-    <link name="${name}_rgb_frame"/>
+    <link name="${name}_rgb_frame">
+      <inertial>
+        <origin xyz="0 0 0" rpy="0 0 0"/>
+        <mass value="0.001"/>
+        <inertia ixx="0.00001" ixy="0" ixz="0"
+                 iyy="0.00001" iyz="0"
+                 izz="0.00001"/>
+      </inertial>
+    </link>
     <joint name="${name}_rgb_optical_joint" type="fixed">
       <origin xyz="0 0 0" rpy="${-90.0 * deg_to_rad} 0.0 ${-90.0 * deg_to_rad}" />
@@ -76,5 +108,13 @@
       <child link="${name}_rgb_optical_frame"/>
     </joint>
-    <link name="${name}_rgb_optical_frame"/>
+    <link name="${name}_rgb_optical_frame">
+      <inertial>
+        <origin xyz="0 0 0" rpy="0 0 0"/>
+        <mass value="0.001"/>
+        <inertia ixx="0.00001" ixy="0" ixz="0"
+                 iyy="0.00001" iyz="0"
+                 izz="0.00001"/>
+      </inertial>
+    </link>
     <!-- extensions -->
     <xacro:xtion_pro_live_rgbd_camera_gazebo name="${name}" />
