Commit message: fixed the frame wrongly removed previously

File: pmb2_description/urdf/sensors/structure_sensor.urdf.xacro (robot description, xacro)
@@ -44,4 +44,18 @@
       </collision>
     </link>
+    <joint name="${name}_optical_joint" type="fixed">
+      <insert_block name="optical_origin" />
+      <parent link="${name}_link"/>
+      <child link="${name}_optical_frame"/>
+    </joint>
+    <link name="${name}_optical_frame">
+      <inertial>
+        <mass value="0.01" />
+        <origin xyz="0 0 0" rpy="0 0 0"/>
+        <inertia ixx="0.0"  ixy="0.0"  ixz="0.0"
+                 iyy="0.0"  iyz="0.0"
+                 izz="0.0" />
+      </inertial>
+    </link>
     <!-- frames of the depth sensor -->
     <joint name="${name}_depth_joint" type="fixed">
@@ -57,4 +71,17 @@
     </joint>
     <link name="${name}_depth_optical_frame"/>
+    <!-- frames of the rgb sensor -->
+    <joint name="${name}_rgb_joint" type="fixed">
+      <origin xyz="0.0 0.0135 0.0" rpy="0 0 0" />
+      <parent link="${name}_link" />
+      <child link="${name}_rgb_frame"/>
+    </joint>
+    <link name="${name}_rgb_frame"/>
+    <joint name="${name}_rgb_optical_joint" type="fixed">
+      <origin xyz="0 0 0" rpy="${-90.0 * deg_to_rad} 0.0 ${-90.0 * deg_to_rad}" />
+      <parent link="${name}_rgb_frame" />
+      <child link="${name}_rgb_optical_frame"/>
+    </joint>
+    <link name="${name}_rgb_optical_frame"/>
     <!-- extensions -->
     <xacro:structure_sensor_rgbd_camera_gazebo name="${name}" />

Commit message: removed rgb frames that are not present in this sensor

File: pmb2_description/urdf/sensors/structure_sensor.urdf.xacro (robot description, xacro)
@@ -71,17 +71,4 @@
     </joint>
     <link name="${name}_depth_optical_frame"/>
-    <!-- frames of the rgb sensor -->
-    <joint name="${name}_rgb_joint" type="fixed">
-      <origin xyz="0.0 0.0135 0.0" rpy="0 0 0" />
-      <parent link="${name}_link" />
-      <child link="${name}_rgb_frame"/>
-    </joint>
-    <link name="${name}_rgb_frame"/>
-    <joint name="${name}_rgb_optical_joint" type="fixed">
-      <origin xyz="0 0 0" rpy="${-90.0 * deg_to_rad} 0.0 ${-90.0 * deg_to_rad}" />
-      <parent link="${name}_rgb_frame" />
-      <child link="${name}_rgb_optical_frame"/>
-    </joint>
-    <link name="${name}_rgb_optical_frame"/>
     <!-- extensions -->
     <xacro:structure_sensor_rgbd_camera_gazebo name="${name}" />
