Commit message: Add color to gazebo

File: pmb2_description/urdf/sensors/hokuyo_urg_04lx_ug01_laser.gazebo.xacro (robot description, xacro)
@@ -40,4 +40,5 @@
         </plugin>
       </sensor>
+      <material>Gazebo/DarkGrey</material>
     </gazebo>
   </xacro:macro>

File: pmb2_description/urdf/sensors/sick_tim551_laser.gazebo.xacro (robot description, xacro)
@@ -40,4 +40,5 @@
         </plugin>
       </sensor>
+      <material>Gazebo/DarkGrey</material>
     </gazebo>
   </xacro:macro>

Commit message: Fix collision error with the omni base + indetation fix

File: pmb2_description/urdf/sensors/hokuyo_urg_04lx_ug01_laser.gazebo.xacro (robot description, xacro)
@@ -12,5 +12,6 @@
   <xacro:macro name="hokuyo_urg_04lx_ug01_laser_gazebo" params="name ros_topic update_rate min_angle max_angle">
     <gazebo reference="${name}_link">
-      <sensor type="ray" name="${name}">
+      <!-- Using gpu laser instead of normal laser because it was causing issues with the omni_base -->
+      <sensor type="gpu_ray" name="${name}">
         <pose>0 0 0 0 0 0</pose>
         <update_rate>${update_rate}</update_rate>
@@ -32,5 +33,5 @@
           </range>
         </ray>
-        <plugin filename="libgazebo_ros_laser.so" name="gazebo_ros_hokuyo_laser">
+        <plugin filename="libgazebo_ros_gpu_laser.so" name="gazebo_ros_hokuyo_laser">
           <gaussianNoise>0.03</gaussianNoise>
           <alwaysOn>true</alwaysOn>

File: pmb2_description/urdf/sensors/sick_tim551_laser.gazebo.xacro (robot description, xacro)
@@ -12,5 +12,6 @@
   <xacro:macro name="sick_tim551_laser_gazebo" params="name ros_topic update_rate min_angle max_angle">
     <gazebo reference="${name}_link">
-      <sensor type="ray" name="${name}">
+      <!-- Using gpu laser instead of normal laser because it was causing issues with the omni_base -->
+      <sensor type="gpu_ray" name="${name}">
         <pose>0 0 0 0 0 0</pose>
         <update_rate>${update_rate}</update_rate>
@@ -32,5 +33,5 @@
           </range>
         </ray>
-        <plugin filename="libgazebo_ros_laser.so" name="gazebo_ros_sick_laser">
+        <plugin filename="libgazebo_ros_gpu_laser.so" name="gazebo_ros_sick_laser">
           <gaussianNoise>0.06</gaussianNoise>
           <alwaysOn>true</alwaysOn>

File: pmb2_description/urdf/sensors/sick_tim561_laser.gazebo.xacro (robot description, xacro)
@@ -12,5 +12,6 @@
   <xacro:macro name="sick_tim561_laser_gazebo" params="name ros_topic update_rate min_angle max_angle">
     <gazebo reference="${name}_link">
-      <sensor type="ray" name="${name}">
+      <!-- Using gpu laser instead of normal laser because it was causing issues with the omni_base -->
+      <sensor type="gpu_ray" name="${name}">
         <pose>0 0 0 0 0 0</pose>
         <update_rate>${update_rate}</update_rate>
@@ -32,5 +33,5 @@
           </range>
         </ray>
-        <plugin filename="libgazebo_ros_laser.so" name="gazebo_ros_sick_laser">
+        <plugin filename="libgazebo_ros_gpu_laser.so" name="gazebo_ros_sick_laser">
           <gaussianNoise>0.06</gaussianNoise>
           <alwaysOn>true</alwaysOn>

File: pmb2_description/urdf/sensors/sick_tim571_laser.gazebo.xacro (robot description, xacro)
@@ -12,5 +12,6 @@
   <xacro:macro name="sick_tim571_laser_gazebo" params="name ros_topic update_rate min_angle max_angle">
     <gazebo reference="${name}_link">
-      <sensor type="ray" name="${name}">
+      <!-- Using gpu laser instead of normal laser because it was causing issues with the omni_base -->
+      <sensor type="gpu_ray" name="${name}">
         <pose>0 0 0 0 0 0</pose>
         <update_rate>${update_rate}</update_rate>
@@ -32,5 +33,5 @@
           </range>
         </ray>
-        <plugin filename="libgazebo_ros_laser.so" name="gazebo_ros_sick_laser">
+        <plugin filename="libgazebo_ros_gpu_laser.so" name="gazebo_ros_sick_laser">
           <gaussianNoise>0.06</gaussianNoise>
           <alwaysOn>true</alwaysOn>

File: pmb2_description/urdf/wheels/wheel.urdf.xacro (robot description, xacro)
@@ -23,54 +23,54 @@
           iyy="0.00499741733" iyz="${-0.00000000164 * reflect}"
           izz="0.00839239692"/>
-        </inertial>
-        <visual>
-          <origin xyz="0 0 0" rpy="${-90.0 * (1 - reflect) * deg_to_rad} 0 0"/>
-          <geometry>
-            <mesh filename="package://pmb2_description/meshes/wheels/wheel.stl"/>
-          </geometry>
-          <material name="DarkGrey"/>
-        </visual>
-        <collision>
-          <origin xyz="0 0 0" rpy="0 0 0"/>
-          <geometry>
-            <sphere radius="${radius}" /> <!-- length="${width}"/> -->
-          </geometry>
-        </collision>
-      </link>
-      <link name="suspension_${side}_link">
-        <inertial>
-          <origin xyz="0 0 -0.02" rpy="0 0 0"/>
-          <mass value="10"/>
-          <inertia ixx="1.0" ixy="0" ixz="0"
-                   iyy="1.0" iyz="0"
-                   izz="1.0"/>
-         </inertial>
-        <kinematic>0</kinematic>
-        <gravity>1</gravity>
-      </link>
-      <joint name="suspension_${side}_joint" type="prismatic">
+      </inertial>
+      <visual>
+        <origin xyz="0 0 0" rpy="${-90.0 * (1 - reflect) * deg_to_rad} 0 0"/>
+        <geometry>
+          <mesh filename="package://pmb2_description/meshes/wheels/wheel.stl"/>
+        </geometry>
+        <material name="DarkGrey"/>
+      </visual>
+      <collision>
         <origin xyz="0 0 0" rpy="0 0 0"/>
-        <axis xyz="0 0 1"/>
-        <limit effort="100.0" lower="-0.005" upper="0.005" velocity="1.0"/>
-        <child link="suspension_${side}_link"/>
-        <parent link="${parent}_link"/>
-        <calibration rising="0.0" />
-        <dynamics damping="100"/>
-        <safety_controller k_position="0"
-          k_velocity="10"
-          soft_lower_limit="-0.005"
-          soft_upper_limit="0.005" />
-        </joint>
-        <joint name="wheel_${side}_joint" type="continuous">
-          <parent link="suspension_${side}_link"/>
-          <child link="wheel_${side}_link"/>
-          <origin xyz="0 ${-separation / 2 * reflect} 0.0" rpy="${-90.0 * deg_to_rad} 0 0"/>
-          <axis xyz="0 0 1"/>
-          <limit effort="${torque}" velocity="${velocity / radius}"/>
-        </joint>
-        <!-- Transmission -->
-        <xacro:wheel_transmission side="${side}"/>
-        <!-- Gazebo extensions -->
-        <xacro:wheel_gazebo side="${side}"/>
-      </xacro:macro>
-    </robot>
+        <geometry>
+          <sphere radius="${radius}" /> <!-- length="${width}"/> -->
+        </geometry>
+      </collision>
+    </link>
+    <link name="suspension_${side}_link">
+      <inertial>
+        <origin xyz="0 0 -0.02" rpy="0 0 0"/>
+        <mass value="10"/>
+        <inertia ixx="1.0" ixy="0" ixz="0"
+                 iyy="1.0" iyz="0"
+                 izz="1.0"/>
+      </inertial>
+      <kinematic>0</kinematic>
+      <gravity>1</gravity>
+    </link>
+    <joint name="suspension_${side}_joint" type="prismatic">
+      <origin xyz="0 0 0" rpy="0 0 0"/>
+      <axis xyz="0 0 1"/>
+      <limit effort="100.0" lower="-0.005" upper="0.005" velocity="1.0"/>
+      <child link="suspension_${side}_link"/>
+      <parent link="${parent}_link"/>
+      <calibration rising="0.0" />
+      <dynamics damping="100"/>
+      <safety_controller k_position="0"
+        k_velocity="10"
+        soft_lower_limit="-0.005"
+        soft_upper_limit="0.005" />
+    </joint>
+    <joint name="wheel_${side}_joint" type="continuous">
+      <parent link="suspension_${side}_link"/>
+      <child link="wheel_${side}_link"/>
+      <origin xyz="0 ${-separation / 2 * reflect} 0.0" rpy="${-90.0 * deg_to_rad} 0 0"/>
+      <axis xyz="0 0 1"/>
+      <limit effort="${torque}" velocity="${velocity / radius}"/>
+    </joint>
+    <!-- Transmission -->
+    <xacro:wheel_transmission side="${side}"/>
+    <!-- Gazebo extensions -->
+    <xacro:wheel_gazebo side="${side}"/>
+  </xacro:macro>
+</robot>
