Commit message: Fix ELP rgb camera position and add its gazebo plugin

File: pmb2_description/urdf/sensors/courier.urdf.xacro (robot description, xacro)
@@ -22,7 +22,7 @@
   <xacro:property name="roof_rgbd_Y" value="0.0"/>
   <!-- RGB characteristics -->
-  <xacro:property name="rgb_x" value="0.185"/>
+  <xacro:property name="rgb_x" value="0.18752"/>
   <xacro:property name="rgb_y" value="0.0"/>
-  <xacro:property name="rgb_z" value="0.86"/>
+  <xacro:property name="rgb_z" value="0.3301"/>
   <xacro:property name="rgb_R" value="0.0"/>
   <xacro:property name="rgb_P" value="15.0"/>

File: pmb2_description/urdf/sensors/elp_rgb.urdf.xacro (robot description, xacro)
@@ -5,4 +5,5 @@
 -->
 <robot xmlns:xacro="http://ros.org/wiki/xacro">
+ <xacro:include filename="$(find pmb2_description)/urdf/sensors/elp_rgb.gazebo.xacro" />
   <!-- Macro -->
   <xacro:macro name="elp_rgb" params="name parent *origin *optical_origin">
@@ -42,4 +43,6 @@
     </joint>
     <link name="${name}_optical_frame"/>
+    <!-- extensions -->
+    <xacro:elp_sensor_rgb_camera_gazebo name="${name}" />
   </xacro:macro>
 </robot>

Commit message: added rgbd calibration feature for courier

File: pmb2_description/urdf/sensors/courier.urdf.xacro (robot description, xacro)
@@ -7,17 +7,15 @@
   <xacro:include filename="$(find pmb2_description)/urdf/sensors/structure_sensor.urdf.xacro"/>
   <xacro:include filename="$(find pmb2_description)/urdf/sensors/elp_rgb.urdf.xacro"/>
+  <xacro:include filename="$(find pmb2_description)/urdf/base/base_pmb2_calib.urdf.xacro"/>
+  <xacro:property name="default_calibration_path" value="$(find pmb2_description)"/>
+  <xacro:property name="calibration_path" value="$(optenv pmb2_description_calibration_path ${default_calibration_path})"/>
+  <xacro:include filename="${calibration_path}/urdf/base/base_pmb2_calib.urdf.xacro"/>
   <!-- base RGBD characteristics -->
   <xacro:property name="base_rgbd_x" value="0.22697"/>
   <xacro:property name="base_rgbd_y" value="0.0"/>
-  <xacro:property name="base_rgbd_z" value="0.52635"/>
-  <xacro:property name="base_rgbd_R" value="-0.171709"/>
-  <xacro:property name="base_rgbd_P" value="57.9362"/>
   <xacro:property name="base_rgbd_Y" value="0.0"/>
   <!-- roof RGBD characteristics -->
   <xacro:property name="roof_rgbd_x" value="0.18473"/>
   <xacro:property name="roof_rgbd_y" value="0.0"/>
-  <xacro:property name="roof_rgbd_z" value="0.470428"/>
-  <xacro:property name="roof_rgbd_R" value="-0.299256"/>
-  <xacro:property name="roof_rgbd_P" value="10.596"/>
   <xacro:property name="roof_rgbd_Y" value="0.0"/>
   <!-- RGB characteristics -->

Commit message: support to structure cameras in simulation

File: pmb2_description/urdf/sensors/courier.urdf.xacro (robot description, xacro)
@@ -19,7 +19,7 @@
   <xacro:property name="base_rgbd_x" value="0.22697"/>
   <xacro:property name="base_rgbd_y" value="0.0"/>
-  <xacro:property name="base_rgbd_z" value="0.52635"/>
+  <xacro:property name="base_rgbd_z" value="0.535"/>
   <xacro:property name="base_rgbd_R" value="-0.171709"/>
-  <xacro:property name="base_rgbd_P" value="57.9362"/>
+  <xacro:property name="base_rgbd_P" value="60"/>
   <xacro:property name="base_rgbd_Y" value="0.0"/>
   <!-- roof RGBD characteristics -->
@@ -28,5 +28,5 @@
   <xacro:property name="roof_rgbd_z" value="0.470428"/>
   <xacro:property name="roof_rgbd_R" value="-0.299256"/>
-  <xacro:property name="roof_rgbd_P" value="10.596"/>
+  <xacro:property name="roof_rgbd_P" value="12"/>
   <xacro:property name="roof_rgbd_Y" value="0.0"/>
   <!-- RGB characteristics -->

File: pmb2_description/urdf/sensors/structure_sensor.gazebo.xacro (robot description, xacro)
@@ -30,22 +30,25 @@
             <far>10.0</far>
           </clip>
+          <distortion>
+            <k1>0.1</k1>
+            <k2>0.2</k2>
+            <k3>0.3</k3>
+            <p1>0.4</p1>
+            <p2>0.5</p2>
+            <center>0.5 0.5</center>
+          </distortion>
         </camera>
-        <plugin name="${name}_frame_controller" filename="libgazebo_ros_openni_kinect.so">
-          <alwaysOn>true</alwaysOn>
-          <updateRate>6.0</updateRate>
-          <cameraName>${name}</cameraName>
-          <imageTopicName>ir/image_raw</imageTopicName>
-          <cameraInfoTopicName>ir/camera_info</cameraInfoTopicName>
-          <depthImageTopicName>depth/image_raw</depthImageTopicName>
-          <depthImageCameraInfoTopicName>depth/camera_info</depthImageCameraInfoTopicName>
-          <pointCloudTopicName>depth/points</pointCloudTopicName>
-          <frameName>${name}_optical_frame</frameName>
-          <pointCloudCutoff>0.45</pointCloudCutoff>
-          <rangeMax>10.0</rangeMax>
-          <distortionK1>0.00000001</distortionK1>
-          <distortionK2>0.00000001</distortionK2>
-          <distortionK3>0.00000001</distortionK3>
-          <distortionT1>0.00000001</distortionT1>
-          <distortionT2>0.00000001</distortionT2>
+        <plugin name="${name}_ir" filename="libgazebo_ros_camera.so">
+          <camera_name>${name}</camera_name>
+          <frame_name>${name}_optical_frame</frame_name>
+          <max_depth>10.0</max_depth>
+          <ros>
+            <remapping>${name}/image_raw:=${name}/ir/image_raw</remapping>
+            <remapping>${name}/camera_info:=${name}/ir/camera_info</remapping>
+            <remapping>${name}/image_raw/compressed:=${name}/ir/image_raw/compressed</remapping>
+            <remapping>${name}/image_raw/compressedDepth:=${name}/ir/image_raw/compressedDepth</remapping>
+            <remapping>${name}/image_raw/theora:=${name}/ir/image_raw/theora</remapping>
+            <remapping>${name}/points:=${name}/depth/points</remapping>
+          </ros>
         </plugin>
       </sensor>
@@ -65,20 +68,25 @@
             <far>10.0</far>
           </clip>
+          <distortion>
+            <k1>0.1</k1>
+            <k2>0.2</k2>
+            <k3>0.3</k3>
+            <p1>0.4</p1>
+            <p2>0.5</p2>
+            <center>0.5 0.5</center>
+          </distortion>
         </camera>
-        <plugin name="${name}_frame_controller" filename="libgazebo_ros_openni_kinect.so">
-          <alwaysOn>true</alwaysOn>
-          <updateRate>6.0</updateRate>
-          <cameraName>${name}</cameraName>
-          <imageTopicName>rgb/image_raw</imageTopicName>
-          <cameraInfoTopicName>rgb/camera_info</cameraInfoTopicName>
-          <pointCloudTopicName>rgb/points</pointCloudTopicName>
-          <frameName>${name}_optical_frame</frameName>
-          <pointCloudCutoff>0.45</pointCloudCutoff>
-          <rangeMax>10.0</rangeMax>
-          <distortionK1>0.00000001</distortionK1>
-          <distortionK2>0.00000001</distortionK2>
-          <distortionK3>0.00000001</distortionK3>
-          <distortionT1>0.00000001</distortionT1>
-          <distortionT2>0.00000001</distortionT2>
+        <plugin name="${name}_rgb" filename="libgazebo_ros_camera.so">
+          <camera_name>${name}</camera_name>
+          <frame_name>${name}_optical_frame</frame_name>
+          <max_depth>10.0</max_depth>
+          <ros>
+            <remapping>${name}/image_raw:=${name}/rgb/image_raw</remapping>
+            <remapping>${name}/camera_info:=${name}/rgb/camera_info</remapping>
+            <remapping>${name}/image_raw/compressed:=${name}/rgb/image_raw/compressed</remapping>
+            <remapping>${name}/image_raw/compressedDepth:=${name}/rgb/image_raw/compressedDepth</remapping>
+            <remapping>${name}/image_raw/theora:=${name}/rgb/image_raw/theora</remapping>
+            <remapping>${name}/points:=${name}/rgb/points</remapping>
+          </ros>
         </plugin>
       </sensor>
