Commit message: urdf full calls default & add sonar/micro

File: pmb2_description/robots/pmb2_full.urdf.xacro (robot description, xacro)
@@ -17,4 +17,4 @@
   <xacro:include filename="$(find pmb2_description)/urdf/materials.urdf.xacro" />
   <!-- Now we can start using the macros included above to define the actual robot -->
-  <xacro:base name="base"/>
+  <xacro:base_full name="base" laser_sick="false"/>
 </robot>

File: pmb2_description/robots/pmb2_full_sick.urdf.xacro (robot description, xacro)
@@ -11,5 +11,5 @@
   <!-- The following included files set up definitions of parts of the robot body -->
   <!-- Base -->
-  <xacro:include filename="$(find pmb2_description)/urdf/base/base_full_sick.urdf.xacro" />
+  <xacro:include filename="$(find pmb2_description)/urdf/base/base_full.urdf.xacro" />
   <!-- Generic simulator_gazebo plugins -->
   <xacro:include filename="$(find pmb2_description)/gazebo/gazebo.urdf.xacro" />
@@ -17,4 +17,4 @@
   <xacro:include filename="$(find pmb2_description)/urdf/materials.urdf.xacro" />
   <!-- Now we can start using the macros included above to define the actual robot -->
-  <xacro:base name="base"/>
+  <xacro:base_full name="base" laser_sick="true"/>
 </robot>

File: pmb2_description/urdf/base/base_full.urdf.xacro (robot description, xacro)
@@ -8,79 +8,7 @@
 -->
 <robot xmlns:xacro="http://ros.org/wiki/xacro">
-  <xacro:include filename="$(find pmb2_description)/urdf/deg_to_rad.xacro"/>
-  <xacro:include filename="$(find pmb2_description)/urdf/wheels/wheel.urdf.xacro"/>
-  <xacro:include filename="$(find pmb2_description)/urdf/wheels/caster.urdf.xacro"/>
+  <xacro:include filename="$(find pmb2_description)/urdf/base/base_default.urdf.xacro"/>
   <xacro:include filename="$(find pmb2_description)/urdf/sensors/range.urdf.xacro"/>
-  <xacro:include filename="$(find pmb2_description)/urdf/sensors/hokuyo_urg_04lx_ug01_laser.urdf.xacro"/>
-  <xacro:include filename="$(find pmb2_description)/urdf/sensors/imu.urdf.xacro"/>
-  <xacro:include filename="$(find pmb2_description)/urdf/sensors/microphone.urdf.xacro"/>
-  <xacro:include filename="$(find pmb2_description)/urdf/objects/cover.urdf.xacro"/>
-  <xacro:include filename="$(find pmb2_description)/urdf/objects/antenna.urdf.xacro"/>
-  <!-- Wheel characteristics -->
-  <property name="wheel_radius"     value="0.0985"/>
-  <property name="wheel_width"      value="0.040"/>
-  <property name="wheel_separation" value="0.4044"/>
-  <property name="wheel_torque"     value="6.0"/>
-  <property name="wheel_velocity"   value="1.0"/>
-  <!-- Caster wheel characteristics -->
-  <property name="caster_radius"       value="0.025"/>
-  <property name="caster_width"        value="0.015"/>
-  <property name="caster_separation_x" value="0.343"/>
-  <property name="caster_separation_y" value="0.204"/>
-  <property name="caster_offset_x"     value="-0.002"/>
-  <property name="caster_offset_y"     value="0.0"/>
-  <property name="caster_offset_z"     value="-0.0335"/>
-  <!-- Laser characteristics -->
-  <property name="base_laser_x" value="0.202"/>
-  <property name="base_laser_y" value="0.0"/>
-  <property name="base_laser_z" value="-0.004"/>
-  <xacro:macro name="base" params="name">
-    <!-- Base -->
-    <link name="${name}_link">
-      <inertial>
-        <origin xyz="-0.00000106 0.00000109 0.0000387" rpy="0 0 0"/>
-        <mass value="28.26649"/>
-        <inertia ixx="0.465408937" ixy="0.002160024" ixz="-0.001760255"
-                 iyy="0.483193291" iyz="-0.000655952"
-                 izz="0.550939703"/>
-      </inertial>
-      <visual>
-        <origin xyz="0 0 0" rpy="0 0 0" />
-        <geometry>
-          <mesh filename="package://pmb2_description/meshes/base/base.stl" />
-        </geometry>
-        <material name="White" />
-      </visual>
-      <collision>
-        <origin xyz="0 0 0" rpy="0 0 0" />
-        <geometry>
-          <mesh filename="package://pmb2_description/meshes/base/base_collision.stl" />
-        </geometry>
-        <material name="White" />
-      </collision>
-    </link>
-    <gazebo reference="${name}_link">
-      <material>Gazebo/White</material>
-    </gazebo>
-    <!-- Base footprint -->
-    <link name="${name}_footprint"/>
-    <joint name="${name}_footprint_joint" type="fixed">
-      <origin xyz="0 0 ${wheel_radius}" rpy="0 0 0" />
-      <child link="${name}_link" />
-      <parent link="${name}_footprint"/>
-    </joint>
-    <!-- Orange cover & antennas -->
-    <xacro:cover name="${name}_cover" parent="${name}_footprint"/>
-    <xacro:antenna name="${name}_antenna_left" parent="${name}_link">
-      <origin xyz="-0.201 0.1062 0.195" rpy="0 0 0"/>
-    </xacro:antenna>
-    <xacro:antenna name="${name}_antenna_right" parent="${name}_link">
-      <origin xyz="-0.201 -0.1062 0.195" rpy="0 0 0"/>
-    </xacro:antenna>
-    <!-- Laser -->
-    <!-- Theoretic FOV = 220 -->
-    <xacro:hokuyo_urg_04lx_ug01_laser name="${name}_laser" parent="${name}" ros_topic="scan" update_rate="10" min_angle="${-110 * deg_to_rad}" max_angle="${110 * deg_to_rad}" >
-      <origin xyz="${base_laser_x} ${base_laser_y} ${base_laser_z}" rpy="0 0 0" />
-    </xacro:hokuyo_urg_04lx_ug01_laser>
+  <xacro:macro name="base_full" params="name laser_sick">
     <!-- Microphones -->
     <xacro:microphone name="${name}_mic_front_left" parent="${name}">
@@ -96,9 +24,4 @@
       <origin xyz="-0.1082 -0.13789 0.195" rpy="0 0 0"/>
     </xacro:microphone>
-    <!-- IMU -->
-    <!-- @todo pmb2_hardware_gazebo needs an IMU!  -->
-    <xacro:imu_sensor name="${name}_imu" parent="${name}_link" update_rate="100.0">
-      <origin xyz="0.10171 0 0.11282" rpy="0 ${180 * deg_to_rad} ${90 * deg_to_rad}"/>
-    </xacro:imu_sensor>
     <!-- Sonars -->
     <xacro:range_sensor name="${name}_sonar_1" parent="${name}" ros_topic="sonar_${name}" update_rate="5" maxRange="0.75" minRange="0.01" fov="0.5" radiation="ultrasound">
@@ -111,12 +34,5 @@
       <origin xyz="-0.183 -0.183 0.173" rpy="0 0 ${225 * deg_to_rad}"/>
     </xacro:range_sensor>
-    <!-- Wheels -->
-    <xacro:wheel side="right" reflect=" 1.0" radius="${wheel_radius}" width="${wheel_width}" torque="${wheel_torque}" velocity="${wheel_velocity}" separation="${wheel_separation}" parent="${name}"/>
-    <xacro:wheel side="left"  reflect="-1.0" radius="${wheel_radius}" width="${wheel_width}" torque="${wheel_torque}" velocity="${wheel_velocity}" separation="${wheel_separation}" parent="${name}"/>
-    <!-- Casters wheels -->
-    <xacro:caster side="front_right" radius="${caster_radius}" width="${caster_width}" separation_x="${ caster_separation_x}" separation_y="${ caster_separation_y}" offset_x="${caster_offset_x}" offset_y="${caster_offset_y}" offset_z="${caster_offset_z}" parent="${name}"/>
-    <xacro:caster side="front_left"  radius="${caster_radius}" width="${caster_width}" separation_x="${ caster_separation_x}" separation_y="${-caster_separation_y}" offset_x="${caster_offset_x}" offset_y="${caster_offset_y}" offset_z="${caster_offset_z}" parent="${name}"/>
-    <xacro:caster side="back_right"  radius="${caster_radius}" width="${caster_width}" separation_x="${-caster_separation_x}" separation_y="${ caster_separation_y}" offset_x="${caster_offset_x}" offset_y="${caster_offset_y}" offset_z="${caster_offset_z}" parent="${name}"/>
-    <xacro:caster side="back_left"   radius="${caster_radius}" width="${caster_width}" separation_x="${-caster_separation_x}" separation_y="${-caster_separation_y}" offset_x="${caster_offset_x}" offset_y="${caster_offset_y}" offset_z="${caster_offset_z}" parent="${name}"/>
+    <xacro:base_default name="${name}" laser_sick="${laser_sick}"/>
   </xacro:macro>
 </robot>
