Commit message: Parametrize urdf

File: pmb2_description/robots/pmb2.urdf.xacro (robot description, xacro)
@@ -9,4 +9,5 @@
 <robot  xmlns:xacro="http://ros.org/wiki/xacro"
         name="pmb2" >
+  <xacro:arg name="laser_model" default="sick-571"/> <!-- false, hokuyo, sick-551, sick-561, sick-571-->
   <!-- The following included files set up definitions of parts of the robot body -->
   <!-- Base -->
@@ -17,4 +18,4 @@
   <xacro:include filename="$(find pmb2_description)/urdf/materials.urdf.xacro" />
   <!-- Now we can start using the macros included above to define the actual robot -->
-  <xacro:base_sensors name="base" hokuyo="true"/>
+  <xacro:base_sensors name="base" laser_model="$(arg laser_model)"/>
 </robot>

File: pmb2_description/urdf/base/base_sensors.urdf.xacro (robot description, xacro)
@@ -19,6 +19,7 @@
   <xacro:property name="base_laser_y" value="0.0"/>
   <xacro:property name="base_laser_z" value="-0.004"/>
-  <xacro:macro name="base_sensors" params=" name hokuyo:=false sick551:=false sick561:=false sick571:=false sonars:=false microphone:=false ">
-    <xacro:if value="${hokuyo}"> <!-- TODO: find expr that encure only one laser is true -->
+  <!-- laser_model can be: false, hokuyo, sick-551, sick-561, sick-571-->
+  <xacro:macro name="base_sensors" params=" name laser_model:=sick-571 sonars:=false microphone:=false ">
+    <xacro:if value="${laser_model == 'hokuyo'}">
       <!-- Laser -->
       <!-- Theoretic FOV = 220 -->
@@ -27,5 +28,5 @@
       </xacro:hokuyo_urg_04lx_ug01_laser>
     </xacro:if>
-    <xacro:if value="${sick551}">
+    <xacro:if value="${laser_model == 'sick-551'}">
       <!-- Laser -->
       <!-- Theoretic FOV = 220 -->
@@ -34,5 +35,5 @@
       </xacro:sick_tim551_laser>
     </xacro:if>
-    <xacro:if value="${sick561}">
+    <xacro:if value="${laser_model == 'sick-561'}">
       <!-- Laser -->
       <!-- Theoretic FOV = 220 -->
@@ -41,5 +42,5 @@
       </xacro:sick_tim561_laser>
     </xacro:if>
-    <xacro:if value="${sick571}">
+    <xacro:if value="${laser_model == 'sick-571'}">
       <!-- Laser -->
       <!-- Theoretic FOV = 220 -->

Commit message: Change robot parameter name

File: pmb2_description/robots/pmb2.urdf.xacro (robot description, xacro)
@@ -10,4 +10,8 @@
         name="pmb2" >
   <xacro:arg name="laser_model" default="sick-571"/> <!-- false, hokuyo, sick-551, sick-561, sick-571-->
+  <xacro:property name="laser_model" value="$(arg laser_model)" />
+  <xacro:if value="${laser_model not in ['false', 'sick-551', 'sick-561', 'sick-571', 'hokuyo']}">
+    <xacro:wrong_laser_model/>
+  </xacro:if>
   <!-- The following included files set up definitions of parts of the robot body -->
   <!-- Base -->

Commit message: Add rgbd sensors

File: pmb2_description/robots/pmb2.urdf.xacro (robot description, xacro)
@@ -10,5 +10,7 @@
         name="pmb2" >
   <xacro:arg name="laser_model" default="sick-571"/> <!-- false, hokuyo, sick-551, sick-561, sick-571-->
+  <xacro:arg name="rgbd_sensors" default="false"/> <!-- false, true-->
   <xacro:property name="laser_model" value="$(arg laser_model)" />
+  <xacro:property name="rgbd_sensors" value="$(arg rgbd_sensors)"/>
   <xacro:if value="${laser_model not in ['false', 'sick-551', 'sick-561', 'sick-571', 'hokuyo']}">
     <xacro:wrong_laser_model/>
@@ -23,3 +25,8 @@
   <!-- Now we can start using the macros included above to define the actual robot -->
   <xacro:base_sensors name="base" laser_model="$(arg laser_model)"/>
+  <!-- RGBD Sensors -->
+  <xacro:if value="${rgbd_sensors}">
+    <xacro:include filename="$(find pmb2_description)/urdf/cameras_add_on/cameras_add_on.urdf.xacro" />
+    <xacro:cameras_add_on name="cameras_add_on" parent="base_link"/>
+  </xacro:if>
 </robot>

Commit message: All joints now form part of a single ros2_control system

File: pmb2_description/robots/pmb2.urdf.xacro (robot description, xacro)
@@ -25,4 +25,6 @@
   <!-- Generic simulator_gazebo plugins -->
   <xacro:include filename="$(find pmb2_description)/gazebo/gazebo.urdf.xacro" />
+  <!-- ros2_control -->
+  <xacro:include filename="$(find pmb2_description)/ros2_control/ros2_control.urdf.xacro" />
   <!-- Materials for visualization -->
   <xacro:include filename="$(find pmb2_description)/urdf/materials.urdf.xacro" />

File: pmb2_description/urdf/wheels/wheel.ros2_control.xacro (robot description, xacro)
@@ -1,5 +1,5 @@
 <?xml version="1.0"?>
 <!--
-  Copyright (c) 2011-2020, PAL Robotics, S.L.
+  Copyright (c) 2011-2021, PAL Robotics, S.L.
   All rights reserved.
   This work is licensed under the Creative Commons Attribution-NonCommercial-NoDerivs 3.0 Unported License.
@@ -8,28 +8,22 @@
 -->
 <robot xmlns:xacro="http://ros.org/wiki/xacro">
-  <!-- Wheel Joint -->
-  <xacro:macro name="wheel_ros2_control" params="side">
-    <ros2_control name="${name}" type="system">
-      <hardware>
-        <plugin>gazebo_ros2_control/GazeboSystem</plugin>
-      </hardware>
+  <xacro:macro name="ros2_control_wheel" params="side">
+    <joint name="wheel_${side}_joint">
+      <command_interface name="velocity">
+        <param name="min">-1</param>
+        <param name="max">1</param>
+      </command_interface>
+      <state_interface name="position" />
+    </joint>
+    <transmission name="wheel_${side}_trans">
+      <type>transmission_interface/SimpleTransmission</type>
+      <actuator name="wheel_${side}_motor">
+        <mechanicalReduction>1.0</mechanicalReduction>
+      </actuator>
       <joint name="wheel_${side}_joint">
-        <command_interface name="velocity">
-          <param name="min">-1</param>
-          <param name="max">1</param>
-        </command_interface>
-        <state_interface name="position" />
+        <hardwareInterface>hardware_interface/VelocityJointInterface</hardwareInterface>
+        <hardwareInterface>hardware_interface/JointStateInterface</hardwareInterface>
       </joint>
-      <transmission name="wheel_${side}_trans">
-        <type>transmission_interface/SimpleTransmission</type>
-        <actuator name="wheel_${side}_motor">
-          <mechanicalReduction>1.0</mechanicalReduction>
-        </actuator>
-        <joint name="wheel_${side}_joint">
-          <hardwareInterface>hardware_interface/VelocityJointInterface</hardwareInterface>
-          <hardwareInterface>hardware_interface/JointStateInterface</hardwareInterface>
-        </joint>
-      </transmission>
-    </ros2_control>
+    </transmission>
   </xacro:macro>
 </robot>

File: pmb2_description/urdf/wheels/wheel.urdf.xacro (robot description, xacro)
@@ -10,5 +10,4 @@
   <xacro:include filename="$(find pmb2_description)/urdf/wheels/wheel.transmission.xacro"/>
   <xacro:include filename="$(find pmb2_description)/urdf/wheels/wheel.gazebo.xacro"/>
-  <xacro:include filename="$(find pmb2_description)/urdf/wheels/wheel.ros2_control.xacro"/>
   <xacro:macro name="wheel" params="side reflect radius width torque velocity separation parent">
     <link name="wheel_${side}_link">
@@ -65,6 +64,4 @@
           <limit effort="${torque}" velocity="${velocity / radius}"/>
         </joint>
-        <!-- ROS2 Control -->
-	<xacro:wheel_ros2_control side="${side}"/>
         <!-- Gazebo extensions -->
         <xacro:wheel_gazebo side="${side}"/>

Commit message: No laser value is 'no-laser', change rgbd_sensors to courier_rgbd_sensors

File: pmb2_description/robots/pmb2.urdf.xacro (robot description, xacro)
@@ -9,9 +9,9 @@
 <robot  xmlns:xacro="http://ros.org/wiki/xacro"
         name="pmb2" >
-  <xacro:arg name="laser_model" default="sick-571"/> <!-- false, hokuyo, sick-551, sick-561, sick-571-->
-  <xacro:arg name="rgbd_sensors" default="false"/> <!-- false, true-->
+  <xacro:arg name="laser_model" default="sick-571"/> <!-- no-laser, hokuyo, sick-551, sick-561, sick-571-->
+  <xacro:arg name="courier_rgbd_sensors" default="false"/> <!-- false, true-->
   <xacro:property name="laser_model" value="$(arg laser_model)" />
-  <xacro:property name="rgbd_sensors" value="$(arg rgbd_sensors)"/>
-  <xacro:if value="${laser_model not in ['false', False, 'sick-551', 'sick-561', 'sick-571', 'hokuyo']}">
+  <xacro:property name="courier_rgbd_sensors" value="$(arg courier_rgbd_sensors)"/>
+  <xacro:if value="${laser_model not in ['no-laser', 'sick-551', 'sick-561', 'sick-571', 'hokuyo']}">
     <xacro:wrong_laser_model/>
   </xacro:if>
@@ -32,5 +32,5 @@
   <xacro:base_sensors name="base" laser_model="$(arg laser_model)" sonars="true"/>
   <!-- RGBD Sensors -->
-  <xacro:if value="${rgbd_sensors}">
+  <xacro:if value="${courier_rgbd_sensors}">
     <xacro:include filename="$(find pmb2_description)/urdf/cameras_add_on/cameras_add_on.urdf.xacro" />
     <xacro:cameras_add_on name="cameras_add_on" parent="base_link"/>

Commit message: robot control plugin if no simulation

File: pmb2_description/robots/pmb2.urdf.xacro (robot description, xacro)
@@ -9,4 +9,5 @@
 <robot  xmlns:xacro="http://ros.org/wiki/xacro"
         name="pmb2" >
+  <xacro:arg name="use_sim" default="true"/>
   <xacro:arg name="laser_model" default="sick-571"/> <!-- no-laser, hokuyo, sick-551, sick-561, sick-571-->
   <xacro:arg name="courier_rgbd_sensors" default="false"/> <!-- false, true-->
@@ -27,4 +28,6 @@
   <!-- ros2_control -->
   <xacro:include filename="$(find pmb2_description)/ros2_control/ros2_control.urdf.xacro" />
+  <xacro:pmb2_ros2_control
+    use_sim="$(arg use_sim)" />
   <!-- Materials for visualization -->
   <xacro:include filename="$(find pmb2_description)/urdf/materials.urdf.xacro" />

File: pmb2_description/ros2_control/ros2_control.urdf.xacro (robot description, xacro)
@@ -9,14 +9,23 @@
 <robot xmlns:xacro="http://ros.org/wiki/xacro"
        name="pmb2" >
-  <xacro:include filename="$(find pmb2_description)/urdf/wheels/wheel.ros2_control.xacro"/>
-  <xacro:include filename="$(find pmb2_description)/urdf/sensors/sensors.ros2_control.xacro"/>
-  <ros2_control name="ros2_control_pmb2_system" type="system">
-    <hardware>
-      <plugin>gazebo_ros2_control/GazeboSystem</plugin>
-    </hardware>
-    <!-- wheels -->
-    <xacro:ros2_control_wheel side="right" />
-    <xacro:ros2_control_wheel side="left" />
-    <xacro:ros2_control_imu name="base_imu_sensor"/>
-  </ros2_control>
+<xacro:macro name="pmb2_ros2_control" params="use_sim:=^|true">
+    <xacro:include filename="$(find pmb2_description)/urdf/wheels/wheel.ros2_control.xacro"/>
+    <xacro:include filename="$(find pmb2_description)/urdf/sensors/sensors.ros2_control.xacro"/>
+    <ros2_control name="ros2_control_pmb2_system" type="system">
+      <xacro:if value="$(arg use_sim)">
+        <xacro:ros2_control_imu name="base_imu_sensor"/>
+        <hardware>
+          <plugin>gazebo_ros2_control/GazeboSystem</plugin>
+        </hardware>
+      </xacro:if>
+      <xacro:unless value="$(arg use_sim)">
+        <hardware>
+          <plugin>robot_control/RobotControl</plugin>
+        </hardware>
+      </xacro:unless>
+      <!-- wheels -->
+      <xacro:ros2_control_wheel side="right" />
+      <xacro:ros2_control_wheel side="left" />
+    </ros2_control>
+  </xacro:macro>
 </robot>

Commit message: added ydlidar

File: pmb2_description/robots/pmb2.urdf.xacro (robot description, xacro)
@@ -18,5 +18,5 @@
   <xacro:property name="laser_model" value="$(arg laser_model)" />
   <xacro:property name="rgbd_sensors" value="$(arg rgbd_sensors)"/>
-  <xacro:if value="${laser_model not in ['false', False, 'sick-551', 'sick-561', 'sick-571', 'hokuyo']}">
+  <xacro:if value="${laser_model not in ['false', False, 'sick-551', 'sick-561', 'sick-571', 'hokuyo', 'ydlidar-tg30', 'ydlidar-tg15']}">
     <xacro:wrong_laser_model/>
   </xacro:if>

File: pmb2_description/urdf/base/base_sensors.urdf.xacro (robot description, xacro)
@@ -18,4 +18,6 @@
   <xacro:include filename="$(find pmb2_description)/urdf/sensors/sick_tim561_laser.urdf.xacro"/>
   <xacro:include filename="$(find pmb2_description)/urdf/sensors/sick_tim571_laser.urdf.xacro"/>
+  <xacro:include filename="$(find pmb2_description)/urdf/sensors/ydlidar_tg30_laser.urdf.xacro"/>
+  <xacro:include filename="$(find pmb2_description)/urdf/sensors/ydlidar_tg15_laser.urdf.xacro"/>
   <xacro:include filename="$(find pmb2_description)/urdf/sensors/range.urdf.xacro"/>
   <xacro:include filename="$(find pmb2_description)/urdf/sensors/microphone.urdf.xacro"/>
@@ -54,4 +56,18 @@
       </xacro:sick_tim571_laser>
     </xacro:if>
+    <xacro:if value="${laser_model == 'ydlidar-tg30'}">
+      <!-- Laser -->
+      <!-- Theoretic FOV = 360 -->
+      <xacro:ydlidar_tg30_laser name="${name}_laser" parent="${name}" ros_topic="scan_raw" update_rate="10" min_angle="${-180 * deg_to_rad}" max_angle="${180 * deg_to_rad}" >
+        <origin xyz="${base_laser_x} ${base_laser_y} ${base_laser_z}" rpy="0 0 ${ 180 * deg_to_rad }" />
+      </xacro:ydlidar_tg30_laser>
+    </xacro:if>
+    <xacro:if value="${laser_model == 'ydlidar-tg15'}">
+      <!-- Laser -->
+      <!-- Theoretic FOV = 360 -->
+      <xacro:ydlidar_tg15_laser name="${name}_laser" parent="${name}" ros_topic="scan_raw" update_rate="10" min_angle="${-180 * deg_to_rad}" max_angle="${180 * deg_to_rad}" >
+        <origin xyz="${base_laser_x} ${base_laser_y} ${base_laser_z}" rpy="0 0 ${ 180 * deg_to_rad }" />
+      </xacro:ydlidar_tg15_laser>
+    </xacro:if>
     <xacro:if value="${sonars}">
       <!-- Sonars -->

Commit message: Use urdf_utils

File: pmb2_description/robots/pmb2.urdf.xacro (robot description, xacro)
@@ -26,4 +26,6 @@
   <xacro:property name="nsp" value="$(arg namespace)" />
   <!-- The following included files set up definitions of parts of the robot body -->
+  <!--File includes-->
+  <xacro:include filename="$(find pal_urdf_utils)/urdf/deg_to_rad.xacro" />
   <!-- Base -->
   <xacro:include filename="$(find pmb2_description)/urdf/base/base_sensors.urdf.xacro" />
@@ -31,5 +33,5 @@
   <xacro:include filename="$(find pmb2_description)/gazebo/gazebo.urdf.xacro" />
   <!-- Materials for visualization -->
-  <xacro:include filename="$(find pmb2_description)/urdf/materials.urdf.xacro" />
+  <xacro:include filename="$(find pal_urdf_utils)/urdf/materials.urdf.xacro" />
   <!-- Now we can start using the macros included above to define the actual robot -->
   <xacro:base_sensors name="base" laser_model="$(arg laser_model)" sonars="true"/>

File: pmb2_description/urdf/base/base.urdf.xacro (robot description, xacro)
@@ -13,5 +13,4 @@
 -->
 <robot xmlns:xacro="http://ros.org/wiki/xacro">
-  <xacro:include filename="$(find pmb2_description)/urdf/deg_to_rad.xacro"/>
   <xacro:include filename="$(find pmb2_description)/urdf/wheels/wheel.urdf.xacro"/>
   <xacro:include filename="$(find pmb2_description)/urdf/wheels/caster.urdf.xacro"/>

File: pmb2_description/urdf/cameras_add_on/cameras_add_on.urdf.xacro (robot description, xacro)
@@ -13,6 +13,4 @@
 -->
 <robot xmlns:xacro="http://ros.org/wiki/xacro">
-  <!--File includes-->
-  <xacro:include filename="$(find pmb2_description)/urdf/deg_to_rad.xacro" />
   <xacro:macro name="cameras_add_on" params="name parent">
     <link name="${name}_link">

File: pmb2_description/urdf/dock/dock.urdf.xacro (robot description, xacro)
@@ -13,5 +13,4 @@
 -->
 <robot xmlns:xacro="http://ros.org/wiki/xacro">
-  <xacro:include filename="$(find pmb2_description)/urdf/deg_to_rad.xacro"/>
   <xacro:include filename="$(find pmb2_description)/urdf/sensors/ir_emitter.urdf.xacro"/>
   <xacro:macro name="dock" params="name">

File: pmb2_description/urdf/sensors/hokuyo_urg_04lx_ug01_laser.urdf.xacro (robot description, xacro)
@@ -30,4 +30,10 @@
         <material name="DarkGrey"/>
       </visual>
+      <collision>
+        <origin xyz="0 0 0" rpy="0 0 0" />
+        <geometry>
+          <cylinder radius="0.02" length="0.04"/>
+        </geometry>
+      </collision>
     </link>
     <joint name="${name}_joint" type="fixed">

File: pmb2_description/urdf/sensors/sick_tim551_laser.urdf.xacro (robot description, xacro)
@@ -30,4 +30,10 @@
         <material name="DarkGrey"/>
       </visual>
+      <collision>
+        <origin xyz="0 0 0" rpy="0 0 0" />
+        <geometry>
+          <cylinder radius="0.02" length="0.04"/>
+        </geometry>
+      </collision>
     </link>
     <joint name="${name}_joint" type="fixed">

File: pmb2_description/urdf/sensors/sick_tim561_laser.urdf.xacro (robot description, xacro)
@@ -30,4 +30,10 @@
         <material name="DarkGrey"/>
       </visual>
+      <collision>
+        <origin xyz="0 0 0" rpy="0 0 0" />
+        <geometry>
+          <cylinder radius="0.02" length="0.04"/>
+        </geometry>
+      </collision>
     </link>
     <joint name="${name}_joint" type="fixed">

File: pmb2_description/urdf/sensors/sick_tim571_laser.urdf.xacro (robot description, xacro)
@@ -30,4 +30,10 @@
         <material name="DarkGrey"/>
       </visual>
+      <collision>
+        <origin xyz="0 0 0" rpy="0 0 0" />
+        <geometry>
+          <cylinder radius="0.02" length="0.04"/>
+        </geometry>
+      </collision>
     </link>
     <joint name="${name}_joint" type="fixed">

File: pmb2_description/urdf/sensors/ydlidar_tg15_laser.urdf.xacro (robot description, xacro)
@@ -25,4 +25,10 @@
         <material name="DarkGrey"/>
       </visual>
+      <collision>
+        <origin xyz="0 0 0" rpy="0 0 0" />
+        <geometry>
+          <cylinder radius="0.02" length="0.04"/>
+        </geometry>
+      </collision>
     </link>
     <joint name="${name}_joint" type="fixed">

File: pmb2_description/urdf/sensors/ydlidar_tg30_laser.urdf.xacro (robot description, xacro)
@@ -25,4 +25,10 @@
         <material name="DarkGrey"/>
       </visual>
+      <collision>
+        <origin xyz="0 0 0" rpy="0 0 0" />
+        <geometry>
+          <cylinder radius="0.02" length="0.04"/>
+        </geometry>
+      </collision>
     </link>
     <joint name="${name}_joint" type="fixed">

Commit message: support camera_model argument

File: pmb2_description/robots/pmb2.urdf.xacro (robot description, xacro)
@@ -22,4 +22,6 @@
   <!-- false, true-->
   <xacro:arg name="add_on_module" default="no-add-on"/>
+  <!-- no-camera, orbbec-astra, orbbec-astra-pro, asus-xtion -->
+  <xacro:arg name="camera_model" default="no-camera"/>
   <!-- Execution env config -->
   <xacro:arg name="use_sim_time" default="false"/>
@@ -33,4 +35,5 @@
   <xacro:property name="has_microphone" value="$(arg has_microphone)" />
   <xacro:property name="add_on_module" value="$(arg add_on_module)"/>
+  <xacro:property name="camera_model" value="$(arg camera_model)" />
   <!-- HW configuration check -->
   <xacro:if value="${laser_model not in ['no-laser', 'sick-551', 'sick-561', 'sick-571', 'hokuyo']}">
@@ -39,4 +42,7 @@
   <xacro:if value="${add_on_module not in ['no-add-on', 'cobra']}">
     <xacro:wrong_add_on_module/>
+  </xacro:if>
+  <xacro:if value="${camera_model not in ['no-camera', 'structure']}">
+    <xacro:wrong_camera_model/>
   </xacro:if>
   <!-- Execution env configuration -->

File: pmb2_description/urdf/sensors/courier.urdf.xacro (robot description, xacro)
@@ -37,25 +37,27 @@
   <xacro:property name="rgb_P" value="15.0"/>
   <xacro:property name="rgb_Y" value="0.0   "/>
-  <!-- RGBD base -->
-  <xacro:structure_sensor name="base_rgbd_camera" parent="base_link">
-    <!-- Pose of sensor frame wrt to base -->
-    <origin xyz="${base_rgbd_x} ${base_rgbd_y} ${base_rgbd_z}" rpy="${base_rgbd_R * deg_to_rad} ${base_rgbd_P * deg_to_rad} ${base_rgbd_Y * deg_to_rad}"/>
-    <!-- Pose of optical frame wrt to sensor -->
-    <origin xyz="0 0 0" rpy="${-90 * deg_to_rad} 0 ${-90 * deg_to_rad}"/>
-  </xacro:structure_sensor>
-  <!-- RGBD roof -->
-  <xacro:structure_sensor name="roof_rgbd_camera" parent="base_link">
-    <!-- Pose of sensor frame wrt to base -->
-    <origin xyz="${roof_rgbd_x} ${roof_rgbd_y} ${roof_rgbd_z}" rpy="${roof_rgbd_R * deg_to_rad} ${roof_rgbd_P * deg_to_rad} ${roof_rgbd_Y * deg_to_rad}"/>
-    <!-- Pose of optical frame wrt to sensor -->
-    <origin xyz="0 0 0" rpy="${-90 * deg_to_rad} 0 ${-90 * deg_to_rad}"/>
-  </xacro:structure_sensor>
-  <!-- RGB -->
-  <xacro:elp_rgb name="rgb_camera" parent="base_link">
-    <!-- Pose of sensor frame wrt to base -->
-    <origin xyz="${rgb_x} ${rgb_y} ${rgb_z}" rpy="${rgb_R * deg_to_rad} ${rgb_P * deg_to_rad} ${rgb_Y * deg_to_rad}"/>
-    <!-- Pose of optical frame wrt to sensor -->
-    <origin xyz="0 0 0" rpy="${-90 * deg_to_rad} 0 ${-90 * deg_to_rad}"/>
-  </xacro:elp_rgb>
+  <xacro:if value="${camera_model == 'structure'}">
+    <!-- RGBD base -->
+    <xacro:structure_sensor name="base_rgbd_camera" parent="base_link">
+      <!-- Pose of sensor frame wrt to base -->
+      <origin xyz="${base_rgbd_x} ${base_rgbd_y} ${base_rgbd_z}" rpy="${base_rgbd_R * deg_to_rad} ${base_rgbd_P * deg_to_rad} ${base_rgbd_Y * deg_to_rad}"/>
+      <!-- Pose of optical frame wrt to sensor -->
+      <origin xyz="0 0 0" rpy="${-90 * deg_to_rad} 0 ${-90 * deg_to_rad}"/>
+    </xacro:structure_sensor>
+    <!-- RGBD roof -->
+    <xacro:structure_sensor name="roof_rgbd_camera" parent="base_link">
+      <!-- Pose of sensor frame wrt to base -->
+      <origin xyz="${roof_rgbd_x} ${roof_rgbd_y} ${roof_rgbd_z}" rpy="${roof_rgbd_R * deg_to_rad} ${roof_rgbd_P * deg_to_rad} ${roof_rgbd_Y * deg_to_rad}"/>
+      <!-- Pose of optical frame wrt to sensor -->
+      <origin xyz="0 0 0" rpy="${-90 * deg_to_rad} 0 ${-90 * deg_to_rad}"/>
+    </xacro:structure_sensor>
+    <!-- RGB -->
+    <xacro:elp_rgb name="rgb_camera" parent="base_link">
+      <!-- Pose of sensor frame wrt to base -->
+      <origin xyz="${rgb_x} ${rgb_y} ${rgb_z}" rpy="${rgb_R * deg_to_rad} ${rgb_P * deg_to_rad} ${rgb_Y * deg_to_rad}"/>
+      <!-- Pose of optical frame wrt to sensor -->
+      <origin xyz="0 0 0" rpy="${-90 * deg_to_rad} 0 ${-90 * deg_to_rad}"/>
+    </xacro:elp_rgb>
+  </xacro:if>
   <!-- RGBD Laser Link -->
   <joint name="rgbd_laser_joint" type="fixed">
