Commit message: integrating ydlidar in urdf

File: pmb2_description/robots/pmb2.urdf.xacro (robot description, xacro)
@@ -14,5 +14,5 @@
 <robot xmlns:xacro="http://ros.org/wiki/xacro" name="pmb2">
   <!-- ARGUMENTS -->
-  <!-- no-laser, hokuyo, sick-551, sick-561, sick-571-->
+  <!-- no-laser, hokuyo, sick-551, sick-561, sick-571, ydlidar-tg30 -->
   <xacro:arg name="laser_model" default="sick-571"/>
   <!-- false, true -->
@@ -37,5 +37,5 @@
   <xacro:property name="camera_model" value="$(arg camera_model)" />
   <!-- HW configuration check -->
-  <xacro:if value="${laser_model not in ['no-laser', 'sick-551', 'sick-561', 'sick-571', 'hokuyo']}">
+  <xacro:if value="${laser_model not in ['no-laser', 'sick-551', 'sick-561', 'sick-571', 'hokuyo', 'ydlidar-tg30']}">
     <xacro:wrong_laser_model/>
   </xacro:if>

File: pmb2_description/urdf/base/base_sensors.urdf.xacro (robot description, xacro)
@@ -24,4 +24,5 @@
   <xacro:include filename="$(find pal_urdf_utils)/urdf/laser/sick_tim561_laser.urdf.xacro"/>
   <xacro:include filename="$(find pal_urdf_utils)/urdf/laser/sick_tim571_laser.urdf.xacro"/>
+  <xacro:include filename="$(find pal_urdf_utils)/urdf/laser/ydlidar_tg30_laser.urdf.xacro"/>
   <xacro:include filename="$(find pal_urdf_utils)/urdf/laser/range.urdf.xacro"/>
   <xacro:include filename="$(find pal_urdf_utils)/urdf/interaction_sensors/microphone.urdf.xacro"/>
@@ -60,4 +61,10 @@
         <origin xyz="${base_laser_x} ${base_laser_y} ${base_laser_z}" rpy="0 0 0" />
       </xacro:sick_tim571_laser>
+    </xacro:if>
+    <!-- 2D LIDAR: YDLIDAR TG30 -->
+    <xacro:if value="${laser_model == 'ydlidar-tg30'}">
+      <xacro:ydlidar_tg30_laser name="${name}_laser" parent="${name}_link" ros_topic="scan_raw" update_rate="10" min_angle="${-110 * deg_to_rad}" max_angle="${110 * deg_to_rad}" >
+        <origin xyz="${base_laser_x} ${base_laser_y} ${base_laser_z}" rpy="0 0 0" />
+      </xacro:ydlidar_tg30_laser>
     </xacro:if>
     <!-- Sonars -->
