Commit message: rm usuless caster 1 collision mesh

File: pmb2_description/urdf/wheels/caster.urdf.xacro (robot description, xacro)
@@ -25,10 +25,10 @@
         <material name="Grey"/>
       </visual>
-      <collision>
+      <!--collision>
         <origin xyz="0 0 0" rpy="0 0 0"/>
         <geometry>
           <cylinder radius="${radius}" length="${width}"/>
         </geometry>
-      </collision>
+      </collision-->
     </link>
     <link name="caster_${side}_2_link">
