Commit message: Fix color of wheels in gazebo

File: pmb2_description/urdf/wheels/caster.gazebo.xacro (robot description, xacro)
@@ -29,4 +29,5 @@
       <minDepth>0.00</minDepth>
       <implicitSpringDamper>1</implicitSpringDamper>
+      <material>Gazebo/DarkGrey</material>
     </gazebo>
   </xacro:macro>

File: pmb2_description/urdf/wheels/wheel.gazebo.xacro (robot description, xacro)
@@ -19,4 +19,5 @@
       <minDepth>0.00</minDepth>
       <implicitSpringDamper>1</implicitSpringDamper>
+      <material>Gazebo/DarkGrey</material>
     </gazebo>
   </xacro:macro>

Commit message: Replace caster collision with spheres, fix spinning

File: pmb2_description/urdf/wheels/caster.gazebo.xacro (robot description, xacro)
@@ -13,6 +13,6 @@
       <kp>1000000.0</kp>
       <kd>100.0</kd>
-      <mu1>1.0</mu1>
-      <mu2>1.0</mu2>
+      <mu1>0</mu1>
+      <mu2>0</mu2>
       <fdir1>1 0 0</fdir1>
       <maxVel>1.0</maxVel>
@@ -23,6 +23,6 @@
       <kp>1000000.0</kp>
       <kd>100.0</kd>
-      <mu1>1.0</mu1>
-      <mu2>1.0</mu2>
+      <mu1>0</mu1>
+      <mu2>0</mu2>
       <fdir1>1 0 0</fdir1>
       <maxVel>1.0</maxVel>

File: pmb2_description/urdf/wheels/caster.urdf.xacro (robot description, xacro)
@@ -45,17 +45,9 @@
         <origin xyz="0 0 0" rpy="0 0 0"/>
         <geometry>
-          <cylinder radius="${radius}" length="${width}"/>
+          <sphere radius="${radius}"/>
         </geometry>
-        <surface>
-          <friction>
-            <ode>
-              <mu> 0.01</mu>
-              <mu2>0.01</mu2>
-            </ode>
-          </friction>
-        </surface>
       </collision>
     </link>
-    <joint name="caster_${side}_1_joint" type="continuous">
+    <joint name="caster_${side}_1_joint" type="fixed">
       <parent link="${parent}_link"/>
       <child link="caster_${side}_1_link"/>
@@ -63,5 +55,5 @@
       <axis xyz="0 0 1"/>
     </joint>
-    <joint name="caster_${side}_2_joint" type="continuous">
+    <joint name="caster_${side}_2_joint" type="fixed">
       <parent link="caster_${side}_1_link"/>
       <child link="caster_${side}_2_link"/>

File: pmb2_description/urdf/wheels/wheel.gazebo.xacro (robot description, xacro)
@@ -11,4 +11,5 @@
     <!-- Contact model for the wheel surface -->
     <gazebo reference="wheel_${side}_link">
+<!--
       <kp>1000000.0</kp>
       <kd>100.0</kd>
@@ -19,4 +20,5 @@
       <minDepth>0.00</minDepth>
       <implicitSpringDamper>1</implicitSpringDamper>
+-->
       <material>Gazebo/DarkGrey</material>
     </gazebo>

Commit message: virtual suspension and rolling caster wheels

File: pmb2_description/urdf/wheels/caster.gazebo.xacro (robot description, xacro)
@@ -13,6 +13,6 @@
       <kp>1000000.0</kp>
       <kd>1000.0</kd>
-      <mu1>0.3</mu1>
-      <mu2>0.3</mu2>
+      <mu1>0.0</mu1>
+      <mu2>0.0</mu2>
       <fdir1>1 0 0</fdir1>
       <maxVel>1.0</maxVel>
@@ -23,6 +23,6 @@
       <kp>1000000.0</kp>
       <kd>1000.0</kd>
-      <mu1>0.3</mu1>
-      <mu2>0.3</mu2>
+      <mu1>0.0</mu1>
+      <mu2>0.0</mu2>
       <fdir1>1 0 0</fdir1>
       <maxVel>1.0</maxVel>

File: pmb2_description/urdf/wheels/caster.urdf.xacro (robot description, xacro)
@@ -55,5 +55,5 @@
       </collision>
     </link>
-    <joint name="caster_${side}_1_joint" type="fixed">
+    <joint name="caster_${side}_1_joint" type="continuous">
       <parent link="${parent}_link"/>
       <child link="caster_${side}_1_link"/>
@@ -61,5 +61,5 @@
       <axis xyz="0 0 1"/>
     </joint>
-    <joint name="caster_${side}_2_joint" type="fixed">
+    <joint name="caster_${side}_2_joint" type="continuous">
       <parent link="caster_${side}_1_link"/>
       <child link="caster_${side}_2_link"/>
@@ -69,4 +69,7 @@
     <!-- Gazebo extensions -->
     <xacro:caster_gazebo side="${side}"/>
+    <!-- Transmission -->
+    <xacro:caster_transmission name="caster_" side="${side}" number="1" reduction="1.0"/>
+    <xacro:caster_transmission name="caster_" side="${side}" number="2" reduction="1.0"/>
   </xacro:macro>
 </robot>

File: pmb2_description/urdf/wheels/wheel.urdf.xacro (robot description, xacro)
@@ -1,13 +1,14 @@
 <?xml version="1.0"?>
 <!--
-  Copyright (c) 2014, PAL Robotics, S.L.
-  All rights reserved.
-  This work is licensed under the Creative Commons Attribution-NonCommercial-NoDerivs 3.0 Unported License.
-  To view a copy of this license, visit http://creativecommons.org/licenses/by-nc-nd/3.0/ or send a letter to
-  Creative Commons, 444 Castro Street, Suite 900, Mountain View, California, 94041, USA.
+Copyright (c) 2014, PAL Robotics, S.L.
+All rights reserved.
+This work is licensed under the Creative Commons Attribution-NonCommercial-NoDerivs 3.0 Unported License.
+To view a copy of this license, visit http://creativecommons.org/licenses/by-nc-nd/3.0/ or send a letter to
+Creative Commons, 444 Castro Street, Suite 900, Mountain View, California, 94041, USA.
 -->
 <robot xmlns:xacro="http://ros.org/wiki/xacro">
   <xacro:include filename="$(find pmb2_description)/urdf/wheels/wheel.transmission.xacro"/>
   <xacro:include filename="$(find pmb2_description)/urdf/wheels/wheel.gazebo.xacro"/>
+  <xacro:include filename="$(find pmb2_description)/urdf/wheels/suspension.transmission.xacro"/>
   <xacro:macro name="wheel" params="side reflect radius width torque velocity separation parent">
     <link name="wheel_${side}_link">
@@ -16,32 +17,53 @@
         <mass value="1.82362"/>
         <inertia ixx="0.00499743171" ixy="${ 0.00000004464 * reflect}" ixz="-0.00000002245"
-                 iyy="0.00499741733" iyz="${-0.00000000164 * reflect}"
-                 izz="0.00839239692"/>
-      </inertial>
-      <visual>
-        <origin xyz="0 0 0" rpy="${-90.0 * (1 - reflect) * deg_to_rad} 0 0"/>
-        <geometry>
-          <mesh filename="package://pmb2_description/meshes/wheels/wheel.stl"/>
-        </geometry>
-        <material name="DarkGrey"/>
-      </visual>
-      <collision>
+          iyy="0.00499741733" iyz="${-0.00000000164 * reflect}"
+          izz="0.00839239692"/>
+        </inertial>
+        <visual>
+          <origin xyz="0 0 0" rpy="${-90.0 * (1 - reflect) * deg_to_rad} 0 0"/>
+          <geometry>
+            <mesh filename="package://pmb2_description/meshes/wheels/wheel.stl"/>
+          </geometry>
+          <material name="DarkGrey"/>
+        </visual>
+        <collision>
+          <origin xyz="0 0 0" rpy="0 0 0"/>
+          <geometry>
+            <cylinder radius="${radius}" length="${width}"/>
+          </geometry>
+        </collision>
+      </link>
+      <link name="suspension_${side}_link">
+        <inertial>
+          <origin xyz="0 0 0" rpy="0 0 0"/>
+          <mass value="0.01"/>
+          <inertia ixx="0.01" ixy="0" ixz="0" iyy="0.01" iyz="0" izz="0.01"/>
+        </inertial>
+      </link>
+      <joint name="suspension_${side}_joint" type="prismatic">
         <origin xyz="0 0 0" rpy="0 0 0"/>
-        <geometry>
-          <cylinder radius="${radius}" length="${width}"/>
-        </geometry>
-      </collision>
-    </link>
-    <joint name="wheel_${side}_joint" type="continuous">
-      <parent link="${parent}_link"/>
-      <child link="wheel_${side}_link"/>
-      <origin xyz="0 ${-separation / 2 * reflect} 0" rpy="${-90.0 * deg_to_rad} 0 0"/>
-      <axis xyz="0 0 1"/>
-      <limit effort="${torque}" velocity="${velocity / radius}"/>
-    </joint>
-    <!-- Transmission -->
-    <xacro:wheel_transmission side="${side}"/>
-    <!-- Gazebo extensions -->
-    <xacro:wheel_gazebo side="${side}"/>
-  </xacro:macro>
-</robot>
+        <axis xyz="0 0 1"/>
+        <limit effort="2000.0" lower="-0.02" upper="0.02" velocity="1.0"/>
+        <child link="suspension_${side}_link"/>
+        <parent link="${parent}_link"/>
+        <calibration rising="0.0" />
+        <dynamics damping="1000" />
+        <safety_controller k_position="0"
+          k_velocity="20"
+          soft_lower_limit="-0.02"
+          soft_upper_limit="0.02" />
+        </joint>
+        <joint name="wheel_${side}_joint" type="continuous">
+          <parent link="suspension_${side}_link"/>
+          <child link="wheel_${side}_link"/>
+          <origin xyz="0 ${-separation / 2 * reflect} 0" rpy="${-90.0 * deg_to_rad} 0 0"/>
+          <axis xyz="0 0 1"/>
+          <limit effort="${torque}" velocity="${velocity / radius}"/>
+        </joint>
+        <!-- Transmission -->
+        <xacro:wheel_transmission side="${side}"/>
+        <xacro:suspension_transmission side="${side}"/>
+        <!-- Gazebo extensions -->
+        <xacro:wheel_gazebo side="${side}"/>
+      </xacro:macro>
+    </robot>

Commit message: rotate and climb with a virtual suspension system and use caster wheels

File: pmb2_description/urdf/wheels/caster.gazebo.xacro (robot description, xacro)
@@ -13,6 +13,6 @@
       <kp>1000000.0</kp>
       <kd>1000.0</kd>
-      <mu1>0.0</mu1>
-      <mu2>0.0</mu2>
+      <mu1>0.2</mu1>
+      <mu2>0.2</mu2>
       <fdir1>1 0 0</fdir1>
       <maxVel>1.0</maxVel>
@@ -23,6 +23,6 @@
       <kp>1000000.0</kp>
       <kd>1000.0</kd>
-      <mu1>0.0</mu1>
-      <mu2>0.0</mu2>
+      <mu1>0.2</mu1>
+      <mu2>0.2</mu2>
       <fdir1>1 0 0</fdir1>
       <maxVel>1.0</maxVel>

File: pmb2_description/urdf/wheels/caster.urdf.xacro (robot description, xacro)
@@ -70,6 +70,7 @@
     <xacro:caster_gazebo side="${side}"/>
     <!-- Transmission -->
-    <xacro:caster_transmission name="caster_" side="${side}" number="1" reduction="1.0"/>
+  <!--  <xacro:caster_transmission name="caster_" side="${side}" number="1" reduction="1.0"/>
     <xacro:caster_transmission name="caster_" side="${side}" number="2" reduction="1.0"/>
+-->
   </xacro:macro>
 </robot>

File: pmb2_description/urdf/wheels/wheel.urdf.xacro (robot description, xacro)
@@ -37,5 +37,5 @@
         <inertial>
           <origin xyz="0 0 0" rpy="0 0 0"/>
-          <mass value="0.01"/>
+          <mass value="10"/>
           <inertia ixx="0.01" ixy="0" ixz="0" iyy="0.01" iyz="0" izz="0.01"/>
         </inertial>

Commit message: fix castor joints transmission

File: pmb2_description/urdf/wheels/caster.gazebo.xacro (robot description, xacro)
@@ -19,4 +19,5 @@
       <minDepth>0.0</minDepth>
       <implicitSpringDamper>1</implicitSpringDamper>
+      <material>Gazebo/DarkGrey</material>
     </gazebo>
     <gazebo reference="caster_${side}_2_link">

File: pmb2_description/urdf/wheels/caster.transmission.xacro (robot description, xacro)
@@ -12,8 +12,9 @@
     <transmission name="${name}_${side}_${number}_trans">
       <type>transmission_interface/SimpleTransmission</type>
-      <actuator name="${name}_${side}_${number}_motor" >
+        <actuator name="${name}_${side}_${number}_motor" >
         <mechanicalReduction>${reduction}</mechanicalReduction>
       </actuator>
       <joint name="${name}_${side}_${number}_joint" >
+        <hardwareInterface>hardware_interface/PositionJointInterface</hardwareInterface>
         <hardwareInterface>hardware_interface/JointStateInterface</hardwareInterface>
       </joint>

File: pmb2_description/urdf/wheels/caster.urdf.xacro (robot description, xacro)
@@ -70,7 +70,6 @@
     <xacro:caster_gazebo side="${side}"/>
     <!-- Transmission -->
-  <!--  <xacro:caster_transmission name="caster_" side="${side}" number="1" reduction="1.0"/>
-    <xacro:caster_transmission name="caster_" side="${side}" number="2" reduction="1.0"/>
--->
+   <xacro:caster_transmission name="caster" side="${side}" number="1" reduction="1.0"/>
+   <xacro:caster_transmission name="caster" side="${side}" number="2" reduction="1.0"/>
   </xacro:macro>
 </robot>

Commit message: Additional wheel collision and transmission fixes

File: pmb2_description/urdf/wheels/caster.gazebo.xacro (robot description, xacro)
@@ -15,8 +15,8 @@
       <mu1>1.0</mu1>
       <mu2>1.0</mu2>
-      <fdir1>1 0 0</fdir1>
+      <fdir1>0 0 1</fdir1>
       <maxVel>1.0</maxVel>
-      <minDepth>0.005</minDepth>
-      <implicitSpringDamper>1</implicitSpringDamper>
+      <minDepth>0.0</minDepth>
+      <implicitSpringDamper>0</implicitSpringDamper>
       <material>Gazebo/DarkGrey</material>
     </gazebo>
@@ -24,10 +24,10 @@
       <kp>1000000.0</kp>
       <kd>1000.0</kd>
-      <mu1>1.0</mu1>
-      <mu2>1.0</mu2>
+      <mu1>0.7</mu1>
+      <mu2>0.7</mu2>
       <fdir1>1 0 0</fdir1>
       <maxVel>1.0</maxVel>
-      <minDepth>0.005</minDepth>
-      <implicitSpringDamper>1</implicitSpringDamper>
+      <minDepth>0.00</minDepth>
+      <implicitSpringDamper>0</implicitSpringDamper>
       <material>Gazebo/DarkGrey</material>
     </gazebo>

File: pmb2_description/urdf/wheels/wheel.gazebo.xacro (robot description, xacro)
@@ -13,9 +13,9 @@
       <kp>1000000.0</kp>
       <kd>1000.0</kd>
-      <mu1>1000.0</mu1>
-      <mu2>1000.0</mu2>
+      <mu1>1.0</mu1>
+      <mu2>1.0</mu2>
       <fdir1>1 0 0</fdir1>
-      <maxVel>20.0</maxVel>
-      <minDepth>0.0</minDepth>
+      <maxVel>1.0</maxVel>
+      <minDepth>0.00</minDepth>
       <implicitSpringDamper>1</implicitSpringDamper>
       <material>Gazebo/DarkGrey</material>

File: pmb2_description/urdf/wheels/wheel.urdf.xacro (robot description, xacro)
@@ -37,10 +37,10 @@
         <inertial>
           <origin xyz="0 0 -0.02" rpy="0 0 0"/>
-          <mass value="30"/>
+          <mass value="10"/>
           <inertia ixx="1.0" ixy="0" ixz="0"
                    iyy="1.0" iyz="0"
                    izz="1.0"/>
          </inertial>
-        <kinematic>1</kinematic>
+        <kinematic>0</kinematic>
         <gravity>1</gravity>
       </link>
@@ -48,13 +48,13 @@
         <origin xyz="0 0 0" rpy="0 0 0"/>
         <axis xyz="0 0 1"/>
-        <limit effort="10000.0" lower="-0.04" upper="0.04" velocity="1.0"/>
+        <limit effort="100.0" lower="-0.005" upper="0.005" velocity="1.0"/>
         <child link="suspension_${side}_link"/>
         <parent link="${parent}_link"/>
         <calibration rising="0.0" />
-        <dynamics damping="10000"/>
-        <safety_controller k_position="-0.03"
-          k_velocity="100"
-          soft_lower_limit="-0.05"
-          soft_upper_limit="0.05" />
+        <dynamics damping="100"/>
+        <safety_controller k_position="0"
+          k_velocity="10"
+          soft_lower_limit="-0.005"
+          soft_upper_limit="0.005" />
         </joint>
         <joint name="wheel_${side}_joint" type="continuous">

Commit message: Fix inertial parameters of the caster wheels
Also added friction and damping to improve behavior

File: pmb2_description/urdf/wheels/caster.gazebo.xacro (robot description, xacro)
@@ -24,6 +24,6 @@
       <kp>1000000.0</kp>
       <kd>1000.0</kd>
-      <mu1>0.0</mu1>
-      <mu2>0.0</mu2>
+      <mu1>0.4</mu1>
+      <mu2>0.4</mu2>
       <fdir1>1 0 0</fdir1>
       <maxVel>1.0</maxVel>

File: pmb2_description/urdf/wheels/caster.urdf.xacro (robot description, xacro)
@@ -12,9 +12,9 @@
     <link name="caster_${side}_1_link">
       <inertial>
-        <origin xyz="-0.01108 0.00003 -0.030" rpy="0 0 0"/>
-        <mass value="0.101"/>
-        <inertia  ixx="0.00002779423" ixy="-0.00000001384" ixz="0.0000074479"
-                  iyy="0.00002767062" iyz="-0.00000002774"
-                  izz="0.00001727605"/>
+        <origin xyz="-0.00634599 0.00005347 -0.02037519" rpy="0 0 0"/>
+        <mass value="0.05144761"/>
+        <inertia  ixx="0.00001513" ixy="-0.00000003" ixz="0.00000267"
+                  iyy="0.00001309" iyz="-0.00000005"
+                  izz="0.00001198"/>
       </inertial>
       <visual>
@@ -35,8 +35,8 @@
       <inertial>
         <origin xyz="0 0 0" rpy="0 0 0"/>
-        <mass value="0.03677"/>
-        <inertia  ixx="0.00000755221" ixy="0" ixz="0"
-                  iyy="0.00000755221" iyz="0"
-                  izz="0.00001281996"/>
+        <mass value="0.08855784"/>
+        <inertia  ixx="0.00001075" ixy="0" ixz="0"
+                  iyy="0.00001541" iyz="0"
+                  izz="0.00001075"/>
         </inertial>
       <visual>
@@ -59,4 +59,5 @@
       <origin xyz="${offset_x + separation_x / 2} ${offset_y - separation_y / 2} ${offset_z}" rpy="0 0 0"/>
       <axis xyz="0 0 1"/>
+      <dynamics damping="0.005" friction="0.0"/>
     </joint>
     <joint name="caster_${side}_2_joint" type="continuous">

Commit message: test sphere collision mesh and contact parameters

File: pmb2_description/urdf/wheels/caster.gazebo.xacro (robot description, xacro)
@@ -22,11 +22,11 @@
     </gazebo>
     <gazebo reference="caster_${side}_2_link">
-      <kp>1000000.0</kp>
-      <kd>1000.0</kd>
-      <mu1>0.4</mu1>
-      <mu2>0.4</mu2>
+      <kp>100000000.0</kp>
+      <kd>10.0</kd>
+      <mu1>0.1</mu1>
+      <mu2>0.1</mu2>
       <fdir1>1 0 0</fdir1>
-      <maxVel>1.0</maxVel>
-      <minDepth>0.00</minDepth>
+      <maxVel>10.0</maxVel>
+      <minDepth>0.0005</minDepth>
       <implicitSpringDamper>0</implicitSpringDamper>
       <material>Gazebo/DarkGrey</material>

File: pmb2_description/urdf/wheels/caster.urdf.xacro (robot description, xacro)
@@ -50,5 +50,5 @@
         <origin xyz="0 0 0" rpy="0 0 0"/>
         <geometry>
-          <cylinder radius="${radius}" length="${width}"/>
+	  <sphere radius="${radius}" /> <!-- length="${width}"/> -->
         </geometry>
       </collision>

File: pmb2_description/urdf/wheels/wheel.gazebo.xacro (robot description, xacro)
@@ -11,11 +11,11 @@
     <!-- Contact model for the wheel surface -->
     <gazebo reference="wheel_${side}_link">
-      <kp>1000000.0</kp>
-      <kd>1000.0</kd>
-      <mu1>1.0</mu1>
-      <mu2>1.0</mu2>
+      <kp>500000.0</kp>
+      <kd>10.0</kd>
+      <mu1>10.0</mu1>
+      <mu2>10.0</mu2>
       <fdir1>1 0 0</fdir1>
       <maxVel>1.0</maxVel>
-      <minDepth>0.00</minDepth>
+      <minDepth>0.003</minDepth>
       <implicitSpringDamper>1</implicitSpringDamper>
       <material>Gazebo/DarkGrey</material>

File: pmb2_description/urdf/wheels/wheel.urdf.xacro (robot description, xacro)
@@ -29,5 +29,5 @@
           <origin xyz="0 0 0" rpy="0 0 0"/>
           <geometry>
-            <cylinder radius="${radius}" length="${width}"/>
+            <sphere radius="${radius}" /> <!-- length="${width}"/> -->
           </geometry>
         </collision>

Commit message: Uss sphere and tuned contacts for collision links

File: pmb2_description/urdf/wheels/caster.gazebo.xacro (robot description, xacro)
@@ -12,15 +12,4 @@
     <gazebo reference="caster_${side}_1_link">
       <kp>1000000.0</kp>
-      <kd>1000.0</kd>
-      <mu1>1.0</mu1>
-      <mu2>1.0</mu2>
-      <fdir1>0 0 1</fdir1>
-      <maxVel>1.0</maxVel>
-      <minDepth>0.0</minDepth>
-      <implicitSpringDamper>0</implicitSpringDamper>
-      <material>Gazebo/DarkGrey</material>
-    </gazebo>
-    <gazebo reference="caster_${side}_2_link">
-      <kp>100000000.0</kp>
       <kd>10.0</kd>
       <mu1>0.1</mu1>
@@ -29,6 +18,21 @@
       <maxVel>10.0</maxVel>
       <minDepth>0.0005</minDepth>
+      <material>Gazebo/DarkGrey</material>
+    </gazebo>
+    <gazebo reference="caster_${side}_2_link">
+      <kp>1000000.0</kp>
+      <kd>10.0</kd>
+      <mu1>1.0</mu1>
+      <mu2>1.0</mu2>
+      <fdir1>1 0 0</fdir1>
+      <maxVel>10.0</maxVel>
+      <minDepth>0.0005</minDepth>
+      <material>Gazebo/DarkGrey</material>
+    </gazebo>
+    <gazebo reference="caster_{side}_1_joint">
       <implicitSpringDamper>0</implicitSpringDamper>
-      <material>Gazebo/DarkGrey</material>
+    </gazebo>
+    <gazebo reference="caster_{side}_2_joint">
+      <implicitSpringDamper>0</implicitSpringDamper>
     </gazebo>
   </xacro:macro>

File: pmb2_description/urdf/wheels/caster.urdf.xacro (robot description, xacro)
@@ -50,5 +50,5 @@
         <origin xyz="0 0 0" rpy="0 0 0"/>
         <geometry>
-	  <sphere radius="${radius}" /> <!-- length="${width}"/> -->
+	  <sphere radius="${radius}" />
         </geometry>
       </collision>

File: pmb2_description/urdf/wheels/wheel.gazebo.xacro (robot description, xacro)
@@ -16,8 +16,11 @@
       <mu2>10.0</mu2>
       <fdir1>1 0 0</fdir1>
+      <!--<dampingFactor>0.9</dampingFactor>-->
       <maxVel>1.0</maxVel>
-      <minDepth>0.003</minDepth>
+      <minDepth>0.002</minDepth>
+      <material>Gazebo/DarkGrey</material>
+    </gazebo>
+    <gazebo reference="wheel_{side}_joint">
       <implicitSpringDamper>1</implicitSpringDamper>
-      <material>Gazebo/DarkGrey</material>
     </gazebo>
   </xacro:macro>

File: pmb2_description/urdf/wheels/wheel.urdf.xacro (robot description, xacro)
@@ -60,5 +60,5 @@
           <parent link="suspension_${side}_link"/>
           <child link="wheel_${side}_link"/>
-          <origin xyz="0 ${-separation / 2 * reflect} 0" rpy="${-90.0 * deg_to_rad} 0 0"/>
+          <origin xyz="0 ${-separation / 2 * reflect} 0.0" rpy="${-90.0 * deg_to_rad} 0 0"/>
           <axis xyz="0 0 1"/>
           <limit effort="${torque}" velocity="${velocity / radius}"/>

Commit message: Tune a bit physics to avoid joint slippage, specially in TIAGo

File: pmb2_description/urdf/wheels/caster.gazebo.xacro (robot description, xacro)
@@ -12,5 +12,5 @@
     <gazebo reference="caster_${side}_1_link">
       <kp>100000000.0</kp>
-      <kd>10.0</kd>
+      <kd>100000.0</kd>
       <friction>
         <ode>
@@ -20,11 +20,11 @@
       </friction>
       <!--<fdir1>1 0 0</fdir1>-->
-      <max_vel>10.0</max_vel>
-      <min_depth>0.0005</min_depth>
+      <max_vel>1.0</max_vel>
+      <min_depth>0.005</min_depth>
       <material>Gazebo/DarkGrey</material>
     </gazebo>
     <gazebo reference="caster_${side}_2_link">
       <kp>100000000.0</kp>
-      <kd>10.0</kd>
+      <kd>100000.0</kd>
       <friction>
         <ode>
@@ -34,6 +34,6 @@
       </friction>
       <!--<fdir1>1 0 0</fdir1>-->
-      <max_vel>10.0</max_vel>
-      <min_depth>0.0005</min_depth>
+      <max_vel>1.0</max_vel>
+      <min_depth>0.005</min_depth>
       <material>Gazebo/DarkGrey</material>
     </gazebo>

File: pmb2_description/urdf/wheels/caster.urdf.xacro (robot description, xacro)
@@ -59,5 +59,5 @@
       <origin xyz="${offset_x + separation_x / 2} ${offset_y - separation_y / 2} ${offset_z}" rpy="0 0 0"/>
       <axis xyz="0 0 1"/>
-      <dynamics damping="0.005" friction="0.0"/>
+      <dynamics damping="0.015" friction="0.0"/>
     </joint>
     <joint name="caster_${side}_2_joint" type="continuous">
@@ -66,4 +66,5 @@
       <origin xyz="-0.016 0.0000 -0.040" rpy="${-90.0 * deg_to_rad} 0 0"/>
       <axis xyz="0 0 1"/>
+      <dynamics damping="0.015" friction="0.0"/>
     </joint>
     <!-- Gazebo extensions -->

File: pmb2_description/urdf/wheels/wheel.urdf.xacro (robot description, xacro)
@@ -62,4 +62,5 @@
           <axis xyz="0 0 1"/>
           <limit effort="${torque}" velocity="${velocity / radius}"/>
+        <dynamics damping="1.0" friction="0.0"/>
         </joint>
         <!-- Gazebo extensions -->
