Commit message: tune wheels physics to avoid slippage

File: pmb2_description/urdf/wheels/caster.gazebo.xacro (robot description, xacro)
@@ -16,6 +16,6 @@
     <!-- Contact model for the caster wheel surface -->
     <gazebo reference="caster_${side}_1_link">
-      <kp>100000000.0</kp>
-      <kd>100000.0</kd>
+      <kp>1000000.0</kp>
+      <kd>10000.0</kd>
       <friction>
         <ode>
@@ -30,6 +30,6 @@
     </gazebo>
     <gazebo reference="caster_${side}_2_link">
-      <kp>100000000.0</kp>
-      <kd>100000.0</kd>
+      <kp>1000000.0</kp>
+      <kd>10000.0</kd>
       <friction>
         <ode>

File: pmb2_description/urdf/wheels/wheel.urdf.xacro (robot description, xacro)
@@ -67,5 +67,5 @@
           <axis xyz="0 0 1"/>
           <limit effort="${torque}" velocity="${velocity / radius}"/>
-        <dynamics damping="1.0" friction="0.0"/>
+        <dynamics damping="1.0" friction="2.0"/>
         </joint>
         <!-- Gazebo extensions -->
