Commit message: indentation fix

File: pmb2_description/urdf/wheels/wheel.urdf.xacro (robot description, xacro)
@@ -22,53 +22,53 @@
           iyy="0.00499741733" iyz="${-0.00000000164 * reflect}"
           izz="0.00839239692"/>
+      </inertial>
+      <visual>
+        <origin xyz="0 0 0" rpy="${-90.0 * (1 - reflect) * deg_to_rad} 0 0"/>
+        <geometry>
+          <mesh filename="package://pmb2_description/meshes/wheels/wheel.stl"/>
+        </geometry>
+        <material name="DarkGrey"/>
+      </visual>
+      <collision>
+        <origin xyz="0 0 0" rpy="0 0 0"/>
+        <geometry>
+          <sphere radius="${radius}" /> <!-- length="${width}"/> -->
+        </geometry>
+      </collision>
+    </link>
+    <link name="suspension_${side}_link">
+      <inertial>
+        <origin xyz="0 0 -0.02" rpy="0 0 0"/>
+        <mass value="10"/>
+        <inertia ixx="1.0" ixy="0" ixz="0"
+                  iyy="1.0" iyz="0"
+                  izz="1.0"/>
         </inertial>
-        <visual>
-          <origin xyz="0 0 0" rpy="${-90.0 * (1 - reflect) * deg_to_rad} 0 0"/>
-          <geometry>
-            <mesh filename="package://pmb2_description/meshes/wheels/wheel.stl"/>
-          </geometry>
-          <material name="DarkGrey"/>
-        </visual>
-        <collision>
-          <origin xyz="0 0 0" rpy="0 0 0"/>
-          <geometry>
-            <sphere radius="${radius}" /> <!-- length="${width}"/> -->
-          </geometry>
-        </collision>
-      </link>
-      <link name="suspension_${side}_link">
-        <inertial>
-          <origin xyz="0 0 -0.02" rpy="0 0 0"/>
-          <mass value="10"/>
-          <inertia ixx="1.0" ixy="0" ixz="0"
-                   iyy="1.0" iyz="0"
-                   izz="1.0"/>
-         </inertial>
-        <kinematic>0</kinematic>
-        <gravity>1</gravity>
-      </link>
-      <joint name="suspension_${side}_joint" type="prismatic">
-        <origin xyz="0 0 0" rpy="0 0 0"/>
-        <axis xyz="0 0 1"/>
-        <limit effort="100.0" lower="-0.005" upper="0.005" velocity="1.0"/>
-        <child link="suspension_${side}_link"/>
-        <parent link="${parent}_link"/>
-        <calibration rising="0.0" />
-        <dynamics damping="100"/>
-        <safety_controller k_position="0"
-          k_velocity="10"
-          soft_lower_limit="-0.005"
-          soft_upper_limit="0.005" />
-        </joint>
-        <joint name="wheel_${side}_joint" type="continuous">
-          <parent link="suspension_${side}_link"/>
-          <child link="wheel_${side}_link"/>
-          <origin xyz="0 ${-separation / 2 * reflect} 0.0" rpy="${-90.0 * deg_to_rad} 0 0"/>
-          <axis xyz="0 0 1"/>
-          <limit effort="${torque}" velocity="${velocity / radius}"/>
-        <dynamics damping="1.0" friction="2.0"/>
-        </joint>
-        <!-- Gazebo extensions -->
-        <xacro:wheel_gazebo side="${side}"/>
-      </xacro:macro>
-    </robot>
+      <kinematic>0</kinematic>
+      <gravity>1</gravity>
+    </link>
+    <joint name="suspension_${side}_joint" type="prismatic">
+      <origin xyz="0 0 0" rpy="0 0 0"/>
+      <axis xyz="0 0 1"/>
+      <limit effort="100.0" lower="-0.005" upper="0.005" velocity="1.0"/>
+      <child link="suspension_${side}_link"/>
+      <parent link="${parent}_link"/>
+      <calibration rising="0.0" />
+      <dynamics damping="100"/>
+      <safety_controller k_position="0"
+        k_velocity="10"
+        soft_lower_limit="-0.005"
+        soft_upper_limit="0.005" />
+    </joint>
+    <joint name="wheel_${side}_joint" type="continuous">
+      <parent link="suspension_${side}_link"/>
+      <child link="wheel_${side}_link"/>
+      <origin xyz="0 ${-separation / 2 * reflect} 0.0" rpy="${-90.0 * deg_to_rad} 0 0"/>
+      <axis xyz="0 0 1"/>
+      <limit effort="${torque}" velocity="${velocity / radius}"/>
+      <dynamics damping="1.0" friction="2.0"/>
+    </joint>
+    <!-- Gazebo extensions -->
+    <xacro:wheel_gazebo side="${side}"/>
+  </xacro:macro>
+</robot>

Commit message: fix shape of wheel collision

File: pmb2_description/urdf/wheels/wheel.urdf.xacro (robot description, xacro)
@@ -34,5 +34,5 @@
         <origin xyz="0 0 0" rpy="0 0 0"/>
         <geometry>
-          <sphere radius="${radius}" /> <!-- length="${width}"/> -->
+          <cylinder radius="${radius}" length="${width}"/>
         </geometry>
       </collision>
