Commit message: Replace ant -> pmb2

File: pmb2_description/gazebo/gazebo.urdf.xacro (robot description, xacro)
@@ -13,5 +13,5 @@
     <plugin filename="libgazebo_ros_control.so" name="ros_control">
       <ns></ns>
-      <robotSimType>ant_hardware_gazebo/AntHardwareGazebo</robotSimType>
+      <robotSimType>pmb2_hardware_gazebo/Pmb2HardwareGazebo</robotSimType>
       <controlPeriod>0.001</controlPeriod>
     </plugin>

File: pmb2_description/robots/dock_full.urdf.xacro (robot description, xacro)
@@ -11,7 +11,7 @@
   <!-- The following included files set up definitions of parts of the dock body -->
   <!-- Dock -->
-  <xacro:include filename="$(find ant_description)/urdf/dock/dock.urdf.xacro" />
+  <xacro:include filename="$(find pmb2_description)/urdf/dock/dock.urdf.xacro" />
   <!-- Materials for visualization -->
-  <xacro:include filename="$(find ant_description)/urdf/materials.urdf.xacro" />
+  <xacro:include filename="$(find pmb2_description)/urdf/materials.urdf.xacro" />
   <!-- Now we can start using the macros included above to define the actual robot -->
   <xacro:dock name="dock"/>

File: pmb2_description/robots/pmb2_full.urdf.xacro (robot description, xacro)
@@ -8,12 +8,12 @@
 -->
 <robot  xmlns:xacro="http://www.ros.org/wiki/xacro"
-        name="ant" >
+        name="pmb2" >
   <!-- The following included files set up definitions of parts of the robot body -->
   <!-- Base -->
-  <xacro:include filename="$(find ant_description)/urdf/base/base.urdf.xacro" />
+  <xacro:include filename="$(find pmb2_description)/urdf/base/base.urdf.xacro" />
   <!-- Generic simulator_gazebo plugins -->
-  <xacro:include filename="$(find ant_description)/gazebo/gazebo.urdf.xacro" />
+  <xacro:include filename="$(find pmb2_description)/gazebo/gazebo.urdf.xacro" />
   <!-- Materials for visualization -->
-  <xacro:include filename="$(find ant_description)/urdf/materials.urdf.xacro" />
+  <xacro:include filename="$(find pmb2_description)/urdf/materials.urdf.xacro" />
   <!-- Now we can start using the macros included above to define the actual robot -->
   <xacro:base name="base"/>

File: pmb2_description/robots/pmb2_full_v2.urdf.xacro (robot description, xacro)
@@ -8,12 +8,12 @@
 -->
 <robot  xmlns:xacro="http://www.ros.org/wiki/xacro"
-        name="ant" >
+        name="pmb2" >
   <!-- The following included files set up definitions of parts of the robot body -->
   <!-- Base -->
-  <xacro:include filename="$(find ant_description)/urdf/base/base_v2.urdf.xacro" />
+  <xacro:include filename="$(find pmb2_description)/urdf/base/base_v2.urdf.xacro" />
   <!-- Generic simulator_gazebo plugins -->
-  <xacro:include filename="$(find ant_description)/gazebo/gazebo.urdf.xacro" />
+  <xacro:include filename="$(find pmb2_description)/gazebo/gazebo.urdf.xacro" />
   <!-- Materials for visualization -->
-  <xacro:include filename="$(find ant_description)/urdf/materials.urdf.xacro" />
+  <xacro:include filename="$(find pmb2_description)/urdf/materials.urdf.xacro" />
   <!-- Now we can start using the macros included above to define the actual robot -->
   <xacro:base name="base"/>

File: pmb2_description/robots/pmb2_horizontal_xtion_pro_live_v2.urdf.xacro (robot description, xacro)
@@ -8,12 +8,12 @@
 -->
 <robot  xmlns:xacro="http://www.ros.org/wiki/xacro"
-        name="ant" >
+        name="pmb2" >
   <!-- The following included files set up definitions of parts of the robot body -->
   <!-- Base -->
-  <xacro:include filename="$(find ant_description)/urdf/base/base_v2_horizontal_xtion_pro_live.urdf.xacro" />
+  <xacro:include filename="$(find pmb2_description)/urdf/base/base_v2_horizontal_xtion_pro_live.urdf.xacro" />
   <!-- Generic simulator_gazebo plugins -->
-  <xacro:include filename="$(find ant_description)/gazebo/gazebo.urdf.xacro" />
+  <xacro:include filename="$(find pmb2_description)/gazebo/gazebo.urdf.xacro" />
   <!-- Materials for visualization -->
-  <xacro:include filename="$(find ant_description)/urdf/materials.urdf.xacro" />
+  <xacro:include filename="$(find pmb2_description)/urdf/materials.urdf.xacro" />
   <!-- Now we can start using the macros included above to define the actual robot -->
   <xacro:base name="base"/>

File: pmb2_description/robots/pmb2_rebujito.urdf.xacro (robot description, xacro)
@@ -8,12 +8,12 @@
 -->
 <robot  xmlns:xacro="http://www.ros.org/wiki/xacro"
-        name="ant" >
+        name="pmb2" >
   <!-- The following included files set up definitions of parts of the robot body -->
   <!-- Base -->
-  <xacro:include filename="$(find ant_description)/urdf/base/base_rebujito.urdf.xacro" />
+  <xacro:include filename="$(find pmb2_description)/urdf/base/base_rebujito.urdf.xacro" />
   <!-- Generic simulator_gazebo plugins -->
-  <xacro:include filename="$(find ant_description)/gazebo/gazebo.urdf.xacro" />
+  <xacro:include filename="$(find pmb2_description)/gazebo/gazebo.urdf.xacro" />
   <!-- Materials for visualization -->
-  <xacro:include filename="$(find ant_description)/urdf/materials.urdf.xacro" />
+  <xacro:include filename="$(find pmb2_description)/urdf/materials.urdf.xacro" />
   <!-- Now we can start using the macros included above to define the actual robot -->
   <xacro:base name="base"/>

File: pmb2_description/robots/pmb2_rplidar.urdf.xacro (robot description, xacro)
@@ -8,12 +8,12 @@
 -->
 <robot  xmlns:xacro="http://www.ros.org/wiki/xacro"
-        name="ant" >
+        name="pmb2" >
   <!-- The following included files set up definitions of parts of the robot body -->
   <!-- Base -->
-  <xacro:include filename="$(find ant_description)/urdf/base/base_rplidar.urdf.xacro" />
+  <xacro:include filename="$(find pmb2_description)/urdf/base/base_rplidar.urdf.xacro" />
   <!-- Generic simulator_gazebo plugins -->
-  <xacro:include filename="$(find ant_description)/gazebo/gazebo.urdf.xacro" />
+  <xacro:include filename="$(find pmb2_description)/gazebo/gazebo.urdf.xacro" />
   <!-- Materials for visualization -->
-  <xacro:include filename="$(find ant_description)/urdf/materials.urdf.xacro" />
+  <xacro:include filename="$(find pmb2_description)/urdf/materials.urdf.xacro" />
   <!-- Now we can start using the macros included above to define the actual robot -->
   <xacro:base name="base"/>

File: pmb2_description/robots/pmb2_softkinetic_ds311.urdf.xacro (robot description, xacro)
@@ -8,12 +8,12 @@
 -->
 <robot  xmlns:xacro="http://www.ros.org/wiki/xacro"
-        name="ant" >
+        name="pmb2" >
   <!-- The following included files set up definitions of parts of the robot body -->
   <!-- Base -->
-  <xacro:include filename="$(find ant_description)/urdf/base/base_softkinetic_ds311.urdf.xacro" />
+  <xacro:include filename="$(find pmb2_description)/urdf/base/base_softkinetic_ds311.urdf.xacro" />
   <!-- Generic simulator_gazebo plugins -->
-  <xacro:include filename="$(find ant_description)/gazebo/gazebo.urdf.xacro" />
+  <xacro:include filename="$(find pmb2_description)/gazebo/gazebo.urdf.xacro" />
   <!-- Materials for visualization -->
-  <xacro:include filename="$(find ant_description)/urdf/materials.urdf.xacro" />
+  <xacro:include filename="$(find pmb2_description)/urdf/materials.urdf.xacro" />
   <!-- Now we can start using the macros included above to define the actual robot -->
   <xacro:base name="base"/>

File: pmb2_description/robots/pmb2_vertical_xtion_pro_live_v2.urdf.xacro (robot description, xacro)
@@ -8,12 +8,12 @@
 -->
 <robot  xmlns:xacro="http://www.ros.org/wiki/xacro"
-        name="ant" >
+        name="pmb2" >
   <!-- The following included files set up definitions of parts of the robot body -->
   <!-- Base -->
-  <xacro:include filename="$(find ant_description)/urdf/base/base_v2_vertical_xtion_pro_live.urdf.xacro" />
+  <xacro:include filename="$(find pmb2_description)/urdf/base/base_v2_vertical_xtion_pro_live.urdf.xacro" />
   <!-- Generic simulator_gazebo plugins -->
-  <xacro:include filename="$(find ant_description)/gazebo/gazebo.urdf.xacro" />
+  <xacro:include filename="$(find pmb2_description)/gazebo/gazebo.urdf.xacro" />
   <!-- Materials for visualization -->
-  <xacro:include filename="$(find ant_description)/urdf/materials.urdf.xacro" />
+  <xacro:include filename="$(find pmb2_description)/urdf/materials.urdf.xacro" />
   <!-- Now we can start using the macros included above to define the actual robot -->
   <xacro:base name="base"/>

File: pmb2_description/robots/pmb2_xtion_pro_live.urdf.xacro (robot description, xacro)
@@ -8,12 +8,12 @@
 -->
 <robot  xmlns:xacro="http://www.ros.org/wiki/xacro"
-        name="ant" >
+        name="pmb2" >
   <!-- The following included files set up definitions of parts of the robot body -->
   <!-- Base -->
-  <xacro:include filename="$(find ant_description)/urdf/base/base_xtion_pro_live.urdf.xacro" />
+  <xacro:include filename="$(find pmb2_description)/urdf/base/base_xtion_pro_live.urdf.xacro" />
   <!-- Generic simulator_gazebo plugins -->
-  <xacro:include filename="$(find ant_description)/gazebo/gazebo.urdf.xacro" />
+  <xacro:include filename="$(find pmb2_description)/gazebo/gazebo.urdf.xacro" />
   <!-- Materials for visualization -->
-  <xacro:include filename="$(find ant_description)/urdf/materials.urdf.xacro" />
+  <xacro:include filename="$(find pmb2_description)/urdf/materials.urdf.xacro" />
   <!-- Now we can start using the macros included above to define the actual robot -->
   <xacro:base name="base"/>

File: pmb2_description/robots/pmb2_xtion_pro_live_only.urdf.xacro (robot description, xacro)
@@ -8,12 +8,12 @@
 -->
 <robot  xmlns:xacro="http://www.ros.org/wiki/xacro"
-        name="ant" >
+        name="pmb2" >
   <!-- The following included files set up definitions of parts of the robot body -->
   <!-- Base -->
-  <xacro:include filename="$(find ant_description)/urdf/base/base_xtion_pro_live_only.urdf.xacro" />
+  <xacro:include filename="$(find pmb2_description)/urdf/base/base_xtion_pro_live_only.urdf.xacro" />
   <!-- Generic simulator_gazebo plugins -->
-  <xacro:include filename="$(find ant_description)/gazebo/gazebo.urdf.xacro" />
+  <xacro:include filename="$(find pmb2_description)/gazebo/gazebo.urdf.xacro" />
   <!-- Materials for visualization -->
-  <xacro:include filename="$(find ant_description)/urdf/materials.urdf.xacro" />
+  <xacro:include filename="$(find pmb2_description)/urdf/materials.urdf.xacro" />
   <!-- Now we can start using the macros included above to define the actual robot -->
   <xacro:base name="base"/>

File: pmb2_description/robots/pmb2_xtion_pro_live_v2.urdf.xacro (robot description, xacro)
@@ -8,12 +8,12 @@
 -->
 <robot  xmlns:xacro="http://www.ros.org/wiki/xacro"
-        name="ant" >
+        name="pmb2" >
   <!-- The following included files set up definitions of parts of the robot body -->
   <!-- Base -->
-  <xacro:include filename="$(find ant_description)/urdf/base/base_v2_xtion_pro_live.urdf.xacro" />
+  <xacro:include filename="$(find pmb2_description)/urdf/base/base_v2_xtion_pro_live.urdf.xacro" />
   <!-- Generic simulator_gazebo plugins -->
-  <xacro:include filename="$(find ant_description)/gazebo/gazebo.urdf.xacro" />
+  <xacro:include filename="$(find pmb2_description)/gazebo/gazebo.urdf.xacro" />
   <!-- Materials for visualization -->
-  <xacro:include filename="$(find ant_description)/urdf/materials.urdf.xacro" />
+  <xacro:include filename="$(find pmb2_description)/urdf/materials.urdf.xacro" />
   <!-- Now we can start using the macros included above to define the actual robot -->
   <xacro:base name="base"/>

File: pmb2_description/urdf/base/base.urdf.xacro (robot description, xacro)
@@ -8,12 +8,12 @@
 -->
 <robot xmlns:xacro="http://ros.org/wiki/xacro">
-  <xacro:include filename="$(find ant_description)/urdf/deg_to_rad.xacro"/>
-  <xacro:include filename="$(find ant_description)/urdf/wheels/wheel.urdf.xacro"/>
-  <xacro:include filename="$(find ant_description)/urdf/wheels/caster.urdf.xacro"/>
-  <xacro:include filename="$(find ant_description)/urdf/sensors/range.urdf.xacro"/>
-  <xacro:include filename="$(find ant_description)/urdf/sensors/hokuyo_urg_04lx_ug01_laser.urdf.xacro"/>
-  <xacro:include filename="$(find ant_description)/urdf/sensors/imu.urdf.xacro"/>
-  <xacro:include filename="$(find ant_description)/urdf/sensors/bumper.urdf.xacro"/>
-  <xacro:include filename="$(find ant_description)/urdf/sensors/ir_receiver.urdf.xacro"/>
+  <xacro:include filename="$(find pmb2_description)/urdf/deg_to_rad.xacro"/>
+  <xacro:include filename="$(find pmb2_description)/urdf/wheels/wheel.urdf.xacro"/>
+  <xacro:include filename="$(find pmb2_description)/urdf/wheels/caster.urdf.xacro"/>
+  <xacro:include filename="$(find pmb2_description)/urdf/sensors/range.urdf.xacro"/>
+  <xacro:include filename="$(find pmb2_description)/urdf/sensors/hokuyo_urg_04lx_ug01_laser.urdf.xacro"/>
+  <xacro:include filename="$(find pmb2_description)/urdf/sensors/imu.urdf.xacro"/>
+  <xacro:include filename="$(find pmb2_description)/urdf/sensors/bumper.urdf.xacro"/>
+  <xacro:include filename="$(find pmb2_description)/urdf/sensors/ir_receiver.urdf.xacro"/>
   <!-- Wheel characteristics -->
   <property name="wheel_radius"     value="0.100"/>
@@ -48,5 +48,5 @@
         <origin xyz="0 0 0" rpy="0 0 0" />
         <geometry>
-          <mesh filename="package://ant_description/meshes/base/base.stl" />
+          <mesh filename="package://pmb2_description/meshes/base/base.stl" />
         </geometry>
         <material name="DarkGrey" />
@@ -92,5 +92,5 @@
     </xacro:bumper-->
     <!-- IMU -->
-    <!-- @todo ant_hardware_gazebo needs an IMU!  -->
+    <!-- @todo pmb2_hardware_gazebo needs an IMU!  -->
     <xacro:imu_sensor name="base_inclinometer" parent="${name}_link" update_rate="100.0">
       <origin xyz="0 0 ${base_length / 2}" rpy="0 0 0"/>

File: pmb2_description/urdf/base/base_rebujito.urdf.xacro (robot description, xacro)
@@ -8,13 +8,13 @@
 -->
 <robot xmlns:xacro="http://ros.org/wiki/xacro">
-  <xacro:include filename="$(find ant_description)/urdf/deg_to_rad.xacro"/>
-  <xacro:include filename="$(find ant_description)/urdf/wheels/wheel.urdf.xacro"/>
-  <xacro:include filename="$(find ant_description)/urdf/wheels/caster.urdf.xacro"/>
-  <xacro:include filename="$(find ant_description)/urdf/sensors/range.urdf.xacro"/>
-  <xacro:include filename="$(find ant_description)/urdf/sensors/hokuyo_urg_04lx_ug01_laser.urdf.xacro"/>
-  <xacro:include filename="$(find ant_description)/urdf/sensors/imu.urdf.xacro"/>
-  <xacro:include filename="$(find ant_description)/urdf/sensors/bumper.urdf.xacro"/>
-  <xacro:include filename="$(find ant_description)/urdf/sensors/ir_receiver.urdf.xacro"/>
-  <xacro:include filename="$(find ant_description)/urdf/antennas/antenna_array.urdf.xacro"/>
+  <xacro:include filename="$(find pmb2_description)/urdf/deg_to_rad.xacro"/>
+  <xacro:include filename="$(find pmb2_description)/urdf/wheels/wheel.urdf.xacro"/>
+  <xacro:include filename="$(find pmb2_description)/urdf/wheels/caster.urdf.xacro"/>
+  <xacro:include filename="$(find pmb2_description)/urdf/sensors/range.urdf.xacro"/>
+  <xacro:include filename="$(find pmb2_description)/urdf/sensors/hokuyo_urg_04lx_ug01_laser.urdf.xacro"/>
+  <xacro:include filename="$(find pmb2_description)/urdf/sensors/imu.urdf.xacro"/>
+  <xacro:include filename="$(find pmb2_description)/urdf/sensors/bumper.urdf.xacro"/>
+  <xacro:include filename="$(find pmb2_description)/urdf/sensors/ir_receiver.urdf.xacro"/>
+  <xacro:include filename="$(find pmb2_description)/urdf/antennas/antenna_array.urdf.xacro"/>
   <!-- Wheel characteristics -->
   <!-- Note that we temporary use Rebujito's -->
@@ -52,5 +52,5 @@
         <origin xyz="0 0 ${base_offset_z}" rpy="0 0 0" />
         <geometry>
-          <mesh filename="package://ant_description/meshes/base/rebujito.stl" />
+          <mesh filename="package://pmb2_description/meshes/base/rebujito.stl" />
         </geometry>
         <material name="LightGrey" />
@@ -59,5 +59,5 @@
         <origin xyz="0 0 ${base_offset_z}" rpy="0 0 0" />
         <geometry>
-          <mesh filename="package://ant_description/meshes/base/rebujito_collision.stl" />
+          <mesh filename="package://pmb2_description/meshes/base/rebujito_collision.stl" />
         </geometry>
         <material name="LightGrey" />

File: pmb2_description/urdf/base/base_rplidar.urdf.xacro (robot description, xacro)
@@ -8,12 +8,12 @@
 -->
 <robot xmlns:xacro="http://ros.org/wiki/xacro">
-  <xacro:include filename="$(find ant_description)/urdf/deg_to_rad.xacro"/>
-  <xacro:include filename="$(find ant_description)/urdf/wheels/wheel.urdf.xacro"/>
-  <xacro:include filename="$(find ant_description)/urdf/wheels/caster.urdf.xacro"/>
-  <xacro:include filename="$(find ant_description)/urdf/sensors/range.urdf.xacro"/>
-  <xacro:include filename="$(find ant_description)/urdf/sensors/rplidar_laser.urdf.xacro"/>
-  <xacro:include filename="$(find ant_description)/urdf/sensors/imu.urdf.xacro"/>
-  <xacro:include filename="$(find ant_description)/urdf/sensors/bumper.urdf.xacro"/>
-  <xacro:include filename="$(find ant_description)/urdf/sensors/ir_receiver.urdf.xacro"/>
+  <xacro:include filename="$(find pmb2_description)/urdf/deg_to_rad.xacro"/>
+  <xacro:include filename="$(find pmb2_description)/urdf/wheels/wheel.urdf.xacro"/>
+  <xacro:include filename="$(find pmb2_description)/urdf/wheels/caster.urdf.xacro"/>
+  <xacro:include filename="$(find pmb2_description)/urdf/sensors/range.urdf.xacro"/>
+  <xacro:include filename="$(find pmb2_description)/urdf/sensors/rplidar_laser.urdf.xacro"/>
+  <xacro:include filename="$(find pmb2_description)/urdf/sensors/imu.urdf.xacro"/>
+  <xacro:include filename="$(find pmb2_description)/urdf/sensors/bumper.urdf.xacro"/>
+  <xacro:include filename="$(find pmb2_description)/urdf/sensors/ir_receiver.urdf.xacro"/>
   <!-- Wheel characteristics -->
   <property name="wheel_radius"     value="0.100"/>
@@ -48,5 +48,5 @@
         <origin xyz="0 0 0" rpy="0 0 0" />
         <geometry>
-          <mesh filename="package://ant_description/meshes/base/base.stl" />
+          <mesh filename="package://pmb2_description/meshes/base/base.stl" />
         </geometry>
         <material name="DarkGrey" />
@@ -92,5 +92,5 @@
     </xacro:bumper-->
     <!-- IMU -->
-    <!-- @todo ant_hardware_gazebo needs an IMU!  -->
+    <!-- @todo pmb2_hardware_gazebo needs an IMU!  -->
     <xacro:imu_sensor name="base_inclinometer" parent="${name}_link" update_rate="100.0">
       <origin xyz="0 0 ${base_length / 2}" rpy="0 0 0"/>

File: pmb2_description/urdf/base/base_softkinetic_ds311.urdf.xacro (robot description, xacro)
@@ -8,13 +8,13 @@
 -->
 <robot xmlns:xacro="http://ros.org/wiki/xacro">
-  <xacro:include filename="$(find ant_description)/urdf/deg_to_rad.xacro"/>
-  <xacro:include filename="$(find ant_description)/urdf/wheels/wheel.urdf.xacro"/>
-  <xacro:include filename="$(find ant_description)/urdf/wheels/caster.urdf.xacro"/>
-  <xacro:include filename="$(find ant_description)/urdf/sensors/range.urdf.xacro"/>
-  <xacro:include filename="$(find ant_description)/urdf/sensors/hokuyo_urg_04lx_ug01_laser.urdf.xacro"/>
-  <xacro:include filename="$(find ant_description)/urdf/sensors/softkinetic_ds311_rgbd_camera.urdf.xacro"/>
-  <xacro:include filename="$(find ant_description)/urdf/sensors/imu.urdf.xacro"/>
-  <xacro:include filename="$(find ant_description)/urdf/sensors/bumper.urdf.xacro"/>
-  <xacro:include filename="$(find ant_description)/urdf/sensors/ir_receiver.urdf.xacro"/>
+  <xacro:include filename="$(find pmb2_description)/urdf/deg_to_rad.xacro"/>
+  <xacro:include filename="$(find pmb2_description)/urdf/wheels/wheel.urdf.xacro"/>
+  <xacro:include filename="$(find pmb2_description)/urdf/wheels/caster.urdf.xacro"/>
+  <xacro:include filename="$(find pmb2_description)/urdf/sensors/range.urdf.xacro"/>
+  <xacro:include filename="$(find pmb2_description)/urdf/sensors/hokuyo_urg_04lx_ug01_laser.urdf.xacro"/>
+  <xacro:include filename="$(find pmb2_description)/urdf/sensors/softkinetic_ds311_rgbd_camera.urdf.xacro"/>
+  <xacro:include filename="$(find pmb2_description)/urdf/sensors/imu.urdf.xacro"/>
+  <xacro:include filename="$(find pmb2_description)/urdf/sensors/bumper.urdf.xacro"/>
+  <xacro:include filename="$(find pmb2_description)/urdf/sensors/ir_receiver.urdf.xacro"/>
   <!-- Wheel characteristics -->
   <property name="wheel_radius"     value="0.100"/>
@@ -85,5 +85,5 @@
         <origin xyz="0 0 0" rpy="0 0 0" />
         <geometry>
-          <mesh filename="package://ant_description/meshes/base/base.stl" />
+          <mesh filename="package://pmb2_description/meshes/base/base.stl" />
         </geometry>
         <material name="DarkGrey" />
@@ -136,5 +136,5 @@
     </xacro:bumper-->
     <!-- IMU -->
-    <!-- @todo ant_hardware_gazebo needs an IMU!  -->
+    <!-- @todo pmb2_hardware_gazebo needs an IMU!  -->
     <xacro:imu_sensor name="base_inclinometer" parent="${name}_link" update_rate="100.0">
       <origin xyz="0 0 ${base_length / 2}" rpy="0 0 0"/>
