Commit message: Replace ant -> pmb2

File: pmb2_description/urdf/base/base_v2.urdf.xacro (robot description, xacro)
@@ -8,12 +8,12 @@
 -->
 <robot xmlns:xacro="http://ros.org/wiki/xacro">
-  <xacro:include filename="$(find ant_description)/urdf/deg_to_rad.xacro"/>
-  <xacro:include filename="$(find ant_description)/urdf/wheels/wheel_v2.urdf.xacro"/>
-  <xacro:include filename="$(find ant_description)/urdf/wheels/caster_v2.urdf.xacro"/>
-  <xacro:include filename="$(find ant_description)/urdf/sensors/range.urdf.xacro"/>
-  <xacro:include filename="$(find ant_description)/urdf/sensors/sick_tim551_laser.urdf.xacro"/>
-  <xacro:include filename="$(find ant_description)/urdf/sensors/imu.urdf.xacro"/>
-  <xacro:include filename="$(find ant_description)/urdf/sensors/bumper.urdf.xacro"/>
-  <xacro:include filename="$(find ant_description)/urdf/sensors/ir_receiver.urdf.xacro"/>
+  <xacro:include filename="$(find pmb2_description)/urdf/deg_to_rad.xacro"/>
+  <xacro:include filename="$(find pmb2_description)/urdf/wheels/wheel_v2.urdf.xacro"/>
+  <xacro:include filename="$(find pmb2_description)/urdf/wheels/caster_v2.urdf.xacro"/>
+  <xacro:include filename="$(find pmb2_description)/urdf/sensors/range.urdf.xacro"/>
+  <xacro:include filename="$(find pmb2_description)/urdf/sensors/sick_tim551_laser.urdf.xacro"/>
+  <xacro:include filename="$(find pmb2_description)/urdf/sensors/imu.urdf.xacro"/>
+  <xacro:include filename="$(find pmb2_description)/urdf/sensors/bumper.urdf.xacro"/>
+  <xacro:include filename="$(find pmb2_description)/urdf/sensors/ir_receiver.urdf.xacro"/>
   <!-- Wheel characteristics -->
   <property name="wheel_radius"     value="0.0985"/>
@@ -45,5 +45,5 @@
         <origin xyz="0 0 0" rpy="0 0 0" />
         <geometry>
-          <mesh filename="package://ant_description/meshes/base/base_v2.stl" />
+          <mesh filename="package://pmb2_description/meshes/base/base_v2.stl" />
         </geometry>
         <material name="DarkGrey" />
@@ -52,5 +52,5 @@
         <origin xyz="0 0 0" rpy="0 0 0" />
         <geometry>
-          <mesh filename="package://ant_description/meshes/base/base_v2_collision.stl" />
+          <mesh filename="package://pmb2_description/meshes/base/base_v2_collision.stl" />
         </geometry>
         <material name="DarkGrey" />
@@ -90,5 +90,5 @@
     </xacro:bumper-->
     <!-- IMU -->
-    <!-- @todo ant_hardware_gazebo needs an IMU!  -->
+    <!-- @todo pmb2_hardware_gazebo needs an IMU!  -->
     <xacro:imu_sensor name="base_inclinometer" parent="${name}_link" update_rate="100.0">
       <origin xyz="0 0 0" rpy="0 0 0"/>

File: pmb2_description/urdf/base/base_v2_horizontal_xtion_pro_live.urdf.xacro (robot description, xacro)
@@ -8,14 +8,14 @@
 -->
 <robot xmlns:xacro="http://ros.org/wiki/xacro">
-  <xacro:include filename="$(find ant_description)/urdf/deg_to_rad.xacro"/>
-  <xacro:include filename="$(find ant_description)/urdf/wheels/wheel_v2.urdf.xacro"/>
-  <xacro:include filename="$(find ant_description)/urdf/wheels/caster_v2.urdf.xacro"/>
-  <xacro:include filename="$(find ant_description)/urdf/sensors/range.urdf.xacro"/>
-  <xacro:include filename="$(find ant_description)/urdf/sensors/sick_tim551_laser.urdf.xacro"/>
-  <xacro:include filename="$(find ant_description)/urdf/sensors/xtion_pro_live.urdf.xacro"/>
-  <xacro:include filename="$(find ant_description)/urdf/sensors/imu.urdf.xacro"/>
-  <xacro:include filename="$(find ant_description)/urdf/sensors/bumper.urdf.xacro"/>
-  <xacro:include filename="$(find ant_description)/urdf/sensors/ir_receiver.urdf.xacro"/>
-  <xacro:include filename="$(find ant_description)/urdf/antennas/antenna_array.urdf.xacro"/>
+  <xacro:include filename="$(find pmb2_description)/urdf/deg_to_rad.xacro"/>
+  <xacro:include filename="$(find pmb2_description)/urdf/wheels/wheel_v2.urdf.xacro"/>
+  <xacro:include filename="$(find pmb2_description)/urdf/wheels/caster_v2.urdf.xacro"/>
+  <xacro:include filename="$(find pmb2_description)/urdf/sensors/range.urdf.xacro"/>
+  <xacro:include filename="$(find pmb2_description)/urdf/sensors/sick_tim551_laser.urdf.xacro"/>
+  <xacro:include filename="$(find pmb2_description)/urdf/sensors/xtion_pro_live.urdf.xacro"/>
+  <xacro:include filename="$(find pmb2_description)/urdf/sensors/imu.urdf.xacro"/>
+  <xacro:include filename="$(find pmb2_description)/urdf/sensors/bumper.urdf.xacro"/>
+  <xacro:include filename="$(find pmb2_description)/urdf/sensors/ir_receiver.urdf.xacro"/>
+  <xacro:include filename="$(find pmb2_description)/urdf/antennas/antenna_array.urdf.xacro"/>
   <!-- Wheel characteristics -->
   <property name="wheel_radius"     value="0.0985"/>
@@ -59,5 +59,5 @@
         <origin xyz="0 0 0" rpy="0 0 0" />
         <geometry>
-          <mesh filename="package://ant_description/meshes/base/base_v2.stl" />
+          <mesh filename="package://pmb2_description/meshes/base/base_v2.stl" />
         </geometry>
         <material name="DarkGrey" />
@@ -66,5 +66,5 @@
         <origin xyz="0 0 0" rpy="0 0 0" />
         <geometry>
-          <mesh filename="package://ant_description/meshes/base/base_v2_collision.stl" />
+          <mesh filename="package://pmb2_description/meshes/base/base_v2_collision.stl" />
         </geometry>
         <material name="DarkGrey" />
@@ -111,5 +111,5 @@
     </xacro:bumper-->
     <!-- IMU -->
-    <!-- @todo ant_hardware_gazebo needs an IMU!  -->
+    <!-- @todo pmb2_hardware_gazebo needs an IMU!  -->
     <xacro:imu_sensor name="base_inclinometer" parent="${name}_link" update_rate="100.0">
       <origin xyz="0 0 0" rpy="0 0 0"/>

File: pmb2_description/urdf/base/base_v2_vertical_xtion_pro_live.urdf.xacro (robot description, xacro)
@@ -8,14 +8,14 @@
 -->
 <robot xmlns:xacro="http://ros.org/wiki/xacro">
-  <xacro:include filename="$(find ant_description)/urdf/deg_to_rad.xacro"/>
-  <xacro:include filename="$(find ant_description)/urdf/wheels/wheel_v2.urdf.xacro"/>
-  <xacro:include filename="$(find ant_description)/urdf/wheels/caster_v2.urdf.xacro"/>
-  <xacro:include filename="$(find ant_description)/urdf/sensors/range.urdf.xacro"/>
-  <xacro:include filename="$(find ant_description)/urdf/sensors/sick_tim551_laser.urdf.xacro"/>
-  <xacro:include filename="$(find ant_description)/urdf/sensors/xtion_pro_live.urdf.xacro"/>
-  <xacro:include filename="$(find ant_description)/urdf/sensors/imu.urdf.xacro"/>
-  <xacro:include filename="$(find ant_description)/urdf/sensors/bumper.urdf.xacro"/>
-  <xacro:include filename="$(find ant_description)/urdf/sensors/ir_receiver.urdf.xacro"/>
-  <xacro:include filename="$(find ant_description)/urdf/antennas/antenna_array.urdf.xacro"/>
+  <xacro:include filename="$(find pmb2_description)/urdf/deg_to_rad.xacro"/>
+  <xacro:include filename="$(find pmb2_description)/urdf/wheels/wheel_v2.urdf.xacro"/>
+  <xacro:include filename="$(find pmb2_description)/urdf/wheels/caster_v2.urdf.xacro"/>
+  <xacro:include filename="$(find pmb2_description)/urdf/sensors/range.urdf.xacro"/>
+  <xacro:include filename="$(find pmb2_description)/urdf/sensors/sick_tim551_laser.urdf.xacro"/>
+  <xacro:include filename="$(find pmb2_description)/urdf/sensors/xtion_pro_live.urdf.xacro"/>
+  <xacro:include filename="$(find pmb2_description)/urdf/sensors/imu.urdf.xacro"/>
+  <xacro:include filename="$(find pmb2_description)/urdf/sensors/bumper.urdf.xacro"/>
+  <xacro:include filename="$(find pmb2_description)/urdf/sensors/ir_receiver.urdf.xacro"/>
+  <xacro:include filename="$(find pmb2_description)/urdf/antennas/antenna_array.urdf.xacro"/>
   <!-- Wheel characteristics -->
   <property name="wheel_radius"     value="0.0985"/>
@@ -59,5 +59,5 @@
         <origin xyz="0 0 0" rpy="0 0 0" />
         <geometry>
-          <mesh filename="package://ant_description/meshes/base/base_v2.stl" />
+          <mesh filename="package://pmb2_description/meshes/base/base_v2.stl" />
         </geometry>
         <material name="DarkGrey" />
@@ -66,5 +66,5 @@
         <origin xyz="0 0 0" rpy="0 0 0" />
         <geometry>
-          <mesh filename="package://ant_description/meshes/base/base_v2_collision.stl" />
+          <mesh filename="package://pmb2_description/meshes/base/base_v2_collision.stl" />
         </geometry>
         <material name="DarkGrey" />
@@ -111,5 +111,5 @@
     </xacro:bumper-->
     <!-- IMU -->
-    <!-- @todo ant_hardware_gazebo needs an IMU!  -->
+    <!-- @todo pmb2_hardware_gazebo needs an IMU!  -->
     <xacro:imu_sensor name="base_inclinometer" parent="${name}_link" update_rate="100.0">
       <origin xyz="0 0 0" rpy="0 0 0"/>

File: pmb2_description/urdf/base/base_v2_xtion_pro_live.urdf.xacro (robot description, xacro)
@@ -8,13 +8,13 @@
 -->
 <robot xmlns:xacro="http://ros.org/wiki/xacro">
-  <xacro:include filename="$(find ant_description)/urdf/deg_to_rad.xacro"/>
-  <xacro:include filename="$(find ant_description)/urdf/wheels/wheel_v2.urdf.xacro"/>
-  <xacro:include filename="$(find ant_description)/urdf/wheels/caster_v2.urdf.xacro"/>
-  <xacro:include filename="$(find ant_description)/urdf/sensors/range.urdf.xacro"/>
-  <xacro:include filename="$(find ant_description)/urdf/sensors/sick_tim551_laser.urdf.xacro"/>
-  <xacro:include filename="$(find ant_description)/urdf/sensors/xtion_pro_live.urdf.xacro"/>
-  <xacro:include filename="$(find ant_description)/urdf/sensors/imu.urdf.xacro"/>
-  <xacro:include filename="$(find ant_description)/urdf/sensors/bumper.urdf.xacro"/>
-  <xacro:include filename="$(find ant_description)/urdf/sensors/ir_receiver.urdf.xacro"/>
+  <xacro:include filename="$(find pmb2_description)/urdf/deg_to_rad.xacro"/>
+  <xacro:include filename="$(find pmb2_description)/urdf/wheels/wheel_v2.urdf.xacro"/>
+  <xacro:include filename="$(find pmb2_description)/urdf/wheels/caster_v2.urdf.xacro"/>
+  <xacro:include filename="$(find pmb2_description)/urdf/sensors/range.urdf.xacro"/>
+  <xacro:include filename="$(find pmb2_description)/urdf/sensors/sick_tim551_laser.urdf.xacro"/>
+  <xacro:include filename="$(find pmb2_description)/urdf/sensors/xtion_pro_live.urdf.xacro"/>
+  <xacro:include filename="$(find pmb2_description)/urdf/sensors/imu.urdf.xacro"/>
+  <xacro:include filename="$(find pmb2_description)/urdf/sensors/bumper.urdf.xacro"/>
+  <xacro:include filename="$(find pmb2_description)/urdf/sensors/ir_receiver.urdf.xacro"/>
   <!-- Wheel characteristics -->
   <property name="wheel_radius"     value="0.0985"/>
@@ -53,5 +53,5 @@
         <origin xyz="0 0 0" rpy="0 0 0" />
         <geometry>
-          <mesh filename="package://ant_description/meshes/base/base_v2.stl" />
+          <mesh filename="package://pmb2_description/meshes/base/base_v2.stl" />
         </geometry>
         <material name="DarkGrey" />
@@ -60,5 +60,5 @@
         <origin xyz="0 0 0" rpy="0 0 0" />
         <geometry>
-          <mesh filename="package://ant_description/meshes/base/base_v2_collision.stl" />
+          <mesh filename="package://pmb2_description/meshes/base/base_v2_collision.stl" />
         </geometry>
         <material name="DarkGrey" />
@@ -105,5 +105,5 @@
     </xacro:bumper-->
     <!-- IMU -->
-    <!-- @todo ant_hardware_gazebo needs an IMU!  -->
+    <!-- @todo pmb2_hardware_gazebo needs an IMU!  -->
     <xacro:imu_sensor name="base_inclinometer" parent="${name}_link" update_rate="100.0">
       <origin xyz="0 0 0" rpy="0 0 0"/>

Commit message: commit version 0.2.1
Update maintainer email

commit version 0.2.1

File: pmb2_description/gazebo/gazebo.urdf.xacro (robot description, xacro)
@@ -9,9 +9,11 @@
 <robot xmlns:sensor="http://playerstage.sourceforge.net/gazebo/xmlschema/#sensor"
        xmlns:controller="http://playerstage.sourceforge.net/gazebo/xmlschema/#controller"
-       xmlns:interface="http://playerstage.sourceforge.net/gazebo/xmlschema/#interface">
+       xmlns:interface="http://playerstage.sourceforge.net/gazebo/xmlschema/#interface"
+       name="pmb2">
   <gazebo>
-    <plugin filename="libgazebo_ros_control.so" name="ros_control">
+    <plugin filename="libgazebo_ros_control.so" name="gazebo_ros_control">
       <ns></ns>
-      <robotSimType>pmb2_hardware_gazebo/Pmb2HardwareGazebo</robotSimType>
+      <robotSimType>pal_hardware_gazebo/PalHardwareGazebo</robotSimType>
+      <robotNamespace></robotNamespace>
       <controlPeriod>0.001</controlPeriod>
     </plugin>
@@ -23,4 +25,46 @@
     </plugin>
   </gazebo>
+  <gazebo reference="base_imu_link">
+    <!-- this is expected to be reparented to pelvis with appropriate offset
+         when imu_link is reduced by fixed joint reduction -->
+    <!-- todo: this is working with gazebo 1.4, need to write a unit test -->
+    <sensor name="imu_sensor" type="imu">
+      <always_on>1</always_on>
+      <update_rate>1000.0</update_rate>
+      <imu>
+        <noise>
+          <type>gaussian</type>
+          <!-- Noise parameters from Boston Dynamics
+               (http://gazebosim.org/wiki/Sensor_noise):
+                 rates (rad/s): mean=0, stddev=2e-4
+                 accels (m/s/s): mean=0, stddev=1.7e-2
+                 rate bias (rad/s): 5e-6 - 1e-5
+                 accel bias (m/s/s): 1e-1
+               Experimentally, simulation provide rates with noise of
+               about 1e-3 rad/s and accels with noise of about 1e-1 m/s/s.
+               So we don't expect to see the noise unless number of inner iterations
+               are increased.
+               We will add bias.  In this model, bias is sampled once for rates
+               and once for accels at startup; the sign (negative or positive)
+               of each bias is then switched with equal probability.  Thereafter,
+               the biases are fixed additive offsets.  We choose
+               bias means and stddevs to produce biases close to the provided
+               data. -->
+          <rate>
+            <mean>0.0</mean>
+            <stddev>2e-4</stddev>
+            <bias_mean>0.0000075</bias_mean>
+            <bias_stddev>0.0000008</bias_stddev>
+          </rate>
+          <accel>
+            <mean>0.0</mean>
+            <stddev>1.7e-2</stddev>
+            <bias_mean>0.1</bias_mean>
+            <bias_stddev>0.001</bias_stddev>
+          </accel>
+        </noise>
+      </imu>
+    </sensor>
+  </gazebo>
   <!-- define global properties -->
   <property name="M_PI" value="3.1415926535897931" />

File: pmb2_description/urdf/base/base.urdf.xacro (robot description, xacro)
@@ -11,8 +11,5 @@
   <xacro:include filename="$(find pmb2_description)/urdf/wheels/wheel.urdf.xacro"/>
   <xacro:include filename="$(find pmb2_description)/urdf/wheels/caster.urdf.xacro"/>
-  <xacro:include filename="$(find pmb2_description)/urdf/sensors/range.urdf.xacro"/>
-  <xacro:include filename="$(find pmb2_description)/urdf/sensors/hokuyo_urg_04lx_ug01_laser.urdf.xacro"/>
   <xacro:include filename="$(find pmb2_description)/urdf/sensors/imu.urdf.xacro"/>
-  <xacro:include filename="$(find pmb2_description)/urdf/sensors/microphone.urdf.xacro"/>
   <xacro:include filename="$(find pmb2_description)/urdf/objects/cover.urdf.xacro"/>
   <xacro:include filename="$(find pmb2_description)/urdf/objects/antenna.urdf.xacro"/>
@@ -24,5 +21,5 @@
   <property name="wheel_velocity"   value="1.0"/>
   <!-- Caster wheel characteristics -->
-  <property name="caster_radius"       value="0.026"/>
+  <property name="caster_radius"       value="0.025"/>
   <property name="caster_width"        value="0.015"/>
   <property name="caster_separation_x" value="0.343"/>
@@ -31,8 +28,4 @@
   <property name="caster_offset_y"     value="0.0"/>
   <property name="caster_offset_z"     value="-0.0335"/>
-  <!-- Laser characteristics -->
-  <property name="base_laser_x" value="0.202"/>
-  <property name="base_laser_y" value="0.0"/>
-  <property name="base_laser_z" value="-0.004"/>
   <xacro:macro name="base" params="name">
     <!-- Base -->
@@ -55,5 +48,5 @@
         <origin xyz="0 0 0" rpy="0 0 0" />
         <geometry>
-          <mesh filename="package://pmb2_description/meshes/base/base_collision.stl" />
+          <mesh filename="package://pmb2_description/meshes/base/base_collision.dae" />
         </geometry>
         <material name="White" />
@@ -70,4 +63,15 @@
       <parent link="${name}_footprint"/>
     </joint>
+  <!-- gazebo parameters are given here for base_link thru base_footprint -->
+    <gazebo reference="${name}_footprint">
+      <kp>100000000.0</kp>
+      <kd>10.0</kd>
+      <mu1>0.1</mu1>
+      <mu2>0.1</mu2>
+      <fdir1>1 0 0</fdir1>
+      <maxVel>10.0</maxVel>
+      <minDepth>0.0005</minDepth>
+      <laserRetro>0</laserRetro>
+    </gazebo>
     <!-- Orange cover & antennas -->
     <xacro:cover name="${name}_cover" parent="${name}_footprint"/>
@@ -78,36 +82,9 @@
       <origin xyz="-0.201 -0.1062 0.195" rpy="0 0 0"/>
     </xacro:antenna>
-    <!-- Laser -->
-    <!-- Theoretic FOV = 220 -->
-    <xacro:hokuyo_urg_04lx_ug01_laser name="${name}_laser" parent="${name}" ros_topic="scan" update_rate="10" min_angle="${-110 * deg_to_rad}" max_angle="${110 * deg_to_rad}" >
-      <origin xyz="${base_laser_x} ${base_laser_y} ${base_laser_z}" rpy="0 0 0" />
-    </xacro:hokuyo_urg_04lx_ug01_laser>
-    <!-- Microphones -->
-    <xacro:microphone name="${name}_mic_front_left" parent="${name}">
-      <origin xyz="0.23182 0.03902 0.195" rpy="0 0 0"/>
-    </xacro:microphone>
-    <xacro:microphone name="${name}_mic_front_right" parent="${name}">
-      <origin xyz="0.23182 -0.03902 0.195" rpy="0 0 0"/>
-    </xacro:microphone>
-    <xacro:microphone name="${name}_mic_back_left" parent="${name}">
-      <origin xyz="-0.1082 -0.0599 0.195" rpy="0 0 0"/>
-    </xacro:microphone>
-    <xacro:microphone name="${name}_mic_back_right" parent="${name}">
-      <origin xyz="-0.1082 -0.13789 0.195" rpy="0 0 0"/>
-    </xacro:microphone>
     <!-- IMU -->
+    <!-- @todo pmb2_hardware_gazebo needs an IMU!  -->
     <xacro:imu_sensor name="${name}_imu" parent="${name}_link" update_rate="100.0">
-      <origin xyz="0.10171 0 0.11282" rpy="0 ${180 * deg_to_rad} ${90 * deg_to_rad}"/>
+      <origin xyz="0.10171 0 0.11282" rpy="0 0 ${-90 * deg_to_rad}"/>
     </xacro:imu_sensor>
-    <!-- Sonars -->
-    <xacro:range_sensor name="${name}_sonar_1" parent="${name}" ros_topic="sonar_${name}" update_rate="5" maxRange="0.75" minRange="0.01" fov="0.5" radiation="ultrasound">
-      <origin xyz="-0.183 0.183 0.173" rpy="0 0 ${135 * deg_to_rad}"/>
-    </xacro:range_sensor>
-    <xacro:range_sensor name="${name}_sonar_2" parent="${name}" ros_topic="sonar_${name}" update_rate="5" maxRange="0.75" minRange="0.01" fov="0.5" radiation="ultrasound">
-      <origin xyz="-0.259 0.0 0.173" rpy="0 0 ${180 * deg_to_rad}"/>
-    </xacro:range_sensor>
-    <xacro:range_sensor name="${name}_sonar_3" parent="${name}" ros_topic="sonar_${name}" update_rate="5" maxRange="0.75" minRange="0.01" fov="0.5" radiation="ultrasound">
-      <origin xyz="-0.183 -0.183 0.173" rpy="0 0 ${225 * deg_to_rad}"/>
-    </xacro:range_sensor>
     <!-- Wheels -->
     <xacro:wheel side="right" reflect=" 1.0" radius="${wheel_radius}" width="${wheel_width}" torque="${wheel_torque}" velocity="${wheel_velocity}" separation="${wheel_separation}" parent="${name}"/>

File: pmb2_description/urdf/wheels/caster.gazebo.xacro (robot description, xacro)
@@ -13,6 +13,6 @@
       <kp>1000000.0</kp>
       <kd>100.0</kd>
-      <mu1>0.1</mu1>
-      <mu2>0.1</mu2>
+      <mu1>0</mu1>
+      <mu2>0</mu2>
       <fdir1>1 0 0</fdir1>
       <maxVel>1.0</maxVel>
@@ -23,6 +23,6 @@
       <kp>1000000.0</kp>
       <kd>100.0</kd>
-      <mu1>0.25</mu1>
-      <mu2>0.15</mu2>
+      <mu1>0</mu1>
+      <mu2>0</mu2>
       <fdir1>1 0 0</fdir1>
       <maxVel>1.0</maxVel>

File: pmb2_description/urdf/wheels/wheel.gazebo.xacro (robot description, xacro)
@@ -13,9 +13,9 @@
       <kp>1000000.0</kp>
       <kd>100.0</kd>
-      <mu1>200.0</mu1>
-      <mu2>100.0</mu2>
+      <mu1>1.0</mu1>
+      <mu2>1.0</mu2>
       <fdir1>1 0 0</fdir1>
       <maxVel>1.0</maxVel>
-      <minDepth>0.00</minDepth>
+      <minDepth>0.003</minDepth>
       <implicitSpringDamper>1</implicitSpringDamper>
       <material>Gazebo/DarkGrey</material>

Commit message: Changes for multi pmb2 simulation

File: pmb2_description/gazebo/gazebo.urdf.xacro (robot description, xacro)
@@ -16,5 +16,10 @@
       <ns></ns>
       <robotSimType>pal_hardware_gazebo/PalHardwareGazebo</robotSimType>
-      <robotNamespace></robotNamespace>
+      <xacro:if value="${is_multiple}">
+          <robotNamespace>/${nsp}</robotNamespace>
+      </xacro:if>
+      <xacro:unless value="${is_multiple}">
+          <robotNamespace></robotNamespace>
+      </xacro:unless>
       <controlPeriod>0.001</controlPeriod>
     </plugin>
@@ -24,4 +29,7 @@
       <alwaysOn>true</alwaysOn>
       <updateRate>100.0</updateRate>
+      <xacro:if value="${is_multiple}">
+          <robotNamespace>/${nsp}</robotNamespace>
+      </xacro:if>
     </plugin>
   </gazebo>

File: pmb2_description/robots/pmb2.urdf.xacro (robot description, xacro)
@@ -16,4 +16,8 @@
     <xacro:wrong_laser_model/>
   </xacro:if>
+  <xacro:arg name="multiple" default="false"/>
+  <xacro:arg name="namespace" default=""/>
+  <xacro:property name="is_multiple" value="$(arg multiple)" />
+  <xacro:property name="nsp" value="$(arg namespace)" />
   <!-- The following included files set up definitions of parts of the robot body -->
   <!-- Base -->
