Commit message: Further urdf updates

File: pmb2_description/urdf/base/base_sensors.urdf.xacro (robot description, xacro)
@@ -16,7 +16,7 @@
   <xacro:include filename="$(find pmb2_description)/urdf/sensors/microphone.urdf.xacro"/>
   <!-- Laser characteristics -->
-  <property name="base_laser_x" value="0.202"/>
-  <property name="base_laser_y" value="0.0"/>
-  <property name="base_laser_z" value="-0.004"/>
+  <xacro:property name="base_laser_x" value="0.202"/>
+  <xacro:property name="base_laser_y" value="0.0"/>
+  <xacro:property name="base_laser_z" value="-0.004"/>
   <xacro:macro name="base_sensors" params=" name hokuyo:=false sick551:=false sick561:=false sick571:=false sonars:=false microphone:=false ">
     <xacro:if value="${hokuyo}"> <!-- TODO: find expr that encure only one laser is true -->
@@ -50,11 +50,11 @@
     <xacro:if value="${sonars}">
       <!-- Sonars -->
-      <xacro:range_sensor name="${name}_sonar_03" parent="${name}" ros_topic="sonar_${name}" update_rate="5" maxRange="2.0" minRange="0.02" fov="0.5" radiation="ultrasound">
+      <xacro:range_sensor name="${name}_sonar_03" parent="${name}" ros_topic="sonar_${name}" update_rate="5" maxRange="1.0" minRange="0.02" fov="0.5" radiation="ultrasound">
         <origin xyz="-0.183 0.183 0.173" rpy="0 0 ${135 * deg_to_rad}"/>
       </xacro:range_sensor>
-      <xacro:range_sensor name="${name}_sonar_02" parent="${name}" ros_topic="sonar_${name}" update_rate="5" maxRange="2.0" minRange="0.02" fov="0.5" radiation="ultrasound">
+      <xacro:range_sensor name="${name}_sonar_02" parent="${name}" ros_topic="sonar_${name}" update_rate="5" maxRange="1.0" minRange="0.02" fov="0.5" radiation="ultrasound">
         <origin xyz="-0.259 0.0 0.173" rpy="0 0 ${180 * deg_to_rad}"/>
       </xacro:range_sensor>
-      <xacro:range_sensor name="${name}_sonar_01" parent="${name}" ros_topic="sonar_${name}" update_rate="5" maxRange="2.0" minRange="0.02" fov="0.5" radiation="ultrasound">
+      <xacro:range_sensor name="${name}_sonar_01" parent="${name}" ros_topic="sonar_${name}" update_rate="5" maxRange="1.0" minRange="0.02" fov="0.5" radiation="ultrasound">
         <origin xyz="-0.183 -0.183 0.173" rpy="0 0 ${225 * deg_to_rad}"/>
       </xacro:range_sensor>

File: pmb2_description/urdf/wheels/caster.urdf.xacro (robot description, xacro)
@@ -8,5 +8,4 @@
 -->
 <robot xmlns:xacro="http://ros.org/wiki/xacro">
-  <xacro:include filename="$(find pmb2_description)/urdf/wheels/caster.transmission.xacro"/>
   <xacro:include filename="$(find pmb2_description)/urdf/wheels/caster.gazebo.xacro"/>
   <xacro:macro name="caster" params="side radius width separation_x separation_y offset_x offset_y offset_z parent">
@@ -26,10 +25,10 @@
         <material name="Grey"/>
       </visual>
-      <collision>
+      <!--collision>
         <origin xyz="0 0 0" rpy="0 0 0"/>
         <geometry>
           <cylinder radius="${radius}" length="${width}"/>
         </geometry>
-      </collision>
+      </collision-->
     </link>
     <link name="caster_${side}_2_link">
@@ -69,7 +68,4 @@
     <!-- Gazebo extensions -->
     <xacro:caster_gazebo side="${side}"/>
-    <!-- Transmission -->
-   <xacro:caster_transmission name="caster" side="${side}" number="1" reduction="1.0"/>
-   <xacro:caster_transmission name="caster" side="${side}" number="2" reduction="1.0"/>
   </xacro:macro>
 </robot>

Commit message: updated laser mounting angle

File: pmb2_description/urdf/base/base_sensors.urdf.xacro (robot description, xacro)
@@ -60,5 +60,5 @@
       <!-- Theoretic FOV = 360 -->
       <xacro:ydlidar_tg30_laser name="${name}_laser" parent="${name}" ros_topic="scan_raw" update_rate="10" min_angle="${-180 * deg_to_rad}" max_angle="${180 * deg_to_rad}" >
-        <origin xyz="${base_laser_x} ${base_laser_y} ${base_laser_z}" rpy="0 0 ${ 180 * deg_to_rad }" />
+        <origin xyz="${base_laser_x} ${base_laser_y} ${base_laser_z}" rpy="0 0 ${ -30 * deg_to_rad }" />
       </xacro:ydlidar_tg30_laser>
     </xacro:if>
@@ -67,5 +67,5 @@
       <!-- Theoretic FOV = 360 -->
       <xacro:ydlidar_tg15_laser name="${name}_laser" parent="${name}" ros_topic="scan_raw" update_rate="10" min_angle="${-180 * deg_to_rad}" max_angle="${180 * deg_to_rad}" >
-        <origin xyz="${base_laser_x} ${base_laser_y} ${base_laser_z}" rpy="0 0 ${ 180 * deg_to_rad }" />
+        <origin xyz="${base_laser_x} ${base_laser_y} ${base_laser_z}" rpy="0 0 ${ -30 * deg_to_rad }" />
       </xacro:ydlidar_tg15_laser>
     </xacro:if>

Commit message: Fix urdf tg values

File: pmb2_description/urdf/base/base_sensors.urdf.xacro (robot description, xacro)
@@ -60,5 +60,5 @@
       <!-- Theoretic FOV = 360 -->
       <xacro:ydlidar_tg30_laser name="${name}_laser" parent="${name}" ros_topic="scan_raw" update_rate="10" min_angle="${-65* deg_to_rad}" max_angle="${125 * deg_to_rad}" >
-        <origin xyz="${base_laser_x} ${base_laser_y} ${base_laser_z}" rpy="0 0 ${ -30 * deg_to_rad }" />
+        <origin xyz="0.2095 0 0.00890" rpy="0 0 ${ -30 * deg_to_rad }" />
       </xacro:ydlidar_tg30_laser>
     </xacro:if>
@@ -67,5 +67,5 @@
       <!-- Theoretic FOV = 360 -->
       <xacro:ydlidar_tg15_laser name="${name}_laser" parent="${name}" ros_topic="scan_raw" update_rate="10" min_angle="${-65 * deg_to_rad}" max_angle="${125 * deg_to_rad}" >
-        <origin xyz="${base_laser_x} ${base_laser_y} ${base_laser_z}" rpy="0 0 ${ -30 * deg_to_rad }" />
+        <origin xyz="0.2095 0 0.00890" rpy="0 0 ${ -30 * deg_to_rad }" />
       </xacro:ydlidar_tg15_laser>
     </xacro:if>

Commit message: Update urdf tg values

File: pmb2_description/urdf/base/base_sensors.urdf.xacro (robot description, xacro)
@@ -60,5 +60,5 @@
       <!-- Theoretic FOV = 360 -->
       <xacro:ydlidar_tg30_laser name="${name}_laser" parent="${name}" ros_topic="scan_raw" update_rate="10" min_angle="${-65* deg_to_rad}" max_angle="${125 * deg_to_rad}" >
-        <origin xyz="0.2095 0 0.00890" rpy="0 0 ${ -30 * deg_to_rad }" />
+        <origin xyz="0.2195 0 0.00890" rpy="0 0 ${ -30 * deg_to_rad }" />
       </xacro:ydlidar_tg30_laser>
     </xacro:if>
@@ -67,5 +67,5 @@
       <!-- Theoretic FOV = 360 -->
       <xacro:ydlidar_tg15_laser name="${name}_laser" parent="${name}" ros_topic="scan_raw" update_rate="10" min_angle="${-65 * deg_to_rad}" max_angle="${125 * deg_to_rad}" >
-        <origin xyz="0.2095 0 0.00890" rpy="0 0 ${ -30 * deg_to_rad }" />
+        <origin xyz="0.2195 0 0.00890" rpy="0 0 ${ -30 * deg_to_rad }" />
       </xacro:ydlidar_tg15_laser>
     </xacro:if>

Commit message: General case for parameter

File: pmb2_description/urdf/base/base_sensors.urdf.xacro (robot description, xacro)
@@ -26,4 +26,14 @@
   <xacro:property name="base_laser_y" value="0.0"/>
   <xacro:property name="base_laser_z" value="-0.004"/>
+  <xacro:if value="${laser_model == 'ydlidar-tg15' or laser_model == 'ydlidar-tg30'}">
+    <xacro:property name="base_laser_x" value="0.2195"/>
+    <xacro:property name="base_laser_y" value="0.0"/>
+    <xacro:property name="base_laser_z" value="0.00890"/>
+  </xacro:if>
+  <xacro:unless value="${laser_model == 'ydlidar-tg15' or laser_model == 'ydlidar-tg30'}">
+      <xacro:property name="base_laser_x" value="0.202"/>
+      <xacro:property name="base_laser_y" value="0.0"/>
+      <xacro:property name="base_laser_z" value="-0.004"/>
+  </xacro:unless>
   <!-- laser_model can be: false, hokuyo, sick-551, sick-561, sick-571-->
   <xacro:macro name="base_sensors" params=" name laser_model:=sick-571 sonars:=false microphone:=false ">
@@ -60,5 +70,5 @@
       <!-- Theoretic FOV = 360 -->
       <xacro:ydlidar_tg30_laser name="${name}_laser" parent="${name}" ros_topic="scan_raw" update_rate="10" min_angle="${-65* deg_to_rad}" max_angle="${125 * deg_to_rad}" >
-        <origin xyz="0.2195 0 0.00890" rpy="0 0 ${ -30 * deg_to_rad }" />
+        <origin xyz="${base_laser_x} ${base_laser_y} ${base_laser_z}" rpy="0 0 ${ -30 * deg_to_rad }" />
       </xacro:ydlidar_tg30_laser>
     </xacro:if>
@@ -67,5 +77,5 @@
       <!-- Theoretic FOV = 360 -->
       <xacro:ydlidar_tg15_laser name="${name}_laser" parent="${name}" ros_topic="scan_raw" update_rate="10" min_angle="${-65 * deg_to_rad}" max_angle="${125 * deg_to_rad}" >
-        <origin xyz="0.2195 0 0.00890" rpy="0 0 ${ -30 * deg_to_rad }" />
+        <origin xyz="${base_laser_x} ${base_laser_y} ${base_laser_z}" rpy="0 0 ${ -30 * deg_to_rad }" />
       </xacro:ydlidar_tg15_laser>
     </xacro:if>

Commit message: Put theoretical values urdf tg

File: pmb2_description/urdf/base/base_sensors.urdf.xacro (robot description, xacro)
@@ -27,5 +27,5 @@
   <xacro:property name="base_laser_z" value="-0.004"/>
   <xacro:if value="${laser_model == 'ydlidar-tg15' or laser_model == 'ydlidar-tg30'}">
-    <xacro:property name="base_laser_x" value="0.2195"/>
+    <xacro:property name="base_laser_x" value="0.2095"/>
     <xacro:property name="base_laser_y" value="0.0"/>
     <xacro:property name="base_laser_z" value="0.00890"/>

Commit message: Right inicialization laser properties

File: pmb2_description/urdf/base/base_sensors.urdf.xacro (robot description, xacro)
@@ -26,16 +26,16 @@
   <xacro:property name="base_laser_y" value="0.0"/>
   <xacro:property name="base_laser_z" value="-0.004"/>
-  <xacro:if value="${laser_model == 'ydlidar-tg15' or laser_model == 'ydlidar-tg30'}">
-    <xacro:property name="base_laser_x" value="0.2095"/>
-    <xacro:property name="base_laser_y" value="0.0"/>
-    <xacro:property name="base_laser_z" value="0.00890"/>
-  </xacro:if>
-  <xacro:unless value="${laser_model == 'ydlidar-tg15' or laser_model == 'ydlidar-tg30'}">
-      <xacro:property name="base_laser_x" value="0.202"/>
-      <xacro:property name="base_laser_y" value="0.0"/>
-      <xacro:property name="base_laser_z" value="-0.004"/>
-  </xacro:unless>
   <!-- laser_model can be: false, hokuyo, sick-551, sick-561, sick-571-->
   <xacro:macro name="base_sensors" params=" name laser_model:=sick-571 sonars:=false microphone:=false ">
+    <xacro:if value="${laser_model == 'ydlidar-tg15' or laser_model == 'ydlidar-tg30'}">
+      <xacro:property name="base_laser_x" value="0.2095"/>
+      <xacro:property name="base_laser_y" value="0.0"/>
+      <xacro:property name="base_laser_z" value="0.00890"/>
+    </xacro:if>
+    <xacro:unless value="${laser_model == 'ydlidar-tg15' or laser_model == 'ydlidar-tg30'}">
+        <xacro:property name="base_laser_x" value="0.202"/>
+        <xacro:property name="base_laser_y" value="0.0"/>
+        <xacro:property name="base_laser_z" value="-0.004"/>
+    </xacro:unless>
     <xacro:if value="${laser_model == 'hokuyo'}">
       <!-- Laser -->
