Commit message: Changes for new Gazebo
Signed-off-by: Juancams <jc.manzanares.serrano@gmail.com>

File: pmb2_description/urdf/base/base.gazebo.xacro (robot description, xacro)
@@ -31,5 +31,5 @@
     </gazebo>
     <!-- Odometry plugin for ground truth -->
-    <gazebo>
+    <!-- <gazebo>
       <plugin filename="libgazebo_world_odometry.so" name="gazebo_ros_odometry">
         <ros>
@@ -41,5 +41,5 @@
         <update_rate>100.0</update_rate>
       </plugin>
-    </gazebo>
+    </gazebo> -->
   </xacro:macro>
 </robot>

File: pmb2_description/urdf/base/base.urdf.xacro (robot description, xacro)
@@ -47,5 +47,5 @@
         <origin xyz="0 0 0" rpy="0 0 0" />
         <geometry>
-          <mesh filename="package://pmb2_description/meshes/base/base.stl" />
+          <mesh filename="file://$(find pmb2_description)/meshes/base/base.stl" />
         </geometry>
         <material name="White" />
@@ -54,5 +54,5 @@
         <origin xyz="0 0 0" rpy="0 0 0" />
         <geometry>
-          <mesh filename="package://pmb2_description/meshes/base/high_resolution/base_collision.stl" />
+          <mesh filename="file://$(find pmb2_description)/meshes/base/high_resolution/base_collision.stl" />
         </geometry>
         <material name="White" />

File: pmb2_description/urdf/cameras_add_on/cameras_add_on.urdf.xacro (robot description, xacro)
@@ -84,5 +84,5 @@
         <origin xyz="0 0 0" rpy="0 0 0"/>
         <geometry>
-          <mesh filename="package://pmb2_description/meshes/cameras_add_on/cameras_add_on.stl" scale="1 1 1"/>
+          <mesh filename="file://$(find pmb2_description)/meshes/cameras_add_on/cameras_add_on.stl" scale="1 1 1"/>
         </geometry>
         <material name="White" />
@@ -91,5 +91,5 @@
         <origin xyz="0 0 0" rpy="0 0 0" />
         <geometry>
-          <mesh filename="package://pmb2_description/meshes/cameras_add_on/cameras_add_on_collision.stl" scale="1 1 1"/>
+          <mesh filename="file://$(find pmb2_description)/meshes/cameras_add_on/cameras_add_on_collision.stl" scale="1 1 1"/>
         </geometry>
         <material name="White" />

File: pmb2_description/urdf/wheels/wheel.urdf.xacro (robot description, xacro)
@@ -24,5 +24,5 @@
         <origin xyz="0 0 0" rpy="${-90.0 * (1 - reflect) * deg_to_rad} 0 0"/>
         <geometry>
-          <mesh filename="package://pmb2_description/meshes/wheels/wheel.stl"/>
+          <mesh filename="file://$(find pmb2_description)/meshes/wheels/wheel.stl"/>
         </geometry>
         <material name="DarkGrey"/>
