Commit message: Update URDF (only locations)

File: pmb2_description/urdf/base/base.urdf.xacro (robot description, xacro)
@@ -9,39 +9,44 @@
 <robot xmlns:xacro="http://ros.org/wiki/xacro">
   <xacro:include filename="$(find pmb2_description)/urdf/deg_to_rad.xacro"/>
-  <xacro:include filename="$(find pmb2_description)/urdf/wheels/wheel.urdf.xacro"/>
-  <xacro:include filename="$(find pmb2_description)/urdf/wheels/caster.urdf.xacro"/>
+  <xacro:include filename="$(find pmb2_description)/urdf/wheels/wheel_v2.urdf.xacro"/>
+  <xacro:include filename="$(find pmb2_description)/urdf/wheels/caster_v2.urdf.xacro"/>
   <xacro:include filename="$(find pmb2_description)/urdf/sensors/range.urdf.xacro"/>
-  <xacro:include filename="$(find pmb2_description)/urdf/sensors/hokuyo_urg_04lx_ug01_laser.urdf.xacro"/>
+  <xacro:include filename="$(find pmb2_description)/urdf/sensors/sick_tim551_laser.urdf.xacro"/>
+  <xacro:include filename="$(find pmb2_description)/urdf/sensors/xtion_pro_live.urdf.xacro"/>
   <xacro:include filename="$(find pmb2_description)/urdf/sensors/imu.urdf.xacro"/>
   <xacro:include filename="$(find pmb2_description)/urdf/sensors/bumper.urdf.xacro"/>
   <xacro:include filename="$(find pmb2_description)/urdf/sensors/ir_receiver.urdf.xacro"/>
   <!-- Wheel characteristics -->
-  <property name="wheel_radius"     value="0.100"/>
-  <property name="wheel_width"      value="0.044"/>
-  <property name="wheel_separation" value="0.43408"/>
+  <property name="wheel_radius"     value="0.0985"/>
+  <property name="wheel_width"      value="0.040"/>
+  <property name="wheel_separation" value="0.4044"/>
   <property name="wheel_torque"     value="6.0"/>
   <property name="wheel_velocity"   value="1.0"/>
   <!-- Caster wheel characteristics -->
   <property name="caster_radius"       value="0.025"/>
-  <property name="caster_width"        value="0.020"/>
-  <property name="caster_separation_x" value="0.36734"/>
-  <property name="caster_separation_y" value="0.20362"/>
-  <property name="caster_offset_z"     value="-0.04252"/>
-  <!-- Base characteristics -->
-  <property name="base_radius" value="${(wheel_separation - wheel_width)/2 - 0.01}"/>
-  <property name="base_length" value="0.04"/>
+  <property name="caster_width"        value="0.015"/>
+  <property name="caster_separation_x" value="0.36384"/>
+  <property name="caster_separation_y" value="0.20000"/>
+  <property name="caster_offset_z"     value="-0.0335"/>
   <!-- Laser characteristics -->
-  <property name="base_laser_x" value="0.185"/>
+  <property name="base_laser_x" value="0.202"/>
   <property name="base_laser_y" value="0.0"/>
-  <property name="base_laser_z" value="0.05275"/>
+  <property name="base_laser_z" value="0.04"/>
+  <!-- RGBD characteristics -->
+  <property name="base_rgbd_x" value="0.202"/>
+  <property name="base_rgbd_y" value="0.0"/>
+  <property name="base_rgbd_z" value="0.0925"/>
+  <property name="base_rgbd_R" value="0.0"/>
+  <property name="base_rgbd_P" value="0.0"/>
+  <property name="base_rgbd_Y" value="0.0"/>
   <xacro:macro name="base" params="name">
     <!-- Base -->
     <link name="${name}_link">
       <inertial>
-        <origin xyz="0.0123 0.0071 0.064" rpy="0 0 0" />
-        <mass value="7.95534" />
-        <inertia ixx="0.19540233297" ixy="-0.00188862789" ixz="-0.00370655921"
-                 iyy="0.23325457568" iyz="0.00387528692"
-                 izz="0.3312456162" />
+        <origin xyz="0.00144 0.00003 0.06711" rpy="0 0 0" />
+        <mass value="24.73813" />
+        <inertia ixx="0.50215676906" ixy="0.00014630224" ixz="-0.00851406322"
+                 iyy="0.41873574615" iyz="0.00001868612"
+                 izz="0.64067017495" />
       </inertial>
       <visual>
@@ -55,5 +60,5 @@
         <origin xyz="0 0 0" rpy="0 0 0" />
         <geometry>
-          <cylinder radius="${base_radius}" length="${base_length}"/>
+          <mesh filename="package://pmb2_description/meshes/base/base_collision.stl" />
         </geometry>
         <material name="DarkGrey" />
@@ -68,7 +73,15 @@
     </joint>
     <!-- Laser -->
-    <xacro:hokuyo_urg_04lx_ug01_laser name="${name}_laser" parent="${name}" ros_topic="scan" update_rate="10" min_angle="${-90 * deg_to_rad}" max_angle="${90 * deg_to_rad}" >
+    <!-- Theoretic FOV = 220º -->
+    <xacro:sick_tim551_laser name="${name}_laser" parent="${name}" ros_topic="scan" update_rate="15" min_angle="${-110 * deg_to_rad}" max_angle="${110 * deg_to_rad}" >
       <origin xyz="${base_laser_x} ${base_laser_y} ${base_laser_z}" rpy="0 0 0" />
-    </xacro:hokuyo_urg_04lx_ug01_laser>
+    </xacro:sick_tim551_laser>
+    <!-- RGBD -->
+    <xacro:xtion_pro_live name="${name}_rgbd_camera" parent="${name}">
+      <!-- Pose of sensor frame wrt to base -->
+      <origin xyz="${base_rgbd_x} ${base_rgbd_y} ${base_rgbd_z}" rpy="${base_rgbd_R * deg_to_rad} ${base_rgbd_P * deg_to_rad} ${base_rgbd_Y * deg_to_rad}"/>
+      <!-- Pose of optical frame wrt to sensor -->
+      <origin xyz="0 0 0" rpy="${-90 * deg_to_rad} 0 ${-90 * deg_to_rad}"/>
+    </xacro:xtion_pro_live>
     <!-- Sonar -->
     <!--xacro:range_sensor name="${name}_sonar_02" parent="${name}" ros_topic="sonar_base" update_rate="10" maxRange="0.75" minRange="0.01" fov="0.5" radiation="ultrasound">
@@ -94,5 +107,5 @@
     <!-- @todo pmb2_hardware_gazebo needs an IMU!  -->
     <xacro:imu_sensor name="base_inclinometer" parent="${name}_link" update_rate="100.0">
-      <origin xyz="0 0 ${base_length / 2}" rpy="0 0 0"/>
+      <origin xyz="0 0 0" rpy="0 0 0"/>
     </xacro:imu_sensor>
     <!-- IR receiver -->

Commit message: Add kinematics and stl files (except for the base)

File: pmb2_description/urdf/base/base.urdf.xacro (robot description, xacro)
@@ -9,6 +9,6 @@
 <robot xmlns:xacro="http://ros.org/wiki/xacro">
   <xacro:include filename="$(find pmb2_description)/urdf/deg_to_rad.xacro"/>
-  <xacro:include filename="$(find pmb2_description)/urdf/wheels/wheel_v2.urdf.xacro"/>
-  <xacro:include filename="$(find pmb2_description)/urdf/wheels/caster_v2.urdf.xacro"/>
+  <xacro:include filename="$(find pmb2_description)/urdf/wheels/wheel.urdf.xacro"/>
+  <xacro:include filename="$(find pmb2_description)/urdf/wheels/caster.urdf.xacro"/>
   <xacro:include filename="$(find pmb2_description)/urdf/sensors/range.urdf.xacro"/>
   <xacro:include filename="$(find pmb2_description)/urdf/sensors/sick_tim551_laser.urdf.xacro"/>
@@ -34,7 +34,7 @@
   <property name="base_laser_z" value="0.04"/>
   <!-- RGBD characteristics -->
-  <property name="base_rgbd_x" value="0.202"/>
+  <property name="base_rgbd_x" value="0.2148"/>
   <property name="base_rgbd_y" value="0.0"/>
-  <property name="base_rgbd_z" value="0.0925"/>
+  <property name="base_rgbd_z" value="0.078"/>
   <property name="base_rgbd_R" value="0.0"/>
   <property name="base_rgbd_P" value="0.0"/>
@@ -44,9 +44,9 @@
     <link name="${name}_link">
       <inertial>
-        <origin xyz="0.00144 0.00003 0.06711" rpy="0 0 0" />
-        <mass value="24.73813" />
-        <inertia ixx="0.50215676906" ixy="0.00014630224" ixz="-0.00851406322"
-                 iyy="0.41873574615" iyz="0.00001868612"
-                 izz="0.64067017495" />
+        <origin xyz="-0.00207000000 -0.00057000000 0.04683000000" rpy="0 0 0"/>
+        <mass value="17.38183000000"/>
+        <inertia ixx="0.38959485090" ixy="0.00018406948" ixz="0.00655155749"
+                 iyy="0.33743896167" iyz="0.00005724656"
+                 izz="0.45143616112"/>
       </inertial>
       <visual>
@@ -85,15 +85,23 @@
     </xacro:xtion_pro_live>
     <!-- Sonar -->
-    <!--xacro:range_sensor name="${name}_sonar_02" parent="${name}" ros_topic="sonar_base" update_rate="10" maxRange="0.75" minRange="0.01" fov="0.5" radiation="ultrasound">
-      <origin xyz="0.18 0.0 0.04" rpy="0.0 ${-10.0 * deg_to_rad} 0.0" />
-    </xacro:range_sensor-->
+    <xacro:range_sensor name="${name}_sonar_01" parent="${name}" ros_topic="sonar_base" update_rate="10" maxRange="2.00" minRange="0.01" fov="0.5" radiation="ultrasound">
+      <origin xyz="-0.17571000000 0.17571000000 0.10150000000" rpy="0.0 0.0 ${135.0 * deg_to_rad}"/>
+    </xacro:range_sensor>
     <!-- Sonar -->
-    <!--xacro:range_sensor name="${name}_sonar_03" parent="${name}" ros_topic="sonar_base" update_rate="10" maxRange="0.75" minRange="0.01" fov="0.5" radiation="ultrasound">
-      <origin xyz="0.15 0.1 0.04" rpy="0.0 ${-10.0 * deg_to_rad} ${40.0 * deg_to_rad}" />
-    </xacro:range_sensor-->
+    <xacro:range_sensor name="${name}_sonar_02" parent="${name}" ros_topic="sonar_base" update_rate="10" maxRange="2.00" minRange="0.01" fov="0.5" radiation="ultrasound">
+      <origin xyz="-0.22958000000 0.09510000000 0.10150000000" rpy="0.0 0.0 ${157.5 * deg_to_rad}"/>
+    </xacro:range_sensor>
     <!-- Sonar -->
-    <!--xacro:range_sensor name="${name}_sonar_01" parent="${name}" ros_topic="sonar_base" update_rate="10" maxRange="0.75" minRange="0.01" fov="0.5" radiation="ultrasound">
-      <origin xyz="0.15 -0.1 0.04" rpy="0.0 ${-10.0 * deg_to_rad} ${-40.0 * deg_to_rad}" />
-    </xacro:range_sensor-->
+    <xacro:range_sensor name="${name}_sonar_03" parent="${name}" ros_topic="sonar_base" update_rate="10" maxRange="2.00" minRange="0.01" fov="0.5" radiation="ultrasound">
+      <origin xyz="-0.24850000000 0.00000000000 0.10150000000" rpy="0.0 0.0 ${180.0 * deg_to_rad}"/>
+    </xacro:range_sensor>
+    <!-- Sonar -->
+    <xacro:range_sensor name="${name}_sonar_04" parent="${name}" ros_topic="sonar_base" update_rate="10" maxRange="2.00" minRange="0.01" fov="0.5" radiation="ultrasound">
+      <origin xyz="-0.22958000000 -0.09510000000 0.10150000000" rpy="0.0 0.0 ${202.5 * deg_to_rad}"/>
+    </xacro:range_sensor>
+    <!-- Sonar -->
+    <xacro:range_sensor name="${name}_sonar_05" parent="${name}" ros_topic="sonar_base" update_rate="10" maxRange="2.00" minRange="0.01" fov="0.5" radiation="ultrasound">
+      <origin xyz="-0.17571000000 -0.17571000000 0.10150000000" rpy="0.0 0.0 ${225.0 * deg_to_rad}"/>
+    </xacro:range_sensor>
     <!-- Bumper right -->
     <!--xacro:bumper name="${name}_bumper_01" parent="${name}" ros_topic="bumper_base" update_rate="25" >
@@ -109,16 +117,4 @@
       <origin xyz="0 0 0" rpy="0 0 0"/>
     </xacro:imu_sensor>
-    <!-- IR receiver -->
-    <!--xacro:ir_receiver name="${name}_ir_receiver_01" parent="${name}" ros_topic="ir_receiver_base" update_rate="10" range_min="0.0" range_max="0.75" fov="0.5">
-      <origin xyz="0.17131 0.0 0.180" rpy="0.0 0.0 0.0" />
-    </xacro:ir_receiver-->
-    <!-- IR receiver -->
-    <!--xacro:ir_receiver name="${name}_ir_receiver_02" parent="${name}" ros_topic="ir_receiver_base" update_rate="10" range_min="0.0" range_max="0.75" fov="0.5">
-      <origin xyz="0.16919 0.14919 0.180" rpy="0.0 0.0 0.349" />
-    </xacro:ir_receiver-->
-    <!-- IR receiver -->
-    <!--xacro:ir_receiver name="${name}_ir_receiver_03" parent="${name}" ros_topic="ir_receiver_base" update_rate="10" range_min="0.0" range_max="0.75" fov="0.5">
-      <origin xyz="0.16919 -0.14919 0.180" rpy="0.0 0.0 -0.349" />
-    </xacro:ir_receiver-->
     <!-- Wheels -->
     <xacro:wheel side="right" reflect=" 1.0" radius="${wheel_radius}" width="${wheel_width}" torque="${wheel_torque}" velocity="${wheel_velocity}" separation="${wheel_separation}" parent="${name}"/>

File: pmb2_description/urdf/sensors/hokuyo_urg_04lx_ug01_laser.urdf.xacro (robot description, xacro)
@@ -12,9 +12,9 @@
      <link name="${name}_link" type="laser">
       <inertial>
-        <origin xyz="0 0 -0.04225" rpy="0 0 0" />
-        <mass value="0.160" />
-        <inertia ixx="0.00008631543" ixy="-0.00000088815" ixz="-0.00000094079"
-                 iyy="0.00008461544" iyz="0.00000139389"
-                 izz="0.00005947238" />
+        <origin xyz="0 0 -0.04480000000" rpy="0 0 0"/>
+        <mass value="0.22963000000"/>
+        <inertia ixx="0.00003393164" ixy="0.00000064943" ixz="0.00000000000"
+                 iyy="0.00001849658" iyz="0.00000000000"
+                 izz="0.00005027615"/>
       </inertial>
       <visual>
@@ -27,10 +27,8 @@
     </link>
     <joint name="${name}_joint" type="fixed">
-      <axis xyz="0 1 0" />
-      <insert_block name="origin" />
+      <axis xyz="0 1 0"/>
+      <insert_block name="origin"/>
       <parent link="${parent}_link"/>
       <child  link="${name}_link"/>
-      <dynamics friction="1.0" damping="1"/>
-      <limit lower="0" upper="0" effort="60" velocity="20" />
     </joint>
     <!-- gazebo extensions -->

File: pmb2_description/urdf/sensors/range.urdf.xacro (robot description, xacro)
@@ -12,11 +12,13 @@
     <link name="${name}_link">
       <inertial>
-        <mass value="0.001" />
-        <origin xyz="0 0 0" rpy="0 0 0" />
-        <inertia ixx="0.0001" ixy="0" ixz="0" iyy="0.000001" iyz="0" izz="0.0001" />
+        <mass value="0.001"/>
+        <origin xyz="0 0 0" rpy="0 0 0"/>
+        <inertia ixx="0.000001" ixy="0" ixz="0"
+                 iyy="0.000001" iyz="0"
+                 izz="0.000001"/>
       </inertial>
     </link>
     <joint name="${name}_joint" type="fixed">
-      <insert_block name="origin" />
+      <insert_block name="origin"/>
       <axis xyz="0 0 1"/>
       <parent link="${parent}_link"/>

File: pmb2_description/urdf/sensors/sick_tim551_laser.urdf.xacro (robot description, xacro)
@@ -12,9 +12,9 @@
      <link name="${name}_link" type="laser">
       <inertial>
-        <origin xyz="0 0 -0.04225" rpy="0 0 0" />
-        <mass value="0.160" />
-        <inertia ixx="0.00008631543" ixy="-0.00000088815" ixz="-0.00000094079"
-                 iyy="0.00008461544" iyz="0.00000139389"
-                 izz="0.00005947238" />
+        <origin xyz="-0.02559000000 -0.00056000000 -0.05732000000" rpy="0 0 0"/>
+        <mass value="0.28922000000"/>
+        <inertia ixx="0.00002628919" ixy="0.00000024298" ixz="-0.00000368129"
+                 iyy="0.00003374542" iyz="-0.00000001330"
+                 izz="0.00005832599"/>
       </inertial>
       <visual>
@@ -27,10 +27,8 @@
     </link>
     <joint name="${name}_joint" type="fixed">
-      <axis xyz="0 1 0" />
-      <insert_block name="origin" />
+      <axis xyz="0 1 0"/>
+      <insert_block name="origin"/>
       <parent link="${parent}_link"/>
       <child  link="${name}_link"/>
-      <dynamics friction="1.0" damping="1"/>
-      <limit lower="0" upper="0" effort="60" velocity="20" />
     </joint>
     <!-- gazebo extensions -->

File: pmb2_description/urdf/sensors/xtion_pro_live.urdf.xacro (robot description, xacro)
@@ -31,10 +31,9 @@
     <link name="${name}_link">
       <inertial>
-        <mass value="0.01" />
-        <origin xyz="0 0 0" rpy="0 0 0"/>
-        <!-- inertia tensor computed analytically for a solid cuboid -->
-        <inertia ixx="0.000030"  ixy="0.0"  ixz="0.0"
-                 iyy="0.000030"  iyz="0.0"
-                 izz="0.000002" />
+        <origin xyz="0.21294000000 -0.00003000000 0.09627000000" rpy="0 0 0"/>
+        <mass value="0.21970000000"/>
+        <inertia ixx="0.00000429247" ixy="0.00000000000" ixz="0.00000002565"
+                 iyy="0.00000008027" iyz="0.00000000000"
+                 izz="0.00000427339"/>
       </inertial>
       <visual>

File: pmb2_description/urdf/wheels/caster.urdf.xacro (robot description, xacro)
@@ -13,14 +13,14 @@
     <link name="caster_${side}_1_link">
       <inertial>
-        <origin xyz="-0.00653 -0.00008 -0.01177" rpy="0 0 0"/>
-        <mass value="0.09556"/>
-        <inertia  ixx="0.00002195406" ixy="0.00000000009" ixz="0.00000370909"
-                  iyy="0.00001717745" iyz="-0.00000000032"
-                  izz="0.00002240463"/>
+        <origin xyz="-0.01108 0.00003 -0.030" rpy="0 0 0"/>
+        <mass value="0.101"/>
+        <inertia  ixx="0.00002779423" ixy="-0.00000001384" ixz="0.0000074479"
+                  iyy="0.00002767062" iyz="-0.00000002774"
+                  izz="0.00001727605"/>
       </inertial>
       <visual>
         <origin xyz="0 0 0" rpy="0 0 0"/>
         <geometry>
-          <mesh filename="package://pmb2_description/meshes/wheels/caster.stl"/>
+          <mesh filename="package://pmb2_description/meshes/wheels/caster_1.stl"/>
         </geometry>
         <material name="Grey"/>
@@ -29,5 +29,5 @@
         <origin xyz="0 0 0" rpy="0 0 0"/>
         <geometry>
-          <mesh filename="package://pmb2_description/meshes/wheels/caster.stl"/>
+          <mesh filename="package://pmb2_description/meshes/wheels/caster_1.stl"/>
         </geometry>
       </collision>
@@ -36,13 +36,13 @@
       <inertial>
         <origin xyz="0 0 0" rpy="0 0 0"/>
-        <mass value="0.02425"/>
-        <inertia  ixx="0.00000464376" ixy="0" ixz="0"
-                  iyy="0.00000464377" iyz="0"
-                  izz="0.00000802779"/>
+        <mass value="0.03677"/>
+        <inertia  ixx="0.00000755221" ixy="0" ixz="0"
+                  iyy="0.00000755221" iyz="0"
+                  izz="0.00001281996"/>
         </inertial>
       <visual>
         <origin xyz="0 0 0" rpy="0 0 0"/>
         <geometry>
-          <cylinder radius="${radius}" length="${width}"/>
+          <mesh filename="package://pmb2_description/meshes/wheels/caster_2.stl"/>
         </geometry>
         <material name="DarkGrey"/>
@@ -72,5 +72,5 @@
       <parent link="caster_${side}_1_link"/>
       <child link="caster_${side}_2_link"/>
-      <origin xyz="-0.017 0.0003 -0.032" rpy="${-90.0 * deg_to_rad} 0 0"/>
+      <origin xyz="-0.016 0.0000 -0.040" rpy="${-90.0 * deg_to_rad} 0 0"/>
       <axis xyz="0 0 1"/>
     </joint>

File: pmb2_description/urdf/wheels/wheel.urdf.xacro (robot description, xacro)
@@ -13,14 +13,14 @@
     <link name="wheel_${side}_link">
       <inertial>
-        <origin xyz="0 0 ${-0.0016 * reflect}" rpy="0 0 0"/>
-        <mass value="3.33926"/>
-        <inertia ixx="0.00668369447" ixy="${ 0.00000007414 * reflect}" ixz="0.00000024433"
-                 iyy="0.00668332554" iyz="${-0.00000005662 * reflect}"
-                 izz="0.01088090651"/>
+        <origin xyz="0 0 ${-0.00207 * reflect}" rpy="0 0 0"/>
+        <mass value="1.82362"/>
+        <inertia ixx="0.00499743171" ixy="${ 0.00000004464 * reflect}" ixz="-0.00000002245"
+                 iyy="0.00499741733" iyz="${-0.00000000164 * reflect}"
+                 izz="0.00839239692"/>
       </inertial>
       <visual>
-        <origin xyz="0 0 0" rpy="0 0 0"/>
+        <origin xyz="0 0 0" rpy="${-90.0 * (1 - reflect) * deg_to_rad} 0 0"/>
         <geometry>
-          <cylinder radius="${radius}" length="${width}"/>
+          <mesh filename="package://pmb2_description/meshes/wheels/wheel.stl"/>
         </geometry>
         <material name="LightGrey"/>
