Commit message: Update meshes

File: pmb2_description/urdf/base/base.urdf.xacro (robot description, xacro)
@@ -16,4 +16,8 @@
   <xacro:include filename="$(find pmb2_description)/urdf/sensors/imu.urdf.xacro"/>
   <xacro:include filename="$(find pmb2_description)/urdf/sensors/bumper.urdf.xacro"/>
+  <xacro:include filename="$(find pmb2_description)/urdf/objects/battery_tlh_2.urdf.xacro"/>
+  <xacro:include filename="$(find pmb2_description)/urdf/objects/charger.urdf.xacro"/>
+  <xacro:include filename="$(find pmb2_description)/urdf/objects/cover.urdf.xacro"/>
+  <xacro:include filename="$(find pmb2_description)/urdf/objects/rear_cover_ultrasound.urdf.xacro"/>
   <!-- Wheel characteristics -->
   <property name="wheel_radius"     value="0.0985"/>
@@ -25,11 +29,13 @@
   <property name="caster_radius"       value="0.025"/>
   <property name="caster_width"        value="0.015"/>
-  <property name="caster_separation_x" value="0.36384"/>
+  <property name="caster_separation_x" value="0.350"/>
   <property name="caster_separation_y" value="0.20000"/>
+  <property name="caster_offset_x"     value="-0.002"/>
+  <property name="caster_offset_y"     value="0.0"/>
   <property name="caster_offset_z"     value="-0.0335"/>
   <!-- Laser characteristics -->
   <property name="base_laser_x" value="0.202"/>
   <property name="base_laser_y" value="0.0"/>
-  <property name="base_laser_z" value="0.04"/>
+  <property name="base_laser_z" value="-0.004"/>
   <!-- RGBD characteristics -->
   <property name="base_rgbd_x" value="0.2148"/>
@@ -65,10 +71,18 @@
     </link>
     <!-- Base footprint -->
-    <link name="${name}_footprint"/>
+    <link name="${name}_footprint_link"/>
     <joint name="${name}_footprint_joint" type="fixed">
       <origin xyz="0 0 ${wheel_radius}" rpy="0 0 0" />
       <child link="${name}_link" />
-      <parent link="${name}_footprint"/>
+      <parent link="${name}_footprint_link"/>
     </joint>
+    <!-- Battery -->
+    <xacro:battery name="${name}_battery" parent="${name}_footprint"/>
+    <!-- Charger -->
+    <xacro:charger name="${name}_charger" parent="${name}_footprint"/>
+    <!-- Cover -->
+    <xacro:cover name="${name}_cover" parent="${name}_footprint"/>
+    <!-- Rear cover -->
+    <xacro:rear_cover name="${name}_rear_cover" parent="${name}_footprint"/>
     <!-- Laser -->
     <!-- Theoretic FOV = 220º -->
@@ -83,29 +97,24 @@
       <origin xyz="0 0 0" rpy="${-90 * deg_to_rad} 0 ${-90 * deg_to_rad}"/>
     </xacro:xtion_pro_live>
-    <!-- Sonar -->
+    <!-- Sonars -->
     <xacro:range_sensor name="${name}_sonar_01" parent="${name}" ros_topic="sonar_base" update_rate="10" maxRange="2.00" minRange="0.01" fov="0.5" radiation="ultrasound">
       <origin xyz="-0.17571000000 0.17571000000 0.10150000000" rpy="0.0 0.0 ${135.0 * deg_to_rad}"/>
     </xacro:range_sensor>
-    <!-- Sonar -->
     <xacro:range_sensor name="${name}_sonar_02" parent="${name}" ros_topic="sonar_base" update_rate="10" maxRange="2.00" minRange="0.01" fov="0.5" radiation="ultrasound">
       <origin xyz="-0.22958000000 0.09510000000 0.10150000000" rpy="0.0 0.0 ${157.5 * deg_to_rad}"/>
     </xacro:range_sensor>
-    <!-- Sonar -->
     <xacro:range_sensor name="${name}_sonar_03" parent="${name}" ros_topic="sonar_base" update_rate="10" maxRange="2.00" minRange="0.01" fov="0.5" radiation="ultrasound">
       <origin xyz="-0.24850000000 0.00000000000 0.10150000000" rpy="0.0 0.0 ${180.0 * deg_to_rad}"/>
     </xacro:range_sensor>
-    <!-- Sonar -->
     <xacro:range_sensor name="${name}_sonar_04" parent="${name}" ros_topic="sonar_base" update_rate="10" maxRange="2.00" minRange="0.01" fov="0.5" radiation="ultrasound">
       <origin xyz="-0.22958000000 -0.09510000000 0.10150000000" rpy="0.0 0.0 ${202.5 * deg_to_rad}"/>
     </xacro:range_sensor>
-    <!-- Sonar -->
     <xacro:range_sensor name="${name}_sonar_05" parent="${name}" ros_topic="sonar_base" update_rate="10" maxRange="2.00" minRange="0.01" fov="0.5" radiation="ultrasound">
       <origin xyz="-0.17571000000 -0.17571000000 0.10150000000" rpy="0.0 0.0 ${225.0 * deg_to_rad}"/>
     </xacro:range_sensor>
-    <!-- Bumper right -->
+    <!-- Bumpers -->
     <!--xacro:bumper name="${name}_bumper_01" parent="${name}" ros_topic="bumper_base" update_rate="25" >
       <origin xyz="0.16 -0.12 0.00" rpy="0 0 ${-20.0 * deg_to_rad}" />
     </xacro:bumper-->
-    <!-- Bumper left -->
     <!--xacro:bumper name="${name}_bumper_02" parent="${name}" ros_topic="bumper_base" update_rate="25" >
       <origin xyz="0.16 0.12 0.00" rpy="0 0 ${20.0 * deg_to_rad}" />
@@ -120,8 +129,8 @@
     <xacro:wheel side="left"  reflect="-1.0" radius="${wheel_radius}" width="${wheel_width}" torque="${wheel_torque}" velocity="${wheel_velocity}" separation="${wheel_separation}" parent="${name}"/>
     <!-- Casters wheels -->
-    <xacro:caster side="front_right" radius="${caster_radius}" width="${caster_width}" separation_x="${ caster_separation_x}" separation_y="${ caster_separation_y}" offset_z="${caster_offset_z}" parent="${name}"/>
-    <xacro:caster side="front_left"  radius="${caster_radius}" width="${caster_width}" separation_x="${ caster_separation_x}" separation_y="${-caster_separation_y}" offset_z="${caster_offset_z}" parent="${name}"/>
-    <xacro:caster side="back_right"  radius="${caster_radius}" width="${caster_width}" separation_x="${-caster_separation_x}" separation_y="${ caster_separation_y}" offset_z="${caster_offset_z}" parent="${name}"/>
-    <xacro:caster side="back_left"   radius="${caster_radius}" width="${caster_width}" separation_x="${-caster_separation_x}" separation_y="${-caster_separation_y}" offset_z="${caster_offset_z}" parent="${name}"/>
+    <xacro:caster side="front_right" radius="${caster_radius}" width="${caster_width}" separation_x="${ caster_separation_x}" separation_y="${ caster_separation_y}" offset_x="${caster_offset_x}" offset_y="${caster_offset_y}" offset_z="${caster_offset_z}" parent="${name}"/>
+    <xacro:caster side="front_left"  radius="${caster_radius}" width="${caster_width}" separation_x="${ caster_separation_x}" separation_y="${-caster_separation_y}" offset_x="${caster_offset_x}" offset_y="${caster_offset_y}" offset_z="${caster_offset_z}" parent="${name}"/>
+    <xacro:caster side="back_right"  radius="${caster_radius}" width="${caster_width}" separation_x="${-caster_separation_x}" separation_y="${ caster_separation_y}" offset_x="${caster_offset_x}" offset_y="${caster_offset_y}" offset_z="${caster_offset_z}" parent="${name}"/>
+    <xacro:caster side="back_left"   radius="${caster_radius}" width="${caster_width}" separation_x="${-caster_separation_x}" separation_y="${-caster_separation_y}" offset_x="${caster_offset_x}" offset_y="${caster_offset_y}" offset_z="${caster_offset_z}" parent="${name}"/>
   </xacro:macro>
 </robot>

File: pmb2_description/urdf/wheels/caster.urdf.xacro (robot description, xacro)
@@ -10,5 +10,5 @@
   <xacro:include filename="$(find pmb2_description)/urdf/wheels/caster.transmission.xacro"/>
   <xacro:include filename="$(find pmb2_description)/urdf/wheels/caster.gazebo.xacro"/>
-  <xacro:macro name="caster" params="side radius width separation_x separation_y offset_z parent">
+  <xacro:macro name="caster" params="side radius width separation_x separation_y offset_x offset_y offset_z parent">
     <link name="caster_${side}_1_link">
       <inertial>
@@ -66,5 +66,5 @@
       <parent link="${parent}_link"/>
       <child link="caster_${side}_1_link"/>
-      <origin xyz="${separation_x / 2} ${-separation_y / 2} ${offset_z}" rpy="0 0 0"/>
+      <origin xyz="${offset_x + separation_x / 2} ${offset_y - separation_y / 2} ${offset_z}" rpy="0 0 0"/>
       <axis xyz="0 0 1"/>
     </joint>

Commit message: Update meshes

File: pmb2_description/urdf/base/base.urdf.xacro (robot description, xacro)
@@ -39,7 +39,7 @@
   <property name="base_laser_z" value="-0.004"/>
   <!-- RGBD characteristics -->
-  <property name="base_rgbd_x" value="0.2148"/>
+  <property name="base_rgbd_x" value="0.2223"/>
   <property name="base_rgbd_y" value="0.0"/>
-  <property name="base_rgbd_z" value="0.078"/>
+  <property name="base_rgbd_z" value="0.099"/>
   <property name="base_rgbd_R" value="0.0"/>
   <property name="base_rgbd_P" value="0.0"/>
@@ -71,9 +71,9 @@
     </link>
     <!-- Base footprint -->
-    <link name="${name}_footprint_link"/>
+    <link name="${name}_footprint"/>
     <joint name="${name}_footprint_joint" type="fixed">
       <origin xyz="0 0 ${wheel_radius}" rpy="0 0 0" />
       <child link="${name}_link" />
-      <parent link="${name}_footprint_link"/>
+      <parent link="${name}_footprint"/>
     </joint>
     <!-- Battery -->
@@ -98,17 +98,17 @@
     </xacro:xtion_pro_live>
     <!-- Sonars -->
-    <xacro:range_sensor name="${name}_sonar_01" parent="${name}" ros_topic="sonar_base" update_rate="10" maxRange="2.00" minRange="0.01" fov="0.5" radiation="ultrasound">
+    <xacro:range_sensor name="${name}_sonar_01" parent="${name}" ros_topic="sonar_base" update_rate="10" maxRange="0.30" minRange="0.01" fov="${60.0 * deg_to_rad}" radiation="ultrasound">
       <origin xyz="-0.17571000000 0.17571000000 0.10150000000" rpy="0.0 0.0 ${135.0 * deg_to_rad}"/>
     </xacro:range_sensor>
-    <xacro:range_sensor name="${name}_sonar_02" parent="${name}" ros_topic="sonar_base" update_rate="10" maxRange="2.00" minRange="0.01" fov="0.5" radiation="ultrasound">
+    <xacro:range_sensor name="${name}_sonar_02" parent="${name}" ros_topic="sonar_base" update_rate="10" maxRange="0.30" minRange="0.01" fov="${60.0 * deg_to_rad}" radiation="ultrasound">
       <origin xyz="-0.22958000000 0.09510000000 0.10150000000" rpy="0.0 0.0 ${157.5 * deg_to_rad}"/>
     </xacro:range_sensor>
-    <xacro:range_sensor name="${name}_sonar_03" parent="${name}" ros_topic="sonar_base" update_rate="10" maxRange="2.00" minRange="0.01" fov="0.5" radiation="ultrasound">
+    <xacro:range_sensor name="${name}_sonar_03" parent="${name}" ros_topic="sonar_base" update_rate="10" maxRange="0.30" minRange="0.01" fov="${60.0 * deg_to_rad}" radiation="ultrasound">
       <origin xyz="-0.24850000000 0.00000000000 0.10150000000" rpy="0.0 0.0 ${180.0 * deg_to_rad}"/>
     </xacro:range_sensor>
-    <xacro:range_sensor name="${name}_sonar_04" parent="${name}" ros_topic="sonar_base" update_rate="10" maxRange="2.00" minRange="0.01" fov="0.5" radiation="ultrasound">
+    <xacro:range_sensor name="${name}_sonar_04" parent="${name}" ros_topic="sonar_base" update_rate="10" maxRange="0.30" minRange="0.01" fov="${60.0 * deg_to_rad}" radiation="ultrasound">
       <origin xyz="-0.22958000000 -0.09510000000 0.10150000000" rpy="0.0 0.0 ${202.5 * deg_to_rad}"/>
     </xacro:range_sensor>
-    <xacro:range_sensor name="${name}_sonar_05" parent="${name}" ros_topic="sonar_base" update_rate="10" maxRange="2.00" minRange="0.01" fov="0.5" radiation="ultrasound">
+    <xacro:range_sensor name="${name}_sonar_05" parent="${name}" ros_topic="sonar_base" update_rate="10" maxRange="0.30" minRange="0.01" fov="${60.0 * deg_to_rad}" radiation="ultrasound">
       <origin xyz="-0.17571000000 -0.17571000000 0.10150000000" rpy="0.0 0.0 ${225.0 * deg_to_rad}"/>
     </xacro:range_sensor>

File: pmb2_description/urdf/objects/battery_atp.urdf.xacro (robot description, xacro)
@@ -24,13 +24,7 @@
         <material name="DarkGrey"/>
       </visual>
-      <collision>
-        <origin xyz="0 0 0" rpy="0 0 0"/>
-        <geometry>
-          <mesh filename="package://pmb2_description/meshes/objects/battery_atp.stl"/>
-        </geometry>
-      </collision>
     </link>
     <joint name="battery_joint" type="fixed">
-      <parent link="${parent}_link"/>
+      <parent link="${parent}"/>
       <child link="${name}_link"/>
       <origin xyz="0 0 0.0985" rpy="0 0 0"/>

File: pmb2_description/urdf/objects/battery_atp_2.urdf.xacro (robot description, xacro)
@@ -24,13 +24,7 @@
         <material name="DarkGrey"/>
       </visual>
-      <collision>
-        <origin xyz="0 0 0" rpy="0 0 0"/>
-        <geometry>
-          <mesh filename="package://pmb2_description/meshes/objects/battery_atp_2.stl"/>
-        </geometry>
-      </collision>
     </link>
     <joint name="battery_joint" type="fixed">
-      <parent link="${parent}_link"/>
+      <parent link="${parent}"/>
       <child link="${name}_link"/>
       <origin xyz="0 0 0.0985" rpy="0 0 0"/>

File: pmb2_description/urdf/objects/battery_tlh.urdf.xacro (robot description, xacro)
@@ -24,13 +24,7 @@
         <material name="DarkGrey"/>
       </visual>
-      <collision>
-        <origin xyz="0 0 0" rpy="0 0 0"/>
-        <geometry>
-          <mesh filename="package://pmb2_description/meshes/objects/battery_tlh.stl"/>
-        </geometry>
-      </collision>
     </link>
     <joint name="battery_joint" type="fixed">
-      <parent link="${parent}_link"/>
+      <parent link="${parent}"/>
       <child link="${name}_link"/>
       <origin xyz="0 0 0.0985" rpy="0 0 0"/>

File: pmb2_description/urdf/objects/battery_tlh_2.urdf.xacro (robot description, xacro)
@@ -24,13 +24,7 @@
         <material name="DarkGrey"/>
       </visual>
-      <collision>
-        <origin xyz="0 0 0" rpy="0 0 0"/>
-        <geometry>
-          <mesh filename="package://pmb2_description/meshes/objects/battery_tlh_2.stl"/>
-        </geometry>
-      </collision>
     </link>
     <joint name="battery_joint" type="fixed">
-      <parent link="${parent}_link"/>
+      <parent link="${parent}"/>
       <child link="${name}_link"/>
       <origin xyz="0 0 0.0985" rpy="0 0 0"/>

File: pmb2_description/urdf/objects/charger.urdf.xacro (robot description, xacro)
@@ -24,13 +24,7 @@
         <material name="DarkGrey"/>
       </visual>
-      <collision>
-        <origin xyz="0 0 0" rpy="0 0 0"/>
-        <geometry>
-          <mesh filename="package://pmb2_description/meshes/objects/charger.stl"/>
-        </geometry>
-      </collision>
     </link>
     <joint name="charger_joint" type="fixed">
-      <parent link="${parent}_link"/>
+      <parent link="${parent}"/>
       <child link="${name}_link"/>
       <origin xyz="0 0 0.0985" rpy="0 0 0"/>

File: pmb2_description/urdf/objects/cover.urdf.xacro (robot description, xacro)
@@ -24,13 +24,7 @@
         <material name="LightGrey"/>
       </visual>
-      <collision>
-        <origin xyz="0 0 0" rpy="0 0 0"/>
-        <geometry>
-          <mesh filename="package://pmb2_description/meshes/objects/cover.stl"/>
-        </geometry>
-      </collision>
     </link>
     <joint name="cover_joint" type="fixed">
-      <parent link="${parent}_link"/>
+      <parent link="${parent}"/>
       <child link="${name}_link"/>
       <origin xyz="0 0 0.0985" rpy="0 0 0"/>

File: pmb2_description/urdf/objects/rear_cover_planar.urdf.xacro (robot description, xacro)
@@ -24,13 +24,7 @@
         <material name="LightGrey"/>
       </visual>
-      <collision>
-        <origin xyz="0 0 0" rpy="0 0 0"/>
-        <geometry>
-          <mesh filename="package://pmb2_description/meshes/objects/rear_cover_planar.stl"/>
-        </geometry>
-      </collision>
     </link>
     <joint name="rear_cover_joint" type="fixed">
-      <parent link="${parent}_link"/>
+      <parent link="${parent}"/>
       <child link="${name}_link"/>
       <origin xyz="0 0 0.0985" rpy="0 0 0"/>

File: pmb2_description/urdf/objects/rear_cover_ultrasound.urdf.xacro (robot description, xacro)
@@ -24,13 +24,7 @@
         <material name="LightGrey"/>
       </visual>
-      <collision>
-        <origin xyz="0 0 0" rpy="0 0 0"/>
-        <geometry>
-          <mesh filename="package://pmb2_description/meshes/objects/rear_cover_ultrasound.stl"/>
-        </geometry>
-      </collision>
     </link>
     <joint name="rear_cover_joint" type="fixed">
-      <parent link="${parent}_link"/>
+      <parent link="${parent}"/>
       <child link="${name}_link"/>
       <origin xyz="0 0 0.0985" rpy="0 0 0"/>

File: pmb2_description/urdf/sensors/xtion_pro_live.urdf.xacro (robot description, xacro)
@@ -31,5 +31,5 @@
     <link name="${name}_link">
       <inertial>
-        <origin xyz="0.21294000000 -0.00003000000 0.09627000000" rpy="0 0 0"/>
+        <origin xyz="-0.00936000000 -0.00003000000 -0.00273000000" rpy="0 0 0"/>
         <mass value="0.21970000000"/>
         <inertia ixx="0.00000429247" ixy="0.00000000000" ixz="0.00000002565"
@@ -40,16 +40,8 @@
         <origin xyz="0 0 0" rpy="0 0 0"/>
         <geometry>
-          <mesh filename="package://pmb2_description/meshes/sensors/xtion_pro_live/xtion_pro_live.dae" />
+          <mesh filename="package://pmb2_description/meshes/sensors/xtion_pro_live.stl"/>
         </geometry>
-        <material name="Grey">
-          <color rgba="0.5 0.5 0.5 1"/>
-        </material>
+        <material name="DarkGrey"/>
       </visual>
-      <collision>
-        <origin xyz="-0.01 0.0025 0" rpy="0 0 0"/>
-        <geometry>
-          <box size="0.04 0.185 0.03"/>
-        </geometry>
-      </collision>
     </link>
     <joint name="${name}_optical_joint" type="fixed">
@@ -58,13 +50,5 @@
       <child link="${name}_optical_frame"/>
     </joint>
-    <link name="${name}_optical_frame">
-      <inertial>
-        <mass value="0.01" />
-        <origin xyz="0 0 0" rpy="0 0 0"/>
-        <inertia ixx="0.0"  ixy="0.0"  ixz="0.0"
-                 iyy="0.0"  iyz="0.0"
-                 izz="0.0" />
-      </inertial>
-    </link>
+    <link name="${name}_optical_frame"/>
     <!-- frames of the depth sensor -->
     <joint name="${name}_depth_joint" type="fixed">

File: pmb2_description/urdf/wheels/caster.urdf.xacro (robot description, xacro)
@@ -26,10 +26,4 @@
         <material name="Grey"/>
       </visual>
-      <collision>
-        <origin xyz="0 0 0" rpy="0 0 0"/>
-        <geometry>
-          <mesh filename="package://pmb2_description/meshes/wheels/caster_1.stl"/>
-        </geometry>
-      </collision>
     </link>
     <link name="caster_${side}_2_link">

File: pmb2_description/urdf/wheels/wheel.urdf.xacro (robot description, xacro)
@@ -24,5 +24,5 @@
           <mesh filename="package://pmb2_description/meshes/wheels/wheel.stl"/>
         </geometry>
-        <material name="LightGrey"/>
+        <material name="DarkGrey"/>
       </visual>
       <collision>
