Commit message: Add bumper

File: pmb2_description/urdf/base/base.urdf.xacro (robot description, xacro)
@@ -49,9 +49,9 @@
     <link name="${name}_link">
       <inertial>
-        <origin xyz="-0.00207000000 -0.00057000000 0.04683000000" rpy="0 0 0"/>
-        <mass value="17.38183000000"/>
-        <inertia ixx="0.38959485090" ixy="0.00018406948" ixz="0.00655155749"
-                 iyy="0.33743896167" iyz="0.00005724656"
-                 izz="0.45143616112"/>
+        <origin xyz="-0.00393000000 -0.00057000000 0.04788000000" rpy="0 0 0"/>
+        <mass value="17.22815000000"/>
+        <inertia ixx="0.38502800825" ixy="0.00017569597" ixz="0.00983980386"
+                 iyy="0.32897158338" iyz="-0.00013935331"
+                 izz="0.44188721859"/>
       </inertial>
       <visual>
@@ -114,10 +114,8 @@
     </xacro:range_sensor>
     <!-- Bumpers -->
-    <!--xacro:bumper name="${name}_bumper_01" parent="${name}" ros_topic="bumper_base" update_rate="25" >
-      <origin xyz="0.16 -0.12 0.00" rpy="0 0 ${-20.0 * deg_to_rad}" />
-    </xacro:bumper-->
-    <!--xacro:bumper name="${name}_bumper_02" parent="${name}" ros_topic="bumper_base" update_rate="25" >
-      <origin xyz="0.16 0.12 0.00" rpy="0 0 ${20.0 * deg_to_rad}" />
-    </xacro:bumper-->
+    257.000.00-64.50
+    <xacro:bumper name="${name}_bumper" parent="${name}" ros_topic="bumper_base" update_rate="10">
+      <origin xyz="0.257 0.00 -0.0645" rpy="0 0 0"/>
+    </xacro:bumper>
     <!-- IMU -->
     <!-- @todo pmb2_hardware_gazebo needs an IMU!  -->

File: pmb2_description/urdf/sensors/bumper.urdf.xacro (robot description, xacro)
@@ -10,30 +10,33 @@
   <xacro:include filename="$(find pmb2_description)/urdf/sensors/bumper.gazebo.xacro" />
   <xacro:macro name="bumper" params="name parent ros_topic update_rate *origin">
-     <joint name="${name}_joint" type="fixed">
-        <axis xyz="0 1 0" />
-        <insert_block name="origin" />
-        <parent link="base_link"/>
-        <child link="${name}_link"/>
-      </joint>
-      <link name="${name}_link">
-         <inertial>
-           <mass value="1.0" />
-           <inertia ixx="0.01" ixy="0.0" ixz="0.0" iyy="0.01" iyz="0.0" izz="0.01" />
-         </inertial>
-         <!--visual>
-           <origin xyz="0 0 0" rpy="0 0 0" />
-           <geometry>
-              <box size="0.01 0.25 0.04"/>
-           </geometry>
-           <material name="DarkGrey"/>
-         </visual-->
-         <collision>
-           <origin xyz="0 0 0" rpy="0 0 0" />
-           <geometry>
-              <box size="0.01 0.25 0.04"/>
-           </geometry>
-           <material name="DarkGrey" />
-         </collision>
-       </link>
+    <link name="${name}_link">
+      <inertial>
+        <origin xyz="-0.05002000000 0.00000000000 0.00000000000" rpy="0 0 0"/>
+        <mass value="0.15368000000"/>
+        <inertia ixx="0.00281031560" ixy="0.00000000000" ixz="0.00000000000"
+                 iyy="0.00021829037" iyz="0.00000000000"
+                 izz="0.00302258512"/>
+      </inertial>
+      <visual>
+        <origin xyz="0 0 0" rpy="0 0 0" />
+        <geometry>
+          <mesh filename="package://pmb2_description/meshes/sensors/bumper.stl"/>
+        </geometry>
+        <material name="DarkGrey"/>
+      </visual>
+      <collision>
+        <origin xyz="0 0 0" rpy="0 0 0" />
+        <geometry>
+          <mesh filename="package://pmb2_description/meshes/sensors/bumper_collision.stl"/>
+        </geometry>
+        <material name="DarkGrey"/>
+      </collision>
+    </link>
+    <joint name="${name}_joint" type="fixed">
+      <axis xyz="0 1 0"/>
+      <insert_block name="origin"/>
+      <parent link="${parent}_link"/>
+      <child  link="${name}_link"/>
+    </joint>
     <!-- gazebo extensions -->
     <xacro:bumper_gazebo name="${name}" ros_topic="${ros_topic}" update_rate="${update_rate}" />

File: pmb2_description/urdf/sensors/hokuyo_urg_04lx_ug01_laser.urdf.xacro (robot description, xacro)
@@ -10,5 +10,5 @@
   <xacro:include filename="$(find pmb2_description)/urdf/sensors/hokuyo_urg_04lx_ug01_laser.gazebo.xacro" />
   <xacro:macro name="hokuyo_urg_04lx_ug01_laser" params="name parent *origin ros_topic update_rate min_angle max_angle">
-     <link name="${name}_link" type="laser">
+    <link name="${name}_link" type="laser">
       <inertial>
         <origin xyz="0 0 -0.04480000000" rpy="0 0 0"/>
@@ -23,5 +23,5 @@
           <mesh filename="package://pmb2_description/meshes/sensors/hokuyo_urg_04lx_ug01.stl"/>
         </geometry>
-        <material name="DarkGrey" />
+        <material name="DarkGrey"/>
       </visual>
     </link>

File: pmb2_description/urdf/sensors/range.urdf.xacro (robot description, xacro)
@@ -11,11 +11,11 @@
   <xacro:macro name="range_sensor" params="name parent *origin ros_topic update_rate maxRange minRange fov radiation">
     <link name="${name}_link">
-      <inertial>
-        <mass value="0.001"/>
-        <origin xyz="0 0 0" rpy="0 0 0"/>
-        <inertia ixx="0.000001" ixy="0" ixz="0"
-                 iyy="0.000001" iyz="0"
-                 izz="0.000001"/>
-      </inertial>
+       <visual>
+        <origin xyz="0 0 0" rpy="0 0 0" />
+        <geometry>
+          <mesh filename="package://pmb2_description/meshes/sensors/srf05.stl"/>
+        </geometry>
+        <material name="DarkGrey"/>
+      </visual>
     </link>
     <joint name="${name}_joint" type="fixed">

File: pmb2_description/urdf/sensors/sick_tim551_laser.urdf.xacro (robot description, xacro)
@@ -23,5 +23,5 @@
           <mesh filename="package://pmb2_description/meshes/sensors/sick_tim551.stl"/>
         </geometry>
-        <material name="DarkGrey" />
+        <material name="DarkGrey"/>
       </visual>
     </link>

Commit message: Add microphones

File: pmb2_description/urdf/base/base.urdf.xacro (robot description, xacro)
@@ -16,4 +16,5 @@
   <xacro:include filename="$(find pmb2_description)/urdf/sensors/imu.urdf.xacro"/>
   <xacro:include filename="$(find pmb2_description)/urdf/sensors/bumper.urdf.xacro"/>
+  <xacro:include filename="$(find pmb2_description)/urdf/sensors/microphone.urdf.xacro"/>
   <xacro:include filename="$(find pmb2_description)/urdf/objects/battery_tlh_2.urdf.xacro"/>
   <xacro:include filename="$(find pmb2_description)/urdf/objects/charger.urdf.xacro"/>
@@ -114,8 +115,20 @@
     </xacro:range_sensor>
     <!-- Bumpers -->
-    257.000.00-64.50
     <xacro:bumper name="${name}_bumper" parent="${name}" ros_topic="bumper_base" update_rate="10">
       <origin xyz="0.257 0.00 -0.0645" rpy="0 0 0"/>
     </xacro:bumper>
+    <!-- Microphones -->
+    <xacro:microphone name="${name}_mic_front_left" parent="${name}">
+      <origin xyz="0 0 0" rpy="0 0 0"/>
+    </xacro:microphone>
+    <xacro:microphone name="${name}_mic_front_right" parent="${name}">
+      <origin xyz="0 0 0" rpy="0 0 0"/>
+    </xacro:microphone>
+    <xacro:microphone name="${name}_mic_back_left" parent="${name}">
+      <origin xyz="0 0 0" rpy="0 0 0"/>
+    </xacro:microphone>
+    <xacro:microphone name="${name}_mic_back_right" parent="${name}">
+      <origin xyz="0 0 0" rpy="0 0 0"/>
+    </xacro:microphone>
     <!-- IMU -->
     <!-- @todo pmb2_hardware_gazebo needs an IMU!  -->

Commit message: Put sonars with its rear cover

File: pmb2_description/urdf/base/base.urdf.xacro (robot description, xacro)
@@ -84,5 +84,5 @@
     <!-- Cover -->
     <xacro:cover name="${name}_cover" parent="${name}_footprint"/>
-    <!-- Rear cover -->
+    <!-- Rear (sonars) cover -->
     <xacro:rear_cover name="${name}_rear_cover" parent="${name}_footprint"/>
     <!-- Laser -->
@@ -98,20 +98,4 @@
       <origin xyz="0 0 0" rpy="${-90 * deg_to_rad} 0 ${-90 * deg_to_rad}"/>
     </xacro:xtion_pro_live>
-    <!-- Sonars -->
-    <xacro:range_sensor name="${name}_sonar_01" parent="${name}" ros_topic="sonar_base" update_rate="10" maxRange="0.30" minRange="0.01" fov="${60.0 * deg_to_rad}" radiation="ultrasound">
-      <origin xyz="-0.17571000000 0.17571000000 0.10150000000" rpy="0.0 0.0 ${135.0 * deg_to_rad}"/>
-    </xacro:range_sensor>
-    <xacro:range_sensor name="${name}_sonar_02" parent="${name}" ros_topic="sonar_base" update_rate="10" maxRange="0.30" minRange="0.01" fov="${60.0 * deg_to_rad}" radiation="ultrasound">
-      <origin xyz="-0.22958000000 0.09510000000 0.10150000000" rpy="0.0 0.0 ${157.5 * deg_to_rad}"/>
-    </xacro:range_sensor>
-    <xacro:range_sensor name="${name}_sonar_03" parent="${name}" ros_topic="sonar_base" update_rate="10" maxRange="0.30" minRange="0.01" fov="${60.0 * deg_to_rad}" radiation="ultrasound">
-      <origin xyz="-0.24850000000 0.00000000000 0.10150000000" rpy="0.0 0.0 ${180.0 * deg_to_rad}"/>
-    </xacro:range_sensor>
-    <xacro:range_sensor name="${name}_sonar_04" parent="${name}" ros_topic="sonar_base" update_rate="10" maxRange="0.30" minRange="0.01" fov="${60.0 * deg_to_rad}" radiation="ultrasound">
-      <origin xyz="-0.22958000000 -0.09510000000 0.10150000000" rpy="0.0 0.0 ${202.5 * deg_to_rad}"/>
-    </xacro:range_sensor>
-    <xacro:range_sensor name="${name}_sonar_05" parent="${name}" ros_topic="sonar_base" update_rate="10" maxRange="0.30" minRange="0.01" fov="${60.0 * deg_to_rad}" radiation="ultrasound">
-      <origin xyz="-0.17571000000 -0.17571000000 0.10150000000" rpy="0.0 0.0 ${225.0 * deg_to_rad}"/>
-    </xacro:range_sensor>
     <!-- Bumpers -->
     <xacro:bumper name="${name}_bumper" parent="${name}" ros_topic="bumper_base" update_rate="10">

File: pmb2_description/urdf/objects/rear_cover_ultrasound.urdf.xacro (robot description, xacro)
@@ -8,4 +8,6 @@
 -->
 <robot xmlns:xacro="http://ros.org/wiki/xacro">
+  <xacro:include filename="$(find pmb2_description)/urdf/deg_to_rad.xacro"/>
+  <xacro:include filename="$(find pmb2_description)/urdf/sensors/range.gazebo.xacro" />
   <xacro:macro name="rear_cover" params="name parent">
     <link name="${name}_link">
@@ -30,4 +32,20 @@
       <origin xyz="0 0 0.0985" rpy="0 0 0"/>
     </joint>
+    <!-- Sonars -->
+    <xacro:range_sensor name="${name}_sonar_01" parent="${name}" ros_topic="sonar_base" update_rate="10" maxRange="0.30" minRange="0.01" fov="${60.0 * deg_to_rad}" radiation="ultrasound">
+      <origin xyz="-0.17571000000 0.17571000000 0.10150000000" rpy="0.0 0.0 ${135.0 * deg_to_rad}"/>
+    </xacro:range_sensor>
+    <xacro:range_sensor name="${name}_sonar_02" parent="${name}" ros_topic="sonar_base" update_rate="10" maxRange="0.30" minRange="0.01" fov="${60.0 * deg_to_rad}" radiation="ultrasound">
+      <origin xyz="-0.22958000000 0.09510000000 0.10150000000" rpy="0.0 0.0 ${157.5 * deg_to_rad}"/>
+    </xacro:range_sensor>
+    <xacro:range_sensor name="${name}_sonar_03" parent="${name}" ros_topic="sonar_base" update_rate="10" maxRange="0.30" minRange="0.01" fov="${60.0 * deg_to_rad}" radiation="ultrasound">
+      <origin xyz="-0.24850000000 0.00000000000 0.10150000000" rpy="0.0 0.0 ${180.0 * deg_to_rad}"/>
+    </xacro:range_sensor>
+    <xacro:range_sensor name="${name}_sonar_04" parent="${name}" ros_topic="sonar_base" update_rate="10" maxRange="0.30" minRange="0.01" fov="${60.0 * deg_to_rad}" radiation="ultrasound">
+      <origin xyz="-0.22958000000 -0.09510000000 0.10150000000" rpy="0.0 0.0 ${202.5 * deg_to_rad}"/>
+    </xacro:range_sensor>
+    <xacro:range_sensor name="${name}_sonar_05" parent="${name}" ros_topic="sonar_base" update_rate="10" maxRange="0.30" minRange="0.01" fov="${60.0 * deg_to_rad}" radiation="ultrasound">
+      <origin xyz="-0.17571000000 -0.17571000000 0.10150000000" rpy="0.0 0.0 ${225.0 * deg_to_rad}"/>
+    </xacro:range_sensor>
   </xacro:macro>
 </robot>

Commit message: Add conditional for base rgbd sensor

File: pmb2_description/urdf/base/base.urdf.xacro (robot description, xacro)
@@ -92,10 +92,12 @@
     </xacro:sick_tim551_laser>
     <!-- RGBD -->
-    <xacro:xtion_pro_live name="${name}_rgbd_camera" parent="${name}">
-      <!-- Pose of sensor frame wrt to base -->
-      <origin xyz="${base_rgbd_x} ${base_rgbd_y} ${base_rgbd_z}" rpy="${base_rgbd_R * deg_to_rad} ${base_rgbd_P * deg_to_rad} ${base_rgbd_Y * deg_to_rad}"/>
-      <!-- Pose of optical frame wrt to sensor -->
-      <origin xyz="0 0 0" rpy="${-90 * deg_to_rad} 0 ${-90 * deg_to_rad}"/>
-    </xacro:xtion_pro_live>
+    <xacro:if value="$(arg have_base_rgbd)">
+      <xacro:xtion_pro_live name="${name}_rgbd_camera" parent="${name}">
+        <!-- Pose of sensor frame wrt to base -->
+        <origin xyz="${base_rgbd_x} ${base_rgbd_y} ${base_rgbd_z}" rpy="${base_rgbd_R * deg_to_rad} ${base_rgbd_P * deg_to_rad} ${base_rgbd_Y * deg_to_rad}"/>
+        <!-- Pose of optical frame wrt to sensor -->
+        <origin xyz="0 0 0" rpy="${-90 * deg_to_rad} 0 ${-90 * deg_to_rad}"/>
+      </xacro:xtion_pro_live>
+    </xacro:if>
     <!-- Bumpers -->
     <xacro:bumper name="${name}_bumper" parent="${name}" ros_topic="bumper_base" update_rate="10">

Commit message: Add new cover and orange ring around body

File: pmb2_description/urdf/base/base.urdf.xacro (robot description, xacro)
@@ -61,5 +61,5 @@
           <mesh filename="package://pmb2_description/meshes/base/base.stl" />
         </geometry>
-        <material name="DarkGrey" />
+        <material name="White" />
       </visual>
       <collision>
@@ -68,7 +68,10 @@
           <mesh filename="package://pmb2_description/meshes/base/base_collision.stl" />
         </geometry>
-        <material name="DarkGrey" />
+        <material name="White" />
       </collision>
     </link>
+    <gazebo reference="${name}_link">
+      <material>Gazebo/White</material>
+    </gazebo>
     <!-- Base footprint -->
     <link name="${name}_footprint"/>
@@ -78,8 +81,4 @@
       <parent link="${name}_footprint"/>
     </joint>
-    <!-- Battery -->
-    <xacro:battery name="${name}_battery" parent="${name}_footprint"/>
-    <!-- Charger -->
-    <xacro:charger name="${name}_charger" parent="${name}_footprint"/>
     <!-- Cover -->
     <xacro:cover name="${name}_cover" parent="${name}_footprint"/>

File: pmb2_description/urdf/materials.urdf.xacro (robot description, xacro)
@@ -29,3 +29,6 @@
     <color rgba="1.0 1.0 1.0 1.0"/>
   </material>
+  <material name="Orange">
+    <color rgba="1.0 0.69 0.0 1.0"/>
+  </material>
 </robot>

File: pmb2_description/urdf/objects/cover.urdf.xacro (robot description, xacro)
@@ -20,7 +20,7 @@
         <origin xyz="0 0 0" rpy="0 0 0"/>
         <geometry>
-          <mesh filename="package://pmb2_description/meshes/objects/cover.stl"/>
+          <mesh filename="package://pmb2_description/meshes/base/base_ring.stl"/>
         </geometry>
-        <material name="LightGrey"/>
+        <material name="Orange"/>
       </visual>
     </link>
@@ -28,6 +28,9 @@
       <parent link="${parent}"/>
       <child link="${name}_link"/>
-      <origin xyz="0 0 0.0985" rpy="0 0 0"/>
+      <origin xyz="0 0 0.15" rpy="0 0 0"/>
     </joint>
+    <gazebo reference="${name}_link">
+      <material>Gazebo/Orange</material>
+    </gazebo>
   </xacro:macro>
 </robot>

Commit message: Remove base_rgbd

File: pmb2_description/urdf/base/base.urdf.xacro (robot description, xacro)
@@ -39,11 +39,4 @@
   <property name="base_laser_y" value="0.0"/>
   <property name="base_laser_z" value="-0.004"/>
-  <!-- RGBD characteristics -->
-  <property name="base_rgbd_x" value="0.2223"/>
-  <property name="base_rgbd_y" value="0.0"/>
-  <property name="base_rgbd_z" value="0.099"/>
-  <property name="base_rgbd_R" value="0.0"/>
-  <property name="base_rgbd_P" value="0.0"/>
-  <property name="base_rgbd_Y" value="0.0"/>
   <xacro:macro name="base" params="name">
     <!-- Base -->
@@ -90,13 +83,4 @@
       <origin xyz="${base_laser_x} ${base_laser_y} ${base_laser_z}" rpy="0 0 0" />
     </xacro:sick_tim551_laser>
-    <!-- RGBD -->
-    <xacro:if value="$(arg have_base_rgbd)">
-      <xacro:xtion_pro_live name="${name}_rgbd_camera" parent="${name}">
-        <!-- Pose of sensor frame wrt to base -->
-        <origin xyz="${base_rgbd_x} ${base_rgbd_y} ${base_rgbd_z}" rpy="${base_rgbd_R * deg_to_rad} ${base_rgbd_P * deg_to_rad} ${base_rgbd_Y * deg_to_rad}"/>
-        <!-- Pose of optical frame wrt to sensor -->
-        <origin xyz="0 0 0" rpy="${-90 * deg_to_rad} 0 ${-90 * deg_to_rad}"/>
-      </xacro:xtion_pro_live>
-    </xacro:if>
     <!-- Bumpers -->
     <xacro:bumper name="${name}_bumper" parent="${name}" ros_topic="bumper_base" update_rate="10">

Commit message: Remove bumpers

File: pmb2_description/urdf/base/base.urdf.xacro (robot description, xacro)
@@ -15,5 +15,4 @@
   <xacro:include filename="$(find pmb2_description)/urdf/sensors/xtion_pro_live.urdf.xacro"/>
   <xacro:include filename="$(find pmb2_description)/urdf/sensors/imu.urdf.xacro"/>
-  <xacro:include filename="$(find pmb2_description)/urdf/sensors/bumper.urdf.xacro"/>
   <xacro:include filename="$(find pmb2_description)/urdf/sensors/microphone.urdf.xacro"/>
   <xacro:include filename="$(find pmb2_description)/urdf/objects/cover.urdf.xacro"/>
@@ -78,8 +77,4 @@
       <origin xyz="${base_laser_x} ${base_laser_y} ${base_laser_z}" rpy="0 0 0" />
     </xacro:sick_tim551_laser>
-    <!-- Bumpers -->
-    <xacro:bumper name="${name}_bumper" parent="${name}" ros_topic="bumper_base" update_rate="10">
-      <origin xyz="0.257 0.00 -0.0645" rpy="0 0 0"/>
-    </xacro:bumper>
     <!-- Microphones -->
     <xacro:microphone name="${name}_mic_front_left" parent="${name}">

Commit message: Add inertial params to main body

File: pmb2_description/urdf/base/base.urdf.xacro (robot description, xacro)
@@ -39,9 +39,9 @@
     <link name="${name}_link">
       <inertial>
-        <origin xyz="-0.00393000000 -0.00057000000 0.04788000000" rpy="0 0 0"/>
-        <mass value="17.22815000000"/>
-        <inertia ixx="0.38502800825" ixy="0.00017569597" ixz="0.00983980386"
-                 iyy="0.32897158338" iyz="-0.00013935331"
-                 izz="0.44188721859"/>
+        <origin xyz="-0.00000106 0.00000109 0.0000387" rpy="0 0 0"/>
+        <mass value="28.26649"/>
+        <inertia ixx="0.465408937" ixy="0.002160024" ixz="-0.001760255"
+                 iyy="0.483193291" iyz="-0.000655952"
+                 izz="0.550939703"/>
       </inertial>
       <visual>

Commit message: Add antennas

File: pmb2_description/urdf/base/base.urdf.xacro (robot description, xacro)
@@ -16,4 +16,5 @@
   <xacro:include filename="$(find pmb2_description)/urdf/sensors/microphone.urdf.xacro"/>
   <xacro:include filename="$(find pmb2_description)/urdf/objects/cover.urdf.xacro"/>
+  <xacro:include filename="$(find pmb2_description)/urdf/objects/antenna.urdf.xacro"/>
   <!-- Wheel characteristics -->
   <property name="wheel_radius"     value="0.0985"/>
@@ -69,6 +70,12 @@
       <parent link="${name}_footprint"/>
     </joint>
-    <!-- Cover -->
+    <!-- Orange cover & antennas -->
     <xacro:cover name="${name}_cover" parent="${name}_footprint"/>
+    <xacro:antenna name="${name}_antenna_left" parent="${name}_link">
+      <origin xyz="-0.201 0.1062 0.195" rpy="0 0 0"/>
+    </xacro:antenna>
+    <xacro:antenna name="${name}_antenna_right" parent="${name}_link">
+      <origin xyz="-0.201 -0.1062 0.195" rpy="0 0 0"/>
+    </xacro:antenna>
     <!-- Laser -->
     <!-- Theoretic FOV = 220º -->

Commit message: Added sonars with proper colors

File: pmb2_description/urdf/base/base.urdf.xacro (robot description, xacro)
@@ -101,4 +101,14 @@
       <origin xyz="0 0 0" rpy="0 0 0"/>
     </xacro:imu_sensor>
+    <!-- Sonars -->
+    <xacro:range_sensor name="${name}_sonar_1" parent="${name}" ros_topic="sonar_${name}" update_rate="5" maxRange="0.75" minRange="0.01" fov="0.5" radiation="ultrasound">
+      <origin xyz="-0.183 0.183 0.173" rpy="0 0 ${135 * deg_to_rad}"/>
+    </xacro:range_sensor>
+    <xacro:range_sensor name="${name}_sonar_2" parent="${name}" ros_topic="sonar_${name}" update_rate="5" maxRange="0.75" minRange="0.01" fov="0.5" radiation="ultrasound">
+      <origin xyz="-0.259 0.0 0.173" rpy="0 0 ${180 * deg_to_rad}"/>
+    </xacro:range_sensor>
+    <xacro:range_sensor name="${name}_sonar_3" parent="${name}" ros_topic="sonar_${name}" update_rate="5" maxRange="0.75" minRange="0.01" fov="0.5" radiation="ultrasound">
+      <origin xyz="-0.183 -0.183 0.173" rpy="0 0 ${225 * deg_to_rad}"/>
+    </xacro:range_sensor>
     <!-- Wheels -->
     <xacro:wheel side="right" reflect=" 1.0" radius="${wheel_radius}" width="${wheel_width}" torque="${wheel_torque}" velocity="${wheel_velocity}" separation="${wheel_separation}" parent="${name}"/>

File: pmb2_description/urdf/sensors/range.gazebo.xacro (robot description, xacro)
@@ -47,4 +47,5 @@
         </plugin>
       </sensor>
+      <material>Gazebo/DarkGrey</material>
     </gazebo>
   </xacro:macro>

Commit message: Add microphone locations

File: pmb2_description/urdf/base/base.urdf.xacro (robot description, xacro)
@@ -85,14 +85,14 @@
     <!-- Microphones -->
     <xacro:microphone name="${name}_mic_front_left" parent="${name}">
-      <origin xyz="0 0 0" rpy="0 0 0"/>
+      <origin xyz="0.23182 0.03902 0.195" rpy="0 0 0"/>
     </xacro:microphone>
     <xacro:microphone name="${name}_mic_front_right" parent="${name}">
-      <origin xyz="0 0 0" rpy="0 0 0"/>
+      <origin xyz="0.23182 -0.03902 0.195" rpy="0 0 0"/>
     </xacro:microphone>
     <xacro:microphone name="${name}_mic_back_left" parent="${name}">
-      <origin xyz="0 0 0" rpy="0 0 0"/>
+      <origin xyz="-0.1082 -0.0599 0.195" rpy="0 0 0"/>
     </xacro:microphone>
     <xacro:microphone name="${name}_mic_back_right" parent="${name}">
-      <origin xyz="0 0 0" rpy="0 0 0"/>
+      <origin xyz="-0.1082 -0.13789 0.195" rpy="0 0 0"/>
     </xacro:microphone>
     <!-- IMU -->

Commit message: Update placement and name of base imu

File: pmb2_description/urdf/base/base.urdf.xacro (robot description, xacro)
@@ -98,6 +98,6 @@
     <!-- IMU -->
     <!-- @todo pmb2_hardware_gazebo needs an IMU!  -->
-    <xacro:imu_sensor name="${name}_inclinometer" parent="${name}_link" update_rate="100.0">
-      <origin xyz="0 0 0" rpy="0 0 0"/>
+    <xacro:imu_sensor name="${name}_imu" parent="${name}_link" update_rate="100.0">
+      <origin xyz="0.10171 0 0.11282" rpy="0 ${180 * deg_to_rad} ${90 * deg_to_rad}"/>
     </xacro:imu_sensor>
     <!-- Sonars -->
