Commit message: Simplified base collision
Now the base_link has a mesh that touches with the ground

File: pmb2_description/urdf/base/base.urdf.xacro (robot description, xacro)
@@ -48,5 +48,5 @@
         <origin xyz="0 0 0" rpy="0 0 0" />
         <geometry>
-          <mesh filename="package://pmb2_description/meshes/base/base_collision.stl" />
+          <mesh filename="package://pmb2_description/meshes/base/base_collision.dae" />
         </geometry>
         <material name="White" />
@@ -63,4 +63,15 @@
       <parent link="${name}_footprint"/>
     </joint>
+  <!-- gazebo parameters are given here for base_link thru base_footprint -->
+    <gazebo reference="${name}_footprint">
+      <kp>100000000.0</kp>
+      <kd>10.0</kd>
+      <mu1>0.1</mu1>
+      <mu2>0.1</mu2>
+      <fdir1>1 0 0</fdir1>
+      <maxVel>10.0</maxVel>
+      <minDepth>0.0005</minDepth>
+      <laserRetro>0</laserRetro>
+    </gazebo>
     <!-- Orange cover & antennas -->
     <xacro:cover name="${name}_cover" parent="${name}_footprint"/>

File: pmb2_description/urdf/wheels/caster.urdf.xacro (robot description, xacro)
@@ -9,5 +9,4 @@
 <robot xmlns:xacro="http://ros.org/wiki/xacro">
   <xacro:include filename="$(find pmb2_description)/urdf/wheels/caster.transmission.xacro"/>
-  <xacro:include filename="$(find pmb2_description)/urdf/wheels/caster.gazebo.xacro"/>
   <xacro:macro name="caster" params="side radius width separation_x separation_y offset_x offset_y offset_z parent">
     <link name="caster_${side}_1_link">
@@ -42,10 +41,4 @@
         <material name="DarkGrey"/>
       </visual>
-      <collision>
-        <origin xyz="0 0 0" rpy="0 0 0"/>
-        <geometry>
-          <sphere radius="${radius}"/>
-        </geometry>
-      </collision>
     </link>
     <joint name="caster_${side}_1_joint" type="fixed">
@@ -61,8 +54,4 @@
       <axis xyz="0 0 1"/>
     </joint>
-    <!-- Transmission -->
-    <!--xacro:caster_transmission name="" side="${side}" number="" reduction=""-->
-    <!-- Gazebo extensions -->
-    <xacro:caster_gazebo side="${side}"/>
   </xacro:macro>
 </robot>

File: pmb2_description/urdf/wheels/wheel.gazebo.xacro (robot description, xacro)
@@ -11,5 +11,4 @@
     <!-- Contact model for the wheel surface -->
     <gazebo reference="wheel_${side}_link">
-<!--
       <kp>1000000.0</kp>
       <kd>100.0</kd>
@@ -18,7 +17,6 @@
       <fdir1>1 0 0</fdir1>
       <maxVel>1.0</maxVel>
-      <minDepth>0.00</minDepth>
+      <minDepth>0.003</minDepth>
       <implicitSpringDamper>1</implicitSpringDamper>
--->
       <material>Gazebo/DarkGrey</material>
     </gazebo>

Commit message: corrected imu frame, z always point upwards
this is because the imu 6050 zeros itself (at least wrt pitch)

File: pmb2_description/urdf/base/base.urdf.xacro (robot description, xacro)
@@ -85,5 +85,5 @@
     <!-- @todo pmb2_hardware_gazebo needs an IMU!  -->
     <xacro:imu_sensor name="${name}_imu" parent="${name}_link" update_rate="100.0">
-      <origin xyz="0.10171 0 0.11282" rpy="0 ${180 * deg_to_rad} ${90 * deg_to_rad}"/>
+      <origin xyz="0.10171 0 0.11282" rpy="0 0 ${-90 * deg_to_rad}"/>
     </xacro:imu_sensor>
     <!-- Wheels -->

Commit message: caster wheels and base collision
Note: Frictin coeffs mu1, mu2 in caster.gazebo.xacro can me adjusted to make robot stopping immideately

File: pmb2_description/urdf/base/base.urdf.xacro (robot description, xacro)
@@ -48,5 +48,5 @@
         <origin xyz="0 0 0" rpy="0 0 0" />
         <geometry>
-          <mesh filename="package://pmb2_description/meshes/base/base_collision.dae" />
+          <mesh filename="package://pmb2_description/meshes/base/base_collision.stl" />
         </geometry>
         <material name="White" />

File: pmb2_description/urdf/wheels/caster.gazebo.xacro (robot description, xacro)
@@ -13,7 +13,8 @@
       <kp>1000000.0</kp>
       <kd>100.0</kd>
-      <mu1>0</mu1>
-      <mu2>0</mu2>
+      <mu1>0.2</mu1>
+      <mu2>0.2</mu2>
       <fdir1>1 0 0</fdir1>
+      <fdir2>0 1 0</fdir2>
       <maxVel>1.0</maxVel>
       <minDepth>0.00</minDepth>
@@ -23,9 +24,10 @@
       <kp>1000000.0</kp>
       <kd>100.0</kd>
-      <mu1>0</mu1>
-      <mu2>0</mu2>
+      <mu1>0.2</mu1>
+      <mu2>0.2</mu2>
       <fdir1>1 0 0</fdir1>
+      <fdir2>0 1 0</fdir2>
       <maxVel>1.0</maxVel>
-      <minDepth>0.00</minDepth>
+      <minDepth>0.05</minDepth>
       <implicitSpringDamper>1</implicitSpringDamper>
       <material>Gazebo/DarkGrey</material>

File: pmb2_description/urdf/wheels/caster.urdf.xacro (robot description, xacro)
@@ -9,4 +9,5 @@
 <robot xmlns:xacro="http://ros.org/wiki/xacro">
   <xacro:include filename="$(find pmb2_description)/urdf/wheels/caster.transmission.xacro"/>
+  <xacro:include filename="$(find pmb2_description)/urdf/wheels/caster.gazebo.xacro"/>
   <xacro:macro name="caster" params="side radius width separation_x separation_y offset_x offset_y offset_z parent">
     <link name="caster_${side}_1_link">
@@ -25,4 +26,10 @@
         <material name="Grey"/>
       </visual>
+      <collision>
+        <origin xyz="0 0 0" rpy="0 0 0"/>
+        <geometry>
+          <cylinder radius="${radius}" length="${width}"/>
+        </geometry>
+      </collision>
     </link>
     <link name="caster_${side}_2_link">
@@ -41,4 +48,10 @@
         <material name="DarkGrey"/>
       </visual>
+      <collision>
+        <origin xyz="0 0 0" rpy="0 0 0"/>
+        <geometry>
+          <cylinder radius="${radius}" length="${width}"/>
+        </geometry>
+      </collision>
     </link>
     <joint name="caster_${side}_1_joint" type="fixed">
@@ -54,4 +67,6 @@
       <axis xyz="0 0 1"/>
     </joint>
+    <!-- Gazebo extensions -->
+    <xacro:caster_gazebo side="${side}"/>
   </xacro:macro>
 </robot>

Commit message: Fix collision and friction issues
Work from andrei@pasnicen.co

File: pmb2_description/urdf/base/base.urdf.xacro (robot description, xacro)
@@ -48,5 +48,5 @@
         <origin xyz="0 0 0" rpy="0 0 0" />
         <geometry>
-          <mesh filename="package://pmb2_description/meshes/base/base_collision.dae" />
+          <mesh filename="package://pmb2_description/meshes/base/high_resolution/base_collision.stl" />
         </geometry>
         <material name="White" />

File: pmb2_description/urdf/wheels/caster.gazebo.xacro (robot description, xacro)
@@ -12,20 +12,21 @@
     <gazebo reference="caster_${side}_1_link">
       <kp>1000000.0</kp>
-      <kd>100.0</kd>
-      <mu1>0</mu1>
-      <mu2>0</mu2>
+      <kd>1000.0</kd>
+      <mu1>1.0</mu1>
+      <mu2>1.0</mu2>
       <fdir1>1 0 0</fdir1>
       <maxVel>1.0</maxVel>
-      <minDepth>0.00</minDepth>
+      <minDepth>0.005</minDepth>
       <implicitSpringDamper>1</implicitSpringDamper>
+      <material>Gazebo/DarkGrey</material>
     </gazebo>
     <gazebo reference="caster_${side}_2_link">
       <kp>1000000.0</kp>
-      <kd>100.0</kd>
-      <mu1>0</mu1>
-      <mu2>0</mu2>
+      <kd>1000.0</kd>
+      <mu1>1.0</mu1>
+      <mu2>1.0</mu2>
       <fdir1>1 0 0</fdir1>
       <maxVel>1.0</maxVel>
-      <minDepth>0.00</minDepth>
+      <minDepth>0.005</minDepth>
       <implicitSpringDamper>1</implicitSpringDamper>
       <material>Gazebo/DarkGrey</material>

File: pmb2_description/urdf/wheels/caster.urdf.xacro (robot description, xacro)
@@ -9,4 +9,5 @@
 <robot xmlns:xacro="http://ros.org/wiki/xacro">
   <xacro:include filename="$(find pmb2_description)/urdf/wheels/caster.transmission.xacro"/>
+  <xacro:include filename="$(find pmb2_description)/urdf/wheels/caster.gazebo.xacro"/>
   <xacro:macro name="caster" params="side radius width separation_x separation_y offset_x offset_y offset_z parent">
     <link name="caster_${side}_1_link">
@@ -25,4 +26,10 @@
         <material name="Grey"/>
       </visual>
+      <collision>
+        <origin xyz="0 0 0" rpy="0 0 0"/>
+        <geometry>
+          <cylinder radius="${radius}" length="${width}"/>
+        </geometry>
+      </collision>
     </link>
     <link name="caster_${side}_2_link">
@@ -41,6 +48,12 @@
         <material name="DarkGrey"/>
       </visual>
+      <collision>
+        <origin xyz="0 0 0" rpy="0 0 0"/>
+        <geometry>
+          <cylinder radius="${radius}" length="${width}"/>
+        </geometry>
+      </collision>
     </link>
-    <joint name="caster_${side}_1_joint" type="fixed">
+    <joint name="caster_${side}_1_joint" type="continuous">
       <parent link="${parent}_link"/>
       <child link="caster_${side}_1_link"/>
@@ -48,5 +61,5 @@
       <axis xyz="0 0 1"/>
     </joint>
-    <joint name="caster_${side}_2_joint" type="fixed">
+    <joint name="caster_${side}_2_joint" type="continuous">
       <parent link="caster_${side}_1_link"/>
       <child link="caster_${side}_2_link"/>
@@ -54,4 +67,9 @@
       <axis xyz="0 0 1"/>
     </joint>
+    <!-- Gazebo extensions -->
+    <xacro:caster_gazebo side="${side}"/>
+    <!-- Transmission -->
+   <xacro:caster_transmission name="caster" side="${side}" number="1" reduction="1.0"/>
+   <xacro:caster_transmission name="caster" side="${side}" number="2" reduction="1.0"/>
   </xacro:macro>
 </robot>

File: pmb2_description/urdf/wheels/suspension.transmission.xacro (robot description, xacro)
@@ -8,13 +8,14 @@
 -->
 <robot xmlns:xacro="http://ros.org/wiki/xacro">
-  <!-- Caster transmissions -->
-  <xacro:macro name="caster_transmission" params="name side number reduction" >
-    <transmission name="${name}_${side}_${number}_trans">
+  <!-- suspension transmission -->
+  <xacro:macro name="suspension_transmission" params="side">
+    <transmission name="suspension_${side}_trans">
       <type>transmission_interface/SimpleTransmission</type>
-        <actuator name="${name}_${side}_${number}_motor" >
-        <mechanicalReduction>${reduction}</mechanicalReduction>
+      <actuator name="suspension_${side}_motor" >
+        <mechanicalReduction>1.0</mechanicalReduction>
       </actuator>
-      <joint name="${name}_${side}_${number}_joint" >
-        <hardwareInterface>hardware_interface/VelocityJointInterface</hardwareInterface>
+      <joint name="suspension_${side}_joint" >
+        <hardwareInterface>hardware_interface/PositionJointInterface</hardwareInterface>
+        <hardwareInterface>hardware_interface/JointStateInterface</hardwareInterface>
       </joint>
     </transmission>

File: pmb2_description/urdf/wheels/wheel.gazebo.xacro (robot description, xacro)
@@ -12,10 +12,10 @@
     <gazebo reference="wheel_${side}_link">
       <kp>1000000.0</kp>
-      <kd>100.0</kd>
-      <mu1>1.0</mu1>
-      <mu2>1.0</mu2>
+      <kd>1000.0</kd>
+      <mu1>1000.0</mu1>
+      <mu2>1000.0</mu2>
       <fdir1>1 0 0</fdir1>
-      <maxVel>1.0</maxVel>
-      <minDepth>0.003</minDepth>
+      <maxVel>20.0</maxVel>
+      <minDepth>0.0</minDepth>
       <implicitSpringDamper>1</implicitSpringDamper>
       <material>Gazebo/DarkGrey</material>

File: pmb2_description/urdf/wheels/wheel.urdf.xacro (robot description, xacro)
@@ -1,13 +1,14 @@
 <?xml version="1.0"?>
 <!--
-  Copyright (c) 2014, PAL Robotics, S.L.
-  All rights reserved.
-  This work is licensed under the Creative Commons Attribution-NonCommercial-NoDerivs 3.0 Unported License.
-  To view a copy of this license, visit http://creativecommons.org/licenses/by-nc-nd/3.0/ or send a letter to
-  Creative Commons, 444 Castro Street, Suite 900, Mountain View, California, 94041, USA.
+Copyright (c) 2014, PAL Robotics, S.L.
+All rights reserved.
+This work is licensed under the Creative Commons Attribution-NonCommercial-NoDerivs 3.0 Unported License.
+To view a copy of this license, visit http://creativecommons.org/licenses/by-nc-nd/3.0/ or send a letter to
+Creative Commons, 444 Castro Street, Suite 900, Mountain View, California, 94041, USA.
 -->
 <robot xmlns:xacro="http://ros.org/wiki/xacro">
   <xacro:include filename="$(find pmb2_description)/urdf/wheels/wheel.transmission.xacro"/>
   <xacro:include filename="$(find pmb2_description)/urdf/wheels/wheel.gazebo.xacro"/>
+  <xacro:include filename="$(find pmb2_description)/urdf/wheels/suspension.transmission.xacro"/>
   <xacro:macro name="wheel" params="side reflect radius width torque velocity separation parent">
     <link name="wheel_${side}_link">
@@ -16,32 +17,57 @@
         <mass value="1.82362"/>
         <inertia ixx="0.00499743171" ixy="${ 0.00000004464 * reflect}" ixz="-0.00000002245"
-                 iyy="0.00499741733" iyz="${-0.00000000164 * reflect}"
-                 izz="0.00839239692"/>
-      </inertial>
-      <visual>
-        <origin xyz="0 0 0" rpy="${-90.0 * (1 - reflect) * deg_to_rad} 0 0"/>
-        <geometry>
-          <mesh filename="package://pmb2_description/meshes/wheels/wheel.stl"/>
-        </geometry>
-        <material name="DarkGrey"/>
-      </visual>
-      <collision>
+          iyy="0.00499741733" iyz="${-0.00000000164 * reflect}"
+          izz="0.00839239692"/>
+        </inertial>
+        <visual>
+          <origin xyz="0 0 0" rpy="${-90.0 * (1 - reflect) * deg_to_rad} 0 0"/>
+          <geometry>
+            <mesh filename="package://pmb2_description/meshes/wheels/wheel.stl"/>
+          </geometry>
+          <material name="DarkGrey"/>
+        </visual>
+        <collision>
+          <origin xyz="0 0 0" rpy="0 0 0"/>
+          <geometry>
+            <cylinder radius="${radius}" length="${width}"/>
+          </geometry>
+        </collision>
+      </link>
+      <link name="suspension_${side}_link">
+        <inertial>
+          <origin xyz="0 0 -0.02" rpy="0 0 0"/>
+          <mass value="30"/>
+          <inertia ixx="1.0" ixy="0" ixz="0"
+                   iyy="1.0" iyz="0"
+                   izz="1.0"/>
+         </inertial>
+        <kinematic>1</kinematic>
+        <gravity>1</gravity>
+      </link>
+      <joint name="suspension_${side}_joint" type="prismatic">
         <origin xyz="0 0 0" rpy="0 0 0"/>
-        <geometry>
-          <cylinder radius="${radius}" length="${width}"/>
-        </geometry>
-      </collision>
-    </link>
-    <joint name="wheel_${side}_joint" type="continuous">
-      <parent link="${parent}_link"/>
-      <child link="wheel_${side}_link"/>
-      <origin xyz="0 ${-separation / 2 * reflect} 0" rpy="${-90.0 * deg_to_rad} 0 0"/>
-      <axis xyz="0 0 1"/>
-      <limit effort="${torque}" velocity="${velocity / radius}"/>
-    </joint>
-    <!-- Transmission -->
-    <xacro:wheel_transmission side="${side}"/>
-    <!-- Gazebo extensions -->
-    <xacro:wheel_gazebo side="${side}"/>
-  </xacro:macro>
-</robot>
+        <axis xyz="0 0 1"/>
+        <limit effort="10000.0" lower="-0.04" upper="0.04" velocity="1.0"/>
+        <child link="suspension_${side}_link"/>
+        <parent link="${parent}_link"/>
+        <calibration rising="0.0" />
+        <dynamics damping="10000"/>
+        <safety_controller k_position="-0.03"
+          k_velocity="100"
+          soft_lower_limit="-0.05"
+          soft_upper_limit="0.05" />
+        </joint>
+        <joint name="wheel_${side}_joint" type="continuous">
+          <parent link="suspension_${side}_link"/>
+          <child link="wheel_${side}_link"/>
+          <origin xyz="0 ${-separation / 2 * reflect} 0" rpy="${-90.0 * deg_to_rad} 0 0"/>
+          <axis xyz="0 0 1"/>
+          <limit effort="${torque}" velocity="${velocity / radius}"/>
+        </joint>
+        <!-- Transmission -->
+        <xacro:wheel_transmission side="${side}"/>
+        <xacro:suspension_transmission side="${side}"/>
+        <!-- Gazebo extensions -->
+        <xacro:wheel_gazebo side="${side}"/>
+      </xacro:macro>
+    </robot>

Commit message: Friction coeffs adjusted

File: pmb2_description/urdf/base/base.urdf.xacro (robot description, xacro)
@@ -41,5 +41,5 @@
         <origin xyz="0 0 0" rpy="0 0 0" />
         <geometry>
-          <mesh filename="package://pmb2_description/meshes/base/base.stl" />
+          <mesh filename="package://pmb2_description/meshes/base/high_resolution/base_collision.stl" />
         </geometry>
         <material name="White" />
@@ -48,5 +48,5 @@
         <origin xyz="0 0 0" rpy="0 0 0" />
         <geometry>
-          <mesh filename="package://pmb2_description/meshes/base/base_collision.stl" />
+          <mesh filename="package://pmb2_description/meshes/base/high_resolution/base_collision.stl" />
         </geometry>
         <material name="White" />

File: pmb2_description/urdf/wheels/caster.gazebo.xacro (robot description, xacro)
@@ -12,22 +12,20 @@
     <gazebo reference="caster_${side}_1_link">
       <kp>1000000.0</kp>
-      <kd>100.0</kd>
-      <mu1>0.2</mu1>
-      <mu2>0.2</mu2>
+      <kd>1000.0</kd>
+      <mu1>0.3</mu1>
+      <mu2>0.3</mu2>
       <fdir1>1 0 0</fdir1>
-      <fdir2>0 1 0</fdir2>
       <maxVel>1.0</maxVel>
-      <minDepth>0.00</minDepth>
+      <minDepth>0.0</minDepth>
       <implicitSpringDamper>1</implicitSpringDamper>
     </gazebo>
     <gazebo reference="caster_${side}_2_link">
       <kp>1000000.0</kp>
-      <kd>100.0</kd>
-      <mu1>0.2</mu1>
-      <mu2>0.2</mu2>
+      <kd>1000.0</kd>
+      <mu1>0.3</mu1>
+      <mu2>0.3</mu2>
       <fdir1>1 0 0</fdir1>
-      <fdir2>0 1 0</fdir2>
       <maxVel>1.0</maxVel>
-      <minDepth>0.05</minDepth>
+      <minDepth>0.0</minDepth>
       <implicitSpringDamper>1</implicitSpringDamper>
       <material>Gazebo/DarkGrey</material>

File: pmb2_description/urdf/wheels/wheel.gazebo.xacro (robot description, xacro)
@@ -17,5 +17,5 @@
       <fdir1>1 0 0</fdir1>
       <maxVel>1.0</maxVel>
-      <minDepth>0.003</minDepth>
+      <minDepth>0.000</minDepth>
       <implicitSpringDamper>1</implicitSpringDamper>
       <material>Gazebo/DarkGrey</material>

Commit message: high-res mesh of the base for visual geometry

File: pmb2_description/urdf/base/base.urdf.xacro (robot description, xacro)
@@ -41,5 +41,5 @@
         <origin xyz="0 0 0" rpy="0 0 0" />
         <geometry>
-          <mesh filename="package://pmb2_description/meshes/base/high_resolution/base_collision.stl" />
+          <mesh filename="package://pmb2_description/meshes/base/base.stl" />
         </geometry>
         <material name="White" />

Commit message: sufficient for tests

File: pmb2_description/urdf/base/base.urdf.xacro (robot description, xacro)
@@ -18,5 +18,5 @@
   <property name="wheel_width"      value="0.040"/>
   <property name="wheel_separation" value="0.4044"/>
-  <property name="wheel_torque"     value="6.0"/>
+  <property name="wheel_torque"     value="10006.0"/>
   <property name="wheel_velocity"   value="1.0"/>
   <!-- Caster wheel characteristics -->

File: pmb2_description/urdf/wheels/caster.gazebo.xacro (robot description, xacro)
@@ -13,9 +13,9 @@
       <kp>1000000.0</kp>
       <kd>1000.0</kd>
-      <mu1>0.2</mu1>
-      <mu2>0.2</mu2>
+      <mu1>1.0</mu1>
+      <mu2>1.0</mu2>
       <fdir1>1 0 0</fdir1>
       <maxVel>1.0</maxVel>
-      <minDepth>0.0</minDepth>
+      <minDepth>0.005</minDepth>
       <implicitSpringDamper>1</implicitSpringDamper>
       <material>Gazebo/DarkGrey</material>
@@ -24,9 +24,9 @@
       <kp>1000000.0</kp>
       <kd>1000.0</kd>
-      <mu1>0.2</mu1>
-      <mu2>0.2</mu2>
+      <mu1>1.0</mu1>
+      <mu2>1.0</mu2>
       <fdir1>1 0 0</fdir1>
       <maxVel>1.0</maxVel>
-      <minDepth>0.0</minDepth>
+      <minDepth>0.005</minDepth>
       <implicitSpringDamper>1</implicitSpringDamper>
       <material>Gazebo/DarkGrey</material>

File: pmb2_description/urdf/wheels/wheel.gazebo.xacro (robot description, xacro)
@@ -12,10 +12,10 @@
     <gazebo reference="wheel_${side}_link">
       <kp>1000000.0</kp>
-      <kd>100.0</kd>
-      <mu1>1.0</mu1>
-      <mu2>1.0</mu2>
+      <kd>1000.0</kd>
+      <mu1>1000.0</mu1>
+      <mu2>1000.0</mu2>
       <fdir1>1 0 0</fdir1>
-      <maxVel>1.0</maxVel>
-      <minDepth>0.000</minDepth>
+      <maxVel>20.0</maxVel>
+      <minDepth>0.0</minDepth>
       <implicitSpringDamper>1</implicitSpringDamper>
       <material>Gazebo/DarkGrey</material>

File: pmb2_description/urdf/wheels/wheel.urdf.xacro (robot description, xacro)
@@ -36,21 +36,25 @@
       <link name="suspension_${side}_link">
         <inertial>
-          <origin xyz="0 0 0" rpy="0 0 0"/>
-          <mass value="10"/>
-          <inertia ixx="0.01" ixy="0" ixz="0" iyy="0.01" iyz="0" izz="0.01"/>
-        </inertial>
+          <origin xyz="0 0 -0.02" rpy="0 0 0"/>
+          <mass value="30"/>
+          <inertia ixx="1.0" ixy="0" ixz="0"
+                   iyy="1.0" iyz="0"
+                   izz="1.0"/>
+         </inertial>
+        <kinematic>1</kinematic>
+        <gravity>1</gravity>
       </link>
       <joint name="suspension_${side}_joint" type="prismatic">
         <origin xyz="0 0 0" rpy="0 0 0"/>
         <axis xyz="0 0 1"/>
-        <limit effort="2000.0" lower="-0.02" upper="0.02" velocity="1.0"/>
+        <limit effort="10000.0" lower="-0.04" upper="0.04" velocity="1.0"/>
         <child link="suspension_${side}_link"/>
         <parent link="${parent}_link"/>
         <calibration rising="0.0" />
-        <dynamics damping="1000" />
-        <safety_controller k_position="0"
-          k_velocity="20"
-          soft_lower_limit="-0.02"
-          soft_upper_limit="0.02" />
+        <dynamics damping="10000"/>
+        <safety_controller k_position="-0.03"
+          k_velocity="100"
+          soft_lower_limit="-0.05"
+          soft_upper_limit="0.05" />
         </joint>
         <joint name="wheel_${side}_joint" type="continuous">
