Commit message: linear move test passed

File: pmb2_description/urdf/base/base.urdf.xacro (robot description, xacro)
@@ -18,5 +18,5 @@
   <property name="wheel_width"      value="0.040"/>
   <property name="wheel_separation" value="0.4044"/>
-  <property name="wheel_torque"     value="6.0"/>
+  <property name="wheel_torque"     value="60.0"/>
   <property name="wheel_velocity"   value="1.0"/>
   <!-- Caster wheel characteristics -->

File: pmb2_description/urdf/wheels/caster.gazebo.xacro (robot description, xacro)
@@ -13,10 +13,10 @@
       <kp>1000000.0</kp>
       <kd>1000.0</kd>
-      <mu1>1.0</mu1>
-      <mu2>1.0</mu2>
-      <fdir1>1 0 0</fdir1>
+      <mu1>0.0</mu1>
+      <mu2>0.0</mu2>
+      <fdir1>0 0 1</fdir1>
       <maxVel>1.0</maxVel>
-      <minDepth>0.005</minDepth>
-      <implicitSpringDamper>1</implicitSpringDamper>
+      <minDepth>0.0</minDepth>
+      <implicitSpringDamper>0</implicitSpringDamper>
       <material>Gazebo/DarkGrey</material>
     </gazebo>
@@ -28,6 +28,6 @@
       <fdir1>1 0 0</fdir1>
       <maxVel>1.0</maxVel>
-      <minDepth>0.005</minDepth>
-      <implicitSpringDamper>1</implicitSpringDamper>
+      <minDepth>0.00</minDepth>
+      <implicitSpringDamper>0</implicitSpringDamper>
       <material>Gazebo/DarkGrey</material>
     </gazebo>

File: pmb2_description/urdf/wheels/wheel.gazebo.xacro (robot description, xacro)
@@ -16,6 +16,6 @@
       <mu2>1000.0</mu2>
       <fdir1>1 0 0</fdir1>
-      <maxVel>20.0</maxVel>
-      <minDepth>0.0</minDepth>
+      <maxVel>40.0</maxVel>
+      <minDepth>0.002</minDepth>
       <implicitSpringDamper>1</implicitSpringDamper>
       <material>Gazebo/DarkGrey</material>

File: pmb2_description/urdf/wheels/wheel.urdf.xacro (robot description, xacro)
@@ -42,5 +42,5 @@
                    izz="1.0"/>
          </inertial>
-        <kinematic>1</kinematic>
+        <kinematic>0</kinematic>
         <gravity>1</gravity>
       </link>
@@ -48,13 +48,13 @@
         <origin xyz="0 0 0" rpy="0 0 0"/>
         <axis xyz="0 0 1"/>
-        <limit effort="10000.0" lower="-0.04" upper="0.04" velocity="1.0"/>
+        <limit effort="10000.0" lower="-0.03" upper="0.03" velocity="1.0"/>
         <child link="suspension_${side}_link"/>
         <parent link="${parent}_link"/>
         <calibration rising="0.0" />
-        <dynamics damping="10000"/>
-        <safety_controller k_position="-0.03"
-          k_velocity="100"
-          soft_lower_limit="-0.05"
-          soft_upper_limit="0.05" />
+        <dynamics damping="1000"/>
+        <safety_controller k_position="0"
+          k_velocity="20"
+          soft_lower_limit="-0.03"
+          soft_upper_limit="0.03" />
         </joint>
         <joint name="wheel_${side}_joint" type="continuous">

Commit message: gtests passed on the flat surface

File: pmb2_description/urdf/base/base.urdf.xacro (robot description, xacro)
@@ -18,5 +18,5 @@
   <property name="wheel_width"      value="0.040"/>
   <property name="wheel_separation" value="0.4044"/>
-  <property name="wheel_torque"     value="60.0"/>
+  <property name="wheel_torque"     value="6.0"/>
   <property name="wheel_velocity"   value="1.0"/>
   <!-- Caster wheel characteristics -->

File: pmb2_description/urdf/wheels/caster.gazebo.xacro (robot description, xacro)
@@ -13,6 +13,6 @@
       <kp>1000000.0</kp>
       <kd>1000.0</kd>
-      <mu1>0.0</mu1>
-      <mu2>0.0</mu2>
+      <mu1>1.0</mu1>
+      <mu2>1.0</mu2>
       <fdir1>0 0 1</fdir1>
       <maxVel>1.0</maxVel>
@@ -24,6 +24,6 @@
       <kp>1000000.0</kp>
       <kd>1000.0</kd>
-      <mu1>1.0</mu1>
-      <mu2>1.0</mu2>
+      <mu1>0.7</mu1>
+      <mu2>0.7</mu2>
       <fdir1>1 0 0</fdir1>
       <maxVel>1.0</maxVel>

File: pmb2_description/urdf/wheels/caster.transmission.xacro (robot description, xacro)
@@ -17,4 +17,5 @@
       <joint name="${name}_${side}_${number}_joint" >
         <hardwareInterface>hardware_interface/VelocityJointInterface</hardwareInterface>
+        <hardwareInterface>hardware_interface/JointStateInterface</hardwareInterface>
       </joint>
     </transmission>

File: pmb2_description/urdf/wheels/wheel.gazebo.xacro (robot description, xacro)
@@ -13,9 +13,9 @@
       <kp>1000000.0</kp>
       <kd>1000.0</kd>
-      <mu1>1000.0</mu1>
-      <mu2>1000.0</mu2>
+      <mu1>1.0</mu1>
+      <mu2>1.0</mu2>
       <fdir1>1 0 0</fdir1>
-      <maxVel>40.0</maxVel>
-      <minDepth>0.002</minDepth>
+      <maxVel>1.0</maxVel>
+      <minDepth>0.00</minDepth>
       <implicitSpringDamper>1</implicitSpringDamper>
       <material>Gazebo/DarkGrey</material>

File: pmb2_description/urdf/wheels/wheel.transmission.xacro (robot description, xacro)
@@ -17,4 +17,5 @@
       <joint name="wheel_${side}_joint" >
         <hardwareInterface>hardware_interface/VelocityJointInterface</hardwareInterface>
+        <hardwareInterface>hardware_interface/JointStateInterface</hardwareInterface>
       </joint>
     </transmission>

File: pmb2_description/urdf/wheels/wheel.urdf.xacro (robot description, xacro)
@@ -37,5 +37,5 @@
         <inertial>
           <origin xyz="0 0 -0.02" rpy="0 0 0"/>
-          <mass value="30"/>
+          <mass value="10"/>
           <inertia ixx="1.0" ixy="0" ixz="0"
                    iyy="1.0" iyz="0"
@@ -48,13 +48,13 @@
         <origin xyz="0 0 0" rpy="0 0 0"/>
         <axis xyz="0 0 1"/>
-        <limit effort="10000.0" lower="-0.03" upper="0.03" velocity="1.0"/>
+        <limit effort="100.0" lower="-0.005" upper="0.005" velocity="1.0"/>
         <child link="suspension_${side}_link"/>
         <parent link="${parent}_link"/>
         <calibration rising="0.0" />
-        <dynamics damping="1000"/>
+        <dynamics damping="100"/>
         <safety_controller k_position="0"
-          k_velocity="20"
-          soft_lower_limit="-0.03"
-          soft_upper_limit="0.03" />
+          k_velocity="10"
+          soft_lower_limit="-0.005"
+          soft_upper_limit="0.005" />
         </joint>
         <joint name="wheel_${side}_joint" type="continuous">

Commit message: fix xacro warning
  deprecated: xacro tags should be prepended with 'xacro' xml namespace.
  Use the following script to fix incorrect usage:
          find . -iname "*.xacro" | xargs sed -i 's#<\([/]\?\)\(if\|unless\|include\|arg\|property\|macro\|insert_block\)#<\1xacro:\2#g'

File: pmb2_description/urdf/base/base.urdf.xacro (robot description, xacro)
@@ -15,17 +15,17 @@
   <xacro:include filename="$(find pmb2_description)/urdf/objects/antenna.urdf.xacro"/>
   <!-- Wheel characteristics -->
-  <property name="wheel_radius"     value="0.0985"/>
-  <property name="wheel_width"      value="0.040"/>
-  <property name="wheel_separation" value="0.4044"/>
-  <property name="wheel_torque"     value="6.0"/>
-  <property name="wheel_velocity"   value="1.0"/>
+  <xacro:property name="wheel_radius"     value="0.0985"/>
+  <xacro:property name="wheel_width"      value="0.040"/>
+  <xacro:property name="wheel_separation" value="0.4044"/>
+  <xacro:property name="wheel_torque"     value="6.0"/>
+  <xacro:property name="wheel_velocity"   value="1.0"/>
   <!-- Caster wheel characteristics -->
-  <property name="caster_radius"       value="0.025"/>
-  <property name="caster_width"        value="0.015"/>
-  <property name="caster_separation_x" value="0.343"/>
-  <property name="caster_separation_y" value="0.204"/>
-  <property name="caster_offset_x"     value="-0.002"/>
-  <property name="caster_offset_y"     value="0.0"/>
-  <property name="caster_offset_z"     value="-0.0335"/>
+  <xacro:property name="caster_radius"       value="0.025"/>
+  <xacro:property name="caster_width"        value="0.015"/>
+  <xacro:property name="caster_separation_x" value="0.343"/>
+  <xacro:property name="caster_separation_y" value="0.204"/>
+  <xacro:property name="caster_offset_x"     value="-0.002"/>
+  <xacro:property name="caster_offset_y"     value="0.0"/>
+  <xacro:property name="caster_offset_z"     value="-0.0335"/>
   <xacro:macro name="base" params="name">
     <!-- Base -->

File: pmb2_description/urdf/base/base_sensors.urdf.xacro (robot description, xacro)
@@ -16,7 +16,7 @@
   <xacro:include filename="$(find pmb2_description)/urdf/sensors/microphone.urdf.xacro"/>
   <!-- Laser characteristics -->
-  <property name="base_laser_x" value="0.202"/>
-  <property name="base_laser_y" value="0.0"/>
-  <property name="base_laser_z" value="-0.004"/>
+  <xacro:property name="base_laser_x" value="0.202"/>
+  <xacro:property name="base_laser_y" value="0.0"/>
+  <xacro:property name="base_laser_z" value="-0.004"/>
   <xacro:macro name="base_sensors" params=" name hokuyo:=false sick551:=false sick561:=false sick571:=false sonars:=false microphone:=false ">
     <xacro:if value="${hokuyo}"> <!-- TODO: find expr that encure only one laser is true -->

File: pmb2_description/urdf/objects/antenna.urdf.xacro (robot description, xacro)
@@ -38,5 +38,5 @@
       <parent link="${parent}"/>
       <child link="${name}_link"/>
-      <insert_block name="origin"/>
+      <xacro:insert_block name="origin"/>
     </joint>
   </xacro:macro>

File: pmb2_description/urdf/sensors/bumper.urdf.xacro (robot description, xacro)
@@ -35,5 +35,5 @@
     <joint name="${name}_joint" type="fixed">
       <axis xyz="0 1 0"/>
-      <insert_block name="origin"/>
+      <xacro:insert_block name="origin"/>
       <parent link="${parent}_link"/>
       <child  link="${name}_link"/>

File: pmb2_description/urdf/sensors/elp_rgb.urdf.xacro (robot description, xacro)
@@ -9,5 +9,5 @@
     <!-- frames in the center of the camera -->
     <joint name="${name}_joint" type="fixed">
-      <insert_block name="origin"/>
+      <xacro:insert_block name="origin"/>
       <axis xyz="0 0 1"/>
       <parent link="${parent}_link"/>

File: pmb2_description/urdf/sensors/hokuyo_urg_04lx_ug01_laser.urdf.xacro (robot description, xacro)
@@ -28,5 +28,5 @@
     <joint name="${name}_joint" type="fixed">
       <axis xyz="0 1 0"/>
-      <insert_block name="origin"/>
+      <xacro:insert_block name="origin"/>
       <parent link="${parent}_link"/>
       <child  link="${name}_link"/>

File: pmb2_description/urdf/sensors/imu.urdf.xacro (robot description, xacro)
@@ -25,5 +25,5 @@
       <parent link="${parent}"/>
       <child link="${name}_link"/>
-      <insert_block name="origin"/>
+      <xacro:insert_block name="origin"/>
     </joint>
     <gazebo reference="${name}_link">

File: pmb2_description/urdf/sensors/microphone.urdf.xacro (robot description, xacro)
@@ -12,5 +12,5 @@
     <link name="${name}_link"/>
     <joint name="${name}_joint" type="fixed">
-      <insert_block name="origin"/>
+      <xacro:insert_block name="origin"/>
       <child link="${name}_link"/>
       <parent link="${parent}_link"/>

File: pmb2_description/urdf/sensors/range.urdf.xacro (robot description, xacro)
@@ -27,5 +27,5 @@
     </link>
     <joint name="${name}_joint" type="fixed">
-      <insert_block name="origin"/>
+      <xacro:insert_block name="origin"/>
       <axis xyz="0 0 1"/>
       <parent link="${parent}_link"/>

File: pmb2_description/urdf/sensors/sick_tim551_laser.urdf.xacro (robot description, xacro)
@@ -28,5 +28,5 @@
     <joint name="${name}_joint" type="fixed">
       <axis xyz="0 1 0"/>
-      <insert_block name="origin"/>
+      <xacro:insert_block name="origin"/>
       <parent link="${parent}_link"/>
       <child  link="${name}_link"/>

File: pmb2_description/urdf/sensors/sick_tim561_laser.urdf.xacro (robot description, xacro)
@@ -28,5 +28,5 @@
     <joint name="${name}_joint" type="fixed">
       <axis xyz="0 1 0"/>
-      <insert_block name="origin"/>
+      <xacro:insert_block name="origin"/>
       <parent link="${parent}_link"/>
       <child  link="${name}_link"/>

File: pmb2_description/urdf/sensors/sick_tim571_laser.urdf.xacro (robot description, xacro)
@@ -28,5 +28,5 @@
     <joint name="${name}_joint" type="fixed">
       <axis xyz="0 1 0"/>
-      <insert_block name="origin"/>
+      <xacro:insert_block name="origin"/>
       <parent link="${parent}_link"/>
       <child  link="${name}_link"/>

File: pmb2_description/urdf/sensors/structure_sensor.urdf.xacro (robot description, xacro)
@@ -23,5 +23,5 @@
     <!-- frames in the center of the camera -->
     <joint name="${name}_joint" type="fixed">
-      <insert_block name="origin"/>
+      <xacro:insert_block name="origin"/>
       <axis xyz="0 0 1"/>
       <!-- <limit lower="0" upper="0.001" effort="100" velocity="0.01"/> -->
@@ -55,5 +55,5 @@
     </link>
     <joint name="${name}_optical_joint" type="fixed">
-      <insert_block name="optical_origin" />
+      <xacro:insert_block name="optical_origin" />
       <parent link="${name}_link"/>
       <child link="${name}_optical_frame"/>

Commit message: Use bigger mesh for collisions

File: pmb2_description/urdf/base/base.urdf.xacro (robot description, xacro)
@@ -48,5 +48,5 @@
         <origin xyz="0 0 0" rpy="0 0 0" />
         <geometry>
-          <mesh filename="package://pmb2_description/meshes/base/high_resolution/base_collision.stl" />
+          <mesh filename="package://pmb2_description/meshes/base/base_collision.stl" />
         </geometry>
         <material name="White" />

Commit message: fix width of wheels

File: pmb2_description/urdf/base/base.urdf.xacro (robot description, xacro)
@@ -21,5 +21,5 @@
   <!-- Wheel characteristics -->
   <xacro:property name="wheel_radius"     value="0.0985"/>
-  <xacro:property name="wheel_width"      value="0.040"/>
+  <xacro:property name="wheel_width"      value="0.020"/>
   <xacro:property name="wheel_separation" value="0.4044"/>
   <xacro:property name="wheel_torque"     value="6.0"/>

Commit message: Use package instead of find for meshes lookup
This change avoids errors when visualizing the robot in rviz2 from a
remote host instead of directly inside the robot

File: pmb2_description/urdf/base/base.urdf.xacro (robot description, xacro)
@@ -47,5 +47,5 @@
         <origin xyz="0 0 0" rpy="0 0 0" />
         <geometry>
-          <mesh filename="file://$(find pmb2_description)/meshes/base/base.stl" />
+          <mesh filename="package://pmb2_description/meshes/base/base.stl" />
         </geometry>
         <material name="White" />
@@ -54,5 +54,5 @@
         <origin xyz="0 0 0" rpy="0 0 0" />
         <geometry>
-          <mesh filename="file://$(find pmb2_description)/meshes/base/high_resolution/base_collision.stl" />
+          <mesh filename="package://pmb2_description/meshes/base/high_resolution/base_collision.stl" />
         </geometry>
         <material name="White" />

File: pmb2_description/urdf/cameras_add_on/cameras_add_on.urdf.xacro (robot description, xacro)
@@ -84,5 +84,5 @@
         <origin xyz="0 0 0" rpy="0 0 0"/>
         <geometry>
-          <mesh filename="file://$(find pmb2_description)/meshes/cameras_add_on/cameras_add_on.stl" scale="1 1 1"/>
+          <mesh filename="package://pmb2_description/meshes/cameras_add_on/cameras_add_on.stl" scale="1 1 1"/>
         </geometry>
         <material name="White" />
@@ -91,5 +91,5 @@
         <origin xyz="0 0 0" rpy="0 0 0" />
         <geometry>
-          <mesh filename="file://$(find pmb2_description)/meshes/cameras_add_on/cameras_add_on_collision.stl" scale="1 1 1"/>
+          <mesh filename="package://pmb2_description/meshes/cameras_add_on/cameras_add_on_collision.stl" scale="1 1 1"/>
         </geometry>
         <material name="White" />

File: pmb2_description/urdf/dock/dock.urdf.xacro (robot description, xacro)
@@ -27,5 +27,5 @@
         <origin xyz="0 0 0" rpy="0 0 0" />
         <geometry>
-          <mesh filename="file://$(find pmb2_description)/meshes/dock/dock.stl" />
+          <mesh filename="package://pmb2_description/meshes/dock/dock.stl" />
         </geometry>
         <material name="LightGrey" />
@@ -34,5 +34,5 @@
         <origin xyz="0 0 0" rpy="0 0 0" />
         <geometry>
-          <mesh filename="file://$(find pmb2_description)/meshes/dock/dock_collision.stl" />
+          <mesh filename="package://pmb2_description/meshes/dock/dock_collision.stl" />
         </geometry>
         <material name="LightGrey" />

File: pmb2_description/urdf/objects/antenna.urdf.xacro (robot description, xacro)
@@ -24,5 +24,5 @@
         <origin xyz="0 0 0" rpy="0 0 0"/>
         <geometry>
-          <mesh filename="file://$(find pmb2_description)/meshes/objects/antenna.stl"/>
+          <mesh filename="package://pmb2_description/meshes/objects/antenna.stl"/>
         </geometry>
         <material name="Black"/>

File: pmb2_description/urdf/objects/cover.urdf.xacro (robot description, xacro)
@@ -24,5 +24,5 @@
         <origin xyz="0 0 0" rpy="0 0 0"/>
         <geometry>
-          <mesh filename="file://$(find pmb2_description)/meshes/base/base_ring.stl"/>
+          <mesh filename="package://pmb2_description/meshes/base/base_ring.stl"/>
         </geometry>
         <material name="Orange"/>

File: pmb2_description/urdf/wheels/caster.urdf.xacro (robot description, xacro)
@@ -24,5 +24,5 @@
         <origin xyz="0 0 0" rpy="0 0 0"/>
         <geometry>
-          <mesh filename="file://$(find pmb2_description)/meshes/wheels/caster_1.stl"/>
+          <mesh filename="package://pmb2_description/meshes/wheels/caster_1.stl"/>
         </geometry>
         <material name="Grey"/>
@@ -44,5 +44,5 @@
         <origin xyz="0 0 0" rpy="0 0 0"/>
         <geometry>
-          <mesh filename="file://$(find pmb2_description)/meshes/wheels/caster_2.stl"/>
+          <mesh filename="package://pmb2_description/meshes/wheels/caster_2.stl"/>
         </geometry>
         <material name="DarkGrey"/>

File: pmb2_description/urdf/wheels/wheel.urdf.xacro (robot description, xacro)
@@ -24,5 +24,5 @@
         <origin xyz="0 0 0" rpy="${-90.0 * (1 - reflect) * deg_to_rad} 0 0"/>
         <geometry>
-          <mesh filename="file://$(find pmb2_description)/meshes/wheels/wheel.stl"/>
+          <mesh filename="package://pmb2_description/meshes/wheels/wheel.stl"/>
         </geometry>
         <material name="DarkGrey"/>
