Commit message: Change path from sensor courier to add_on cameras

File: pmb2_description/urdf/cameras_add_on/cameras_add_on.urdf.xacro (robot description, xacro)
@@ -13,6 +13,64 @@
 -->
 <robot xmlns:xacro="http://ros.org/wiki/xacro">
-  <!-- INCLUDES -->
-  <xacro:include filename="$(find pal_urdf_utils)/urdf/sensors/bases/pmb2/courier.urdf.xacro" />
+  <xacro:include filename="$(find pmb2_description)/urdf/sensors/structure_sensor.urdf.xacro"/>
+  <xacro:include filename="$(find pmb2_description)/urdf/sensors/elp_rgb.urdf.xacro"/>
+  <xacro:include filename="$(find pal_urdf_utils)/urdf/deg_to_rad.urdf.xacro" />
+  <!-- base RGBD characteristics -->
+  <xacro:property name="base_rgbd_x" value="0.22697"/>
+  <xacro:property name="base_rgbd_y" value="0.0"/>
+  <xacro:property name="base_rgbd_z" value="0.535"/>
+  <xacro:property name="base_rgbd_R" value="-0.171709"/>
+  <xacro:property name="base_rgbd_P" value="60"/>
+  <xacro:property name="base_rgbd_Y" value="0.0"/>
+  <!-- roof RGBD characteristics -->
+  <xacro:property name="roof_rgbd_x" value="0.18473"/>
+  <xacro:property name="roof_rgbd_y" value="0.0"/>
+  <xacro:property name="roof_rgbd_z" value="0.470428"/>
+  <xacro:property name="roof_rgbd_R" value="-0.299256"/>
+  <xacro:property name="roof_rgbd_P" value="12"/>
+  <xacro:property name="roof_rgbd_Y" value="0.0"/>
+  <!-- RGB characteristics -->
+  <xacro:property name="rgb_x" value="0.18752"/>
+  <xacro:property name="rgb_y" value="0.0"/>
+  <xacro:property name="rgb_z" value="0.3301"/>
+  <xacro:property name="rgb_R" value="0.0"/>
+  <xacro:property name="rgb_P" value="15.0"/>
+  <xacro:property name="rgb_Y" value="0.0   "/>
+  <xacro:if value="${camera_model == 'structure'}">
+    <!-- RGBD base -->
+    <xacro:structure_sensor name="base_rgbd_camera" parent="base_link">
+      <!-- Pose of sensor frame wrt to base -->
+      <origin xyz="${base_rgbd_x} ${base_rgbd_y} ${base_rgbd_z}" rpy="${base_rgbd_R * deg_to_rad} ${base_rgbd_P * deg_to_rad} ${base_rgbd_Y * deg_to_rad}"/>
+      <!-- Pose of optical frame wrt to sensor -->
+      <origin xyz="0 0 0" rpy="${-90 * deg_to_rad} 0 ${-90 * deg_to_rad}"/>
+    </xacro:structure_sensor>
+    <!-- RGBD roof -->
+    <xacro:structure_sensor name="roof_rgbd_camera" parent="base_link">
+      <!-- Pose of sensor frame wrt to base -->
+      <origin xyz="${roof_rgbd_x} ${roof_rgbd_y} ${roof_rgbd_z}" rpy="${roof_rgbd_R * deg_to_rad} ${roof_rgbd_P * deg_to_rad} ${roof_rgbd_Y * deg_to_rad}"/>
+      <!-- Pose of optical frame wrt to sensor -->
+      <origin xyz="0 0 0" rpy="${-90 * deg_to_rad} 0 ${-90 * deg_to_rad}"/>
+    </xacro:structure_sensor>
+    <!-- RGB -->
+    <xacro:elp_rgb name="rgb_camera" parent="base_link">
+      <!-- Pose of sensor frame wrt to base -->
+      <origin xyz="${rgb_x} ${rgb_y} ${rgb_z}" rpy="${rgb_R * deg_to_rad} ${rgb_P * deg_to_rad} ${rgb_Y * deg_to_rad}"/>
+      <!-- Pose of optical frame wrt to sensor -->
+      <origin xyz="0 0 0" rpy="${-90 * deg_to_rad} 0 ${-90 * deg_to_rad}"/>
+    </xacro:elp_rgb>
+  </xacro:if>
+  <!-- RGBD Laser Link -->
+  <joint name="rgbd_laser_joint" type="fixed">
+    <parent link="base_footprint"/>
+    <child link="rgbd_laser_link"/>
+    <origin xyz="-0.9 0 0" rpy="0 0 0" />
+  </joint>
+  <link name="rgbd_laser_link">
+    <inertial>
+      <origin xyz="0 0 0" rpy="0 0 0"/>
+      <mass value="0.0001" />
+      <inertia ixx="0.0001" ixy="0" ixz="0" iyy="0.0001" iyz="0" izz="0.0001" />
+    </inertial>
+  </link>
   <!-- MACRO DEFINITION-->
   <xacro:macro name="cameras_add_on" params="name parent">
